File: PCB/PC110.kicad_sch (KiCad schematic)
At the start: 11 parts, among them U1 74LS32, U10 74HC74, U11 TL3414AID, U2 74LS08, U3 74LS126, U4 74LS02, U5 74LVC2G32, U6 74LS125, U7 74LS32, U8 74LS244, U9 74LS125

Commit message: add initial schematic from the sandy river project
The entire schematic needs to be redesigned/reassigned
Parts:
- removed U1: 74LS32, PC110:TSSOP-14_4.4x5mm_P0.65mm, symbol 74xx:74LS32
- removed U10: 74HC74, symbol 74xx:74HC74
- removed U11: TL3414AID, PCM_Package_SO_AKL:SO-8_3.9x4.9mm_P1.27mm, symbol PCM_Amplifier_Operational_AKL:TL3414AID
- removed U2: 74LS08, Package_SO:TSSOP-14_4.4x5mm_P0.65mm, symbol 74xx:74LS08
- removed U3: 74LS126, Package_SO:TSSOP-14_4.4x5mm_P0.65mm, symbol 74xx:74LS126
- removed U4: 74LS02, symbol 74xx:74LS02
- removed U5: 74LVC2G32, symbol 74xGxx:74LVC2G32
- removed U6, U9: 74LS125, symbol 74xx:74LS125
- removed U7: 74LS32, symbol 74xx:74LS32
- removed U8: 74LS244, symbol 74xx:74LS244
Other:
- added sheet Audio Controller (Audio.kicad_sch)
- added sheet Buffers (Buffers.kicad_sch)
- added sheet Chipset (Chipset.kicad_sch)
- added sheet Decoupling Dapacitors (Decoup_caps.kicad_sch)
- added sheet Keyboard and BIOS (Keyboard_BIOS.kicad_sch)
- added sheet Local Bus IDE (VLB_IDE.kicad_sch)
- added sheet Memory (Memory.kicad_sch)
- added sheet Power (Power.kicad_sch)
- added sheet Processor (Processor.kicad_sch)
- added sheet Pull-ups (Pull-ups.kicad_sch)
- added sheet Super I/O (Super_IO.kicad_sch)
- added sheet VGA Controller (VGA.kicad_sch)
- note added: "TODO - Schematic: - update all the schematics to be compatible with the PC110"
- title: (none) -> PC110 Motherboard
