File: Modifications/CPU Upgrade/pcb-bga-adapter/pcb-bga-adapter.kicad_pcb (KiCad board)
At the start: 2 copper layers, 23 x 23 mm, 2 parts, among them J1 51338-1074

Commit message: Initial commit of  cpu adapter
Parts:
- turned J1 to 90 degrees
Connections:
- J1 pad 1: unconnected-(J1-Pad1) -> D29
- J1 pad 10: unconnected-(J1-Pad10) -> D17
- J1 pad 100: unconnected-(J1-Pad100) -> A12
- J1 pad 11: unconnected-(J1-Pad11) -> STPCLK#
- J1 pad 12: unconnected-(J1-Pad12) -> D24
- J1 pad 13: unconnected-(J1-Pad13) -> D31
- J1 pad 14: unconnected-(J1-Pad14) -> D23
- J1 pad 15: unconnected-(J1-Pad15) -> D30
- J1 pad 16: unconnected-(J1-Pad16) -> D21
- J1 pad 17: unconnected-(J1-Pad17) -> SMIACT#
- J1 pad 18: unconnected-(J1-Pad18) -> D19
- J1 pad 19: unconnected-(J1-Pad19) -> SRESET
- J1 pad 2: unconnected-(J1-Pad2) -> DP3
- J1 pad 20: unconnected-(J1-Pad20) -> D11
- J1 pad 21: unconnected-(J1-Pad21) -> NMI
- J1 pad 22: unconnected-(J1-Pad22) -> D16
- J1 pad 23: unconnected-(J1-Pad23) -> SMI#
- J1 pad 24: unconnected-(J1-Pad24) -> DP2
- J1 pad 25: unconnected-(J1-Pad25) -> FLUSH#
- J1 pad 26: unconnected-(J1-Pad26) -> D15
- J1 pad 27: unconnected-(J1-Pad27) -> INTR
- J1 pad 28: unconnected-(J1-Pad28) -> D12
- J1 pad 29: unconnected-(J1-Pad29) -> RESET
- J1 pad 3: unconnected-(J1-Pad3) -> D27
- J1 pad 30: unconnected-(J1-Pad30) -> D13
- J1 pad 31: unconnected-(J1-Pad31) -> A20M#
- J1 pad 32: unconnected-(J1-Pad32) -> D14
- J1 pad 33: unconnected-(J1-Pad33) -> EADS#
- J1 pad 34: unconnected-(J1-Pad34) -> D10
- J1 pad 35: unconnected-(J1-Pad35) -> DC#
- J1 pad 36: unconnected-(J1-Pad36) -> DP1
- J1 pad 37: unconnected-(J1-Pad37) -> BE2#
- J1 pad 38: unconnected-(J1-Pad38) -> D8
- J1 pad 39: unconnected-(J1-Pad39) -> BE3#
- J1 pad 4: unconnected-(J1-Pad4) -> D22
- J1 pad 40: unconnected-(J1-Pad40) -> D9
- J1 pad 41: unconnected-(J1-Pad41) -> MIO#
- J1 pad 42: unconnected-(J1-Pad42) -> D5
- J1 pad 43: unconnected-(J1-Pad43) -> BE0#
- J1 pad 44: unconnected-(J1-Pad44) -> D2
- J1 pad 45: unconnected-(J1-Pad45) -> BE1#
- J1 pad 46: unconnected-(J1-Pad46) -> D7
- J1 pad 47: unconnected-(J1-Pad47) -> CLK
- J1 pad 48: unconnected-(J1-Pad48) -> D6
- J1 pad 49: unconnected-(J1-Pad49) -> VCC
- J1 pad 5: unconnected-(J1-Pad5) -> D25
- J1 pad 50: unconnected-(J1-Pad50) -> D3
- J1 pad 51: unconnected-(J1-Pad51) -> VCC
- J1 pad 52: unconnected-(J1-Pad52) -> D4
- J1 pad 53: unconnected-(J1-Pad53) -> VCC
- J1 pad 54: unconnected-(J1-Pad54) -> DP0
- J1 pad 55: unconnected-(J1-Pad55) -> HLDA
- J1 pad 56: unconnected-(J1-Pad56) -> D0
- J1 pad 57: unconnected-(J1-Pad57) -> WR#
- J1 pad 58: unconnected-(J1-Pad58) -> D1
- J1 pad 59: unconnected-(J1-Pad59) -> AHOLD
- J1 pad 6: unconnected-(J1-Pad6) -> D20
- J1 pad 60: unconnected-(J1-Pad60) -> A30
- J1 pad 61: unconnected-(J1-Pad61) -> KEN#
- J1 pad 62: unconnected-(J1-Pad62) -> A27
- J1 pad 63: unconnected-(J1-Pad63) -> RDY#
- J1 pad 64: unconnected-(J1-Pad64) -> A31
- J1 pad 65: unconnected-(J1-Pad65) -> HOLD
- J1 pad 66: unconnected-(J1-Pad66) -> A28
- J1 pad 67: unconnected-(J1-Pad67) -> GND
- J1 pad 68: unconnected-(J1-Pad68) -> A29
- J1 pad 69: unconnected-(J1-Pad69) -> GND
- J1 pad 7: unconnected-(J1-Pad7) -> D28
- J1 pad 70: unconnected-(J1-Pad70) -> A25
- J1 pad 71: unconnected-(J1-Pad71) -> GND
- J1 pad 72: unconnected-(J1-Pad72) -> A24
- J1 pad 73: unconnected-(J1-Pad73) -> BS16#
- J1 pad 74: unconnected-(J1-Pad74) -> A21
- J1 pad 75: unconnected-(J1-Pad75) -> BRDY#
- J1 pad 76: unconnected-(J1-Pad76) -> A26
- J1 pad 77: unconnected-(J1-Pad77) -> A2
- J1 pad 78: unconnected-(J1-Pad78) -> A22
- J1 pad 79: unconnected-(J1-Pad79) -> ADS#
- J1 pad 8: unconnected-(J1-Pad8) -> D18
- J1 pad 80: unconnected-(J1-Pad80) -> A23
- J1 pad 81: unconnected-(J1-Pad81) -> BLAST#
- J1 pad 82: unconnected-(J1-Pad82) -> A19
- J1 pad 83: unconnected-(J1-Pad83) -> A3
- J1 pad 84: unconnected-(J1-Pad84) -> A20
- J1 pad 85: unconnected-(J1-Pad85) -> A5
- J1 pad 86: unconnected-(J1-Pad86) -> A17
- J1 pad 87: unconnected-(J1-Pad87) -> A6
- J1 pad 88: unconnected-(J1-Pad88) -> A15
- J1 pad 89: unconnected-(J1-Pad89) -> A4
- J1 pad 9: unconnected-(J1-Pad9) -> D26
- J1 pad 90: unconnected-(J1-Pad90) -> A18
- J1 pad 91: unconnected-(J1-Pad91) -> A10
- J1 pad 92: unconnected-(J1-Pad92) -> A16
- J1 pad 94: unconnected-(J1-Pad94) -> A13
- J1 pad 95: unconnected-(J1-Pad95) -> A7
- J1 pad 96: unconnected-(J1-Pad96) -> A8
- J1 pad 97: unconnected-(J1-Pad97) -> A9
- J1 pad 98: unconnected-(J1-Pad98) -> A14
- J1 pad 99: unconnected-(J1-Pad99) -> A11
- U1 pad A11: unconnected-(U1-BE2#-PadA11) -> BE2#
- U1 pad A12: unconnected-(U1-DC#-PadA12) -> DC#
- U1 pad A13: unconnected-(U1-EADS#-PadA13) -> EADS#
- U1 pad A3: unconnected-(U1-A2-PadA3) -> A2
- U1 pad A6: unconnected-(U1-BS16#-PadA6) -> BS16#
- U1 pad A7: unconnected-(U1-RDY#-PadA7) -> RDY#
- U1 pad A8: unconnected-(U1-AHOLD-PadA8) -> AHOLD
- U1 pad A9: unconnected-(U1-CLK-PadA9) -> CLK
- U1 pad B10: unconnected-(U1-BE0#-PadB10) -> BE0#
- U1 pad B11: unconnected-(U1-BE3#-PadB11) -> BE3#
- U1 pad B13: unconnected-(U1-A20M#-PadB13) -> A20M#
- U1 pad B3: unconnected-(U1-ADS#-PadB3) -> ADS#
- U1 pad B5: unconnected-(U1-BRDY#-PadB5) -> BRDY#
- U1 pad B7: unconnected-(U1-KEN#-PadB7) -> KEN#
- U1 pad B9: unconnected-(U1-HLDA-PadB9) -> HLDA
- U1 pad C10: unconnected-(U1-BE1#-PadC10) -> BE1#
- U1 pad C11: unconnected-(U1-MIO#-PadC11) -> MIO#
- U1 pad C13: unconnected-(U1-RESET-PadC13) -> RESET
- U1 pad C16: unconnected-(U1-FLUSH#-PadC16) -> FLUSH#
- U1 pad C3: unconnected-(U1-BLAST#-PadC3) -> BLAST#
- U1 pad C7: unconnected-(U1-HOLD-PadC7) -> HOLD
- U1 pad C9: unconnected-(U1-WR#-PadC9) -> WR#
- U1 pad D1: unconnected-(U1-A4-PadD1) -> A4
- U1 pad D10: Net-(U1-VCC-PadD10) -> VCC
- U1 pad D11: Net-(U1-VCC-PadD10) -> VCC
- U1 pad D12: Net-(U1-VCC-PadD10) -> VCC
- U1 pad D13: Net-(U1-VCC-PadD10) -> VCC
- U1 pad D14: Net-(U1-VCC-PadD10) -> VCC
- U1 pad D15: unconnected-(U1-INTR-PadD15) -> INTR
- U1 pad D16: unconnected-(U1-NMI-PadD16) -> NMI
- U1 pad D2: unconnected-(U1-A3-PadD2) -> A3
- U1 pad D3: Net-(U1-VCC-PadD10) -> VCC
- U1 pad D4: Net-(U1-VCC-PadD10) -> VCC
- U1 pad D5: Net-(U1-VCC-PadD10) -> VCC
- U1 pad D6: Net-(U1-VCC-PadD10) -> VCC
- U1 pad D7: Net-(U1-VCC-PadD10) -> VCC
- U1 pad D8: Net-(U1-VCC-PadD10) -> VCC
- U1 pad D9: Net-(U1-VCC-PadD10) -> VCC
- U1 pad E10: Net-(U1-VCC-PadD10) -> VCC
- U1 pad E11: Net-(U1-VCC-PadD10) -> VCC
- U1 pad E12: Net-(U1-VCC-PadD10) -> VCC
- U1 pad E13: Net-(U1-VCC-PadD10) -> VCC
- U1 pad E14: Net-(U1-VCC-PadD10) -> VCC
- U1 pad E15: unconnected-(U1-SRESET-PadE15) -> SRESET
- U1 pad E16: unconnected-(U1-SMIACT#-PadE16) -> SMIACT#
- U1 pad E2: unconnected-(U1-A5-PadE2) -> A5
- U1 pad E3: Net-(U1-VCC-PadD10) -> VCC
- U1 pad E4: Net-(U1-VCC-PadD10) -> VCC
- U1 pad E5: Net-(U1-VCC-PadD10) -> VCC
- U1 pad E6: Net-(U1-VCC-PadD10) -> VCC
- U1 pad E7: Net-(U1-VCC-PadD10) -> VCC
- U1 pad E8: Net-(U1-VCC-PadD10) -> VCC
- U1 pad E9: Net-(U1-VCC-PadD10) -> VCC
- U1 pad F1: unconnected-(U1-A7-PadF1) -> A7
- U1 pad F14: Net-(U1-VCC-PadD10) -> VCC
- U1 pad F15: unconnected-(U1-SMI#-PadF15) -> SMI#
- U1 pad F2: unconnected-(U1-A6-PadF2) -> A6
- U1 pad F3: Net-(U1-VCC-PadD10) -> VCC
- U1 pad G1: unconnected-(U1-A9-PadG1) -> A9
- U1 pad G14: Net-(U1-VCC-PadD10) -> VCC
- U1 pad G15: unconnected-(U1-STPCLK#-PadG15) -> STPCLK#
- U1 pad G16: unconnected-(U1-D31-PadG16) -> D31
- U1 pad G2: unconnected-(U1-A8-PadG2) -> A8
- U1 pad G3: Net-(U1-VCC-PadD10) -> VCC
- U1 pad H1: unconnected-(U1-A11-PadH1) -> A11
- U1 pad H14: Net-(U1-VCC-PadD10) -> VCC
- U1 pad H15: unconnected-(U1-D30-PadH15) -> D30
- U1 pad H16: unconnected-(U1-D29-PadH16) -> D29
- U1 pad H2: unconnected-(U1-A10-PadH2) -> A10
- U1 pad H3: Net-(U1-VCC-PadD10) -> VCC
- U1 pad J1: unconnected-(U1-A12-PadJ1) -> A12
- U1 pad J14: Net-(U1-VCC-PadD10) -> VCC
- U1 pad J15: unconnected-(U1-D28-PadJ15) -> D28
- U1 pad J16: unconnected-(U1-D27-PadJ16) -> D27
- U1 pad J3: Net-(U1-VCC-PadD10) -> VCC
- U1 pad K1: unconnected-(U1-A14-PadK1) -> A14
- U1 pad K14: Net-(U1-VCC-PadD10) -> VCC
- U1 pad K15: unconnected-(U1-D26-PadK15) -> D26
- U1 pad K16: unconnected-(U1-D25-PadK16) -> D25
- U1 pad K2: unconnected-(U1-A13-PadK2) -> A13
- U1 pad K3: Net-(U1-VCC-PadD10) -> VCC
- U1 pad L1: unconnected-(U1-A16-PadL1) -> A16
- U1 pad L14: Net-(U1-VCC-PadD10) -> VCC
- U1 pad L15: unconnected-(U1-D24-PadL15) -> D24
- U1 pad L16: unconnected-(U1-DP3-PadL16) -> DP3
- U1 pad L2: unconnected-(U1-A15-PadL2) -> A15
- U1 pad L3: Net-(U1-VCC-PadD10) -> VCC
- U1 pad M10: Net-(U1-VCC-PadD10) -> VCC
- U1 pad M11: Net-(U1-VCC-PadD10) -> VCC
- U1 pad M12: Net-(U1-VCC-PadD10) -> VCC
- U1 pad M13: Net-(U1-VCC-PadD10) -> VCC
- U1 pad M14: Net-(U1-VCC-PadD10) -> VCC
- U1 pad M15: unconnected-(U1-D23-PadM15) -> D23
- U1 pad M16: unconnected-(U1-D22-PadM16) -> D22
- U1 pad M2: unconnected-(U1-A17-PadM2) -> A17
- U1 pad M3: Net-(U1-VCC-PadD10) -> VCC
- U1 pad M4: Net-(U1-VCC-PadD10) -> VCC
- U1 pad M5: Net-(U1-VCC-PadD10) -> VCC
- U1 pad M6: Net-(U1-VCC-PadD10) -> VCC
- U1 pad M7: Net-(U1-VCC-PadD10) -> VCC
- U1 pad M8: Net-(U1-VCC-PadD10) -> VCC
- U1 pad M9: Net-(U1-VCC-PadD10) -> VCC
- U1 pad N1: unconnected-(U1-A18-PadN1) -> A18
- U1 pad N10: Net-(U1-VCC-PadD10) -> VCC
- U1 pad N11: Net-(U1-VCC-PadD10) -> VCC
- U1 pad N12: Net-(U1-VCC-PadD10) -> VCC
- U1 pad N13: Net-(U1-VCC-PadD10) -> VCC
- U1 pad N14: Net-(U1-VCC-PadD10) -> VCC
- U1 pad N15: unconnected-(U1-D21-PadN15) -> D21
- U1 pad N16: unconnected-(U1-D20-PadN16) -> D20
- U1 pad N3: Net-(U1-VCC-PadD10) -> VCC
- U1 pad N4: Net-(U1-VCC-PadD10) -> VCC
- U1 pad N5: Net-(U1-VCC-PadD10) -> VCC
- U1 pad N6: Net-(U1-VCC-PadD10) -> VCC
- U1 pad N7: Net-(U1-VCC-PadD10) -> VCC
- U1 pad N8: Net-(U1-VCC-PadD10) -> VCC
- U1 pad N9: Net-(U1-VCC-PadD10) -> VCC
- U1 pad P1: unconnected-(U1-A20-PadP1) -> A20
- U1 pad P10: unconnected-(U1-D9-PadP10) -> D9
- U1 pad P11: unconnected-(U1-D11-PadP11) -> D11
- U1 pad P12: unconnected-(U1-D14-PadP12) -> D14
- U1 pad P13: unconnected-(U1-D16-PadP13) -> D16
- U1 pad P15: unconnected-(U1-D19-PadP15) -> D19
- U1 pad P16: unconnected-(U1-D18-PadP16) -> D18
- U1 pad P2: unconnected-(U1-A19-PadP2) -> A19
- U1 pad P3: unconnected-(U1-A23-PadP3) -> A23
- U1 pad P4: unconnected-(U1-A26-PadP4) -> A26
- U1 pad P5: unconnected-(U1-A29-PadP5) -> A29
- U1 pad P7: unconnected-(U1-D1-PadP7) -> D1
- U1 pad P8: unconnected-(U1-D4-PadP8) -> D4
- U1 pad P9: unconnected-(U1-D7-PadP9) -> D7
- U1 pad R10: unconnected-(U1-D8-PadR10) -> D8
- U1 pad R11: unconnected-(U1-D10-PadR11) -> D10
- U1 pad R12: unconnected-(U1-D13-PadR12) -> D13
- U1 pad R13: unconnected-(U1-DP2-PadR13) -> DP2
- U1 pad R16: unconnected-(U1-D17-PadR16) -> D17
- U1 pad R3: unconnected-(U1-A22-PadR3) -> A22
- U1 pad R4: unconnected-(U1-A25-PadR4) -> A25
- U1 pad R5: unconnected-(U1-A28-PadR5) -> A28
- U1 pad R6: unconnected-(U1-A31-PadR6) -> A31
- U1 pad R7: unconnected-(U1-D0-PadR7) -> D0
- U1 pad R8: unconnected-(U1-D3-PadR8) -> D3
- U1 pad R9: unconnected-(U1-D6-PadR9) -> D6
- U1 pad T10: unconnected-(U1-DP1-PadT10) -> DP1
- U1 pad T12: unconnected-(U1-D12-PadT12) -> D12
- U1 pad T13: unconnected-(U1-D15-PadT13) -> D15
- U1 pad T3: unconnected-(U1-A21-PadT3) -> A21
- U1 pad T4: unconnected-(U1-A24-PadT4) -> A24
- U1 pad T5: unconnected-(U1-A27-PadT5) -> A27
- U1 pad T6: unconnected-(U1-A30-PadT6) -> A30
- U1 pad T7: unconnected-(U1-DP0-PadT7) -> DP0
- U1 pad T8: unconnected-(U1-D2-PadT8) -> D2
- U1 pad T9: unconnected-(U1-D5-PadT9) -> D5
Routing:
- net GND: track 0.00 -> 141.8 mm, vias 0 -> 4
- net VCC: track 0.00 -> 90.2 mm, vias 0 -> 5
- net DP2: track 0.00 -> 12.8 mm, vias 0 -> 1
- net EADS#: track 0.00 -> 11.5 mm, vias 0 -> 1
- net D15: track 0.00 -> 11.1 mm, vias 0 -> 1
- net DP0: track 0.00 -> 11.0 mm, vias 0 -> 1
- net A30: track 0.00 -> 11.0 mm, vias 0 -> 1
- net A20M#: track 0.00 -> 10.6 mm, vias 0 -> 1
- net D2: track 0.00 -> 10.6 mm, vias 0 -> 1
- net A24: track 0.00 -> 10.4 mm, vias 0 -> 1
- net D12: track 0.00 -> 10.4 mm, vias 0 -> 1
- net A27: track 0.00 -> 10.3 mm, vias 0 -> 1
- net D30: track 0.00 -> 10.1 mm, vias 0 -> 1
- net D5: track 0.00 -> 10.1 mm, vias 0 -> 1
- net D11: track 0.00 -> 10.1 mm, vias 0 -> 1
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
Commit message: silkscreen update
Routing:
- net GND: track 141.8 -> 157.0 mm, vias 4 -> 5
- net VCC: track 90.2 -> 94.1 mm, vias 5 -> 4
- net HLDA: track 9.53 -> 8.26 mm
- net A2: track 8.90 -> 9.92 mm
- net ADS#: track 7.49 -> 8.48 mm
- net BRDY#: track 7.46 -> 8.27 mm
- net RDY#: track 9.27 -> 10.0 mm
- net CLK: track 9.04 -> 8.52 mm
- net KEN#: track 7.86 -> 7.33 mm
- net BS16#: track 9.09 -> 8.57 mm
Other:
- board text added: "1"
- board text added: "A1"
- board text added: "PC110 CPU INTERPOSER v1"
