File: PSU/PSU.kicad_pcb (KiCad board)
At the start: 4 copper layers, 72.3 x 45 mm, 183 parts, among them J1 PSU_Connector_Receptor, Q1 SOT-23, Q1 SOT-powerT, Q10 SOT-89-3, Q11 SOT-416, Q12 SOT-416, Q13 SOT-416, Q14 SOT-23, Q16 SOT-416, Q19 SOT-416, Q2 SOT-416, Q2 SOT-powerT, Q21 SOT-416, Q22 SOT-416, Q23 SOT-416, Q24 SOT-416, Q25 SOT-416, Q26 SOT-23, Q28 SOT-416, Q3 SOT-416, Q30 SOT-23, Q32 SOT-416, Q33 SOT-416, Q4 SOT-23, Q5 SOT-416, Q6 SOT-416, Q7 SOT-416, Q8 SOT-23-3, Q9 SOT-23, U1 SOT-23-5, U2 SOT-23-6_Handsoldering

Commit message: Add files via upload
Parts:
- removed the Q26 at (136.7, 115.2)
- removed Q30: SOT-23, Package_TO_SOT_SMD:SOT-23
- removed Q8: SOT-23-3, Package_TO_SOT_SMD:SOT-23-3
- removed the REF** at (145.0, 93.3)
- added J2: Backllight_Connector, Connector_JST:Backllight_Connector, F.Cu at (145.0, 93.2)
- added Q26: SOT-23-PC110, Package_TO_SOT_SMD:SOT-23-PC110, F.Cu at (140.7, 115.4)
- added Q26: SOT-23-PC110, Package_TO_SOT_SMD:SOT-23-PC110, F.Cu at (136.6, 115.2)
- added U1: SOT-23-5, Package_TO_SOT_SMD:SOT-23-5, F.Cu at (127.7, 95.4)
- renumbered REF** to Q1, REF** to Q2, REF** to Q4
Connections:
- C15 pad 1: (no net) -> GND
- C22 pad 1: (no net) -> GND
- C38 pad 2: (no net) -> GND
- C39 pad 1: (no net) -> GND
- C40 pad 1: (no net) -> GND
- J1 pad 19: (no net) -> J1_19
- Q1 pad 1: (no net) -> J1_38
- Q14 pad 2: (no net) -> GND
- Q2 pad 1: (no net) -> J1_19
- R28 pad 1: (no net) -> GND
Routing:
- net (no net): track 1572.0 -> 1798.6 mm, vias 144 -> 140
- net GND: track 280.3 -> 343.3 mm, vias 53 -> 54
- net J1_19: track 0.00 -> 47.8 mm, vias 0 -> 2
- net J1_38: track 0.00 -> 35.7 mm, vias 0 -> 1

Commit message: Add files via upload
Parts:
- added C24: C_0603_1608Metric, Capacitor_SMD:C_0603_1608Metric, B.Cu at (156.6, 112.0)
- added C24: C_0603_1608Metric, Capacitor_SMD:C_0603_1608Metric, B.Cu at (108.7, 92.1)
- added C24: C_0603_1608Metric, Capacitor_SMD:C_0603_1608Metric, B.Cu at (157.5, 104.0)
- added C24: C_0603_1608Metric, Capacitor_SMD:C_0603_1608Metric, B.Cu at (165.7, 110.4)
- added C24: C_0603_1608Metric, Capacitor_SMD:C_0603_1608Metric, B.Cu at (113.0, 108.2)
- added C24: C_0603_1608Metric, Capacitor_SMD:C_0603_1608Metric, B.Cu at (159.6, 112.1)
- added C24: C_0603_1608Metric, Capacitor_SMD:C_0603_1608Metric, B.Cu at (163.9, 90.6)
- added C24: C_0603_1608Metric, Capacitor_SMD:C_0603_1608Metric, B.Cu at (111.0, 97.8)
- added C24: C_0603_1608Metric, Capacitor_SMD:C_0603_1608Metric, B.Cu at (154.7, 98.8)
- added C24: C_0603_1608Metric, Capacitor_SMD:C_0603_1608Metric, B.Cu at (117.8, 89.1)
- added C24: C_0603_1608Metric, Capacitor_SMD:C_0603_1608Metric, B.Cu at (159.1, 104.7)
- added C24: C_0603_1608Metric, Capacitor_SMD:C_0603_1608Metric, B.Cu at (151.9, 100.9)
- added C24: C_0603_1608Metric, Capacitor_SMD:C_0603_1608Metric, B.Cu at (155.0, 87.5)
- added C24: C_0603_1608Metric, Capacitor_SMD:C_0603_1608Metric, B.Cu at (153.5, 81.8)
- added C24: C_0603_1608Metric, Capacitor_SMD:C_0603_1608Metric, B.Cu at (164.2, 100.1)
- added C24: C_0603_1608Metric, Capacitor_SMD:C_0603_1608Metric, B.Cu at (109.1, 103.5)
- added C24: C_0603_1608Metric, Capacitor_SMD:C_0603_1608Metric, B.Cu at (112.5, 97.8)
- added C24: C_0603_1608Metric, Capacitor_SMD:C_0603_1608Metric, B.Cu at (117.6, 94.4)
- added C24: C_0603_1608Metric, Capacitor_SMD:C_0603_1608Metric, B.Cu at (169.7, 98.5)
- added C25: C_0805_2012Metric, Capacitor_SMD:C_0805_2012Metric, B.Cu at (158.4, 87.3)
- added C25: C_0805_2012Metric, Capacitor_SMD:C_0805_2012Metric, B.Cu at (117.9, 87.3)
- added C25: C_0805_2012Metric, Capacitor_SMD:C_0805_2012Metric, B.Cu at (118.0, 90.8)
- added C25: C_0805_2012Metric, Capacitor_SMD:C_0805_2012Metric, B.Cu at (158.0, 98.8)
- added F1: Fuse_1206_3216Metric, Fuse:Fuse_1206_3216Metric, B.Cu at (124.1, 107.6)
- added F2: Fuse_1210_3225Metric, Fuse:Fuse_1210_3225Metric, B.Cu at (109.7, 107.2)
- added F3: Fuse_2010_5025Metric, Fuse:Fuse_2010_5025Metric, B.Cu at (147.2, 96.6)
- added F3: Fuse_2010_5025Metric, Fuse:Fuse_2010_5025Metric, B.Cu at (169.8, 90.3)
- added F3: Fuse_2010_5025Metric, Fuse:Fuse_2010_5025Metric, B.Cu at (176.5, 115.3)
- added J3: PSU_Jack, PSU:PSU_Jack, B.Cu at (165.7, 82.0)
- added Q23: SOT-416, Package_TO_SOT_SMD:SOT-416, B.Cu at (159.0, 108.5)
- added Q23: SOT-416, Package_TO_SOT_SMD:SOT-416, B.Cu at (153.4, 85.2)
- added R1: C_1206_3216Metric, Capacitor_SMD:C_1206_3216Metric, B.Cu at (177.5, 98.4)
- added R1: C_1206_3216Metric, Capacitor_SMD:C_1206_3216Metric, B.Cu at (174.8, 98.5)
- added R72: R_0603_1608Metric, Resistor_SMD:R_0603_1608Metric, B.Cu at (153.6, 80.2)
- added R72: R_0603_1608Metric, Resistor_SMD:R_0603_1608Metric, B.Cu at (158.1, 112.1)
- added R72: R_0603_1608Metric, Resistor_SMD:R_0603_1608Metric, B.Cu at (154.2, 107.9)
- added R72: R_0603_1608Metric, Resistor_SMD:R_0603_1608Metric, B.Cu at (151.9, 102.3)
- added R72: R_0603_1608Metric, Resistor_SMD:R_0603_1608Metric, B.Cu at (108.8, 89.3)
- added R72: R_0603_1608Metric, Resistor_SMD:R_0603_1608Metric, B.Cu at (151.9, 105.2)
- added R72: R_0603_1608Metric, Resistor_SMD:R_0603_1608Metric, B.Cu at (149.9, 92.1)
- added R72: R_0603_1608Metric, Resistor_SMD:R_0603_1608Metric, B.Cu at (155.7, 107.9)
- added R72: R_0603_1608Metric, Resistor_SMD:R_0603_1608Metric, B.Cu at (157.1, 107.9)
- added R72: R_0603_1608Metric, Resistor_SMD:R_0603_1608Metric, B.Cu at (108.9, 100.6)
- added R72: R_0603_1608Metric, Resistor_SMD:R_0603_1608Metric, B.Cu at (151.4, 95.0)
- added R72: R_0603_1608Metric, Resistor_SMD:R_0603_1608Metric, B.Cu at (153.6, 78.7)
- added R72: R_0603_1608Metric, Resistor_SMD:R_0603_1608Metric, B.Cu at (153.6, 83.2)
- added R72: R_0603_1608Metric, Resistor_SMD:R_0603_1608Metric, B.Cu at (168.8, 96.3)
- added R72: R_0603_1608Metric, Resistor_SMD:R_0603_1608Metric, B.Cu at (113.9, 97.8)
- added R72: R_0603_1608Metric, Resistor_SMD:R_0603_1608Metric, B.Cu at (164.2, 98.2)
- added R72: R_0603_1608Metric, Resistor_SMD:R_0603_1608Metric, B.Cu at (151.5, 92.1)
- added R72: R_0603_1608Metric, Resistor_SMD:R_0603_1608Metric, B.Cu at (114.4, 100.9)
- added R72: R_0603_1608Metric, Resistor_SMD:R_0603_1608Metric, B.Cu at (164.1, 110.3)
- added R72: R_0603_1608Metric, Resistor_SMD:R_0603_1608Metric, B.Cu at (151.9, 103.7)
- added R72: R_0603_1608Metric, Resistor_SMD:R_0603_1608Metric, B.Cu at (150.3, 98.7)
- added R72: R_0603_1608Metric, Resistor_SMD:R_0603_1608Metric, B.Cu at (162.5, 110.3)
- added R72: R_0603_1608Metric, Resistor_SMD:R_0603_1608Metric, B.Cu at (108.9, 97.8)
- added SW1: PSU-SW1, PSU:PSU-SW1, B.Cu at (158.7, 80.3)
- added U1: SOP-8_3.9x4.9mm_P1.27mm, Package_SO:SOP-8_3.9x4.9mm_P1.27mm, B.Cu at (141.0, 93.1)
- added U1: SOP-8_3.9x4.9mm_P1.27mm, Package_SO:SOP-8_3.9x4.9mm_P1.27mm, B.Cu at (163.9, 116.9)
- added U1: TSSOP-28_6.1x9.7mm_P0.65mm, Package_SO:TSSOP-28_6.1x9.7mm_P0.65mm, B.Cu at (157.6, 93.1)
- added U1: SOP-8_3.9x4.9mm_P1.27mm, Package_SO:SOP-8_3.9x4.9mm_P1.27mm, B.Cu at (123.5, 93.0)
- added U1: SOP-8_3.9x4.9mm_P1.27mm, Package_SO:SOP-8_3.9x4.9mm_P1.27mm, B.Cu at (132.5, 92.9)
- added U1: SOP-8_3.9x4.9mm_P1.27mm, Package_SO:SOP-8_3.9x4.9mm_P1.27mm, B.Cu at (152.1, 117.3)
- added U1: SSOP-8_2.95x2.8mm_P0.65mm, Package_SO:SSOP-8_2.95x2.8mm_P0.65mm, B.Cu at (111.8, 103.0)
- added U1: SSOP-16_3.9x4.9mm_P0.635mm, Package_SO:SSOP-16_3.9x4.9mm_P0.635mm, B.Cu at (113.2, 91.3)
- added U3: TSSOP-14_4.4x5mm_P0.65mm, Package_SO:TSSOP-14_4.4x5mm_P0.65mm, B.Cu at (162.6, 105.1)
- added U3: SSOP-8_2.95x2.8mm_P0.65mm, Package_SO:SSOP-8_2.95x2.8mm_P0.65mm, B.Cu at (155.0, 103.6)
Connections:
- C12 pad 1: (no net) -> C12_1
- C12 pad 2: (no net) -> GND
- C16 pad 1: (no net) -> C16_1
- C16 pad 2: (no net) -> C16_2
- Q14 pad 1: (no net) -> GND
- Q26 pad 2: (no net) -> GND
- Q5 pad 2: (no net) -> GND
- R44 pad 1: (no net) -> GND
Routing:
- net (no net): track 1798.6 -> 1877.4 mm
- net GND: track 343.3 -> 364.1 mm
- net C12_1: track 0.00 -> 1.57 mm, vias 0 -> 1
- net C16_1: track 0.00 -> 1.47 mm, vias 0 -> 1
- net C16_2: track 0.00 -> 1.45 mm, vias 0 -> 1

Commit message: Add files via upload
Parts:
- removed the U1 at (111.8, 103.0)
- removed the U1 at (113.2, 91.3)
- removed the U3 at (155.0, 103.6)
- added U10: SSOP-8-PSU, PSU:SSOP-8-PSU, B.Cu at (111.6, 102.9)
- added U11: SSOP-16_4.4x5.2mm_P0.65mm, Package_SO:SSOP-16_4.4x5.2mm_P0.65mm, B.Cu at (113.0, 91.7)
- added U6: SSOP-8-PSU, PSU:SSOP-8-PSU, B.Cu at (155.0, 103.7)
- renumbered C17 to C10, C10 to C11, C11 to C12, C12 to C13, C13 to C14, C14 to C15, C15 to C16, C16 to C17, C19 to C18, C20 to C19, C21 to C20, C22 to C21, C18 to C22, C26 to C23, C23 to C24, C24 to C26, C30 to C29, C29 to C30, C32 to C31, C34 to C32, C31 to C34, C36 to C35, C35 to C36, C24 to C38, C24 to C39, C9 to C4, C25 to C40, C25 to C41, C24 to C42, C24 to C43, C24 to C44, C40 to C45, C24 to C46, C24 to C47, C24 to C48, C24 to C49, C6 to C5, C38 to C50, C39 to C51, C24 to C52, C41 to C53, C24 to C54, C24 to C55, C25 to C56, C25 to C57, C42 to C58, C43 to C59, C7 to C6, C44 to C60, C24 to C61, C24 to C62, C45 to C63, C24 to C64, C24 to C65, C24 to C66, C24 to C67, C24 to C68, C46 to C69, C4 to C7, C5 to C9, F3 to F1, F3 to F2, F1 to F3, F2 to F4, F3 to F5, J2 to J1, J3 to J2, J1 to J3, L3 to L2, L2 to L3, Q11 to Q10, Q2 to Q11, Q9 to Q12, Q1 to Q13, Q13 to Q14, Q14 to Q15, Q4 to Q17, Q19 to Q18, Q23 to Q19, Q21 to Q20, Q24 to Q21, Q26 to Q23, Q25 to Q24, Q2 to Q25, Q4 to Q27, Q1 to Q29, Q4 to Q3, Q33 to Q30, Q32 to Q31, Q23 to Q32, Q23 to Q33, Q3 to Q4, Q12 to Q8, Q10 to Q9, R11 to R10, R72 to R100, R72 to R101, R72 to R102, R72 to R103, R72 to R104, R72 to R105, R72 to R106, R72 to R107, R72 to R108, R72 to R109, R12 to R11, R72 to R110, R72 to R111, R72 to R112, R72 to R113, R72 to R114, R72 to R115, R72 to R116, R15 to R12, R14 to R13, R16 to R14, R18 to R15, R19 to R16, R10 to R17, R17 to R18, R13 to R19, R29 to R22, R35 to R23, R26 to R25, R25 to R26, R22 to R27, R27 to R28, R30 to R29, R31 to R30, R23 to R31, R34 to R32, R28 to R33, R33 to R34, R32 to R35, R41 to R39, R5 to R4, R67 to R40, R43 to R41, R45 to R43, R47 to R45, R48 to R46, R49 to R47, R50 to R48, R46 to R49, R4 to R5, R51 to R50, R52 to R51, R55 to R52, R56 to R55, R60 to R56, R61 to R59, R62 to R60, R65 to R61, R59 to R62, R66 to R65, R39 to R66, R69 to R67, R40 to R69, R72 to R70, R70 to R71, R75 to R72, R77 to R73, R71 to R74, R73 to R75, R78 to R76, R76 to R77, R74 to R78, R81 to R80, R80 to R81, R88 to R87, R89 to R88, R91 to R89, R87 to R91, R72 to R92, R72 to R93, R72 to R94, R1 to R95, R1 to R96, R72 to R97, R72 to R98, R72 to R99, U1 to U12, U1 to U13, U1 to U2, U2 to U3, U1 to U4, U1 to U5, U3 to U7, U1 to U8, U1 to U9
Connections:
- C11 pad 1: (no net) -> D28_1_PC110
- C13 pad 1: C12_1 -> R284_2_PC110
- C15 pad 2: (no net) -> GND
- C16 pad 2: (no net) -> Q43_2_PC110
- C17 pad 1: C16_1 -> R284_2_PC110
- C20 pad 1: (no net) -> M38_P63_PC110
- C22 pad 1: (no net) -> PNET1_PC110
- C28 pad 2: (no net) -> PNET5_PC110
- C34 pad 2: (no net) -> Q43_2_PC110
- C35 pad 1: (no net) -> PNET4_PC110
- C38 pad 1: (no net) -> GND
- C39 pad 1: (no net) -> J5_33_PC110
- C39 pad 2: (no net) -> GND
- C40 pad 2: (no net) -> GND
- C41 pad 1: (no net) -> GND
- C43 pad 2: (no net) -> GND
- C44 pad 2: (no net) -> GND
- C45 pad 2: (no net) -> R284_2_PC110
- C46 pad 2: (no net) -> GND
- C47 pad 1: (no net) -> GND
- C48 pad 2: (no net) -> GND
- C50 pad 1: (no net) -> PNET1_PC110
- C51 pad 2: (no net) -> R284_2_PC110
- C54 pad 2: (no net) -> GND
- C55 pad 1: (no net) -> M38_P61_PC110
- C56 pad 1: (no net) -> GND
- C57 pad 1: (no net) -> GND
- C58 pad 1: (no net) -> D28_1_PC110
- C59 pad 1: (no net) -> GND
- C59 pad 2: (no net) -> PNET5_PC110
- C6 pad 2: (no net) -> D28_1_PC110
- C61 pad 1: (no net) -> GND
- C62 pad 2: (no net) -> GND
- C63 pad 1: (no net) -> PNET5_PC110
- C66 pad 2: (no net) -> GND
- C67 pad 1: (no net) -> GND
- C67 pad 2: (no net) -> PNET5_PC110
- C68 pad 2: (no net) -> GND
- C69 pad 2: (no net) -> Q43_2_PC110
- D2 pad 1: (no net) -> PNET4_PC110
- D4 pad 2: (no net) -> Q49_1_PC110
- F3 pad 2: (no net) -> R284_2_PC110
- F4 pad 2: (no net) -> R284_2_PC110
- F5 pad 1: (no net) -> GND
- J1 pad 1: (no net) -> D18_2_3_PC110
- J2 pad 2: (no net) -> PWR_IN_NEG
- J2 pad 3: (no net) -> PWR_IN_NEG
- J3 pad 1: (no net) -> M38_P60_PC110
- J3 pad 10: (no net) -> PNET5_PC110
- J3 pad 11: (no net) -> PNET5_PC110
- J3 pad 12: (no net) -> D28_1_PC110
- J3 pad 13: (no net) -> Q43_2_PC110
- J3 pad 14: (no net) -> R284_2_PC110
- J3 pad 15: (no net) -> R73_2_PC110
- J3 pad 16: (no net) -> U54_VCC_PC110
- J3 pad 17: (no net) -> U54_1D_PC110
- J3 pad 18: (no net) -> M38_P52_PC110
- J3 pad 19: J1_19 -> M38_P20_PC110
- J3 pad 2: (no net) -> M38_P61_PC110
- J3 pad 21: (no net) -> M38_P63_PC110
- J3 pad 22: (no net) -> Q49_1_PC110
- J3 pad 23: (no net) -> PNET4_PC110
- J3 pad 24: (no net) -> GND
- J3 pad 25: (no net) -> GND
- J3 pad 26: (no net) -> D2_3_PC110
- J3 pad 27: (no net) -> M38_P64_PC110
- J3 pad 28: (no net) -> PNET1_PC110
- J3 pad 3: (no net) -> PNET4_PC110
- J3 pad 30: GND -> M38_VREF_PC110
- J3 pad 31: (no net) -> PNET5_PC110
- J3 pad 33: (no net) -> J5_33_PC110
- J3 pad 34: (no net) -> U21_131_PC110
- J3 pad 35: (no net) -> F65_ENAVEE_PC110
- J3 pad 36: (no net) -> U54_1Q_PC110
- J3 pad 38: (no net) -> M38_P53_PC110
- J3 pad 39: (no net) -> M38_P21_PC110
- J3 pad 4: (no net) -> PNET4_PC110
- J3 pad 40: (no net) -> D18_2_3_PC110
- J3 pad 5: (no net) -> GND
- J3 pad 6: (no net) -> J5_6_PC110
- J3 pad 7: (no net) -> GND
- J3 pad 8: (no net) -> PNET1_PC110
- L1 pad 2: (no net) -> L1_2
- Q1 pad 1: GND -> M38_VREF_PC110
- Q10 pad 2: (no net) -> PNET4_PC110
- Q11 pad 4: (no net) -> D28_1_PC110
- Q13 pad 4: (no net) -> Q43_2_PC110
- Q14 pad 2: GND -> M38_VREF_PC110
- Q16 pad 3: (no net) -> PNET5_PC110
- Q20 pad 3: (no net) -> D2_3_PC110
- Q25 pad 1: J1_19 -> M38_P20_PC110
- Q26 pad 2: (no net) -> PNET4_PC110
- Q27 pad 1: (no net) -> J5_6_PC110
- Q29 pad 1: J1_38 -> M38_P53_PC110
- Q32 pad 2: (no net) -> GND
- Q33 pad 1: (no net) -> M38_P20_PC110
- Q33 pad 2: (no net) -> GND
- R100 pad 1: (no net) -> M38_P61_PC110
- R103 pad 2: (no net) -> GND
- R105 pad 1: (no net) -> GND
- R106 pad 2: (no net) -> GND
- R110 pad 2: (no net) -> GND
- R111 pad 1: (no net) -> GND
- R112 pad 2: (no net) -> GND
- R113 pad 1: (no net) -> GND
- R114 pad 2: (no net) -> GND
- R17 pad 2: (no net) -> PNET5_PC110
- R21 pad 1: (no net) -> PNET5_PC110
- R24 pad 1: (no net) -> PNET5_PC110
- R25 pad 1: (no net) -> PNET5_PC110
- R26 pad 2: (no net) -> PNET5_PC110
- R3 pad 1: GND -> M38_P52_PC110
- R32 pad 1: (no net) -> PNET1_PC110
- R34 pad 1: (no net) -> PNET5_PC110
- R39 pad 1: (no net) -> M38_P61_PC110
- R42 pad 1: (no net) -> PNET1_PC110
- R51 pad 1: (no net) -> M38_P64_PC110
- R52 pad 1: (no net) -> M38_P63_PC110
- R55 pad 1: (no net) -> PNET1_PC110
- R60 pad 2: (no net) -> PNET4_PC110
- R66 pad 1: (no net) -> M38_P64_PC110
- R67 pad 2: (no net) -> M38_P63_PC110
- R79 pad 2: (no net) -> Q43_2_PC110
- R80 pad 2: (no net) -> R73_2_PC110
- R81 pad 2: (no net) -> U54_1Q_PC110
- R82 pad 2: (no net) -> PNET5_PC110
- R83 pad 1: (no net) -> PNET4_PC110
- R85 pad 2: (no net) -> Q49_1_PC110
- R9 pad 2: (no net) -> PNET5_PC110
- R92 pad 2: (no net) -> GND
- R93 pad 1: (no net) -> J5_33_PC110
- R94 pad 2: (no net) -> J5_33_PC110
- R96 pad 2: (no net) -> GND
- R97 pad 2: (no net) -> GND
- U1 pad 3: (no net) -> GND
- U12 pad 1: (no net) -> PNET4_PC110
- U12 pad 2: (no net) -> PNET4_PC110
- U12 pad 3: (no net) -> PNET4_PC110
- U12 pad 5: (no net) -> L1_2
- U12 pad 6: (no net) -> L1_2
- U12 pad 7: (no net) -> L1_2
- U12 pad 8: (no net) -> L1_2
- U13 pad 1: (no net) -> PNET4_PC110
- U13 pad 2: (no net) -> PNET4_PC110
- U13 pad 3: (no net) -> PNET4_PC110
- U13 pad 5: (no net) -> R284_2_PC110
- U13 pad 6: (no net) -> R284_2_PC110
- U13 pad 7: (no net) -> R284_2_PC110
- U13 pad 8: (no net) -> R284_2_PC110
- U2 pad 5: (no net) -> PNET5_PC110
- U4 pad 1: (no net) -> GND
- U4 pad 5: (no net) -> R284_2_PC110
- U4 pad 6: (no net) -> R284_2_PC110
- U5 pad 20: (no net) -> GND
- U5 pad 4: (no net) -> GND
- U5 pad 5: (no net) -> GND
- U5 pad 9: (no net) -> GND
- U7 pad 1: (no net) -> M38_P63_PC110
- U7 pad 11: (no net) -> GND
- U7 pad 14: (no net) -> M38_P61_PC110
- U7 pad 7: (no net) -> M38_P64_PC110
- U7 pad 8: (no net) -> M38_P60_PC110
- U8 pad 5: (no net) -> R284_2_PC110
- U8 pad 6: (no net) -> R284_2_PC110
- U8 pad 7: (no net) -> R284_2_PC110
- U8 pad 8: (no net) -> R284_2_PC110
- U9 pad 1: (no net) -> GND
- U9 pad 2: (no net) -> GND
- U9 pad 3: (no net) -> GND
Routing:
- net (no net): track 1877.4 -> 1444.8 mm, vias 140 -> 84
- net GND: track 364.1 -> 549.1 mm, vias 54 -> 56
- net PNET5_PC110: track 0.00 -> 124.1 mm, vias 0 -> 7
- net PNET4_PC110: track 0.00 -> 101.7 mm, vias 0 -> 3
- net R284_2_PC110: track 0.00 -> 100.4 mm, vias 0 -> 9
- net J5_33_PC110: track 0.00 -> 83.6 mm, vias 0 -> 2
- net M38_VREF_PC110: track 0.00 -> 81.1 mm, vias 0 -> 4
- net M38_P61_PC110: track 0.00 -> 53.6 mm, vias 0 -> 3
- net M38_P63_PC110: track 0.00 -> 53.3 mm, vias 0 -> 3
- net J5_6_PC110: track 0.00 -> 53.1 mm, vias 0 -> 4
- net M38_P20_PC110: track 0.00 -> 50.9 mm, vias 0 -> 2
- net D2_3_PC110: track 0.00 -> 48.6 mm, vias 0 -> 2
- net J1_19: track 47.8 -> 0.00 mm, vias 2 -> 0
- net D18_2_3_PC110: track 0.00 -> 46.4 mm, vias 0 -> 3
- net M38_P52_PC110: track 0.00 -> 44.2 mm, vias 0 -> 2
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- added copper zone on In1.Cu, net PWR_IN_NEG
Other:
- outline, holes or cut-outs redrawn

Commit message: Add files via upload
Parts:
- removed the Q12 at (131.5, 103.7)
- removed the Q3 at (117.3, 80.0)
- added Q10: 3D, PC110:3D, F.Cu at (131.4, 103.8)
- added Q2: 3D, PC110:3D, F.Cu at (117.2, 80.3)
- C2: renamed from C1; value C_0603_1608Metric -> 150nF
- Q1: value SOT-23 -> 3D; footprint Package_TO_SOT_SMD:SOT-23 -> PC110:3D
- R3: renamed from R6; value R_0603_1608Metric -> 470
- moved Q1 0.37 mm to (113.8, 83.6), turned to 180 degrees
- moved Q6 0.22 mm to (109.8, 100.3)
- renumbered C2 to C1, C11 to C10, C15 to C11, C16 to C12, C12 to C14, C17 to C15, C14 to C16, C10 to C17, C28 to C18, C23 to C19, C21 to C20, C22 to C21, C18 to C22, C24 to C23, C26 to C24, C19 to C26, C20 to C28, C30 to C29, C29 to C30, C32 to C31, C33 to C32, C31 to C33, C7 to C4, C46 to C44, C47 to C45, C45 to C46, C48 to C47, C50 to C48, C8 to C5, C52 to C50, C53 to C51, C44 to C52, C51 to C53, C61 to C57, C9 to C6, C62 to C61, C63 to C62, C57 to C63, C66 to C64, C64 to C65, C65 to C66, C6 to C7, C5 to C8, C4 to C9, Q9 to Q11, Q10 to Q12, Q8 to Q13, Q16 to Q14, Q14 to Q15, Q15 to Q16, Q21 to Q19, Q22 to Q21, Q19 to Q22, Q24 to Q23, Q23 to Q24, Q28 to Q25, Q27 to Q26, Q26 to Q27, Q25 to Q28, Q4 to Q3, Q31 to Q30, Q30 to Q31, Q2 to Q4, Q7 to Q6, Q6 to Q7, Q13 to Q8, Q11 to Q9, R20 to R10, R104 to R103, R105 to R104, R106 to R105, R107 to R106, R108 to R107, R109 to R108, R110 to R109, R9 to R11, R111 to R110, R99 to R111, R116 to R115, R115 to R116, R13 to R12, R10 to R13, R11 to R14, R14 to R15, R19 to R16, R15 to R17, R16 to R18, R17 to R19, R18 to R20, R35 to R22, R24 to R23, R31 to R24, R28 to R25, R30 to R26, R32 to R27, R25 to R28, R27 to R29, R33 to R30, R22 to R31, R38 to R32, R34 to R33, R23 to R34, R36 to R35, R37 to R36, R29 to R37, R26 to R38, R69 to R40, R45 to R41, R41 to R42, R42 to R43, R43 to R44, R44 to R45, R51 to R46, R52 to R47, R46 to R48, R47 to R49, R3 to R5, R48 to R50, R56 to R51, R66 to R52, R67 to R53, R59 to R54, R53 to R55, R54 to R56, R60 to R57, R57 to R58, R58 to R59, R5 to R6, R61 to R60, R62 to R61, R65 to R62, R55 to R63, R63 to R64, R64 to R65, R40 to R66, R50 to R67, R49 to R68, R68 to R69, R74 to R70, R77 to R71, R70 to R72, R75 to R73, R76 to R74, R71 to R75, R73 to R76, R78 to R77, R72 to R78, R81 to R79, R79 to R81, R86 to R82, R85 to R83, R82 to R84, R83 to R85, R84 to R86, R89 to R87, R91 to R88, R87 to R89, R12 to R9, R88 to R90, R90 to R91, R103 to R98, R98 to R99, U11 to U10, U10 to U11, U7 to U5, U5 to U7, U9 to U8, U8 to U9
Connections:
- C2 pad 2: (no net) -> M38_VREF_PC110
- C23 pad 1: (no net) -> M38_P60_PC110
- C29 pad 1: (no net) -> PWR_IN_NEG
- C3 pad 2: (no net) -> U54_VCC_PC110
- C30 pad 2: (no net) -> GND
- C9 pad 1: (no net) -> GND
- D1 pad 1: (no net) -> J5_6_PC110
- Q1 pad 1: M38_VREF_PC110 -> GND
- Q1 pad 2: GND -> (no net)
- Q1 pad 3: (no net) -> M38_VREF_PC110
- Q4 pad 2: (no net) -> U54_VCC_PC110
- R10 pad 1: (no net) -> GND
- R13 pad 2: (no net) -> U21_131_PC110
- R2 pad 2: (no net) -> R2_2
- R20 pad 2: (no net) -> GND
- R3 pad 1: (no net) -> M38_VREF_PC110
- R41 pad 1: (no net) -> M38_P60_PC110
- R42 pad 1: (no net) -> BATT_POS
- R50 pad 2: (no net) -> BATT_POS
- R64 pad 1: (no net) -> GND
- R66 pad 2: (no net) -> BATT_POS
- R68 pad 1: (no net) -> GND
- R7 pad 1: (no net) -> GND
- R7 pad 2: (no net) -> BATT_POS
- R8 pad 1: (no net) -> GND
- R8 pad 2: (no net) -> BATT_POS
- SW1 pad 1: (no net) -> U54_VCC_PC110
Routing:
- net U54_VCC_PC110: track 40.4 -> 104.0 mm, vias 3 -> 5
- net BATT_POS: track 0.00 -> 49.1 mm, vias 0 -> 1
- net GND: track 549.1 -> 595.2 mm
- net (no net): track 1444.8 -> 1405.5 mm, vias 84 -> 82
- net J5_6_PC110: track 53.1 -> 57.7 mm
- net M38_VREF_PC110: track 81.1 -> 85.6 mm
- net M38_P60_PC110: track 34.6 -> 37.0 mm
- net PWR_IN_NEG: track 19.4 -> 21.4 mm
- net R2_2: track 0.00 -> 1.71 mm
- net U21_131_PC110: track 38.7 -> 40.4 mm
- net PNET5_PC110: track 124.1 -> 125.3 mm
Other:
- outline, holes or cut-outs redrawn

Commit message: Add files via upload
Parts:
- removed the Q16 at (144.1, 100.2)
- removed the R96 at (174.8, 98.5)
- added Q17: 3D, PC110:3D, F.Cu at (144.0, 100.5)
- added R97: R_1206_3216Metric, Resistor_SMD:R_1206_3216Metric, B.Cu at (177.6, 98.4)
- R95: value C_1206_3216Metric -> R_1206_3216Metric; footprint Capacitor_SMD:C_1206_3216Metric -> Resistor_SMD:R_1206_3216Metric
- moved R95 2.84 mm to (174.7, 98.4)
- renumbered C12 to C10, C17 to C12, C10 to C15, C15 to C17, C28 to C18, C26 to C19, C19 to C23, C25 to C24, C27 to C25, C18 to C26, C23 to C27, C24 to C28, C33 to C32, C32 to C33, C40 to C38, C38 to C39, C39 to C40, C43 to C42, C42 to C43, C51 to C44, C56 to C45, C44 to C46, C46 to C47, C45 to C48, C47 to C49, C8 to C5, C49 to C50, C55 to C51, C50 to C52, C52 to C53, C48 to C54, C54 to C55, C53 to C56, C59 to C57, C57 to C59, C7 to C6, C61 to C60, C62 to C61, C63 to C62, C60 to C63, C66 to C65, C67 to C66, C68 to C67, C65 to C68, C6 to C7, C5 to C8, L3 to L2, L2 to L3, Q11 to Q10, Q9 to Q11, REF** to Q14, Q14 to Q16, REF** to Q19, Q17 to Q20, REF** to Q21, Q21 to Q23, Q20 to Q24, Q19 to Q25, Q23 to Q26, Q24 to Q27, Q25 to Q28, Q28 to Q30, Q27 to Q31, Q26 to Q32, Q30 to Q33, Q31 to Q34, Q32 to Q35, Q33 to Q36, Q10 to Q8, Q8 to Q9, R15 to R10, R101 to R100, R102 to R101, R104 to R102, R105 to R104, R106 to R105, R107 to R106, R108 to R107, R109 to R108, R98 to R109, R9 to R11, R99 to R111, R116 to R115, R115 to R116, R16 to R13, R13 to R14, R11 to R15, R14 to R16, R5 to R2, R22 to R21, R24 to R22, R29 to R23, R21 to R24, R32 to R25, R27 to R26, R28 to R27, R26 to R28, R31 to R29, R2 to R3, R34 to R31, R23 to R32, R38 to R33, R33 to R34, R25 to R35, R37 to R36, R35 to R37, R36 to R38, R55 to R39, R63 to R40, R39 to R41, R40 to R42, R53 to R43, R56 to R44, R43 to R45, R44 to R46, R41 to R47, R45 to R48, R47 to R49, R6 to R5, R48 to R50, R49 to R51, R50 to R52, R46 to R53, R51 to R54, R52 to R55, R54 to R56, R67 to R57, R57 to R58, R58 to R59, R3 to R6, R59 to R60, R60 to R61, R61 to R63, R42 to R64, R64 to R65, R65 to R66, R66 to R67, R69 to R68, R68 to R69, R8 to R7, R77 to R70, R76 to R71, R75 to R73, R78 to R74, R74 to R75, R73 to R76, R71 to R77, R70 to R78, R81 to R79, R7 to R8, R79 to R80, R80 to R81, R84 to R82, R85 to R83, R86 to R84, R83 to R85, R82 to R86, R88 to R87, R89 to R88, R90 to R89, R10 to R9, R87 to R90, R93 to R92, R94 to R93, R92 to R94, R97 to R96, R111 to R98, R100 to R99, U11 to U10, U10 to U11, U13 to U12, U12 to U13, U9 to U8, U8 to U9
Connections:
- C1 pad 1: (no net) -> C1_1
- C1 pad 2: (no net) -> C1_2
- C11 pad 1: (no net) -> R31_1
- C12 pad 1: (no net) -> R24_2
- C12 pad 2: (no net) -> R36_2
- C14 pad 2: (no net) -> C14_2
- C16 pad 1: (no net) -> C16_1
- C17 pad 2: C16_2 -> GND
- C18 pad 2: (no net) -> U5_2
- C19 pad 1: (no net) -> U6_6
- C19 pad 2: (no net) -> U6_7
- C20 pad 2: (no net) -> J1_4
- C21 pad 2: (no net) -> C21_2
- C22 pad 1: (no net) -> C63_2
- C22 pad 2: (no net) -> U7_18
- C23 pad 1: (no net) -> Q17_2
- C23 pad 2: (no net) -> U7_25
- C24 pad 2: (no net) -> U7_6
- C25 pad 1: (no net) -> U6_2
- C25 pad 2: (no net) -> Q20_1
- C27 pad 2: (no net) -> C27_2
- C28 pad 1: (no net) -> R56_1
- C28 pad 2: (no net) -> R56_2
- C29 pad 2: (no net) -> PWR_IN_POS_Fuse
- C30 pad 1: (no net) -> GND
- C30 pad 2: GND -> PWR_IN_10v5
- C31 pad 1: (no net) -> C31_1
- C31 pad 2: (no net) -> C32_1
- C32 pad 1: (no net) -> C33_1
- C33 pad 1: (no net) -> C32_1
- C34 pad 1: (no net) -> R80_1
- C35 pad 2: (no net) -> C35_2
- C36 pad 1: (no net) -> C36_1
- C36 pad 2: (no net) -> C36_2
- C37 pad 1: (no net) -> GND
- C37 pad 2: (no net) -> Q33_2
- C38 pad 1: (no net) -> U7_10
- C39 pad 2: (no net) -> U7_2
- C4 pad 1: (no net) -> Q7_1
- C41 pad 2: (no net) -> U11_15
- C42 pad 1: (no net) -> R72_2
- C43 pad 1: (no net) -> U5_3
- C43 pad 2: (no net) -> Q33_3
- C44 pad 1: (no net) -> Q17_2
- C44 pad 2: (no net) -> R56_1
- C45 pad 2: (no net) -> R63_1
- C46 pad 1: (no net) -> R111_!
- C48 pad 2: (no net) -> U7_23
- C49 pad 1: (no net) -> U7_14
- C5 pad 1: (no net) -> Q6_2
- C5 pad 2: (no net) -> R20_1
- C50 pad 1: (no net) -> R106_2
- C50 pad 2: (no net) -> PNET4_PC110
- C51 pad 2: (no net) -> R65_2
- C52 pad 1: (no net) -> GND
- C52 pad 2: (no net) -> R106_1
- C53 pad 1: (no net) -> Q4_3
- C55 pad 1: (no net) -> Q4_3
- C59 pad 2: (no net) -> U11_1
- C6 pad 1: (no net) -> Q7_3
- C60 pad 1: (no net) -> Q6_2
- C61 pad 2: (no net) -> GND
- C62 pad 2: (no net) -> Q6_2
- C63 pad 1: (no net) -> C63_1
- C63 pad 2: (no net) -> C63_2
- C64 pad 1: (no net) -> U11_9
- C65 pad 1: (no net) -> U11_5
- C65 pad 2: (no net) -> R36_1
- C67 pad 1: (no net) -> R284_2_PC110_Fuse
- C68 pad 1: (no net) -> U11_5
- C68 pad 2: (no net) -> R115_2
- C7 pad 1: (no net) -> C6_1
- C7 pad 2: (no net) -> C6_2
- C8 pad 1: (no net) -> C8_1
- C8 pad 2: (no net) -> Q6_2
- C9 pad 2: (no net) -> R17_2
- D1 pad 2: (no net) -> D1_2
- D2 pad 2: (no net) -> R35_2
- D3 pad 1: (no net) -> PWR_IN_10v5
- D3 pad 2: (no net) -> R72_1
- D4 pad 1: (no net) -> Q14_2
- F1 pad 1: (no net) -> PWR_IN_POS_Fuse
- F1 pad 2: (no net) -> PWR_IN_POS
- F2 pad 1: (no net) -> J1_4
- F2 pad 2: (no net) -> R284_2_PC110
- F3 pad 1: (no net) -> F3_1
- F4 pad 1: (no net) -> R284_2_PC110_Fuse
- F5 pad 1: GND -> F2_1
- F5 pad 2: (no net) -> Q33_2
- J1 pad 2: (no net) -> J1_2
- J1 pad 4: (no net) -> J1_4
- J1 pad MP: (no net) -> J1_MP2
- J2 pad 1: (no net) -> PWR_IN_POS
- J3 pad 20: (no net) -> J1_2
- L1 pad 1: (no net) -> Q33_2
- L2 pad 1: (no net) -> F3_1
- L2 pad 2: (no net) -> L2_2
- L3 pad 1: (no net) -> Q8_5
- L3 pad 2: (no net) -> R284_2_PC110_Fuse
- Q1 pad 2: (no net) -> Q1_2
- Q10 pad 1: (no net) -> U54_VCC_PC110
- Q10 pad 3: (no net) -> C14_2
- Q11 pad 1: (no net) -> Q9_1
- Q11 pad 3: (no net) -> L2_2
- Q11 pad 5: (no net) -> L2_2
- Q12 pad 1: (no net) -> R35_2
- Q12 pad 3: (no net) -> C14_2
- Q13 pad 1: (no net) -> R21_1
- Q13 pad 3: (no net) -> Q13_3
- Q14 pad 1: (no net) -> R48_2
- Q14 pad 2: (no net) -> Q14_2
- Q14 pad 3: (no net) -> R38_1
- Q15 pad 1: (no net) -> R68_1
- Q15 pad 3: (no net) -> R111_2
- Q16 pad 1: (no net) -> R61_1
- Q16 pad 2: (no net) -> R51_2
- Q18 pad 1: (no net) -> R59_1
- Q18 pad 3: (no net) -> R68_2
- Q19 pad 1: (no net) -> Q20_1
- Q19 pad 2: (no net) -> R51_1
- Q19 pad 3: (no net) -> U6_7
- Q2 pad 2: (no net) -> R6_2
- Q20 pad 1: (no net) -> U7_18
- Q20 pad 2: (no net) -> R63_1
- Q20 pad 3: (no net) -> U7_25
- Q21 pad 1: (no net) -> U5_12
- Q21 pad 3: (no net) -> C27_2
- Q22 pad 1: (no net) -> Q22_1
- Q22 pad 2: (no net) -> PWR_IN_10v5
- Q22 pad 3: (no net) -> R78_2
- Q23 pad 1: (no net) -> R73_2
- Q23 pad 3: (no net) -> R70_2
- Q24 pad 1: (no net) -> R77_1
- Q25 pad 1: (no net) -> R77_2
- Q25 pad 3: (no net) -> Q3_3
- Q26 pad 1: (no net) -> C32_1
- Q26 pad 3: (no net) -> C31_1
- Q27 pad 1: (no net) -> C33_1
- Q27 pad 3: (no net) -> Q27_3
- Q28 pad 1: (no net) -> R82_1
- Q28 pad 2: (no net) -> R50_1
- Q28 pad 3: (no net) -> C36_2
- Q29 pad 2: (no net) -> Q29_2
- Q29 pad 3: (no net) -> Q30_2
- Q3 pad 1: (no net) -> Q3_1
- Q3 pad 3: (no net) -> Q3_3
- Q30 pad 2: (no net) -> Q30_2
- Q30 pad 3: (no net) -> M38_P21_PC110
- Q31 pad 1: (no net) -> Q27_3
- Q31 pad 3: (no net) -> C35_2
- Q32 pad 2: (no net) -> U3_6
- Q32 pad 3: (no net) -> PWR_IN_10v5
- Q33 pad 1: (no net) -> R91_2
- Q33 pad 2: (no net) -> Q33_2
- Q33 pad 3: (no net) -> Q33_3
- Q34 pad 1: (no net) -> R88_1
- Q34 pad 2: (no net) -> GND
- Q34 pad 3: (no net) -> R91_1
- Q35 pad 1: (no net) -> R92_2
- Q35 pad 3: (no net) -> R77_2
- Q36 pad 3: (no net) -> Q36_3
- Q4 pad 1: (no net) -> Q4_1
- Q4 pad 3: (no net) -> Q4_3
- Q5 pad 1: (no net) -> D1_2
- Q5 pad 3: (no net) -> Q3_3
- Q6 pad 1: (no net) -> R17_2
- Q6 pad 2: (no net) -> Q6_2
- Q6 pad 3: (no net) -> R80_1
- Q7 pad 1: (no net) -> Q7_1
- Q7 pad 2: (no net) -> Q6_2
- Q7 pad 3: (no net) -> Q7_3
- Q8 pad 1: (no net) -> GND
- Q8 pad 2: (no net) -> C63_2
- Q8 pad 3: (no net) -> GND
- Q9 pad 1: (no net) -> Q8_1
- Q9 pad 3: (no net) -> Q8_5
- Q9 pad 5: (no net) -> Q8_5
- R1 pad 1: (no net) -> C1_2
- R1 pad 2: (no net) -> R32_1
- R10 pad 1: (no net) -> Q6_2
- R10 pad 2: (no net) -> C8_1
- R100 pad 1: (no net) -> R111_!
- R100 pad 2: (no net) -> R111_2
- R101 pad 1: (no net) -> U7_23
- R101 pad 2: (no net) -> R284_2_PC110
- R102 pad 2: (no net) -> R56_2
- R103 pad 1: (no net) -> U5_3
- R103 pad 2: (no net) -> GND
- R104 pad 1: (no net) -> R104_1
- R105 pad 1: (no net) -> R104_1
- R105 pad 2: (no net) -> Q36_3
- R106 pad 1: (no net) -> R106_1
- R106 pad 2: (no net) -> R106_2
- R107 pad 1: (no net) -> R104_1
- R107 pad 2: (no net) -> R111_2
- R108 pad 1: (no net) -> R111_!
- R109 pad 1: (no net) -> C21_2
- R11 pad 1: (no net) -> Q6_2
- R11 pad 2: (no net) -> R36_1
- R110 pad 2: (no net) -> R56_2
- R111 pad 1: (no net) -> R111_!
- R111 pad 2: (no net) -> R111_2
- R112 pad 1: (no net) -> U11_2
- R113 pad 2: (no net) -> Q7_3
- R114 pad 1: (no net) -> R80_1
- R115 pad 1: (no net) -> R36_1
- R115 pad 2: (no net) -> R115_2
- R116 pad 1: (no net) -> PNET5_PC110
- R116 pad 2: (no net) -> U11_9
- R12 pad 1: (no net) -> R32_1
- R12 pad 2: (no net) -> Q6_2
- R13 pad 1: (no net) -> R20_1
- R13 pad 2: (no net) -> Q6_2
- R14 pad 1: (no net) -> Q7_1
- R15 pad 1: (no net) -> R11_1
- R16 pad 1: (no net) -> Q8_1
- R16 pad 2: (no net) -> C6_2
- R17 pad 1: (no net) -> F65_ENAVEE_PC110
- R17 pad 2: (no net) -> R17_2
- R18 pad 1: (no net) -> Q7_3
- R18 pad 2: (no net) -> D28_1_PC110
- R19 pad 1: (no net) -> R19_1
- R2 pad 2: (no net) -> Q3_1
- R20 pad 1: (no net) -> R20_1
- R21 pad 1: (no net) -> R21_1
- R21 pad 2: (no net) -> R21_2
- R22 pad 1: (no net) -> Q9_1
- R22 pad 2: (no net) -> R24_2
- R23 pad 1: (no net) -> Q8_1
- R23 pad 2: (no net) -> C6_1
- R24 pad 2: (no net) -> C63_1
- R25 pad 1: (no net) -> R32_1
- R26 pad 2: (no net) -> R56_1
- R27 pad 2: (no net) -> C63_1
- R28 pad 1: (no net) -> R21_2
- R28 pad 2: (no net) -> R26_2
- R29 pad 1: (no net) -> R31_1
- R29 pad 2: (no net) -> R26_2
- R3 pad 1: (no net) -> Q4_3
- R30 pad 2: (no net) -> R38_1
- R31 pad 1: (no net) -> R31_1
- R31 pad 2: (no net) -> PNET4_PC110
- R32 pad 2: (no net) -> R48_2
- R33 pad 1: (no net) -> R38_1
- R34 pad 2: (no net) -> C63_1
- R35 pad 1: (no net) -> Q13_3
- R35 pad 2: (no net) -> R35_2
- R36 pad 1: (no net) -> R36_1
- R37 pad 1: (no net) -> C33_1
- R37 pad 2: (no net) -> U54_1D_PC110
- R38 pad 1: (no net) -> Q9_1
- R38 pad 2: (no net) -> R36_2
- R39 pad 1: (no net) -> U6_2
- R39 pad 2: (no net) -> Q20_1
- R4 pad 1: (no net) -> Q4_1
- R4 pad 2: (no net) -> Q3_3
- R40 pad 2: (no net) -> R56_1
- R41 pad 2: (no net) -> U6_6
- R42 pad 1: (no net) -> R54_2
- R43 pad 1: (no net) -> U6_2
- R44 pad 1: (no net) -> R56_1
- R44 pad 2: (no net) -> R56_2
- R45 pad 2: (no net) -> C21_2
- R46 pad 2: (no net) -> U5_6
- R47 pad 2: (no net) -> C27_2
- R48 pad 2: (no net) -> R48_2
- R49 pad 2: (no net) -> U5_2
- R5 pad 1: (no net) -> C1_1
- R5 pad 2: (no net) -> R32_1
- R50 pad 1: (no net) -> R50_1
- R50 pad 2: (no net) -> R50_2
- R51 pad 1: (no net) -> R51_1
- R51 pad 2: (no net) -> R51_2
- R52 pad 1: (no net) -> U5_12
- R53 pad 2: (no net) -> U5_6
- R54 pad 1: (no net) -> U3_6
- R54 pad 2: (no net) -> R54_2
- R55 pad 2: (no net) -> U5_6
- R56 pad 2: (no net) -> U5_10
- R57 pad 1: (no net) -> U5_12
- R58 pad 1: (no net) -> Q27_3
- R59 pad 1: (no net) -> R59_1
- R59 pad 2: (no net) -> Q30_2
- R6 pad 2: (no net) -> R6_2
- R60 pad 1: (no net) -> C36_1
- R60 pad 2: (no net) -> U3_6
- R61 pad 1: (no net) -> R61_1
- R61 pad 2: (no net) -> Q30_2
- R62 pad 1: (no net) -> R51_1
- R63 pad 1: (no net) -> R63_1
- R63 pad 2: (no net) -> U7_6
- R64 pad 2: (no net) -> U5_2
- R65 pad 2: (no net) -> R65_2
- R66 pad 1: (no net) -> U11_1
- R66 pad 2: (no net) -> R50_2
- R67 pad 1: (no net) -> C27_2
- R68 pad 1: (no net) -> R68_1
- R68 pad 2: (no net) -> R68_2
- R69 pad 2: (no net) -> U5_10
- R70 pad 1: (no net) -> Q22_1
- R70 pad 2: (no net) -> R70_2
- R71 pad 1: (no net) -> R76_1
- R71 pad 2: (no net) -> PWR_IN_10v5
- R72 pad 1: (no net) -> R72_1
- R72 pad 2: (no net) -> R72_2
- R73 pad 1: (no net) -> Q29_2
- R73 pad 2: (no net) -> R73_2
- R74 pad 1: (no net) -> R78_1
- R75 pad 2: (no net) -> R77_1
- R76 pad 1: (no net) -> R76_1
- R76 pad 2: (no net) -> R77_1
- R77 pad 1: (no net) -> R77_1
- R77 pad 2: (no net) -> R77_2
- R78 pad 1: (no net) -> R78_1
- R78 pad 2: (no net) -> R78_2
- R79 pad 1: (no net) -> R80_1
- R80 pad 1: (no net) -> C32_1
- R81 pad 1: (no net) -> R80_1
- R82 pad 1: (no net) -> R82_1
- R83 pad 2: (no net) -> C35_2
- R84 pad 1: (no net) -> C36_2
- R84 pad 2: (no net) -> C36_1
- R85 pad 1: (no net) -> Q14_2
- R86 pad 1: (no net) -> C35_2
- R86 pad 2: (no net) -> C31_1
- R87 pad 1: (no net) -> R89_1
- R87 pad 2: (no net) -> Q33_2
- R88 pad 1: (no net) -> R88_1
- R88 pad 2: (no net) -> Q29_2
- R89 pad 1: (no net) -> GND
- R89 pad 2: (no net) -> R89_1
- R9 pad 2: (no net) -> C8_1
- R90 pad 1: (no net) -> GND
- R90 pad 2: (no net) -> Q33_2
- R91 pad 1: (no net) -> R91_1
- R91 pad 2: (no net) -> R91_2
- R92 pad 2: (no net) -> R92_2
- R93 pad 1: (no net) -> SW1_2
- R94 pad 1: (no net) -> SW1_2
- R95 pad 1: (no net) -> PWR_IN_NEG
- R95 pad 2: (no net) -> GND
- R96 pad 1: (no net) -> R72_2
- R98 pad 1: (no net) -> U5_3
- R98 pad 2: (no net) -> Q33_3
- R99 pad 2: (no net) -> R65_2
- SW1 pad 2: (no net) -> SW1_2
- SW1 pad 3: (no net) -> SW1_3
- SW1 pad 4: (no net) -> SW1_4
- U1 pad 1: (no net) -> R21_2
- U1 pad 2: (no net) -> R31_1
- U1 pad 4: (no net) -> U1_4
- U1 pad 5: (no net) -> U1_5
- U10 pad 1: (no net) -> R19_1
- U10 pad 2: (no net) -> C6_2
- U10 pad 3: (no net) -> R19_1
- U10 pad 5: (no net) -> R24_2
- U10 pad 6: (no net) -> R11_1
- U10 pad 7: (no net) -> R24_2
- U11 pad 1: (no net) -> U11_1
- U11 pad 10: (no net) -> R19_1
- U11 pad 11: (no net) -> R20_1
- U11 pad 12: (no net) -> C1_2
- U11 pad 13: (no net) -> R32_1
- U11 pad 14: (no net) -> Q7_3
- U11 pad 15: (no net) -> U11_15
- U11 pad 16: (no net) -> Q6_2
- U11 pad 2: (no net) -> U11_2
- U11 pad 3: (no net) -> R80_1
- U11 pad 4: (no net) -> R36_1
- U11 pad 5: (no net) -> U11_5
- U11 pad 6: (no net) -> C8_1
- U11 pad 7: (no net) -> R11_1
- U11 pad 8: (no net) -> U11_8
- U11 pad 9: (no net) -> U11_9
- U12 pad 4: (no net) -> C35_2
- U13 pad 4: (no net) -> U3_1
- U2 pad 1: (no net) -> R51_1
- U2 pad 3: (no net) -> R50_2
- U2 pad 4: (no net) -> R50_1
- U3 pad 1: (no net) -> U3_1
- U3 pad 2: (no net) -> C36_1
- U3 pad 4: (no net) -> U3_1
- U3 pad 5: (no net) -> C36_1
- U3 pad 6: (no net) -> U3_6
- U4 pad 2: (no net) -> U7_24
- U4 pad 3: (no net) -> Q17_2
- U4 pad 4: (no net) -> U7_27
- U4 pad 7: (no net) -> Q17_2
- U4 pad 8: (no net) -> Q17_2
- U5 pad 10: (no net) -> U5_10
- U5 pad 12: (no net) -> U5_12
- U5 pad 13: (no net) -> R65_2
- U5 pad 2: (no net) -> U5_2
- U5 pad 3: (no net) -> U5_3
- U5 pad 4: (no net) -> Q4_3
- U5 pad 5: (no net) -> R78_1
- U5 pad 6: (no net) -> U5_6
- U5 pad 9: (no net) -> C27_2
- U6 pad 1: (no net) -> Q20_1
- U6 pad 2: (no net) -> U6_2
- U6 pad 3: (no net) -> R111_!
- U6 pad 5: (no net) -> R104_1
- U6 pad 6: (no net) -> U6_6
- U6 pad 7: (no net) -> U6_7
- U6 pad 8: (no net) -> Q4_3
- U7 pad 1: (no net) -> R56_2
- U7 pad 10: (no net) -> U7_10
- U7 pad 11: (no net) -> GND
- U7 pad 12: (no net) -> U7_6
- U7 pad 13: (no net) -> U7_6
- U7 pad 14: (no net) -> U7_14
- U7 pad 15: (no net) -> C63_1
- U7 pad 16: (no net) -> U8_4
- U7 pad 17: (no net) -> C63_2
- U7 pad 18: (no net) -> U7_18
- U7 pad 19: (no net) -> U9_4
- U7 pad 2: (no net) -> U7_2
- U7 pad 21: (no net) -> PNET5_PC110
- U7 pad 22: (no net) -> R63_1
- U7 pad 23: (no net) -> U7_23
- U7 pad 24: (no net) -> U7_24
- U7 pad 25: (no net) -> U7_25
- U7 pad 26: (no net) -> Q17_2
- U7 pad 27: (no net) -> U7_27
- U7 pad 28: (no net) -> C21_2
- U7 pad 3: (no net) -> U7_6
- U7 pad 6: (no net) -> U7_6
- U7 pad 7: (no net) -> U7_7
- U7 pad 8: (no net) -> U7_8
- U8 pad 1: (no net) -> C63_2
- U8 pad 2: (no net) -> C63_2
- U8 pad 3: (no net) -> C63_2
- U8 pad 4: (no net) -> U8_4
- U9 pad 4: (no net) -> U9_4
- U9 pad 5: (no net) -> C63_2
- U9 pad 6: (no net) -> C63_2
- U9 pad 7: (no net) -> C63_2
- U9 pad 8: (no net) -> C63_2
Routing:
- net (no net): track 1405.5 -> 0.00 mm, vias 82 -> 0
- net Q4_3: track 0.00 -> 83.9 mm, vias 0 -> 2
- net Q3_3: track 0.00 -> 74.3 mm, vias 0 -> 3
- net C63_2: track 0.00 -> 62.9 mm, vias 0 -> 2
- net C63_1: track 0.00 -> 54.4 mm, vias 0 -> 2
- net U11_1: track 0.00 -> 53.3 mm, vias 0 -> 2
- net U9_4: track 0.00 -> 50.5 mm, vias 0 -> 2
- net U8_4: track 0.00 -> 46.6 mm, vias 0 -> 2
- net J1_2: track 0.00 -> 44.5 mm, vias 0 -> 2
- net PNET5_PC110: track 125.3 -> 168.9 mm, vias 7 -> 9
- net PWR_IN_10v5: track 0.00 -> 43.3 mm, vias 0 -> 8
- net R80_1: track 0.00 -> 43.2 mm, vias 0 -> 2
- net Q17_2: track 0.00 -> 41.8 mm, vias 0 -> 2
- net R77_2: track 0.00 -> 32.8 mm, vias 0 -> 3
- net R38_1: track 0.00 -> 27.6 mm
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- added copper zone on In1.Cu, net GND
- added copper zone on In1.Cu, net PNET5_PC110
- added copper zone on In1.Cu, net PWR_IN_10v5
