File: PSU/PSU.kicad_pcb (KiCad board)
At the start: 4 copper layers, 72.3 x 45 mm, 250 parts, among them J1 Backllight_Connector, J2 PSU_Jack, J3 PSU_Connector_Receptor, Q1 3D, Q10 SOT-89-3, Q11 SOT-powerT, Q12 SOT-416, Q13 SOT-416, Q14 3D, Q15 SOT-416, Q16 SOT-416, Q17 3D, Q18 SOT-416, Q19 3D, Q2 3D, Q20 3D, Q21 3D, Q22 SOT-416, Q23 SOT-416, Q24 SOT-416, Q25 SOT-416, Q26 SOT-416, Q27 SOT-23-PC110, Q28 SOT-416, Q29 3D, Q3 SOT-416, Q30 3D, Q31 SOT-23-PC110, Q32 3D, Q33 SOT-416, Q34 SOT-416, Q35 SOT-416, Q36 SOT-416, Q4 SOT-416, Q5 SOT-416, Q6 SOT-416, Q7 SOT-416, Q8 3D, Q9 SOT-powerT, SW1 PSU-SW1, U1 SOT-23-5, U10 SSOP-8-PSU, U11 SSOP-16_4.4x5.2mm_P0.65mm, U12 SOP-8_3.9x4.9mm_P1.27mm, U13 SOP-8_3.9x4.9mm_P1.27mm, U2 SOT-23-5, U3 SOT-23-6_Handsoldering, U4 SOP-8_3.9x4.9mm_P1.27mm, U5 TSSOP-14_4.4x5mm_P0.65mm, U6 SSOP-8-PSU, U7 TSSOP-28_6.1x9.7mm_P0.65mm, U8 SOP-8_3.9x4.9mm_P1.27mm, U9 SOP-8_3.9x4.9mm_P1.27mm

Commit message: Add files via upload
Parts:
- removed the C44 at (141.2, 99.3)
- removed the C63 at (125.5, 100.5)
- added D3: DNP, Diode_SMD:D_1206_3216Metric, F.Cu at (120.5, 96.9)
- added D6: DNP, Diode_SMD:D_1206_3216Metric, B.Cu at (169.6, 119.2)
- added D7: D_1206_3216Metric, Diode_SMD:D_1206_3216Metric, B.Cu at (159.5, 117.7)
- added D8: D_1206_3216Metric, Diode_SMD:D_1206_3216Metric, B.Cu at (156.5, 117.7)
- added L2: 10uH, Inductor_THT:L_Radial_D10.0mm_P5.00mm_Fastron_07M, B.Cu at (141.2, 99.3)
- added L5: 10uH, Inductor_THT:L_Radial_D10.0mm_P5.00mm_Fastron_07M, B.Cu at (125.6, 100.5)
- added Q36: 3P4J, Package_TO_SOT_SMD:TO-252-2, B.Cu at (169.7, 105.0)
- added R95: DNP, Resistor_SMD:R_1206_3216Metric, B.Cu at (176.3, 102.4)
- added R97: DNP, Resistor_SMD:R_1206_3216Metric, B.Cu at (176.2, 94.3)
- C10: renamed from C12; value C_0603_1608Metric -> 3.6nF
- C11: renamed from C15; value C_0603_1608Metric -> 180nF
- C12: renamed from C14; value C_1206_3216Metric -> 1.2uF
- C13: value C_1206_3216Metric -> 1.5uF
- C14: renamed from C17; value C_1206_3216Metric -> 1.5uF
- C15: renamed from C16; value C_0603_1608Metric -> 180nF
- C16: renamed from C11; value C_0603_1608Metric -> 150nF
- C17: renamed from C10; value C_0603_1608Metric -> 10nF
- C18: renamed from C22; value C_0603_1608Metric -> 120nF
- C19: renamed from C23; value C_0603_1608Metric -> 18nF
- C2: renamed from C1; value C_0603_1608Metric -> 4.7nF
- C20: renamed from C18; value C_0603_1608Metric -> 100pF
- C21: renamed from C19; value C_0603_1608Metric -> 12nF
- C22: renamed from C21; value C_0603_1608Metric -> 10nF
- C23: renamed from C24; value C_0805_2012Metric -> 1.5uF
- C24: renamed from C20; value C_0603_1608Metric -> 150nF
- C25: renamed from C27; value C_0603_1608Metric -> 1.2nF
- C26: renamed from C28; value C_0603_1608Metric -> 10nF
- C27: renamed from C25; value C_0603_1608Metric -> 1.2nF
- C28: renamed from C26; value C_0603_1608Metric -> 150nF
- C29, C30, C9: value C_0603_1608Metric -> 10nF
- C3: value C_1206_3216Metric -> 5.2uF
- C31: renamed from C32; value C_0603_1608Metric -> 1.2nF
- C32: renamed from C34; value C_0603_1608Metric -> 10nF
- C33: renamed from C31; value C_0603_1608Metric -> 24nF
- C34: renamed from C33; value C_0805_2012Metric -> 1.5uF
- C35: renamed from C36; value C_0603_1608Metric -> 1.2nF
- C36: renamed from C35; value C_0603_1608Metric -> 150nF
- C37: value C_0603_1608Metric -> 180nF
- C38, C41: value C_0805_2012Metric -> 1.5uF
- C39: renamed from C40; value C_0603_1608Metric -> 10nF
- C4: renamed from C7; value C_0603_1608Metric -> 2.5nF
- C40: renamed from C39; value C_0603_1608Metric -> 10nF
- C42, C64: value C_0603_1608Metric -> 120nF
- C43: value C_0603_1608Metric -> 10pF
- C44: renamed from C55; value C_0603_1608Metric -> 180nF
- C45: renamed from C56; value C_Disc_D3.0mm_W1.6mm_P2.50mm -> 33uF 20V
- C46, C5: value C_0603_1608Metric -> 150nF
- C47: renamed from C48; value C_0603_1608Metric -> 150nF
- C48: renamed from C49; value C_0603_1608Metric -> 10nF
- C49: renamed from C53; value C_0603_1608Metric -> 180nF
- C50: renamed from C47; value EC -> 56uF 25V EC
- C51: renamed from C52; value C_0603_1608Metric -> 120nF
- C52: renamed from C51; value C_0603_1608Metric -> 1nF
- C53: renamed from C50; value C_0603_1608Metric -> 120nF
- C54, C61: value C_Radial_D6.3mm_H11.0mm_P2.50mm -> 47uF 6.3v
- C55: renamed from C45; value C_0805_2012Metric -> 1.5uF
- C56: renamed from C57; value C_Radial_D6.3mm_H11.0mm_P2.50mm -> 47uF 6.3V
- C57: renamed from C58; value C_Radial_D6.3mm_H11.0mm_P2.50mm -> 15uF 16V
- C58: renamed from C62; value C_0805_2012Metric -> 1.5uF
- C59: renamed from C60; value C_0603_1608Metric -> 150nF
- C6: value C_0603_1608Metric -> 100pF
- C62: renamed from C66; value C_0603_1608Metric -> 100nF
- C63: renamed from C65; value C_0603_1608Metric -> 5.1nF
- C65: renamed from C67; value C_0603_1608Metric -> 100nF
- C66: renamed from C68; value C_0603_1608Metric -> 1.2nF
- C67: renamed from C69; value C_Radial_D6.3mm_H11.0mm_P2.50mm -> 18uF 50V
- C7: renamed from C8; value C_0603_1608Metric -> 150nF
- C8: renamed from C4; value C_0603_1608Metric -> 24nF
- D1: value D_0603_1608Metric -> 8-2
- D2: value D_0603_1608Metric -> 5-9
- D4: renamed from D3; value D_0603_1608Metric -> 18
- D5: renamed from D4; value D_0603_1608Metric -> 3^9
- F1, F5: value Fuse_2010_5025Metric -> 2.5A
- F2: value Fuse_2010_5025Metric -> 830mA
- F3: value Fuse_1206_3216Metric -> 15
- F4: value Fuse_1210_3225Metric -> 10
- L1: value L_Radial_D7.5mm_P5.00mm_Fastron_07P -> 10uH
- L3: renamed from L2; value L_Coilcraft_LPS5030 -> 68uH
- L4: renamed from L3; value L_Coilcraft_LPS5030 -> 470uH
- Q1: value 3D -> R4C
- Q10: renamed from Q11; value SOT-powerT -> 103 5G
- Q11: renamed from Q12; value SOT-416 -> 6LS
- Q12: renamed from Q8; value 3D -> Q
- Q13: value SOT-416 -> 8LR
- Q14: renamed from Q15; value SOT-416 -> 6LS
- Q15: renamed from Q16; value SOT-416 -> 8LR
- Q16: renamed from Q19; value 3D -> M2P
- Q17: renamed from Q20; value 3D -> M2P
- Q18: renamed from Q17; value 3D -> Q
- Q19: renamed from Q21; value 3D -> M2P
- Q2, Q32: value 3D -> K
- Q20: renamed from Q14; value 3D -> W6
- Q21: renamed from Q18; value SOT-416 -> 8C
- Q22: renamed from Q25; value SOT-416 -> 8C
- Q23: renamed from Q24; value SOT-416 -> 8C
- Q24: renamed from Q22; value SOT-416 -> 6LS
- Q25: renamed from Q23; value SOT-416 -> 8LB
- Q26: renamed from Q27; value SOT-23-PC110 -> G16
- Q27: renamed from Q26; value SOT-416 -> 8C
- Q28: renamed from Q30; value 3D -> W6
- Q29: renamed from Q31; value SOT-23-PC110 -> H15
- Q3: renamed from Q4; value SOT-416 -> 6LS
- Q30: renamed from Q28; value SOT-416 -> 8C
- Q31: renamed from Q29; value 3D -> W6
- Q33: renamed from Q34; value SOT-416 -> 8LR
- Q34: renamed from Q33; value SOT-416 -> 6LS
- Q35, Q5: value SOT-416 -> 8C
- Q37: renamed from Q36; value SOT-416 -> 8LR
- Q4: renamed from Q3; value SOT-416 -> 8LR
- Q6: renamed from Q7; value SOT-416 -> 6LS
- Q7: renamed from Q6; value SOT-416 -> 6LS
- Q8: renamed from Q9; value SOT-powerT -> 303 5H
- Q9: renamed from Q10; value SOT-89-3 -> KD 3.E
- R1, R50: value R_0603_1608Metric -> DNP
- R10: renamed from R14; value R_0603_1608Metric -> 470k
- R100: renamed from R109; value R_0603_1608Metric -> 7.5k
- R101: renamed from R99; value R_0603_1608Metric -> 200k
- R102: renamed from R98; value R_0603_1608Metric -> 300k
- R103: renamed from R100; value R_0603_1608Metric -> 10k
- R104: renamed from R101; value R_0603_1608Metric -> 100
- R105: renamed from R103; value R_0603_1608Metric -> 100k
- R106: renamed from R104; value R_0603_1608Metric -> 4.7k
- R107: renamed from R105; value R_0603_1608Metric -> 2k
- R108: renamed from R110; value R_0603_1608Metric -> DNP
- R109: renamed from R111; value R_0603_1608Metric -> 200k
- R11: renamed from R12; value R_0603_1608Metric -> 10k
- R110: renamed from R102; value R_0603_1608Metric -> 7.5k
- R111: renamed from R106; value R_0603_1608Metric -> 33
- R112: renamed from R107; value R_0603_1608Metric -> 20k
- R113: renamed from R108; value R_0603_1608Metric -> 20k
- R114: renamed from R112; value R_0603_1608Metric -> 10k
- R115: renamed from R114; value R_0603_1608Metric -> 11K
- R116: renamed from R113; value R_0603_1608Metric -> 15k
- R117: renamed from R115; value R_0603_1608Metric -> 10k
- R118: renamed from R116; value R_0603_1608Metric -> 100
- R12: renamed from R16; value R_0603_1608Metric -> 2.2k
- R13: renamed from R11; value R_0603_1608Metric -> 10k
- R14: renamed from R10; value R_0603_1608Metric -> 12k
- R15: renamed from R17; value R_0603_1608Metric -> 100k
- R16: renamed from R18; value R_0603_1608Metric -> 130k
- R17: renamed from R19; value R_0603_1608Metric -> 10k
- R18: renamed from R20; value R_0603_1608Metric -> 20k
- R19: renamed from R13; value R_0603_1608Metric -> 10k
- R2, R83: value R_0603_1608Metric -> 470k
- R20: renamed from R15; value R_0603_1608Metric -> 10k
- R21: renamed from R29; value R_0603_1608Metric -> 470k
- R22: renamed from R31; value R_0603_1608Metric -> 100k
- R23: renamed from R24; value R_1206_3216Metric -> 0.1
- R24: renamed from R23; value R_0603_1608Metric -> 220
- R25: renamed from R27; value R_1206_3216Metric -> 0.1
- R26: renamed from R32; value R_1206_3216Metric -> 103 (RT1)
- R27: renamed from R30; value R_0603_1608Metric -> 4.7k
- R28: value R_0603_1608Metric -> 0
- R29: renamed from R33; value R_1206_3216Metric -> 103 (RT2)
- R3, R93: value R_0603_1608Metric -> 1k
- R30: renamed from R35; value R_0603_1608Metric -> 10k
- R31: renamed from R21; value R_0603_1608Metric -> 470k
- R33: renamed from R36; value R_0603_1608Metric -> 10k
- R34: value R_1206_3216Metric -> 0.1
- R35: renamed from R25; value R_0603_1608Metric -> 10k
- R36: renamed from R37; value R_0603_1608Metric -> 1k
- R37: renamed from R38; value R_0603_1608Metric -> 120
- R38: renamed from R22; value R_0603_1608Metric -> 470
- R39: renamed from R42; value R_0603_1608Metric -> 4.7k
- R4: renamed from R5; value R_0603_1608Metric -> 10k
- R41: renamed from R54; value R_0603_1608Metric -> 4.7k
- R42: renamed from R41; value R_0603_1608Metric -> 47k
- R43: renamed from R45; value R_0603_1608Metric -> 300
- R44: renamed from R69; value R_0603_1608Metric -> 10k
- R45: renamed from R56; value R_0603_1608Metric -> 200k
- R46: renamed from R58; value R_0603_1608Metric -> 1M
- R47: renamed from R61; value R_0603_1608Metric -> 47k
- R48: renamed from R63; value R_0603_1608Metric -> 100
- R49: renamed from R64; value R_0603_1608Metric -> 300k
- R5: renamed from R4; value R_0603_1608Metric -> 100k
- R51: value R_0603_1608Metric -> 4.7k
- R52, R86: value R_0603_1608Metric -> 10k
- R53: renamed from R46; value R_0603_1608Metric -> 300k
- R54: renamed from R53; value R_0603_1608Metric -> 100k
- R55: renamed from R39; value R_0603_1608Metric -> 1M
- R56: renamed from R44; value R_0603_1608Metric -> 300
- R57: renamed from R49; value R_0603_1608Metric -> 100k
- R58: renamed from R48; value R_0603_1608Metric -> 4.7k
- R59, R80, R92: value R_0603_1608Metric -> 100k
- R60: renamed from R62; value R_0603_1608Metric -> 4.7k
- R61: renamed from R60; value R_0603_1608Metric -> 10k
- R62: renamed from R47; value R_0603_1608Metric -> 200k
- R63: renamed from R67; value R_0603_1608Metric -> 10k
- R64: renamed from R65; value R_0603_1608Metric -> 10k
- R65: renamed from R66; value R_0603_1608Metric -> 1k
- R66: renamed from R55; value R_0603_1608Metric -> DNP
- R67: renamed from R43; value R_0603_1608Metric -> 47k
- R68, R94: value R_0603_1608Metric -> 47k
- R69: renamed from R57; value R_0603_1608Metric -> 200k
- R7: renamed from R8; value R_1210_3225Metric -> 0.1
- R70: renamed from R73; value R_0603_1608Metric -> 470k
- R71: renamed from R76; value R_0603_1608Metric -> 1k
- R72: renamed from R75; value R_0603_1608Metric -> 1k
- R73: renamed from R77; value R_0603_1608Metric -> 47k
- R74: renamed from R70; value R_0603_1608Metric -> 470k
- R75: renamed from R71; value R_0603_1608Metric -> 1k
- R76: renamed from R72; value R_0603_1608Metric -> 1k
- R77: renamed from R74; value R_0603_1608Metric -> 100k
- R78: value R_0603_1608Metric -> 300k
- R79: renamed from R81; value R_0603_1608Metric -> 47k
- R8: renamed from R7; value R_1210_3225Metric -> 0.1
- R81: renamed from R79; value R_0603_1608Metric -> 200k
- R82: renamed from R85; value R_0603_1608Metric -> DNP
- R84: renamed from R82; value R_0603_1608Metric -> 100k
- R85: renamed from R84; value R_0603_1608Metric -> 10k
- R87: renamed from R88; value R_0603_1608Metric -> 470k
- R88: renamed from R89; value R_0603_1608Metric -> 1M
- R89: renamed from R87; value R_0603_1608Metric -> 1M
- R9: value R_0603_1608Metric -> 20k
- R90: renamed from R91; value R_0603_1608Metric -> 470k
- R91: renamed from R90; value R_1206_3216Metric -> DNP
- R96: value R_0603_1608Metric -> 1.8k
- R98: renamed from R95; value R_1206_3216Metric -> 0
- R99: renamed from R97; value R_1206_3216Metric -> 0
- U1: value SOT-23-5 -> D9D
- U10: renamed from U11; value SSOP-16_4.4x5.2mm_P0.65mm -> 9742
- U11: renamed from U10; value SSOP-8-PSU -> 7W14
- U12, U13: value SOP-8_3.9x4.9mm_P1.27mm -> J421
- U2: value SOT-23-5 -> TA
- U3: value SOT-23-6_Handsoldering -> 6.5 5F
- U4: renamed from U7; value TSSOP-28_6.1x9.7mm_P0.65mm -> MAX786CAI
- U5: renamed from U4; value SOP-8_3.9x4.9mm_P1.27mm -> K2337
- U6: renamed from U5; value TSSOP-14_4.4x5mm_P0.65mm -> 7064
- U7: renamed from U6; value SSOP-8-PSU -> 5W01
- U8: renamed from U9; value SOP-8_3.9x4.9mm_P1.27mm -> 2556
- U9: renamed from U8; value SOP-8_3.9x4.9mm_P1.27mm -> 2556
- renumbered C2 to C1, C59 to C60, R26 to R32
Routing:
- net GND: track 586.1 -> 592.6 mm
- net R72_2: track 4.91 -> 9.07 mm
- net C14_2: track 7.04 -> 11.0 mm
- net PWR_IN_10v5: track 43.3 -> 46.8 mm
- net PNET4_PC110: track 103.4 -> 105.7 mm
- net PWR_IN_NEG: track 21.4 -> 22.9 mm
- net Q4_3: track 83.9 -> 84.8 mm
- net L1_2: track 11.4 -> 12.1 mm

Commit message: Add files via upload
Parts:
- added G***: LOGO, PC110:logo, F.Cu at (170.6, 86.4)
- D7, D8: value D_1206_3216Metric -> s.3 4F
Other:
- board text added: "Recreated with Love by Ahmad Byagowi"

Commit message: Add files via upload
Parts:
- C60: value C_0603_1608Metric -> 1nF
- R32: value R_1206_3216Metric -> 0.1
- R40: value R_1206_3216Metric -> 0.22
Connections:
- net C21_2 renamed MAX_FB3
- net C27_2 renamed JRC_IN3-
- net C63_1 renamed MAX_CS5
- net C63_2 renamed MAX_LX5
- net Q17_2 renamed MAX_LX3
- net Q4_3 renamed JRC_VDD
- net R56_2 renamed MAX_CS3
- net R63_1 renamed MAX_VL
- net R65_2 renamed JRC_IN4-
- net R78_1 renamed JRC_IN2+
- net U5_10 renamed JRC_IN3+
- net U5_12 renamed JRC_IN4+
- net U5_2 renamed JRC_IN1-
- net U5_3 renamed JRC_IN1+
- net U5_6 renamed JRC_IN2-
- net U7_10 renamed MAX_REF
- net U7_14 renamed MAX_SS5
- net U7_18 renamed MAX_BST5
- net U7_2 renamed MAX_SS3
- net U7_23 renamed MAX_VL+
- net U7_24 renamed MAX_DL3
- net U7_25 renamed MAX_BST3
- net U7_27 renamed MAX_DH3
- net U7_6 renamed ON3_ON5_VH_SHDN#
- net U7_7 renamed MAX_Q2
- net U7_8 renamed MAX_Q1
- net U8_4 renamed MAX_DH5
- net U9_4 renamed MAX_DL5
