File: PCB/PSU/PSU.kicad_pcb (KiCad board)
At the start: 4 copper layers, 72.3 x 45 mm, 258 parts, among them J1 Backllight_Connector, J2 PSU_Jack, J3 PSU_Connector_Receptor, Q1 R4C, Q10 103 5G, Q11 6LS, Q12 Q, Q13 8LR, Q14 6LS, Q15 8LR, Q16 M2P, Q17 M2P, Q18 Q, Q19 M2P, Q2 K, Q20 W6, Q21 8C, Q22 8C, Q23 8C, Q24 6LS, Q25 8LB, Q26 G16, Q27 8C, Q28 W6, Q29 H15, Q3 6LS, Q30 8C, Q31 W6, Q32 K, Q33 8LR, Q34 6LS, Q35 8C, Q36 3P4J, Q37 8LR, Q4 8LR, Q5 8C, Q6 6LS, Q7 6LS, Q8 303 5H, Q9 KD 3.E, SW1 PSU-SW1, U1 D9D, U10 9742, U11 7W14, U12 J421, U13 J421, U2 TA, U3 6.5 5F, U4 MAX786CAI, U5 K2337, U6 7064, U7 5W01, U8 2556, U9 2556

Commit message: Add files via upload
Routing:
- net GND: track 594.6 -> 599.0 mm
- added copper zone on F.Cu, net BATT_POS
- added copper zone on B.Cu, net F2_1
- added copper zone on B.Cu, net GND
- added copper zone on F.Cu, net GND
- added copper zone on B.Cu, net L1_2
- added copper zone on B.Cu, net MAX_LX5
- added copper zone on B.Cu, net PNET1_PC110
- added copper zone on B.Cu, net PNET4_PC110
- added copper zone on B.Cu, net PNET5_PC110
- added copper zone on B.Cu, net PWR_IN_NEG
- added copper zone on B.Cu, net PWR_IN_POS
- added copper zone on B.Cu, net Q33_2
- added copper zone on B.Cu, net R284_2_PC110

Commit message: Add files via upload
Routing:
- net GND: track 599.0 -> 603.4 mm
- added copper zone on F.Cu, net MAX_LX3
- added copper zone on F.Cu, net PNET1_PC110
- added copper zone on F.Cu, net Q33_2
- added copper zone on F.Cu, net R56_1
- added copper zone on F.Cu, net U3_1

Commit message: Add files via upload
Connections:
- net J1_2 renamed R412_1_PC110
Changed lines of the file:
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@@
 	(net 72 "C14_2")
 	(net 73 "R31_1")
-	(net 74 "J1_2")
+	(net 74 "R412_1_PC110")
 	(net 75 "J1_4")
 	(net 76 "R284_2_PC110_Fuse")
@@
 			(layers "F.Cu" "F.Mask" "F.Paste")
 			(roundrect_rratio 0.25)
-			(net 74 "J1_2")
+			(net 74 "R412_1_PC110")
 		)
 		(pad "3" smd roundrect
@@
 			(size 2.1 0.5)
 			(layers "B.Cu" "B.Mask" "B.Paste")
-			(net 74 "J1_2")
+			(net 74 "R412_1_PC110")
 			(thermal_bridge_angle 45)
 		)
