File: PCB/PSU/PSU.kicad_pcb (KiCad board)
At the start: 4 copper layers, 72.3 x 45 mm, 258 parts, among them J1 Backllight_Connector, J2 PSU_Jack, J3 PSU_Connector_Receptor, Q1 R4C, Q10 103 5G, Q11 6LS, Q12 Q, Q13 8LR, Q14 6LS, Q15 8LR, Q16 M2P, Q17 M2P, Q18 Q, Q19 M2P, Q2 K, Q20 W6, Q21 8C, Q22 8C, Q23 8C, Q24 6LS, Q25 8LB, Q26 G16, Q27 8C, Q28 W6, Q29 H15, Q3 6LS, Q30 8C, Q31 W6, Q32 K, Q33 8LR, Q34 6LS, Q35 8C, Q36 3P4J, Q37 8LR, Q4 8LR, Q5 8C, Q6 6LS, Q7 6LS, Q8 303 5H, Q9 KD 3.E, SW1 PSU-SW1, U1 D9D, U10 9742, U11 7W14, U12 J421, U13 J421, U2 TA, U3 6.5 5F, U4 MAX786CAI, U5 K2337, U6 7064, U7 5W01, U8 2556, U9 2556

Commit message: Add files via upload
Parts:
- G1: renamed from G***; moved to B.Cu
- moved G1 51.8 mm to (119.0, 82.1), turned to 180 degrees

Commit message: Add files via upload
Connections:
- C15 pad 1: C16_1 -> F3_1
Routing:
- net F3_1: track 3.44 -> 8.01 mm, vias 0 -> 1
- net C16_1: track 1.21 -> 0.00 mm, vias 1 -> 0
