File: PCB/PSU/PSU.kicad_sch (KiCad schematic)
At the start: 258 parts, among them J1 Backllight_Connector, J2 PSU_Jack, J3 PSU_Connector_Receptor, Q1 R4C, Q10 103 5G, Q11 6LS, Q12 Q, Q13 8LR, Q14 6LS, Q15 8LR, Q16 M2P, Q17 M2P, Q18 Q, Q19 M2P, Q2 K, Q20 W6, Q21 8C, Q22 8C, Q23 8C, Q24 6LS, Q25 8LB, Q26 G16, Q27 8C, Q28 W6, Q29 H15, Q3 6LS, Q30 8C, Q31 W6, Q32 K, Q33 8LR, Q34 6LS, Q35 8C, Q36 3P4J, Q37 8LR, Q4 8LR, Q5 8C, Q6 6LS, Q7 6LS, Q8 303 5H, Q9 KD 3.E, SW1 PSU-SW1, U1 D9D, U10 9742, U11 7W14, U12 J421, U13 J421, U2 TA, U3 6.5 5F, U4 MAX786CAI, U5 K2337, U6 7064, U7 5W01, U8 2556, U9 2556

Commit message: Personal notes for PSU understanding
Parts:
- D1: value 8-2 -> 8.2V
- Q12: symbol Device:D_Zener_Dual_CommonAnode_KAK -> Device:D_Zener_Dual_CommonCathode_AKA
- Q2: symbol Device:D_Dual_Series_KAC_Parallel -> Device:D_Dual_CommonCathode_AKA
- Q21: symbol Simulation_SPICE:NPN -> Transistor_BJT:Q_NPN_BEC
- Q22, Q4, Q5: symbol PCM_Transistor_BJT_AKL:Q_NPN_Generic_CEB -> Transistor_BJT:Q_NPN_BEC
- Q3, Q34: symbol Simulation_SPICE:PNP -> Transistor_BJT:Q_PNP_BEC
- Q32: symbol Device:D_Dual_Series_ACK_Parallel -> Device:D_Dual_CommonCathode_AKA
Connections:
- net PNET5_PC110 is gone; now on net PNET5_PC110_5V: C28.2 (-), C56.2 (-), C61.1 (+), C62.2 (-), J3.10 (Pin_10), J3.11 (Pin_11), J3.31 (Pin_31), Q15.3 (C), Q2.3 (A), R118.1 (+), R17.2 (-), R20.2 (-), R23.1 (+), R25.1 (+), R26.1 (+), R29.2 (-), R34.1 (+), R84.2 (-), U11.8 (VCC), U2.5 (VCC)
- net GND: now also Q21.2 (E); no longer Q21.3 (E)
- net at C37.2 (-), F5.2, L1.1 (+)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: now also Q34.2 (E); no longer Q34.3 (E)
- net at C9.2 (-), Q7.1 (C), R15.2 (-): no longer U10.7 (OUT1)
- net PNET4_PC110_RAW_AlwaysON: now reaches U13.5 (D), U13.6 (D), U13.7 (D), U13.8 (D)
- net PNET4_PC110_RAW_AlwaysON: now also C36.1 (+), C53.2 (-), D2.1 (K-), D7.1 (K-), D8.1 (K-), J3.23 (Pin_23), J3.3 (Pin_3), J3.4 (Pin_4), Q11.2 (E), Q29.2 (S), R22.2 (-), R46.2 (-), R83.1 (+), U12.1 (S), U12.2 (S), U12.3 (S); no longer D6.2 (-), L1.2 (-)
- net at R68.2 (-): now also Q21.3 (C); no longer Q21.2 (B)
- net Switched_Vref: now reaches Q14.3 (C), R103.2 (-), R109.2 (-), R112.2 (-)
- net at R20.1 (+), U11.6: now also U10.7 (OUT1)
- net at R78.2 (-): now also Q24.1 (C); no longer Q24.3 (B)
- net at C43.2 (-), R102.2 (-): now also Q34.3 (C); no longer Q34.1 (C)
- net at R90.1 (+): now also Q34.1 (B); no longer Q34.2 (B)
- net at R74.1 (+): now also Q24.3 (B); no longer Q24.1 (C)
- net D18_2_3_PC110 renamed D18_2_3_PC110_Backlight_EN3V3
- net D28_1_PC110 renamed D28_1_PC110_PWR12V
- net J5_33_PC110 renamed PSU_AUX_SW1
- net M38_P52_PC110 renamed M38_P52_PC110_JRC_VCC_Enable
- net M38_P53_PC110 renamed M38_P53_PC110_EN_PWR_Source_V_Sense
- net M38_P60_PC110 renamed M38_P60_PC110_Bat_NegCurrent_Sense
- net M38_P61_PC110 renamed M38_P61_PC110_Bat_PosCurrent_Sense
- net M38_P63_PC110 renamed M38_P63_PC110_Bat_VSense
- net M38_P64_PC110 renamed M38_P64_PC110_PWR_IN_Sense
- net PNET1 renamed PNET1_PC110_3V3_3V3
- net PNET1_PC110_3V3_3V3: now also C54.2 (-), R32.1 (+), R40.1 (+)
- removed net PNET1_PC110: C54.2 (-), J3.28 (Pin_28), J3.8 (Pin_8), R32.1 (+), R40.1 (+)
- removed net PNET4_PC110: C36.1 (+), C53.2 (-), D2.1 (K-), D7.1 (K-), D8.1 (K-), J3.23 (Pin_23), J3.3 (Pin_3), J3.4 (Pin_4), Q11.2 (E), Q29.2 (S), R22.2 (-), R46.2 (-), R83.1 (+), U12.1 (S), U12.2 (S), U12.3 (S), U13.1 (S), U13.2 (S), U13.3 (S)
- net PNET5 renamed PNET5_PC110_5V
- net Q43_2_PC110 renamed Q43_2_PC110_PWR25V
- net R284_2_PC110 renamed R284_2_PC110_BAT_or_PWR_IN_RAW
- net R412_1_PC110 renamed R412_1_PC110_Backlight_low_switch
- net U54_VCC_PC110 renamed U54_VCC_PC110_5V_AlwaysON
- new net: D6.2 (-), L1.2 (-), U13.1 (S), U13.2 (S), U13.3 (S)
- new net PNET1_PC110_3V3: J3.28 (Pin_28), J3.8 (Pin_8)
Other:
- moved on the sheet: D1, Q14, Q2, Q22, Q24, Q3, Q32, Q4, Q5, Q7, R115, R2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
