File: PCB/DockingStation/DockingStation.kicad_pcb (KiCad board)
At the start: 2 copper layers, 147.2 x 63.2 mm, 249 parts, among them CN1 DSUB-15-HD_Socket_Horizontal_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, CN2 FDC_Connector, CN4 DSUB-25_Socket_Horizontal_P2.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, CN5 DSUB-9_Pins_Horizontal_P2.77x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, CN6 PS2 Connector, CN7 PS2 Connector, CN8 BarrelJack_Horizontal_PC110, Q1 TO-252-2, Q2 SOT-323_SC-70, U1 SSOP-20_4.4x6.5mm_P0.65mm, U2 SSOP-28_5.3x10.2mm_P0.65mm, U3 SSOP-28_5.3x10.2mm_P0.65mm, U4 SOT-23-5

Commit message: Add files via upload
Parts:
- added J1: PCB Edge, Connector_FFC-FPC:TE_2-1734839-5_1x25-1MP_P0.5mm_Horizontal, B.Cu at (178.3, 100.2)
- added J2: PCB Edge, Connector_FFC-FPC:TE_2-1734839-5_1x25-1MP_P0.5mm_Horizontal, B.Cu at (202.2, 100.2)
- added J3: PCB Edge, Connector_FFC-FPC:TE_2-1734839-5_1x25-1MP_P0.5mm_Horizontal, B.Cu at (202.2, 113.2)
- added J4: PCB Edge, Connector_FFC-FPC:TE_2-1734839-5_1x25-1MP_P0.5mm_Horizontal, B.Cu at (178.3, 113.3)
Routing:
- net (no net): track 94.1 -> 3827.2 mm, vias 40 -> 239

Commit message: Add files via upload
Parts:
- added ?: , , F.Cu at (172.5, 115.6)
- added ?: , , F.Cu at (174.6, 115.6)
- J1, J2, J3, J4: footprint Connector_FFC-FPC:TE_2-1734839-5_1x25-1MP_P0.5mm_Horizontal -> DockingStation:25-1MP_P0.5mm_Horizontal_PC110_dock
Routing:
- net (no net): track 3827.2 -> 6802.4 mm, vias 239 -> 271
- net PWR_IN-_EMI: track 7.32 -> 121.8 mm, vias 2 -> 17

Commit message: Add files via upload
Parts:
- added G1: LOGO, DockingStation:logo, F.Cu at (103.4, 94.9)
- moved D3 0.21 mm to (141.4, 120.4)
Connections:
- ? pad 2: (no net) -> PWR_IN+_Diode (x2)
- C1 pad 1: (no net) -> GND
- C1 pad 2: (no net) -> PNET1_Dock
- C10 pad 1: (no net) -> GND
- C11 pad 1: (no net) -> GND
- C12 pad 1: (no net) -> GND
- C13 pad 2: (no net) -> GND
- C14 pad 2: (no net) -> GND
- C15 pad 1: (no net) -> GND
- C16 pad 2: (no net) -> GND
- C17 pad 1: (no net) -> GND
- C18 pad 2: (no net) -> GND
- C19 pad 1: (no net) -> GND
- C2 pad 1: (no net) -> GND
- C2 pad 2: (no net) -> PNET1_Dock
- C20 pad 2: (no net) -> GND
- C21 pad 1: (no net) -> GND
- C22 pad 2: (no net) -> GND
- C23 pad 1: (no net) -> GND
- C24 pad 2: (no net) -> GND
- C25 pad 1: (no net) -> GND
- C26 pad 2: (no net) -> GND
- C27 pad 1: (no net) -> GND
- C28 pad 2: (no net) -> GND
- C29 pad 1: (no net) -> GND
- C3 pad 2: (no net) -> GND
- C30 pad 2: (no net) -> GND
- C31 pad 1: (no net) -> GND
- C32 pad 1: (no net) -> PNET1_Dock
- C32 pad 2: (no net) -> GND
- C33 pad 1: (no net) -> PNET1_Dock
- C33 pad 2: (no net) -> GND
- C34 pad 1: (no net) -> GND
- C34 pad 2: (no net) -> PNET3_Dock
- C35 pad 2: (no net) -> PNET3_Dock
- C36 pad 1: (no net) -> GND
- C36 pad 2: (no net) -> PNET2_Dock
- C37 pad 2: (no net) -> GND
- C38 pad 2: (no net) -> GND
- C39 pad 2: (no net) -> GND
- C4 pad 2: (no net) -> GND
- C40 pad 2: (no net) -> GND
- C41 pad 2: (no net) -> GND
- C42 pad 1: (no net) -> GND
- C43 pad 2: (no net) -> GND
- C44 pad 2: (no net) -> GND
- C45 pad 1: (no net) -> GND
- C46 pad 1: (no net) -> GND
- C47 pad 1: (no net) -> GND
- C48 pad 1: (no net) -> GND
- C49 pad 1: (no net) -> GND
- C50 pad 1: (no net) -> GND
- C51 pad 1: (no net) -> GND
- C52 pad 1: (no net) -> GND
- C53 pad 1: (no net) -> GND
- C54 pad 1: (no net) -> GND
- C55 pad 1: (no net) -> GND
- C56 pad 1: (no net) -> GND
- C57 pad 1: (no net) -> GND
- C58 pad 1: (no net) -> GND
- C59 pad 1: (no net) -> GND
- C60 pad 1: (no net) -> GND
- C61 pad 1: (no net) -> GND
- C62 pad 2: (no net) -> GND
- C63 pad 1: (no net) -> GND
- C64 pad 1: (no net) -> GND
- C65 pad 1: (no net) -> GND
- C66 pad 1: (no net) -> GND
- C67 pad 2: (no net) -> GND
- C68 pad 2: (no net) -> GND
- C69 pad 2: (no net) -> GND
- C71 pad 2: (no net) -> GND
- C73 pad 2: (no net) -> GND
- C74 pad 2: (no net) -> GND
- C75 pad 2: (no net) -> PWR_IN-_EMI
- C78 pad 1: (no net) -> GND
- C80 pad 2: (no net) -> GND
- C83 pad 1: (no net) -> GND
- C9 pad 1: (no net) -> GND
- CN1 pad 0: (no net) -> GND
- CN1 pad 5: (no net) -> GND
- CN1 pad 6: (no net) -> GND
- CN1 pad 7: (no net) -> GND
- CN1 pad 8: (no net) -> GND
- CN2 pad : (no net) -> GND
- CN2 pad 1: (no net) -> GND
- CN2 pad 19: (no net) -> GND
- CN2 pad 5: (no net) -> GND
- CN2 pad 7: (no net) -> GND
- CN4 pad 0: (no net) -> GND
- CN4 pad 18: (no net) -> GND
- CN4 pad 19: (no net) -> GND
- CN4 pad 20: (no net) -> GND
- CN4 pad 21: (no net) -> GND
- CN4 pad 22: (no net) -> GND
- CN4 pad 23: (no net) -> GND
- CN4 pad 24: (no net) -> GND
- CN4 pad 25: (no net) -> GND
- CN5 pad 0: (no net) -> GND
- CN5 pad 5: (no net) -> GND
- CN6 pad : (no net) -> GND
- CN6 pad 3: (no net) -> GND
- CN7 pad : (no net) -> GND
- CN7 pad 3: (no net) -> GND
- D2 pad 1: (no net) -> PWR_IN+_Diode
- D2 pad 2: (no net) -> PWR_IN+_Fuse
- D3 pad 1: (no net) -> PWR_IN+_Diode
- D3 pad 2: (no net) -> PWR_IN+_Fuse
- DA1 pad 1: (no net) -> GND
- DA10 pad 1: (no net) -> GND
- DA11 pad 1: (no net) -> PNET1_Dock
- DA11 pad 2: (no net) -> PNET1_Dock
- DA12 pad 1: (no net) -> PNET1_Dock
- DA12 pad 2: (no net) -> PNET1_Dock
- DA2 pad 1: (no net) -> GND
- DA3 pad 1: (no net) -> GND
- DA4 pad 2: (no net) -> GND
- DA6 pad 1: (no net) -> GND
- DA9 pad 2: (no net) -> GND
- F1 pad 1: (no net) -> PWR_IN+_EMI
- F1 pad 2: (no net) -> PWR_IN+_Fuse
- J1 pad 1: (no net) -> GND
- J1 pad 10: (no net) -> GND
- J1 pad 12: (no net) -> GND
- J1 pad 19: (no net) -> PWR_IN-_EMI
- J1 pad 20: (no net) -> PWR_IN-_EMI
- J1 pad 21: (no net) -> PWR_IN-_EMI
- J1 pad 22: (no net) -> PWR_IN-_EMI
- J1 pad 23: (no net) -> PWR_IN-_EMI
- J1 pad 25: (no net) -> GND
- J1 pad 6: (no net) -> GND
- J1 pad 8: (no net) -> GND
- J2 pad 1: (no net) -> GND
- J2 pad 12: (no net) -> PNET3_Dock
- J2 pad 13: (no net) -> PNET3_Dock
- J2 pad 16: (no net) -> GND
- J2 pad 21: (no net) -> PNET1_Dock
- J3 pad 1: (no net) -> GND
- J3 pad 13: (no net) -> PNET3_Dock
- J3 pad 21: (no net) -> PNET1_Dock
- J4 pad 15: (no net) -> PNET2_Dock
- J4 pad 19: (no net) -> PWR_IN+_Diode
- J4 pad 20: (no net) -> PWR_IN+_Diode
- J4 pad 21: (no net) -> PWR_IN+_Diode
- J4 pad 22: (no net) -> PWR_IN+_Diode
- J4 pad 23: (no net) -> PWR_IN+_Diode
- J4 pad 25: (no net) -> GND
- L11 pad 1: (no net) -> PNET3_Dock
- Q1 pad 1: (no net) -> PWR_IN-_EMI
- Q1 pad 2: (no net) -> PWR_IN+_Fuse
- Q2 pad 2: (no net) -> GND
- R10 pad 2: (no net) -> PNET1_Dock
- R11 pad 1: (no net) -> PNET2_Dock
- R31 pad 1: (no net) -> PWR_IN-_EMI
- R32 pad 2: (no net) -> PWR_IN+_Fuse
- R34 pad 1: (no net) -> PWR_IN-_EMI
- R35 pad 1: (no net) -> PWR_IN-_EMI
- R36 pad 2: (no net) -> PWR_IN+_Fuse
- R38 pad 2: (no net) -> PWR_IN+_Fuse
- R39 pad 1: (no net) -> PNET2_Dock
- R42 pad 1: (no net) -> PNET2_Dock
- R5 pad 1: (no net) -> GND
- R6 pad 1: (no net) -> GND
- R7 pad 2: (no net) -> GND
- R8 pad 2: (no net) -> GND
- R9 pad 2: (no net) -> GND
- RA3 pad 1: (no net) -> PNET3_Dock
- RA3 pad 2: (no net) -> PNET3_Dock
- RA3 pad 3: (no net) -> PNET3_Dock
- RA3 pad 4: (no net) -> PNET3_Dock
- RA4 pad 1: (no net) -> PNET3_Dock
- RA4 pad 2: (no net) -> PNET3_Dock
- RA4 pad 3: (no net) -> PNET3_Dock
- RA4 pad 4: (no net) -> PNET3_Dock
- RA5 pad 1: (no net) -> PNET3_Dock
- RA5 pad 2: (no net) -> PNET3_Dock
- RA5 pad 3: (no net) -> PNET3_Dock
- RA5 pad 4: (no net) -> PNET3_Dock
- RA6 pad 1: (no net) -> PNET3_Dock
- RA6 pad 2: (no net) -> PNET3_Dock
- RA6 pad 3: (no net) -> PNET3_Dock
- RA6 pad 4: (no net) -> PNET3_Dock
- SSFC pad 1: (no net) -> PWR_IN+_EMI
- SSFC pad 2: (no net) -> PWR_IN+_Fuse
- U1 pad 1: (no net) -> GND
- U1 pad 10: (no net) -> GND
- U1 pad 19: (no net) -> GND
- U1 pad 20: (no net) -> PNET1_Dock
- U3 pad 27: (no net) -> GND
- U3 pad 5: (no net) -> GND
- U4 pad 3: (no net) -> GND
- ZD1 pad 1: (no net) -> PWR_IN+_Fuse
- ZD4 pad 2: (no net) -> PWR_IN-_EMI
Routing:
- net (no net): track 6802.4 -> 5430.9 mm, vias 271 -> 126
- net GND: track 0.00 -> 1268.4 mm, vias 0 -> 110
- net PNET1_Dock: track 0.00 -> 157.3 mm, vias 0 -> 12
- net PNET3_Dock: track 0.00 -> 92.8 mm, vias 0 -> 10
- net PNET2_Dock: track 0.00 -> 81.9 mm, vias 0 -> 6
- net PWR_IN-_EMI: track 121.8 -> 192.2 mm, vias 17 -> 21
- net PWR_IN+_Diode: track 0.00 -> 56.4 mm
- net PWR_IN+_EMI: track 7.47 -> 53.9 mm, vias 2 -> 5
- net PWR_IN+_Fuse: track 0.00 -> 30.6 mm
- added copper zone on B.Cu, net GND
- added copper zone on F.Cu, net GND
- added copper zone on In1.Cu, net GND
- added copper zone on F.Cu, net PNET1_Dock
- added copper zone on In2.Cu, net PNET1_Dock
- added copper zone on F.Cu, net PNET2_Dock
- added copper zone on In2.Cu, net PNET2_Dock
- added copper zone on F.Cu, net PNET3_Dock
- added copper zone on In2.Cu, net PNET3_Dock
- added copper zone on F.Cu, net PWR_IN+_Diode
- added copper zone on In2.Cu, net PWR_IN+_EMI
- added copper zone on F.Cu, net PWR_IN+_Fuse
- added copper zone on B.Cu, net PWR_IN-_EMI
Other:
- copper layers 2 -> 4
- board text added: "Recreated with love by Ahmad Byagowi"

Commit message: Add files via upload
Parts:
- C1: value C_0805_2012Metric -> 330nF
- C10: value C_0603_1608Metric -> 1nF
- C11: value C_1206_3216Metric -> 2.5uF
- C12, C15, C17, C19, C21, C23, C25, C27, C29, C31, C32, C34, C35, C36, C9: value C_0603_1608Metric -> 280nF
- C13, C14, C16, C18, C20, C22, C24, C26, C28, C30: value C_0603_1608Metric -> 82pF
- C2: value C_0805_2012Metric -> 1nF
- C3, C4: value C_0805_2012Metric -> 200pF
- C33: value C_0603_1608Metric -> 330nF
- C37, C38, C39, C40, C41, C42, C43, C44, C63, C64, C65, C66: value C_0603_1608Metric -> 200pF
- C45, C46, C47, C48, C49, C50, C51, C52, C53, C54, C55, C56, C57, C58, C59, C60, C61: value C_0603_1608Metric -> 200nF
- C62, C67, C78: value C_0603_1608Metric -> 250nF
- C68, C73, C74, C83: value C_0603_1608Metric -> DNP
- C69, C71: value C_1206_3216Metric -> DNP
- C70, C72: value C_0805_2012Metric -> DNP
- C75: value C_0603_1608Metric -> 150nF
- C76, C77: value C_0603_1608Metric -> 10nF
- C79, C80, C81, C82: value C_0805_2012Metric -> 360nF
- D2, D3: value D_2010_5025Metric -> s.3 5J
- DA1, DA10, DA2, DA3, DA4, DA6, DA7, DA8: value SOT-323_SC-70 -> 1W
- DA11, DA12: value SOT-23W -> DNP
- F1: value Fuse_Littelfuse_395Series -> 50v x1G0 JX30
- L1, L2, L3, L34, L37, L38: value L_0805_2012Metric -> 300nH
- L11, L13, L14, L15, L16, L17, L18, L19, L20, L21, L22, L23, L24, L25, L26, L27, L28, L29, L30, L31, L39, L40, L41, L42, L43, L44, L45, L46, L47, L48, L49, L5, L50, L51, L52, L53, L54, L55, L56, L57, L58, L59, L6, L60, L61, L62, L63, L64, L65, L66, L67: value L_0805_2012Metric -> 680nH
- Q1: value TO-252-2 -> 3P4J
- Q2: value SOT-323_SC-70 -> 8C
- R1, R2: value R_0805_2012Metric -> 33
- R10, R11, R29, R40, R42, R43, R44, R45, R46, R47, R48, R49, R50, R51, R60, R61, R62, R63, R64, R65, R66, R67: value R_0603_1608Metric -> DNP
- R12, R13, R14, R15, R16, R17, R18, R19, R20, R21, R22, R23, R24, R25, R26, R27, R28: value R_0603_1608Metric -> 10
- R3, R4: value R_0603_1608Metric -> 33
- R30, R31, R32, R33, R34, R35, R36, R37: value R_0805_2012Metric -> 1k
- R38: value R_0805_2012Metric -> 0
- R39, R41, R5, R52, R53, R54, R55, R56, R57, R58, R59, R68, R69, R7, R70, R71, R72, R73, R74, R75, R8: value R_0603_1608Metric -> 0
- R6, R9: value R_0603_1608Metric -> 470k
- RA2, RA3, RA4: value R_Array_Concave_4x0603 -> 47k
- RA5, RA6: value R_Array_Concave_4x0603 -> 470k
- RA7, RA8: value R_Array_Concave_4x0603 -> DNP
- U1: value SSOP-20_4.4x6.5mm_P0.65mm -> 74VHCT244
- U2: value SSOP-28_5.3x10.2mm_P0.65mm -> DNP (LT1237CS)
- U3: value SSOP-28_5.3x10.2mm_P0.65mm -> DS14C535MSA
- U4: value SOT-23-5 -> DNP
- ZD1: value D_0805_2012Metric -> 18-
- ZD4: value D_0805_2012Metric -> 5_1
Routing:
- net (no net): track 5430.9 -> 5439.2 mm

Commit message: Add files via upload
Parts:
- J1, J2, J3, J4: value PCB Edge -> 25-1MP_P0.5mm_Horizontal
Changed lines of the file:
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@@
 			)
 		)
-		(property "Value" "PCB Edge"
+		(property "Value" "25-1MP_P0.5mm_Horizontal"
 			(at 0 -3.25 0)
 			(layer "Dwgs.User")
@@
 			)
 		)
-		(property "Value" "PCB Edge"
+		(property "Value" "25-1MP_P0.5mm_Horizontal"
 			(at 0 -3.25 0)
 			(layer "Dwgs.User")
@@
 			)
 		)
-		(property "Value" "PCB Edge"
+		(property "Value" "25-1MP_P0.5mm_Horizontal"
 			(at 0 -3.25 0)
 			(layer "Dwgs.User")
@@
 			)
 		)
-		(property "Value" "PCB Edge"
+		(property "Value" "25-1MP_P0.5mm_Horizontal"
 			(at 0 -3.25 0)
 			(layer "Dwgs.User")

Commit message: Add files via upload
Connections:
- net PNET1_Dock renamed PNET2
- net PNET2_Dock renamed PNET5
- C31 pad 2: (no net) -> PNET5_Q1_F2
- DA1 pad 3: (no net) -> VGA_RED
- DA2 pad 3: (no net) -> VGA_GREEN
- DA3 pad 3: (no net) -> VGA_BLUE
- J1 pad 11: (no net) -> VGA_BLUE
- J1 pad 13: (no net) -> R269_1_PC110
- J1 pad 14: (no net) -> M38_P16_R80_PC110
- J1 pad 15: (no net) -> M38_P67
- J1 pad 16: (no net) -> J13_60_PC110
- J1 pad 17: (no net) -> J13_59_PC110
- J1 pad 18: (no net) -> J13_58_PC110
- J1 pad 2: (no net) -> FDC_SLCTIN#
- J1 pad 24: (no net) -> J13_52_PC110
- J1 pad 3: (no net) -> FDC_AUTOFD#
- J1 pad 4: (no net) -> FDC_INIT#
- J1 pad 5: (no net) -> FDC_ACK#
- J1 pad 7: (no net) -> VGA_RED
- J1 pad 9: (no net) -> VGA_GREEN
- J2 pad 10: (no net) -> FDC_RDATA#
- J2 pad 11: (no net) -> J13_90_PC110
- J2 pad 14: (no net) -> KB_INT4
- J2 pad 15: (no net) -> KB_INT3
- J2 pad 17: (no net) -> FDC_DSR2#
- J2 pad 18: (no net) -> FDC_RTS2#
- J2 pad 19: (no net) -> FDC_CTS2#
- J2 pad 2: (no net) -> J13_99_PC110
- J2 pad 20: (no net) -> FDC_RI2#
- J2 pad 22: (no net) -> J13_79_PC110
- J2 pad 23: (no net) -> FDC_PE
- J2 pad 24: (no net) -> FDC_ERROR#
- J2 pad 25: (no net) -> FDC_PD6
- J2 pad 3: (no net) -> J13_98_PC110
- J2 pad 4: (no net) -> J13_97_PC110
- J2 pad 5: (no net) -> FDC_MEDIA2
- J2 pad 6: (no net) -> J13_95_PC110
- J2 pad 7: (no net) -> FDC_STEP#
- J2 pad 8: (no net) -> FDC_WGATE#
- J2 pad 9: (no net) -> J13_92_PC110
- J3 pad 10: (no net) -> FDC_WRTPRT#
- J3 pad 11: (no net) -> FDC_HDSEL#
- J3 pad 12: (no net) -> FDC_DSKCHG#
- J3 pad 14: (no net) -> KB_INT1
- J3 pad 15: (no net) -> KB_INT2
- J3 pad 16: (no net) -> PNET5_Q1_F2
- J3 pad 17: (no net) -> FDC_DCD2#
- J3 pad 18: (no net) -> U29_A2_FDC_IRRX_RXD2_InBuff
- J3 pad 19: (no net) -> U29_Y1_FDC_IRTX_TXD2_BufSW
- J3 pad 2: (no net) -> J13_2_PC110
- J3 pad 20: (no net) -> FDC_DTR2#
- J3 pad 22: (no net) -> FDC_BUSY
- J3 pad 23: (no net) -> FDC_SLCT
- J3 pad 24: (no net) -> FDC_PD7
- J3 pad 25: (no net) -> FDC_PD5
- J3 pad 3: (no net) -> FDC_MEDIA
- J3 pad 4: (no net) -> FDC_INDEX#
- J3 pad 5: (no net) -> FDC_DS0#
- J3 pad 6: (no net) -> FDC_MTR0#
- J3 pad 7: (no net) -> FDC_DIR#
- J3 pad 8: (no net) -> FDC_WDATA#
- J3 pad 9: (no net) -> FDC_TRK0
- J4 pad 1: (no net) -> FDC_PD4
- J4 pad 10: (no net) -> J13_35_PC110
- J4 pad 11: (no net) -> VGA_Hsync
- J4 pad 12: (no net) -> J13_37_PC110
- J4 pad 13: (no net) -> M38_P46_P34
- J4 pad 14: (no net) -> M38_P46_P34
- J4 pad 16: (no net) -> J13_41_PC110
- J4 pad 17: (no net) -> J13_42_PC110
- J4 pad 18: (no net) -> J13_43_PC110
- J4 pad 2: (no net) -> FDC_PD3
- J4 pad 24: (no net) -> J13_49_PC110
- J4 pad 3: (no net) -> FDC_PD2
- J4 pad 4: (no net) -> FDC_PD1
- J4 pad 5: (no net) -> FDC_PD0
- J4 pad 6: (no net) -> FDC_STROBE#
- J4 pad 7: (no net) -> J13_32_PC110
- J4 pad 8: (no net) -> VGA_Vsync
- J4 pad 9: (no net) -> J13_34_PC110
- L1 pad 1: (no net) -> VGA_GREEN
- L13 pad 1: (no net) -> FDC_MEDIA
- L14 pad 1: (no net) -> FDC_INDEX#
- L15 pad 1: (no net) -> FDC_DS0#
- L16 pad 1: (no net) -> FDC_MTR0#
- L17 pad 1: (no net) -> FDC_DIR#
- L18 pad 1: (no net) -> FDC_WDATA#
- L19 pad 1: (no net) -> FDC_TRK0
- L2 pad 1: (no net) -> VGA_BLUE
- L20 pad 1: (no net) -> FDC_WRTPRT#
- L21 pad 1: (no net) -> FDC_HDSEL#
- L22 pad 1: (no net) -> FDC_DSKCHG#
- L23 pad 1: (no net) -> J13_98_PC110
- L24 pad 1: (no net) -> J13_97_PC110
- L25 pad 1: (no net) -> FDC_MEDIA2
- L26 pad 1: (no net) -> J13_95_PC110
- L27 pad 1: (no net) -> FDC_STEP#
- L28 pad 1: (no net) -> FDC_WGATE#
- L29 pad 1: (no net) -> J13_92_PC110
- L3 pad 1: (no net) -> VGA_RED
- L31 pad 2: (no net) -> J13_90_PC110
- L38 pad 2: (no net) -> PNET5_Q1_F2
- L39 pad 2: (no net) -> KB_INT3
- L40 pad 2: (no net) -> KB_INT2
- L41 pad 2: (no net) -> KB_INT4
- L42 pad 2: (no net) -> KB_INT1
- Q2 pad 3: (no net) -> M38_P46_P34
- R12 pad 1: (no net) -> FDC_PD7
- R13 pad 1: (no net) -> FDC_PD5
- R14 pad 1: (no net) -> FDC_PD3
- R15 pad 1: (no net) -> FDC_PD1
- R16 pad 1: (no net) -> FDC_STROBE#
- R17 pad 1: (no net) -> FDC_INIT#
- R18 pad 1: (no net) -> FDC_SLCT
- R19 pad 1: (no net) -> FDC_ERROR#
- R20 pad 1: (no net) -> FDC_BUSY
- R21 pad 2: (no net) -> FDC_PD6
- R22 pad 1: (no net) -> FDC_PD4
- R23 pad 1: (no net) -> FDC_PD2
- R24 pad 1: (no net) -> FDC_PD0
- R25 pad 1: (no net) -> FDC_AUTOFD#
- R26 pad 1: (no net) -> FDC_SLCTIN#
- R27 pad 1: (no net) -> FDC_PE
- R28 pad 1: (no net) -> FDC_ACK#
- R3 pad 1: (no net) -> VGA_Hsync
- R33 pad 1: (no net) -> M38_P67
- R34 pad 2: (no net) -> M38_P67
- R38 pad 1: (no net) -> R269_1_PC110
- R4 pad 1: (no net) -> VGA_Vsync
- R41 pad 1: (no net) -> J13_79_PC110
- R43 pad 2: (no net) -> J13_79_PC110
- R44 pad 2: (no net) -> FDC_DTR2#
- R45 pad 2: (no net) -> U29_Y1_FDC_IRTX_TXD2_BufSW
- R46 pad 2: (no net) -> FDC_CTS2#
- R47 pad 2: (no net) -> U29_A2_FDC_IRRX_RXD2_InBuff
- R49 pad 2: (no net) -> FDC_DCD2#
- R50 pad 2: (no net) -> FDC_DSR2#
- R51 pad 1: (no net) -> FDC_RI2#
- R52 pad 1: (no net) -> FDC_DTR2#
- R54 pad 1: (no net) -> U29_Y1_FDC_IRTX_TXD2_BufSW
- R55 pad 1: (no net) -> FDC_DCD2#
- R56 pad 1: (no net) -> FDC_CTS2#
- R57 pad 1: (no net) -> FDC_DSR2#
- R58 pad 1: (no net) -> U29_A2_FDC_IRRX_RXD2_InBuff
- R59 pad 2: (no net) -> FDC_RI2#
- R7 pad 1: (no net) -> J13_2_PC110
- R8 pad 1: (no net) -> J13_99_PC110
- R9 pad 1: (no net) -> FDC_CTS2#
- RA2 pad 5: (no net) -> FDC_DSKCHG#
- RA2 pad 6: (no net) -> FDC_HDSEL#
- RA2 pad 8: (no net) -> FDC_WRTPRT#
- RA3 pad 6: (no net) -> FDC_MTR0#
- RA3 pad 7: (no net) -> FDC_DS0#
- RA3 pad 8: (no net) -> FDC_INDEX#
- RA4 pad 5: (no net) -> FDC_TRK0
- RA4 pad 6: (no net) -> FDC_WGATE#
- RA4 pad 7: (no net) -> FDC_WDATA#
- RA4 pad 8: (no net) -> FDC_STEP#
- RA5 pad 5: (no net) -> J13_92_PC110
- RA5 pad 6: (no net) -> FDC_DIR#
- RA5 pad 7: (no net) -> J13_95_PC110
- RA6 pad 5: (no net) -> FDC_MEDIA2
- RA6 pad 6: (no net) -> J13_97_PC110
- RA6 pad 7: (no net) -> J13_98_PC110
- RA6 pad 8: (no net) -> FDC_MEDIA
- RA7 pad 5: (no net) -> FDC_PD7
- RA7 pad 6: (no net) -> FDC_PD6
- RA7 pad 7: (no net) -> FDC_PD5
- RA7 pad 8: (no net) -> FDC_PD4
- RA8 pad 5: (no net) -> FDC_PD3
- RA8 pad 6: (no net) -> FDC_PD2
- RA8 pad 7: (no net) -> FDC_PD1
- RA8 pad 8: (no net) -> FDC_PD0
- ZD4 pad 1: (no net) -> M38_P67
Routing:
- net (no net): track 5439.2 -> 1658.9 mm, vias 126 -> 44
- net KB_INT4: track 0.00 -> 128.9 mm, vias 0 -> 3
- net KB_INT3: track 0.00 -> 126.4 mm, vias 0 -> 3
- net PNET5_Q1_F2: track 0.00 -> 125.7 mm, vias 0 -> 6
- net KB_INT1: track 0.00 -> 123.0 mm, vias 0 -> 3
- net KB_INT2: track 0.00 -> 122.6 mm, vias 0 -> 3
- net M38_P46_P34: track 0.00 -> 112.3 mm, vias 0 -> 1
- net VGA_RED: track 0.00 -> 99.2 mm, vias 0 -> 1
- net FDC_ERROR#: track 0.00 -> 98.9 mm, vias 0 -> 1
- net FDC_PD6: track 0.00 -> 94.9 mm, vias 0 -> 1
- net VGA_GREEN: track 0.00 -> 94.3 mm, vias 0 -> 1
- net VGA_BLUE: track 0.00 -> 89.2 mm, vias 0 -> 1
- net FDC_PD7: track 0.00 -> 86.1 mm, vias 0 -> 1
- net FDC_PD5: track 0.00 -> 78.9 mm, vias 0 -> 1
- net VGA_Hsync: track 0.00 -> 78.8 mm, vias 0 -> 1
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