File: PCB/DockingStation/DockingStation.kicad_sch (KiCad schematic)
At the start: 221 parts, among them CN1 VGA, CN2 FDC_Connector, CN4 LPT, CN5 Serial Port, CN6 PS/2, CN7 PS/2, CN8 BarrelJack_Horizontal_PC110, J1 Dock Connector, J2 Dock Connector, J3 Dock Connector, J4 Dock Connector, Q1 3PJ4, Q2 8C, U1 74HCT244

Commit message: Add files via upload
Connections:
- net at C44.1 (+), L43.1 (+): now also CN5.1
- no-connect marks 24 -> 23
Changed lines of the file:
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@@
 	)
 	(junction
+		(at 69.85 294.64)
+		(diameter 0)
+		(color 0 0 0 0)
+	)
+	(junction
 		(at 534.67 535.94)
 		(diameter 0)
@@
 	)
 	(no_connect
-		(at 57.15 294.64)
-	)
-	(no_connect
 		(at 516.89 69.85)
 	)
@@
 	(wire
 		(pts
+			(xy 57.15 294.64) (xy 69.85 294.64)
+		)
+		(stroke
+			(width 0)
+			(type default)
+		)
+	)
+	(wire
+		(pts
 			(xy 137.16 224.79) (xy 198.12 224.79)
 		)
@@
 	(wire
 		(pts
-			(xy 69.85 254) (xy 69.85 298.45)
+			(xy 69.85 254) (xy 69.85 294.64)
 		)
 		(stroke
@@
 		)
 		(stroke
+			(width 0)
+			(type default)
+		)
+	)
+	(wire
+		(pts
+			(xy 69.85 294.64) (xy 69.85 298.45)
+		)
+		(stroke

Commit message: Add files via upload
Parts:
- removed CN6, CN7: PS/2, symbol Connector_Generic:Conn_01x06
- added C35: 280nF, symbol PCM_Elektuur:C
- added C68, C69, C70, C71, C72, C73, C74, C83: DNP, symbol PCM_Elektuur:C
- added C77: 10nF, symbol PCM_Elektuur:C
- added C78: 250nF, symbol PCM_Elektuur:C
- added CN6, CN7: PS/2, symbol Connector:Mini-DIN-6
- added DA1, DA10, DA2, DA3, DA4, DA6, DA7, DA8, DA9: 1W, symbol Device:D_Dual_Series_ACK
- added R10, R11, R29, R40, R42, R43: DNP, symbol PCM_Elektuur:R
- added R39, R5: 0, symbol PCM_Elektuur:R
- added R9: 470k, symbol PCM_Elektuur:R
- added U2: ~, symbol DockingStation:LT1237
- added U4: DNP, symbol 74xGxx:74AHC1G14
Connections:
- net CTS2#: now also R9.1 (+)
- net DS_VCC: now also C78.1 (+), R39.2 (-), R40.2 (-)
- net FDD_PWR: now also C35.1 (+)
- net GND: now also C35.2 (-), C68.2 (-), C69.2 (-), C71.2 (-), C73.2 (-), C74.2 (-), C78.2 (-), C83.2 (-), CN6.3, CN7.3, DA1.1 (A), DA10.1 (A), DA2.1 (A), DA3.1 (A), DA4.1 (A), DA6.1 (A), DA9.1 (A), R29.2 (-), R5.2 (-), R9.2 (-), U2.17 (GND), U4.3 (GND)
- net PNET2: now also R10.1 (+), R40.1 (+)
- net PNET5: now also R11.1 (+), R39.1 (+), R42.1 (+)
- net PWR_IN-: now also C77.2 (-)
- net at CN1.2, L1.1 (+): now also DA2.2 (common)
- net at C66.1 (+), L42.2 (-): now also CN6.1
- net at C64.1 (+), L41.2 (-): now also CN6.2, CN7.1
- net at L34.2 (-): now also CN6.4
- net at C65.1 (+), L40.2 (-): now also CN6.5
- net at C63.1 (+), L39.2 (-): now also CN6.6, CN7.5
- net at CN1.1, L3.1 (+): now also DA1.2 (common)
- net at F1.1 (+), L68.4, SSFC.1 (+): now also C77.1 (+)
- net LT_DR1_OUT: now reaches R60.2 (-)
- net LT_DR1_OUT: now also U2.11 (DR3_OUT), U2.5 (DR1_OUT), U2.7 (DR2_OUT)
- net at R4.2 (-), U1.11 (2A3), U1.13 (2A2)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: now also DA10.2 (common)
- net at R3.2 (-), U1.2 (1A0), U1.4 (1A1)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: now also DA6.2 (common)
- net LT_RX5_OUT: now reaches R51.2 (-)
- net LT_RX5_OUT: now also U2.18 (RX5_OUT)
- net LT_DR2_IN: now reaches R48.2 (-)
- net LT_DR1_IN: now reaches R44.2 (-)
- net LT_DR1_IN: now also U2.19 (DR3_IN), U2.23 (DR2_IN), U2.25 (DR1_IN)
- net LT_RX1_IN: now reaches R65.2 (-)
- net LT_RX1_IN: now also U2.6 (RX1_IN)
- net LT_DR3_OUT: now reaches R61.2 (-)
- net at L37.2 (-): now also CN7.4
- net LT_RX2_IN: now reaches R62.2 (-)
- net LT_RX2_IN: now also U2.8 (RX2_IN)
- net LT_RX1_OUT: now reaches R49.2 (-)
- net LT_RX1_OUT: now also U2.24 (RX1_OUT)
- net LT_DR3_IN: now reaches R45.2 (-)
- net LT_RX5_IN: now reaches R67.2 (-)
- net LT_RX5_IN: now also U2.12 (RX5_IN)
- net LT_RX3_IN: now reaches R66.2 (-)
- net LT_RX3_IN: now also U2.9 (RX3_IN)
- net LT_RX3_OUT: now reaches R50.2 (-)
- net LT_RX3_OUT: now also U2.21 (RX3_OUT)
- net LT_RX4_IN: now reaches R63.2 (-)
- net LT_RX4_IN: now also U2.10 (RX4_IN)
- net at CN1.3, L2.1 (+): now also DA3.2 (common)
- net LT_RX2_OUT: now reaches R46.2 (-)
- net LT_RX2_OUT: now also U2.22 (RX2_OUT)
- net LT_RX4_OUT: now reaches R47.2 (-)
- net LT_RX4_OUT: now also U2.20 (RX4_OUT)
- net LT_DR2_OUT: now reaches R64.2 (-)
- net J13_79_PC110 renamed EN_RS232
- net EN_RS232: now also R43.2 (-)
- new net: C68.1 (+), R10.2 (-), R11.2 (-), U2.2 (VCC)
- new net: R29.1 (+), U2.16 (DRV_DIS)
- new net: C83.1 (+), R42.2 (-), U4.5 (VCC)
- new net: DA10.3 (K), DA6.3 (K), DA7.3 (K)
- new net: C69.1 (+), C71.1 (+), U2.1 (V+)
- new net: R43.1 (+), U4.2
- new net: DA1.3 (K), DA2.3 (K), DA3.3 (K), DA4.3 (K)
- new net: DA8.1 (A), DA9.3 (K), R5.1 (+)
- new net: DA7.1 (A), DA8.3 (K)
- new net: C70.1 (+), U2.3 (C1+)
- new net: C70.2 (-), U2.4 (C1-)
- new net: U2.13 (ON/OFF), U4.4
- new net: C72.2 (-), U2.26 (C2+)
- new net: C72.1 (+), U2.27 (C2-)
- new net: C73.1 (+), C74.1 (+), U2.28 (V-)
- no-connect marks 23 -> 31
Other:
- moved on the sheet: C1, C2, C3, C31, C4, C62, C63, C64, C65, C66, C67, CN1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

Commit message: Add files via upload
Parts:
- U2: value ~ -> DNP; now fitted
- renumbered SSFC to SSFC1
Connections:
- net LT_DR1_IN: no longer U2.19 (DR3_IN), U2.23 (DR2_IN)
- net LT_DR1_OUT: no longer U2.11 (DR3_OUT), U2.7 (DR2_OUT)
- net LT_DR2_IN: now also U2.23 (DR2_IN)
- net LT_DR2_OUT: now also U2.7 (DR2_OUT)
- net LT_DR3_IN: now also U2.19 (DR3_IN)
- net LT_DR3_OUT: now also U2.11 (DR3_OUT)
- no-connect marks 31 -> 29

Commit message: Add files via upload
Parts:
- removed DA1, DA10, DA2, DA3, DA4, DA6, DA7, DA8, DA9: 1W, symbol Device:D_Dual_Series_ACK
- removed Q2: 8C, symbol Simulation_SPICE:NPN
- added DA1, DA10, DA2, DA3, DA4, DA6, DA7, DA8, DA9: 1W, symbol Device:D_Dual_Series_KAC
- added Q2: 8C, symbol PCM_Transistor_BJT_AKL:Q_NPN_Generic_BEC
Connections:
- net CTS2#: now also R46.2 (-); no longer R46.1 (+)
- net DSR2#: now also R50.2 (-); no longer R50.1 (+)
- net DS_VCC: now also C78.2 (-), R40.1 (+); no longer C78.1 (+), R40.2 (-)
- net DTR2#: now also R44.2 (-); no longer R44.1 (+)
- net EN_RS232: now also R41.1 (+); no longer R41.2 (-)
- net FDC_ACK#: now also R28.1 (+); no longer R28.2 (-)
- net FDC_AUTOFD#: now also R25.1 (+); no longer R25.2 (-)
- net FDC_BUSY: now also R20.1 (+); no longer R20.2 (-)
- net FDC_DCD2#: now also R49.2 (-); no longer R49.1 (+)
- net FDC_ERROR#: now also R19.1 (+); no longer R19.2 (-)
- net FDC_INIT#: now also R17.1 (+); no longer R17.2 (-)
- net FDC_PE: now also R27.1 (+); no longer R27.2 (-)
- net FDC_SLCT: now also R18.1 (+); no longer R18.2 (-)
- net FDC_SLCTIIN#: now also R26.1 (+); no longer R26.2 (-)
- net FDC_STROBE#: now also R16.1 (+); no longer R16.2 (-)
- net FDD_Bowman: now also L31.2 (-); no longer L31.1 (+)
- net FDD_PWR: now also C34.2 (-), C35.2 (-); no longer C11.1 (+), C34.1 (+), C35.1 (+)
- net GND: now also C1.1 (+), C10.1 (+), C11.1 (+), C12.1 (+), C15.1 (+), C17.1 (+), C19.1 (+), C2.1 (+), C21.1 (+), C23.1 (+), C25.1 (+), C27.1 (+), C29.1 (+), C31.1 (+), C34.1 (+), C35.1 (+), C45.1 (+), C46.1 (+), C47.1 (+), C48.1 (+), C49.1 (+), C50.1 (+), C51.1 (+), C52.1 (+), C53.1 (+), C54.1 (+), C55.1 (+), C56.1 (+), C57.1 (+), C58.1 (+), C59.1 (+), C60.1 (+), C61.1 (+), C62.2 (-), C63.1 (+), C64.1 (+), C65.1 (+), C66.1 (+), C78.1 (+), C83.1 (+), C9.1 (+), R29.1 (+), R5.1 (+), R6.1 (+), DA1.1 (K), DA10.1 (K), DA2.1 (K), DA3.1 (K), DA4.2 (A), DA6.1 (K), DA9.2 (A), Q2.2 (E); no longer C1.2 (-), C10.2 (-), C11.2 (-), C12.2 (-), C15.2 (-), C17.2 (-), C19.2 (-), C2.2 (-), C21.2 (-), C23.2 (-), C25.2 (-), C27.2 (-), C29.2 (-), C31.2 (-), C34.2 (-), C35.2 (-), C45.2 (-), C46.2 (-), C47.2 (-), C48.2 (-), C49.2 (-), C50.2 (-), C51.2 (-), C52.2 (-), C53.2 (-), C54.2 (-), C55.2 (-), C56.2 (-), C57.2 (-), C58.2 (-), C59.2 (-), C60.2 (-), C61.2 (-), C62.1 (+), C63.2 (-), C64.2 (-), C65.2 (-), C66.2 (-), C78.2 (-), C83.2 (-), C9.2 (-), R29.2 (-), R5.2 (-), R6.2 (-)
- net KB_INIT1: now also L42.2 (-); no longer L42.1 (+)
- net KB_INIT2: now also L40.2 (-); no longer L40.1 (+)
- net KB_INIT3: now also L39.2 (-); no longer L39.1 (+)
- net KB_INIT4: now also L41.2 (-); no longer L41.1 (+)
- net LT_DR1_IN: now also R44.1 (+); no longer R44.2 (-)
- net LT_DR2_IN: now also R48.1 (+); no longer R48.2 (-)
- net LT_DR3_IN: now also R45.1 (+); no longer R45.2 (-)
- net LT_RX1_OUT: now also R49.1 (+); no longer R49.2 (-)
- net LT_RX2_OUT: now also R46.1 (+); no longer R46.2 (-)
- net LT_RX3_OUT: now also R50.1 (+); no longer R50.2 (-)
- net LT_RX4_OUT: now also R47.1 (+); no longer R47.2 (-)
- net M38_P46_PC110: now also Q2.3 (C)
- net M38_P67_PC110: now also R33.1 (+), R34.2 (-); no longer R33.2 (-), R34.1 (+)
- net PD0: now also R24.1 (+); no longer R24.2 (-)
- net PD1: now also R15.1 (+); no longer R15.2 (-)
- net PD2: now also R23.1 (+); no longer R23.2 (-)
- net PD3: now also R14.1 (+); no longer R14.2 (-)
- net PD4: now also R22.1 (+); no longer R22.2 (-)
- net PD5: now also R13.1 (+); no longer R13.2 (-)
- net PD7: now also R12.1 (+); no longer R12.2 (-)
- net PNET2: now also C1.2 (-), C2.2 (-), R10.2 (-), R40.2 (-); no longer C1.1 (+), C2.1 (+), R10.1 (+), R40.1 (+)
- net PNET5_Q1: now also C31.2 (-), L38.2 (-); no longer C31.1 (+), L38.1 (+)
- net PWR_IN-: now also R31.1 (+), R34.1 (+), R35.1 (+); no longer R31.2 (-), R34.2 (-), R35.2 (-)
- net R269_1_PC110: now also R38.1 (+); no longer R38.2 (-)
- net RI2#: now also R59.2 (-); no longer R59.1 (+)
- net ROUT5: now also R59.1 (+); no longer R59.2 (-)
- net RTS2#: now also R48.2 (-); no longer R48.1 (+)
- net RXD2: now also R47.2 (-); no longer R47.1 (+)
- net TXD2: now also R45.2 (-); no longer R45.1 (+)
- net at C68.1 (+), R11.2 (-), U2.2 (VCC): now also R10.1 (+); no longer R10.2 (-)
- net at R32.2 (-): now also D2.2 (A), D3.2 (A), F1.2 (-), Q1.2 (A+), R36.2 (-), R38.2 (-), SSFC1.2 (-), ZD1.1 (K); no longer R33.1 (+)
- net at L66.2 (-): now also C46.2 (-), CN4.10; no longer R28.1 (+)
- net at L57.2 (-): now also C55.2 (-), CN4.3; no longer R15.1 (+)
- net at CN2.18 (Pin_18), CN2.2 (Pin_2), L11.2 (-): now also C10.2 (-), C11.2 (-), C9.2 (-), R6.2 (-); no longer C10.1 (+), C9.1 (+), R6.1 (+)
- net at CN1.2, L1.1 (+): now also DA2.3 (common)
- net at U2.16 (DRV_DIS): now also R29.2 (-); no longer R29.1 (+)
- net at R42.2 (-), U4.5 (VCC): now also C83.2 (-); no longer C83.1 (+)
- net at L63.2 (-): now also C49.2 (-), CN4.13; no longer R18.1 (+)
- net at L60.2 (-): now also C52.2 (-), CN4.14 (P14); no longer R25.1 (+)
- net at CN1.1, L3.1 (+): now also DA1.3 (common)
- net at L65.2 (-): now also C47.2 (-), CN4.15 (P15); no longer R19.1 (+)
- net at U3.23 (SHUTDOWN): now also R41.2 (-); no longer R41.1 (+)
- net at CN6.2, CN7.1: now also C64.2 (-), L41.1 (+); no longer C64.1 (+), L41.2 (-)
- net at L37.2 (-): now also C62.1 (+), C67.1 (+), L34.2 (-), L38.1 (+); no longer CN7.4
- net at CN6.6, CN7.5: now also C63.2 (-), L39.1 (+); no longer C63.1 (+), L39.2 (-)
- net at R4.2 (-), U1.11 (2A3), U1.13 (2A2)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: now also DA10.3 (common)
- net at CN2.22 (Pin_22), L28.2 (-): now also C19.2 (-); no longer C19.1 (+)
- net at L62.2 (-): now also C50.2 (-), CN4.17 (P17); no longer R26.1 (+)
- net at CN2.20 (Pin_20), L26.2 (-): now also C23.2 (-); no longer C23.1 (+)
- net at L64.2 (-): now also C48.2 (-), CN4.12; no longer R27.1 (+)
- net at R3.2 (-), U1.2 (1A0), U1.4 (1A1)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: now also DA6.3 (common)
- net at CN8.2, L68.1: now also C76.1 (+); no longer C76.2 (-)
- net at CN8.1, L68.3: now also C76.2 (-); no longer C76.1 (+)
- net at L58.2 (-): now also C54.2 (-), CN4.2; no longer R24.1 (+)
- net at L55.2 (-): now also C57.2 (-), CN4.5; no longer R14.1 (+)
- net at L54.2 (-): now also C58.2 (-), CN4.6; no longer R22.1 (+)
- net at C75.1 (+), Q1.3 (G), R30.1 (+): now also R31.2 (-); no longer R31.1 (+)
- net at L67.2 (-): now also C45.2 (-), CN4.11; no longer R20.1 (+)
- net at CN1.3, L2.1 (+): now also DA3.3 (common)
- net at C70.1 (+): now also U2.4 (C1-); no longer U2.3 (C1+)
- net at C70.2 (-): now also U2.3 (C1+); no longer U2.4 (C1-)
- net at R37.2 (-): now also R36.1 (+); no longer R35.1 (+)
- net at CN2.26 (Pin_26), L22.2 (-): now also C12.2 (-); no longer C12.1 (+)
- net at U2.26 (C2+): now also C72.1 (+); no longer C72.2 (-)
- net at U2.27 (C2-): now also C72.2 (-); no longer C72.1 (+)
- net at CN2.15 (Pin_15), L23.2 (-): now also C29.2 (-); no longer C29.1 (+)
- net at CN2.21 (Pin_21), L27.2 (-): now also C21.2 (-); no longer C21.1 (+)
- net at CN6.4: now also L34.1 (+); no longer L34.2 (-)
- net at CN2.5 (Pin_5), L24.2 (-): now also C27.2 (-); no longer C27.1 (+)
- net at L61.2 (-): now also C51.2 (-), CN4.16 (P16); no longer R17.1 (+)
- net at CN2.19 (Pin_19), L25.2 (-): now also C25.2 (-); no longer C25.1 (+)
- net at R21.1 (+): now also L52.1 (+); no longer L52.2 (-)
- net at R37.1 (+): now also R35.2 (-), Q2.1 (B); no longer R36.2 (-)
- net at CN2.11 (Pin_11), L29.2 (-): now also C17.2 (-); no longer C17.1 (+)
- net at CN2.12 (Pin_12), L30.2 (-): now also C15.2 (-); no longer C15.1 (+)
- net at C13.1 (+), CN2.13 (Pin_13): now also L31.1 (+); no longer L31.2 (-)
- net at L56.2 (-): now also C56.2 (-), CN4.4; no longer R23.1 (+)
- net at L51.2 (-): now also C61.2 (-), CN4.9; no longer R12.1 (+)
- net at L53.2 (-): now also C59.2 (-), CN4.7; no longer R13.1 (+)
- net at L59.2 (-): now also C53.2 (-), CN4.1; no longer R16.1 (+)
- new net: R32.1 (+), R33.2 (-)
- new net: L66.1 (+), R28.2 (-)
- new net: L57.1 (+), R15.2 (-)
- new net: L63.1 (+), R18.2 (-)
- new net: L60.1 (+), R25.2 (-)
- new net: L65.1 (+), R19.2 (-)
- new net: CN7.4, L37.1 (+)
- new net: DA7.2 (A), DA8.1 (K)
- new net: DA8.2 (A), DA9.1 (K), R5.2 (-)
- new net: DA10.2 (A), DA6.2 (A), DA7.1 (K)
- new net: DA1.2 (A), DA2.2 (A), DA3.2 (A), DA4.1 (K)
- new net: L62.1 (+), R26.2 (-)
- new net: L64.1 (+), R27.2 (-)
- new net: L58.1 (+), R24.2 (-)
- new net: L55.1 (+), R14.2 (-)
- new net: C65.2 (-), CN6.5, L40.1 (+)
- new net: L54.1 (+), R22.2 (-)
- new net: L67.1 (+), R20.2 (-)
- new net: C66.2 (-), CN6.1, L42.1 (+)
- new net: L61.1 (+), R17.2 (-)
- new net: C60.2 (-), CN4.8, L52.2 (-)
- new net: L56.1 (+), R23.2 (-)
- new net: L51.1 (+), R12.2 (-)
- new net: L53.1 (+), R13.2 (-)
- new net: L59.1 (+), R16.2 (-)
Other:
- moved on the sheet: C11, C34, L11, L31, L34, L37, L38, L39, L40, L41, L42, L51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

Commit message: Add files via upload
Parts:
- C1, C2, C3, C4, C79, C80, C81, C82: footprint (none) -> Capacitor_SMD:C_0805_2012Metric; Indicator + -> (none); Rating V -> (none)
- C10, C15, C17, C19, C20, C21, C22, C23, C24, C25, C26, C29, C30, C31, C32, C33, C34, C35, C37, C38, C39, C40, C41, C42, C43, C44, C62, C63, C64, C65, C66, C67, C75, C76, C77, C78, C9: footprint (none) -> Capacitor_SMD:C_0603_1608Metric; Indicator + -> (none); Rating V -> (none)
- C11: value 1.5uF -> 2.5uF; footprint (none) -> Capacitor_SMD:C_1206_3216Metric; Indicator + -> (none); Rating V -> (none)
- C12: value 82nF -> 280nF; footprint (none) -> Capacitor_SMD:C_0603_1608Metric; Indicator + -> (none); Rating V -> (none)
- C13, C14, C16, C18: value 82nF -> 82pF; footprint (none) -> Capacitor_SMD:C_0603_1608Metric; Indicator + -> (none); Rating V -> (none)
- C27: value 82pF -> 280nF; footprint (none) -> Capacitor_SMD:C_0603_1608Metric; Indicator + -> (none); Rating V -> (none)
- C28: value 280nF -> 82pF; footprint (none) -> Capacitor_SMD:C_0603_1608Metric; Indicator + -> (none); Rating V -> (none)
- C45, C46, C47, C48, C49, C50, C51, C52, C53, C54, C55, C56, C57, C58, C59, C60, C61: value 200pF -> 200nF; footprint (none) -> Capacitor_SMD:C_0603_1608Metric; Indicator + -> (none); Rating V -> (none)
- C68, C73, C74, C83: footprint (none) -> Capacitor_SMD:C_0603_1608Metric; Indicator + -> (none); Rating V -> (none); now not fitted
- C69, C71: footprint (none) -> Capacitor_SMD:C_1206_3216Metric; Indicator + -> (none); Rating V -> (none); now not fitted
- C70, C72: footprint (none) -> Capacitor_SMD:C_0805_2012Metric; Indicator + -> (none); Rating V -> (none); now not fitted
- CN1: value VGA -> DSUB-15-HD_Socket_Horizontal_P2.29x1.90mm_EdgePinOffset3.03mm_Housed_MountingHolesOffset4.94mm; footprint (none) -> Connector_Dsub:DSUB-15-HD_Socket_Horizontal_P2.29x1.90mm_EdgePinOffset3.03mm_Housed_MountingHolesOffset4.94mm
- CN2: footprint (none) -> DockingStation:FDC_Connector
- CN4: value LPT -> DSUB-25_Socket_Horizontal_P2.77x2.84mm_EdgePinOffset4.94mm_Housed_MountingHolesOffset4.94mm; footprint (none) -> Connector_Dsub:DSUB-25_Socket_Horizontal_P2.77x2.84mm_EdgePinOffset4.94mm_Housed_MountingHolesOffset4.94mm
- CN5: value Serial Port -> DSUB-9_Pins_Horizontal_P2.77x2.84mm_EdgePinOffset4.94mm_Housed_MountingHolesOffset4.94mm; footprint (none) -> Connector_Dsub:DSUB-9_Pins_Horizontal_P2.77x2.84mm_EdgePinOffset4.94mm_Housed_MountingHolesOffset4.94mm
- CN6, CN7: value PS/2 -> PS2 Connector; footprint (none) -> DockingStation:PS2 Connector
- CN8: footprint (none) -> DockingStation:BarrelJack_Horizontal_PC110
- D2, D3: footprint (none) -> Diode_SMD:D_2010_5025Metric
- DA1, DA10, DA2, DA3, DA4, DA6, DA7, DA8, Q2: footprint (none) -> Package_TO_SOT_SMD:SOT-323_SC-70
- DA11, DA12: footprint (none) -> Package_TO_SOT_SMD:SOT-23W; now not fitted
- DA9: value 1W -> SOT-323_SC-70; footprint (none) -> Package_TO_SOT_SMD:SOT-323_SC-70; now not fitted
- F1: footprint (none) -> Fuse:Fuse_Littelfuse_395Series; Indicator ● -> (none); Rating W -> (none)
- J1, J2, J3, J4: value Dock Connector -> 25-1MP_P0.5mm_Horizontal; footprint (none) -> DockingStation:25-1MP_P0.5mm_Horizontal_PC110_dock
- L1, L11, L13, L14, L15, L16, L17, L18, L19, L2, L20, L21, L22, L23, L24, L25, L26, L27, L28, L29, L3, L30, L31, L34, L37, L38, L39, L40, L41, L42, L43, L44, L45, L46, L47, L48, L49, L50, L51, L52, L53, L54, L55, L56, L57, L58, L59, L60, L61, L62, L63, L64, L65, L66, L67: footprint (none) -> Inductor_SMD:L_0805_2012Metric; Indicator ● -> (none); Rating A -> (none)
- L5, L6: value 300nH -> 680nH; footprint (none) -> Inductor_SMD:L_0805_2012Metric; Indicator ● -> (none); Rating A -> (none)
- L68: footprint (none) -> DockingStation:EMI_Transformer
- Q1: value 3PJ4 -> 3P4J; footprint (none) -> Package_TO_SOT_SMD:TO-252-2; Rating V/A -> (none)
- R1, R2, R30, R31, R32, R33, R34, R35, R36, R37, R38: footprint (none) -> Resistor_SMD:R_0805_2012Metric; Indicator + -> (none); Rating W -> (none)
- R10, R11, R29, R40, R42, R43, R44, R45, R46, R47, R48, R49, R50, R51: footprint (none) -> Resistor_SMD:R_0603_1608Metric; Indicator + -> (none); Rating W -> (none); now not fitted
- R12, R13, R14, R15, R16, R17, R18, R19, R20, R21, R22, R23, R24, R25, R26, R27, R28, R3, R39, R4, R41, R5, R52, R53, R54, R55, R56, R57, R58, R59, R6, R60, R61, R62, R63, R64, R65, R66, R67, R68, R69, R7, R70, R71, R72, R73, R74, R75, R8, R9: footprint (none) -> Resistor_SMD:R_0603_1608Metric; Indicator + -> (none); Rating W -> (none)
- RA2, RA3, RA4, RA5, RA6: footprint (none) -> Resistor_SMD:R_Array_Concave_4x0603
- RA7, RA8: footprint (none) -> Resistor_SMD:R_Array_Concave_4x0603; now not fitted
- SSFC1: value Fuse -> Fuse_2010_5025Metric; footprint (none) -> Fuse:Fuse_2010_5025Metric; Indicator ● -> (none); Rating W -> (none)
- U1: value 74HCT244 -> 74VHCT244; footprint (none) -> Package_SO:SSOP-20_4.4x6.5mm_P0.65mm
- U2: value DNP -> DNP (LT1237CS); footprint (none) -> Package_SO:SSOP-28_5.3x10.2mm_P0.65mm; now not fitted
- U3: value ~ -> DS14C535MSA; footprint (none) -> Package_SO:SSOP-28_5.3x10.2mm_P0.65mm
- U4: footprint (none) -> Package_TO_SOT_SMD:SOT-23-5; now not fitted
- ZD1, ZD4: footprint Diode_THT:D_DO-35_SOD27_P10.16mm_Horizontal -> Diode_SMD:D_0805_2012Metric
Connections:
- net DOUT1: now also R68.1 (+); no longer R68.2 (-)
- net DOUT2: now also R70.1 (+); no longer R70.2 (-)
- net DOUT3: now also R72.1 (+); no longer R72.2 (-)
- net GND: now also C42.1 (+); no longer C42.2 (-)
- net RIN1: now also R74.1 (+); no longer R74.2 (-)
- net RIN2: now also R69.1 (+); no longer R69.2 (-)
- net RIN3: now also R71.1 (+); no longer R71.2 (-)
- net RIN4: now also R73.1 (+); no longer R73.2 (-)
- net RIN5: now also R75.1 (+); no longer R75.2 (-)
- net at C44.1 (+), CN5.1: now also L43.2 (-); no longer L43.1 (+)
- net at C39.1 (+), CN5.8: now also L48.2 (-); no longer L48.1 (+)
- net at C38.1 (+), CN5.4: now also L49.2 (-); no longer L49.1 (+)
- net at C37.1 (+), CN5.9: now also L50.2 (-); no longer L50.1 (+)
- net at C40.1 (+), CN5.3: now also L47.2 (-); no longer L47.1 (+)
- net at C43.1 (+), CN5.6: now also L44.2 (-); no longer L44.1 (+)
- net at C41.1 (+), CN5.7: now also L46.2 (-); no longer L46.1 (+)
- new net: L48.1 (+), R62.1 (+), R69.2 (-)
- new net: L49.1 (+), R60.1 (+), R68.2 (-)
- new net: L43.1 (+), R65.1 (+), R74.2 (-)
- new net: L50.1 (+), R67.1 (+), R75.2 (-)
- new net: L47.1 (+), R61.1 (+), R72.2 (-)
- new net: L45.1 (+), R63.1 (+), R73.2 (-)
- new net: L44.1 (+), R66.1 (+), R71.2 (-)
- new net: C42.2 (-), CN5.2, L45.2 (-)
- new net: L46.1 (+), R64.1 (+), R70.2 (-)
Other:
- moved on the sheet: L43, L44, L45, L46, L47, L48, L49, L50, R68, R69, R70, R71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

Commit message: Add files via upload
Parts:
- R60, R61, R62, R63, R64, R65, R66, R67: now not fitted
Connections:
- net VGA_BLUE: now also L2.1 (+); no longer L2.2 (-)
- net VGA_GREEN: now also L1.1 (+); no longer L1.2 (-)
- net VGA_RED: now also L3.1 (+); no longer L3.2 (-)
- net at CN1.2, DA2.3 (common): now also L1.2 (-); no longer L1.1 (+)
- net at CN1.1, DA1.3 (common): now also L3.2 (-); no longer L3.1 (+)
- net at CN1.3, DA3.3 (common): now also L2.2 (-); no longer L2.1 (+)
Other:
- moved on the sheet: L1, L2, L3
Changed lines of the file:
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@@
 	(symbol
 		(lib_id "PCM_Elektuur:L")
-		(at 713.74 389.89 90)
+		(at 713.74 389.89 270)
+		(mirror x)
 		(unit 1)
 		(exclude_from_sim no)
@@
 	(symbol
 		(lib_id "PCM_Elektuur:L")
-		(at 713.74 384.81 90)
+		(at 713.74 384.81 270)
+		(mirror x)
 		(unit 1)
 		(exclude_from_sim no)
@@
 		(in_bom yes)
 		(on_board yes)
-		(dnp no)
+		(dnp yes)
 		(property "Reference" "R60"
 			(at 161.29 230.886 90)
@@
 		(in_bom yes)
 		(on_board yes)
-		(dnp no)
+		(dnp yes)
 		(property "Reference" "R65"
 			(at 90.17 205.486 90)
@@
 		(in_bom yes)
 		(on_board yes)
-		(dnp no)
+		(dnp yes)
 		(property "Reference" "R61"
 			(at 175.26 235.966 90)
@@
 		(in_bom yes)
 		(on_board yes)
-		(dnp no)
+		(dnp yes)
 		(property "Reference" "R62"
 			(at 118.11 215.646 90)
@@
 		(in_bom yes)
 		(on_board yes)
-		(dnp no)
+		(dnp yes)
 		(property "Reference" "R67"
 			(at 104.14 210.566 90)
@@
 		(in_bom yes)
 		(on_board yes)
-		(dnp no)
+		(dnp yes)
 		(property "Reference" "R66"
 			(at 146.05 225.806 90)
@@
 		(in_bom yes)
 		(on_board yes)
-		(dnp no)
+		(dnp yes)
 		(property "Reference" "R63"
 			(at 189.23 241.046 90)
@@
 		(in_bom yes)
 		(on_board yes)
-		(dnp no)
+		(dnp yes)
 		(property "Reference" "R64"
 			(at 132.08 220.726 90)
@@
 	(symbol
 		(lib_id "PCM_Elektuur:L")
-		(at 713.74 394.97 90)
+		(at 713.74 394.97 270)
+		(mirror x)
 		(unit 1)
 		(exclude_from_sim no)
