File: PCB/DockingStation/DockingStation.kicad_sch (KiCad schematic)
At the start: 252 parts, among them CN1 DSUB-15-HD_Socket_Horizontal_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, CN2 FDC_Connector, CN4 DSUB-25_Socket_Horizontal_P2.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, CN5 DSUB-9_Pins_Horizontal_P2.77x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, CN6 PS2 Connector, CN7 PS2 Connector, CN8 BarrelJack_Horizontal_PC110, J1 25-1MP_P0.5mm_Horizontal, J2 25-1MP_P0.5mm_Horizontal, J3 25-1MP_P0.5mm_Horizontal, J4 25-1MP_P0.5mm_Horizontal, Q1 3P4J, Q2 8C, U1 74VHCT244, U2 DNP (LT1237CS), U3 DS14C535MSA, U4 DNP

Commit message: Add files via upload
Connections:
- net VGA_BLUE: now also DA3.3 (common)
- net VGA_GREEN: now also DA2.3 (common)
- net VGA_RED: now also DA1.3 (common)
- net at CN1.2, L1.2 (-): no longer DA2.3 (common)
- net at CN1.1, L3.2 (-): no longer DA1.3 (common)
- net at CN1.3, L2.2 (-): no longer DA3.3 (common)
Changed lines of the file:
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@@
 	)
 	(junction
-		(at 704.85 394.97)
-		(diameter 0)
-		(color 0 0 0 0)
-	)
-	(junction
 		(at 727.71 82.55)
 		(diameter 0)
@@
 	)
 	(junction
-		(at 707.39 384.81)
-		(diameter 0)
-		(color 0 0 0 0)
-	)
-	(junction
 		(at 609.6 401.32)
 		(diameter 0)
@@
 	)
 	(junction
+		(at 744.22 394.97)
+		(diameter 0)
+		(color 0 0 0 0)
+	)
+	(junction
 		(at 125.73 292.1)
 		(diameter 0)
@@
 	)
 	(junction
+		(at 732.79 389.89)
+		(diameter 0)
+		(color 0 0 0 0)
+	)
+	(junction
 		(at 218.44 398.78)
 		(diameter 0)
@@
 	)
 	(junction
-		(at 706.12 389.89)
-		(diameter 0)
-		(color 0 0 0 0)
-	)
-	(junction
 		(at 575.31 285.75)
 		(diameter 0)
@@
 	)
 	(junction
+		(at 721.36 384.81)
+		(diameter 0)
+		(color 0 0 0 0)
+	)
+	(junction
 		(at 314.96 101.6)
 		(diameter 0)
@@
 	(wire
 		(pts
+			(xy 744.22 394.97) (xy 744.22 422.91)
+		)
+		(stroke
+			(width 0)
+			(type default)
+		)
+	)
+	(wire
+		(pts
 			(xy 457.2 378.46) (xy 457.2 379.73)
 		)
@@
 	(wire
 		(pts
-			(xy 718.82 384.81) (xy 759.46 384.81)
+			(xy 718.82 384.81) (xy 721.36 384.81)
 		)
 		(stroke
@@
 	(wire
 		(pts
+			(xy 732.79 389.89) (xy 759.46 389.89)
+		)
+		(stroke
+			(width 0)
+			(type default)
+		)
+	)
+	(wire
+		(pts
 			(xy 697.23 87.63) (xy 770.89 87.63)
 		)
@@
 	(wire
 		(pts
+			(xy 744.22 394.97) (xy 759.46 394.97)
+		)
+		(stroke
+			(width 0)
+			(type default)
+		)
+	)
+	(wire
+		(pts
 			(xy 153.67 284.48) (xy 156.21 284.48)
 		)
@@
 	(wire
 		(pts
-			(xy 727.71 422.91) (xy 727.71 407.67)
+			(xy 336.55 29.21) (xy 336.55 33.02)
 		)
 		(stroke
@@
 	(wire
 		(pts
-			(xy 336.55 29.21) (xy 336.55 33.02)
+			(xy 189.23 530.86) (xy 189.23 549.91)
 		)
 		(stroke
@@
 	(wire
 		(pts
-			(xy 189.23 530.86) (xy 189.23 549.91)
+			(xy 519.43 392.43) (xy 557.53 392.43)
 		)
 		(stroke
@@
 	(wire
 		(pts
-			(xy 519.43 392.43) (xy 557.53 392.43)
+			(xy 567.69 392.43) (xy 570.23 392.43)
 		)
 		(stroke
@@
 	(wire
 		(pts
-			(xy 567.69 392.43) (xy 570.23 392.43)
+			(xy 130.81 81.28) (xy 370.84 81.28)
 		)
 		(stroke
@@
 	(wire
 		(pts
-			(xy 130.81 81.28) (xy 370.84 81.28)
+			(xy 64.77 114.3) (xy 67.31 114.3)
 		)
 		(stroke
@@
 	(wire
 		(pts
-			(xy 64.77 114.3) (xy 67.31 114.3)
+			(xy 252.73 535.94) (xy 252.73 549.91)
 		)
 		(stroke
@@
 	(wire
 		(pts
-			(xy 252.73 535.94) (xy 252.73 549.91)
+			(xy 707.39 405.13) (xy 721.36 405.13)
 		)
 		(stroke
@@
 	(wire
 		(pts
+			(xy 707.39 422.91) (xy 707.39 405.13)
+		)
+		(stroke
+			(width 0)
+			(type default)
+		)
+	)
+	(wire
+		(pts
 			(xy 332.74 116.84) (xy 370.84 116.84)
 		)
@@
 	(wire
 		(pts
-			(xy 707.39 422.91) (xy 707.39 384.81)
-		)
-		(stroke
-			(width 0)
-			(type default)
-		)
-	)
-	(wire
-		(pts
-			(xy 748.03 422.91) (xy 745.49 422.91)
+			(xy 748.03 422.91) (xy 744.22 422.91)
 		)
 		(stroke
@@
 	(wire
 		(pts
-			(xy 706.12 407.67) (xy 706.12 389.89)
-		)
-		(stroke
-			(width 0)
-			(type default)
-		)
-	)
-	(wire
-		(pts
 			(xy 232.41 495.3) (xy 232.41 514.35)
 		)
@@
 	(wire
 		(pts
-			(xy 694.69 394.97) (xy 704.85 394.97)
-		)
-		(stroke
-			(width 0)
-			(type default)
-		)
-	)
-	(wire
-		(pts
 			(xy 713.74 422.91) (xy 707.39 422.91)
 		)
@@
 	(wire
 		(pts
-			(xy 745.49 406.4) (xy 745.49 422.91)
-		)
-		(stroke
-			(width 0)
-			(type default)
-		)
-	)
-	(wire
-		(pts
 			(xy 166.37 96.52) (xy 146.05 96.52)
 		)
@@
 	(wire
 		(pts
+			(xy 732.79 405.13) (xy 732.79 389.89)
+		)
+		(stroke
+			(width 0)
+			(type default)
+		)
+	)
+	(wire
+		(pts
 			(xy 115.57 76.2) (xy 370.84 76.2)
 		)
@@
 	(wire
 		(pts
-			(xy 99.06 214.63) (xy 97.79 214.63)
+			(xy 721.36 405.13) (xy 721.36 384.81)
 		)
 		(stroke
@@
 	(wire
 		(pts
-			(xy 528.32 434.34) (xy 528.32 433.07)
+			(xy 99.06 214.63) (xy 97.79 214.63)
 		)
 		(stroke
@@
 	(wire
 		(pts
-			(xy 181.61 289.56) (xy 184.15 289.56)
+			(xy 528.32 434.34) (xy 528.32 433.07)
 		)
 		(stroke
@@
 	(wire
 		(pts
-			(xy 718.82 389.89) (xy 759.46 389.89)
+			(xy 181.61 289.56) (xy 184.15 289.56)
 		)
 		(stroke
@@
 	(wire
 		(pts
-			(xy 718.82 394.97) (xy 759.46 394.97)
+			(xy 718.82 394.97) (xy 744.22 394.97)
 		)
 		(stroke
@@
 	(wire
 		(pts
-			(xy 707.39 384.81) (xy 708.66 384.81)
+			(xy 694.69 384.81) (xy 708.66 384.81)
 		)
 		(stroke
@@
 	(wire
 		(pts
+			(xy 721.36 384.81) (xy 759.46 384.81)
+		)
+		(stroke
+			(width 0)
+			(type default)
+		)
+	)
+	(wire
+		(pts
 			(xy 473.71 67.31) (xy 473.71 133.35)
 		)
@@
 	(wire
 		(pts
-			(xy 704.85 406.4) (xy 704.85 394.97)
+			(xy 727.71 405.13) (xy 732.79 405.13)
 		)
 		(stroke
@@
 	(wire
 		(pts
+			(xy 727.71 422.91) (xy 727.71 405.13)
+		)
+		(stroke
+			(width 0)
+			(type default)
+		)
+	)
+	(wire
+		(pts
 			(xy 317.5 106.68) (xy 370.84 106.68)
 		)
@@
 	(wire
 		(pts
-			(xy 745.49 406.4) (xy 704.85 406.4)
-		)
-		(stroke
-			(width 0)
-			(type default)
-		)
-	)
-	(wire
-		(pts
 			(xy 128.27 274.32) (xy 125.73 274.32)
 		)
@@
 	(wire
 		(pts
-			(xy 727.71 407.67) (xy 706.12 407.67)
-		)
-		(stroke
-			(width 0)
-			(type default)
-		)
-	)
-	(wire
-		(pts
 			(xy 87.63 81.28) (xy 87.63 142.24)
 		)
@@
 	(wire
 		(pts
-			(xy 694.69 384.81) (xy 707.39 384.81)
-		)
-		(stroke
-			(width 0)
-			(type default)
-		)
-	)
-	(wire
-		(pts
 			(xy 227.33 398.78) (xy 274.32 398.78)
 		)
@@
 	(wire
 		(pts
-			(xy 704.85 394.97) (xy 708.66 394.97)
+			(xy 694.69 394.97) (xy 708.66 394.97)
 		)
 		(stroke
@@
 	(wire
 		(pts
-			(xy 706.12 389.89) (xy 708.66 389.89)
+			(xy 694.69 389.89) (xy 708.66 389.89)
 		)
 		(stroke
@@
 	(wire
 		(pts
-			(xy 694.69 389.89) (xy 706.12 389.89)
-		)
-		(stroke
-			(width 0)
-			(type default)
-		)
-	)
-	(wire
-		(pts
 			(xy 753.11 40.64) (xy 753.11 44.45)
 		)
@@
 		)
 		(stroke
+			(width 0)
+			(type default)
+		)
+	)
+	(wire
+		(pts
+			(xy 718.82 389.89) (xy 732.79 389.89)
+		)
+		(stroke
