File: PCB/Modem/Modem.kicad_pcb (KiCad board)
At the start: 6 copper layers, 64.6 x 58.9 mm, 211 parts, among them IC10 74ACT32, IC11 TSOP-I-32_18.4x8mm_P0.5mm_Rev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, IC12 TSOP-I-32_18.4x8mm_P0.5mm_Rev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, IC13 SOT-353_SC-70-5, IC14 SOT-353_SC-70-5, IC15 SOIC-8_5.3x6.2mm_P1.27mm, IC16 SOT-353_SC-70-5, IC17 SOT-353_SC-70-5, IC18 TSOT-23-5, IC2 SOT-353_SC-70-5, IC3 Line-Module, IC4 SOT-353_SC-70-5, IC5 MN195, IC6 SOT-353_SC-70-5, IC7 SOT-353_SC-70-5, IC8 TA31033F, IC9 SOT-353_SC-70-5, Q1 SOT-323_SC-70, Q2 SOT-89-3, Q3 SOT-323_SC-70, Q4 SOT-323_SC-70, Q7 SOT-323_SC-70, Q9 SOT-323_SC-70, SW2 SW_modem, T1 IsoTransformer

Commit message: Add files via upload
Connections:
- net D3_2 renamed MN195_S12
- net IC3_16 renamed MN195_SHIN
- net IC3_17 renamed MN195_AGCOUT
- net IC3_18 renamed MN195_AGCIN
- net IC5_12 renamed MN195_HDRES#
- net IC5_39 renamed MN195_VREEH
- net IC5_49 renamed MN195_S3
- net IC5_56 renamed MN195_S10
- net IC5_65 renamed FDC_DCD1_PC110
- net IC5_88 renamed MN195_VPDA#
- net IC5_95 renamed MN195_ADCK#
- net PNET2 renamed U54_VCC_PC110
- net PNET3 renamed PNET5_Q31_PC110
- net PNET5 renamed GND
- net R16_2 renamed MN195_S9
- C2 pad 1: (no net) -> MN195_IREF1
- C2 pad 2: (no net) -> MN195_TXLPIN
- C23 pad 2: (no net) -> MN195_DVDD1
- C34 pad 2: (no net) -> IREF2
- C39 pad 1: (no net) -> MN195_DVDD1
- C46 pad 2: (no net) -> MN195_DVDD1
- C47 pad 1: (no net) -> MN195_DVDD1
- C48 pad 2: (no net) -> MN195_DVDD1
- CNP4 pad 10: (no net) -> FDC_RXD1_PC110
- CNP4 pad 11: (no net) -> U100_FDC_TXD1_PC110
- CNP4 pad 16: (no net) -> MN195_VSEN#
- CNP4 pad 17: (no net) -> MN195_VSDA#
- CNP4 pad 18: (no net) -> MN195_VPCK#
- CNP4 pad 20: (no net) -> MN195_IRQ1#
- CNP4 pad 22: (no net) -> J13_58_PC110
- CNP4 pad 23: (no net) -> J13_41_PC110
- CNP4 pad 24: (no net) -> J13_42_PC110
- CNP4 pad 3: (no net) -> U102_6A_PC110
- CNP4 pad 5: (no net) -> FDC_RI1_PC110
- CNP4 pad 6: (no net) -> U100_FDC_DIR1#_PC110
- CNP4 pad 7: (no net) -> FDC_DSR1_PC110
- CNP4 pad 8: (no net) -> FDC_CTS1#
- CNP4 pad 9: (no net) -> U110_FDC_RTS1#_PC110
- D8 pad 2: (no net) -> MN195_S13
- IC10 pad 10: (no net) -> U102_6A_PC110
- IC10 pad 2: (no net) -> FDC_RI1_PC110
- IC10 pad 5: (no net) -> FDC_CTS1#
- IC3 pad 10: (no net) -> MN195_TXOUT
- IC3 pad 11: (no net) -> MN195_MTA1
- IC3 pad 2: (no net) -> MN195_HVDD
- IC3 pad 3: (no net) -> MN195_RXL
- IC3 pad 4: (no net) -> MN195_S1
- IC3 pad 5: (no net) -> MN195_S4
- IC3 pad 6: (no net) -> MN195_HPOUT
- IC3 pad 9: (no net) -> MN195_TXLPIN
- IC4 pad 2: (no net) -> MN195_S2
- IC5 pad 1: (no net) -> MN195_MD7
- IC5 pad 100: (no net) -> MN195_UC0
- IC5 pad 101: (no net) -> MN195_UC2
- IC5 pad 102: (no net) -> MN195_UC3
- IC5 pad 103: (no net) -> MN195_A23
- IC5 pad 104: (no net) -> MN195_A22
- IC5 pad 105: (no net) -> MN195_A21
- IC5 pad 106: (no net) -> MN195_A20
- IC5 pad 107: (no net) -> MN195_A19
- IC5 pad 108: (no net) -> MN195_A18
- IC5 pad 109: (no net) -> MN195_A17
- IC5 pad 11: (no net) -> MN195_CX
- IC5 pad 110: (no net) -> MN195_A16
- IC5 pad 111: (no net) -> MN195_A15
- IC5 pad 113: (no net) -> MN195_DVDD1
- IC5 pad 114: (no net) -> MN195_A14
- IC5 pad 115: (no net) -> MN195_A13
- IC5 pad 116: (no net) -> MN195_A12
- IC5 pad 117: (no net) -> MN195_A11
- IC5 pad 118: (no net) -> MN195_A10
- IC5 pad 119: (no net) -> MN195_A9
- IC5 pad 120: (no net) -> MN195_A8
- IC5 pad 121: (no net) -> MN195_A7
- IC5 pad 122: (no net) -> MN195_A6
- IC5 pad 123: (no net) -> MN195_A5
- IC5 pad 124: (no net) -> MN195_A4
- IC5 pad 125: (no net) -> MN195_A3
- IC5 pad 126: (no net) -> MN195_A2
- IC5 pad 127: (no net) -> MN195_A1
- IC5 pad 128: (no net) -> MN195_A0
- IC5 pad 13: (no net) -> MN195_DVDD1
- IC5 pad 15: (no net) -> MN195_WR#
- IC5 pad 16: (no net) -> MN195_RD#
- IC5 pad 17: (no net) -> MN195_RNW
- IC5 pad 18: (no net) -> MN195_BA
- IC5 pad 2: (no net) -> MN195_MD6
- IC5 pad 20: (no net) -> MN195_EQMD#
- IC5 pad 22: (no net) -> MN195_EYCY#
- IC5 pad 23: (no net) -> MN195_PLSD
- IC5 pad 25: (no net) -> MN195_DVDD1
- IC5 pad 29: (no net) -> MN195_HPOUT
- IC5 pad 3: (no net) -> MN195_MD5
- IC5 pad 30: (no net) -> MN195_RXLPIN
- IC5 pad 31: (no net) -> IREF2
- IC5 pad 32: (no net) -> MN195_RXL
- IC5 pad 33: (no net) -> MN195_HVDD
- IC5 pad 34: (no net) -> MN195_TXOUT
- IC5 pad 36: (no net) -> MN195_TXLPIN
- IC5 pad 37: (no net) -> MN195_IREF1
- IC5 pad 38: (no net) -> MN195_IREF0
- IC5 pad 4: (no net) -> MN195_MD4
- IC5 pad 42: (no net) -> MN195_MOD1,3
- IC5 pad 45: (no net) -> MN195_MOD1,3
- IC5 pad 46: (no net) -> MN195_S0
- IC5 pad 47: (no net) -> MN195_S1
- IC5 pad 48: (no net) -> MN195_S2
- IC5 pad 5: (no net) -> MN195_MD3
- IC5 pad 50: (no net) -> MN195_S4
- IC5 pad 51: (no net) -> FDC_DSR1_PC110
- IC5 pad 52: (no net) -> FDC_RXD1_PC110
- IC5 pad 53: (no net) -> U110_FDC_RTS1#_PC110
- IC5 pad 54: (no net) -> U100_FDC_DIR1#_PC110
- IC5 pad 57: (no net) -> MN195_S11
- IC5 pad 59: (no net) -> MN195_S13
- IC5 pad 6: (no net) -> MN195_MD2
- IC5 pad 60: (no net) -> MN195_S14
- IC5 pad 61: (no net) -> MN195_S14
- IC5 pad 62: (no net) -> MN195_U1ST#
- IC5 pad 63: (no net) -> MN195_U1RD#
- IC5 pad 64: (no net) -> MN195_U1RCK
- IC5 pad 66: (no net) -> MN195_U1TCK#
- IC5 pad 67: (no net) -> MN195_IRQ1#
- IC5 pad 68: (no net) -> MN195_IRQ2#
- IC5 pad 69: (no net) -> MN195_IRQ3#
- IC5 pad 7: (no net) -> MN195_MD1
- IC5 pad 70: (no net) -> MN195_IRQ4#
- IC5 pad 71: (no net) -> MN195_U2ST#
- IC5 pad 72: (no net) -> MN195_U2RD#
- IC5 pad 73: (no net) -> MN195_U2RCK#
- IC5 pad 74: (no net) -> MN195_U2SD#
- IC5 pad 75: (no net) -> MN195_U2TCK#
- IC5 pad 77: (no net) -> MN195_DVDD1
- IC5 pad 78: (no net) -> MN195_MTB4
- IC5 pad 79: (no net) -> MN195_MTB3
- IC5 pad 8: (no net) -> MN195_MD0
- IC5 pad 80: (no net) -> MN195_MTB2
- IC5 pad 81: (no net) -> MN195_MTB1
- IC5 pad 82: (no net) -> MN195_SH4#
- IC5 pad 83: (no net) -> MN195_SH3#
- IC5 pad 84: (no net) -> MN195_SH2#
- IC5 pad 85: (no net) -> MN195_SH1#
- IC5 pad 86: (no net) -> MN195_VPST
- IC5 pad 87: (no net) -> MN195_VPCK#
- IC5 pad 89: (no net) -> MN195_MTA4
- IC5 pad 9: (no net) -> MN195_SYNCA
- IC5 pad 90: (no net) -> MN195_MTA3
- IC5 pad 91: (no net) -> MN195_MTA2
- IC5 pad 92: (no net) -> MN195_MTA1
- IC5 pad 93: (no net) -> MN195_MOT
- IC5 pad 94: (no net) -> MN195_V8CK#
- IC5 pad 96: (no net) -> MN195_VSDA#
- IC5 pad 97: (no net) -> MN195_VIR#
- IC5 pad 98: (no net) -> MN195_VSEN#
- IC5 pad 99: (no net) -> MN195_UC0#
- IC6 pad 1: (no net) -> MN195_S0
- IC9 pad 4: (no net) -> U100_FDC_TXD1_PC110
- Q4 pad 2: (no net) -> J13_58_PC110
- R10 pad 1: (no net) -> MN195_IREF0
- R10 pad 2: (no net) -> MN195_IREF1
- R101 pad 2: (no net) -> MN195_UC0#
- R102 pad 2: (no net) -> MN195_A18
- R103 pad 2: (no net) -> MN195_A16
- R104 pad 2: (no net) -> MN195_A14
- R105 pad 2: (no net) -> MN195_A12
- R106 pad 2: (no net) -> MN195_A10
- R107 pad 2: (no net) -> MN195_A8
- R108 pad 2: (no net) -> MN195_A6
- R11 pad 1: (no net) -> MN195_IREF1
- R11 pad 2: (no net) -> MN195_TXLPIN
- R110 pad 2: (no net) -> MN195_A2
- R111 pad 2: (no net) -> MN195_A0
- R114 pad 2: (no net) -> MN195_A17
- R115 pad 2: (no net) -> MN195_A15
- R116 pad 2: (no net) -> MN195_A13
- R117 pad 2: (no net) -> MN195_A11
- R118 pad 2: (no net) -> MN195_A9
- R119 pad 2: (no net) -> MN195_A7
- R120 pad 2: (no net) -> MN195_A5
- R121 pad 2: (no net) -> MN195_A3
- R122 pad 2: (no net) -> MN195_A1
- R123 pad 2: (no net) -> MN195_RD#
- R124 pad 2: (no net) -> MN195_WR#
- R124 pad 2: (no net) -> MN195_MD3
- R125 pad 2: (no net) -> MN195_MD0
- R126 pad 2: (no net) -> MN195_MD1
- R127 pad 2: (no net) -> MN195_MD2
- R129 pad 2: (no net) -> MN195_MD4
- R130 pad 2: (no net) -> MN195_MD5
- R131 pad 2: (no net) -> MN195_MD6
- R132 pad 2: (no net) -> MN195_MD7
- R19 pad 1: (no net) -> MN195_U1RD#
- R21 pad 2: (no net) -> MN195_S0
- R22 pad 2: (no net) -> FDC_RI1_PC110
- R23 pad 2: (no net) -> FDC_CTS1#
- R26 pad 1: (no net) -> MN195_DVDD1
- R27 pad 1: (no net) -> U102_6A_PC110
- R27 pad 2: (no net) -> MN195_U1RD#
- R3 pad 1: (no net) -> MN195_IRQ1#
- R33 pad 1: (no net) -> MN195_DVDD1
- R34 pad 1: (no net) -> MN195_DVDD1
- R41 pad 2: (no net) -> MN195_MOD1,3
- R43 pad 2: (no net) -> MN195_IRQ2#
- R44 pad 1: (no net) -> MN195_CX
- R47 pad 2: (no net) -> MN195_S2
- R52 pad 2: (no net) -> J13_58_PC110
- R72 pad 2: (no net) -> MN195_S13
- R92 pad 1: (no net) -> MN195_S0
Routing:
- net (no net): track 3153.1 -> 2140.9 mm, vias 207 -> 151
- net MN195_DVDD1: track 0.00 -> 76.2 mm, vias 0 -> 6
- net MN195_S0: track 0.00 -> 59.4 mm, vias 0 -> 2
- net J13_58_PC110: track 0.00 -> 51.3 mm, vias 0 -> 2
- net MN195_S2: track 0.00 -> 47.6 mm, vias 0 -> 2
- net MN195_S13: track 0.00 -> 45.2 mm, vias 0 -> 2
- net MN195_S11: track 0.00 -> 43.9 mm, vias 0 -> 2
- net MN195_MTA1: track 0.00 -> 38.9 mm, vias 0 -> 1
- net MN195_S4: track 0.00 -> 33.2 mm, vias 0 -> 1
- net MN195_PLSD: track 0.00 -> 32.2 mm, vias 0 -> 1
- net FDC_DSR1_PC110: track 0.00 -> 31.6 mm, vias 0 -> 2
- net MN195_S1: track 0.00 -> 31.3 mm, vias 0 -> 1
- net FDC_RXD1_PC110: track 0.00 -> 31.1 mm, vias 0 -> 2
- net U100_FDC_DIR1#_PC110: track 0.00 -> 28.9 mm, vias 0 -> 2
- net U110_FDC_RTS1#_PC110: track 0.00 -> 27.9 mm, vias 0 -> 2
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
Commit message: Add files via upload
Parts:
- C1, C4, C52, C54: value C_0603_1608Metric -> 330nF
- C13: value C_1206_3216Metric -> 822J
- C15, C2, C32: value C_0603_1608Metric -> 1.2uF
- C2, C34: value C_0603_1608Metric -> 1nF
- C23: value C_0805_2012Metric -> 1.2uF
- C24, C37: value C_0603_1608Metric -> 230nF
- C26: value C_0603_1608Metric -> 10nF
- C28: value C_1206_3216Metric -> 8.1uF
- C29, C30: value C_0603_1608Metric -> 1.5uF
- C3: value C_0603_1608Metric -> 30nF
- C31: value C_1206_3216Metric -> 230nF
- C38: value C_0603_1608Metric -> 2.2uF
- C39: value C_0603_1608Metric -> 100nF
- C39, C48: value C_0603_1608Metric -> 25nF
- C40: value C_0603_1608Metric -> 16nF
- C41, C43: value C_0603_1608Metric -> 1uF
- C42, C51: value C_0603_1608Metric -> 1.2nF
- C46, C47: value C_0603_1608Metric -> 24nF
- C5: value C_0603_1608Metric -> 250nF
- C56: value C_0402_1005Metric -> 1.6nF
- C57: value C_1206_3216Metric -> 6.8uF
- C58: value C_0603_1608Metric -> 220nF
- C59, C60, C62: value C_2220_5750Metric -> 280nF
- C70, C72: value C_0603_1608Metric -> 1.8uF
- C71: value C_0805_2012Metric -> 1.3uF
- C73: value C_0402_1005Metric -> 100pF
- C74: value C_0805_2012Metric -> 220nF
- D10: value D_1206_3216Metric -> 152
- D2: value D_SOD-128 -> 1N4148
- D3, D4, D8: value D_1206_3216Metric_modem -> 5
- D5: value SOT-323_SC-70 -> 3D
- D6: value SOT-23-3 -> 30H
- DA1: value DA_Modem -> M1T
- IC10: value 74ACT32 -> AT32 433
- IC11: value TSOP-I-32_18.4x8mm_P0.5mm_Reverse -> 29F040A-12
- IC12: value TSOP-I-32_18.4x8mm_P0.5mm_Reverse -> KM681000BLT-7
- IC13, IC17, IC2, IC7, IC9: value SOT-353_SC-70-5 -> EA
- IC14: value SOT-353_SC-70-5 -> E4
- IC16: value SOT-353_SC-70-5 -> E3
- IC18: value TSOT-23-5 -> 3L01
- IC4: value SOT-353_SC-70-5 -> E5
- IC6: value SOT-353_SC-70-5 -> 54
- L1, L2: value L_1206_3216Metric -> 1.2uH
- L3, L5: value L_0603_1608Metric -> 1.8uH
- L4: value L_0603_1608Metric -> 1.2uH
- NF1: value L_1206_3216Metric -> 300nH
- NF2, NF4: value L_1206_3216Metric -> 4.7nH
- NF3: value L_1206_3216Metric -> 0
- Q1, Q4: value SOT-323_SC-70 -> CQ
- Q2: value SOT-89-3 -> DA QU
- Q3: value SOT-323_SC-70 -> 123
- Q9: value SOT-323_SC-70 -> HP
- R10, R11, R68: value R_0402_1005Metric -> 38k
- R100, R51, R72 (x2): value R_0402_1005Metric -> 470k
- R101, R102, R103, R104, R105, R106, R107, R108, R109, R110, R111, R112, R114, R115, R116, R117, R118, R119, R120, R121, R122, R123, R124 (x2), R125, R126, R127, R129, R130, R131, R132: value R_0402_1005Metric -> 100
- R12, R75: value R_2010_5025Metric -> 2.2k
- R13, R133, R16, R17, R19, R21, R47, R49, R62, R67, R82: value R_0402_1005Metric -> 10k
- R14: value R_0402_1005Metric -> 560k
- R15: value R_0402_1005Metric -> 330k
- R18, R46: value R_0402_1005Metric -> 1.5k
- R2, R28, R29, R3, R30, R31, R32, R36, R37, R38, R41, R43: value R_0402_1005Metric -> 4.7k
- R20, R63, R81, R9: value R_0402_1005Metric -> 100k
- R24: value R_0603_1608Metric -> 200
- R25: value R_0402_1005Metric -> unknown
- R26, R33, R34, R7: value R_1206_3216Metric -> 10
- R35: value R_1206_3216Metric -> 20
- R4: value R_0402_1005Metric -> 330
- R42: value R_0402_1005Metric -> 15k
- R44: value R_0402_1005Metric -> 51
- R48: value R_1206_3216Metric -> 3.3
- R5: value R_0603_1608Metric -> 100
- R50: value R_0603_1608Metric -> 6.2k
- R52, R70, R71: value R_0402_1005Metric -> 1k
- R53: value R_0603_1608Metric -> 11k
- R54: value R_0603_1608Metric -> 1.5k
- R55: value R_2010_5025Metric -> 82
- R56: value R_1206_3216Metric -> 15
- R57: value R_0603_1608Metric -> 150
- R58: value R_0603_1608Metric -> 620
- R59, R60: value R_0402_1005Metric -> 2.2k
- R6: value R_0603_1608Metric -> 3.3k
- R65: value R_0402_1005Metric -> 15
- R68: value R_0402_1005Metric -> 20k
- R73: value R_0603_1608Metric -> 120
- R76: value R_0402_1005Metric -> 2.4k
- R77: value R_0402_1005Metric -> 270k
- R78: value R_0402_1005Metric -> 5.6k
- R98, R99: value R_0805_2012Metric -> 100
- renumbered C56 to 470nF
Connections:
- R51 pad 1: (no net) -> GND
- R51 pad 2: (no net) -> MN195_HDRES#
Routing:
- net MN195_HDRES#: track 12.3 -> 14.8 mm
- net GND: track 230.4 -> 232.4 mm
- net (no net): track 2140.9 -> 2142.7 mm
- net PNET4: track 52.2 -> 54.1 mm
- added copper zone on B.Cu, net GND
- added copper zone on B.Cu, net U54_VCC_PC110

Commit message: Add files via upload
Parts:
- R1: value R_0402_1005Metric -> 12k
- R25: value unknown -> 500k
- R8: value R_0402_1005Metric -> 22k
Changed lines of the file:
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@@
 			)
 		)
-		(property "Value" "R_0402_1005Metric"
+		(property "Value" "22k"
 			(at 0 -1.17 0)
 			(layer "B.Fab")
@@
 			)
 		)
-		(property "Value" "unknown"
+		(property "Value" "500k"
 			(at 0 -1.17 0)
 			(layer "B.Fab")
@@
 			)
 		)
-		(property "Value" "R_0402_1005Metric"
+		(property "Value" "12k"
 			(at 0 -1.17 0)
 			(layer "B.Fab")
@@
 		(start 167.99 117.6)
 		(end 173.09 117.6)
-		(width 0.2)
+		(width 0.5)
 		(layer "F.Cu")
 		(net 2)
@@
 		(start 170.74 103.8)
 		(end 167.99 103.8)
-		(width 0.2)
+		(width 0.5)
 		(layer "F.Cu")
 		(net 5)
@@
 		(start 173.09 103.8)
 		(end 170.86 103.8)
-		(width 0.2)
+		(width 0.5)
 		(layer "F.Cu")
 		(net 5)
@@
 		(start 164.37 110.1)
 		(end 167.99 110.1)
-		(width 0.1)
+		(width 0.2)
 		(layer "F.Cu")
 		(net 27)
@@
 	)
 	(segment
+		(start 170.04 108.99)
+		(end 171.48 107.55)
+		(width 0.2)
+		(layer "F.Cu")
+		(net 33)
+	)
+	(segment
+		(start 171.48 107.55)
+		(end 173.09 107.55)
+		(width 0.2)
+		(layer "F.Cu")
+		(net 33)
+	)
+	(segment
 		(start 156.08 112.54)
 		(end 156.08 111.81)
@@
 	)
 	(segment
-		(start 170.04 109.54)
-		(end 170.04 108.6)
-		(width 0.1)
-		(layer "F.Cu")
-		(net 33)
-	)
-	(segment
 		(start 153.85 119.42)
 		(end 153.85 117.48)
@@
 	)
 	(segment
-		(start 170.04 108.6)
-		(end 171.09 107.55)
-		(width 0.1)
-		(layer "F.Cu")
-		(net 33)
-	)
-	(segment
-		(start 171.09 107.55)
-		(end 173.09 107.55)
+		(start 154.91 121.11)
+		(end 154.91 120.48)
 		(width 0.1)
 		(layer "F.Cu")
@@
 	)
 	(segment
-		(start 154.91 121.11)
-		(end 154.91 120.48)
-		(width 0.1)
+		(start 170.04 109.54)
+		(end 170.04 108.99)
+		(width 0.2)
 		(layer "F.Cu")
 		(net 33)
@@
 		(start 171.11 109.5)
 		(end 171.81 108.8)
-		(width 0.1)
+		(width 0.2)
 		(layer "F.Cu")
 		(net 34)
@@
 		(start 171.81 108.8)
 		(end 173.09 108.8)
-		(width 0.1)
+		(width 0.2)
 		(layer "F.Cu")
 		(net 34)
@@
 		(start 164.42 118.11)
 		(end 162.91 118.11)
-		(width 0.1)
+		(width 0.2)
 		(layer "F.Cu")
 		(net 43)
@@
 		(start 165.13 119.81)
 		(end 165.13 117.95)
-		(width 0.1)
+		(width 0.3)
 		(layer "F.Cu")
 		(net 43)
@@
 		(start 170.96 110.93)
 		(end 170.54 111.35)
-		(width 0.1)
+		(width 0.2)
 		(layer "F.Cu")
 		(net 43)
@@
 		(start 165.13 117.95)
 		(end 164.58 117.95)
-		(width 0.1)
+		(width 0.2)
 		(layer "F.Cu")
 		(net 43)
@@
 		(start 170.54 111.35)
 		(end 167.99 111.35)
-		(width 0.1)
+		(width 0.2)
 		(layer "F.Cu")
 		(net 43)
@@
 		(start 164.58 117.95)
 		(end 164.42 118.11)
-		(width 0.1)
+		(width 0.2)
 		(layer "F.Cu")
 		(net 43)

Commit message: Add files via upload
Parts:
- IC11: value 29F040A-12 -> 29F040A-12 (I-Reverse
- IC12: value KM681000BLT-7 -> KM681000BLT-7 (I-Reverse)
Connections:
- C45 pad 2: (no net) -> MN195_VREEH
- C70 pad 1: (no net) -> C70_1
- C70 pad 2: (no net) -> C70_2
- C74 pad 1: (no net) -> C74_1
- DA1 pad 1: (no net) -> C70_2
- DA1 pad 4: (no net) -> C70_2
- IC10 pad 1: (no net) -> IC10_1
- IC10 pad 11: (no net) -> IC10_11
- IC10 pad 3: (no net) -> IC10_3
- IC10 pad 6: (no net) -> IC10_6
- IC10 pad 8: (no net) -> IC10_8
- IC11 pad 1: (no net) -> 29F_OE#
- IC11 pad 10: (no net) -> 29F_DQ2
- IC11 pad 11: (no net) -> 29F_DQ1
- IC11 pad 12: (no net) -> 29F_DQ0
- IC11 pad 13: (no net) -> 29F_A0
- IC11 pad 14: (no net) -> 29F_A1
- IC11 pad 15: (no net) -> 29F_A2
- IC11 pad 16: (no net) -> 29F_A3
- IC11 pad 17: (no net) -> 29F_A4
- IC11 pad 18: (no net) -> 29F_A5
- IC11 pad 19: IC11_19 -> 29F_A6
- IC11 pad 2: (no net) -> 29F_A10
- IC11 pad 20: (no net) -> 29FA7
- IC11 pad 21: (no net) -> 29F_A12
- IC11 pad 22: (no net) -> 29F_A15
- IC11 pad 23: (no net) -> 29F_A16
- IC11 pad 24: (no net) -> 29F_A18
- IC11 pad 26: (no net) -> 29F_WE#
- IC11 pad 27: (no net) -> 29F_A17
- IC11 pad 28: (no net) -> 29F_A14
- IC11 pad 29: (no net) -> 29F_A13
- IC11 pad 3: (no net) -> 29F_CE#
- IC11 pad 30: (no net) -> 29F_A8
- IC11 pad 31: (no net) -> 29F_A9
- IC11 pad 32: (no net) -> 29F_A11
- IC11 pad 4: (no net) -> 29F_DQ7
- IC11 pad 5: (no net) -> 29F_DQ6
- IC11 pad 6: (no net) -> 29F_DQ5
- IC11 pad 7: (no net) -> 29F_DQ4
- IC11 pad 8: (no net) -> 29F_DQ3
- IC12 pad 1: (no net) -> 29F_A11
- IC12 pad 10: (no net) -> 29F_A16
- IC12 pad 11: (no net) -> 29F_A14
- IC12 pad 12: (no net) -> 29F_A12
- IC12 pad 13: (no net) -> 29FA7
- IC12 pad 14: (no net) -> 29F_A6
- IC12 pad 15: (no net) -> 29F_A5
- IC12 pad 16: (no net) -> 29F_A4
- IC12 pad 17: (no net) -> 29F_A3
- IC12 pad 18: (no net) -> 29F_A2
- IC12 pad 19: IC11_19 -> 29F_A1
- IC12 pad 2: (no net) -> 29F_A9
- IC12 pad 20: (no net) -> 29F_A0
- IC12 pad 21: (no net) -> 29F_DQ0
- IC12 pad 22: (no net) -> 29F_DQ1
- IC12 pad 23: (no net) -> 29F_DQ2
- IC12 pad 24: (no net) -> GND
- IC12 pad 25: U54_VCC_PC110 -> 29F_DQ3
- IC12 pad 26: (no net) -> 29F_DQ4
- IC12 pad 27: U54_VCC_PC110 -> 29F_DQ5
- IC12 pad 28: (no net) -> 29F_DQ6
- IC12 pad 29: (no net) -> 29F_DQ7
- IC12 pad 3: IC12_3 -> 29F_A8
- IC12 pad 30: (no net) -> IC12_3
- IC12 pad 31: (no net) -> 29F_A10
- IC12 pad 32: (no net) -> 29F_OE#
- IC12 pad 4: (no net) -> 29F_A13
- IC12 pad 5: (no net) -> 29F_WE#
- IC12 pad 6: (no net) -> U54_VCC_PC110
- IC12 pad 7: (no net) -> 29F_A15
- IC12 pad 8: (no net) -> U54_VCC_PC110
- IC12 pad 9: GND -> KM68_NC
- IC17 pad 4: (no net) -> C70_1
- IC17 pad 5: (no net) -> C74_1
- NF4 pad 2: (no net) -> GND
- R100 pad 1: (no net) -> C70_1
- R101 pad 1: (no net) -> 29F_CE#
- R102 pad 1: (no net) -> 29F_A18
- R103 pad 1: (no net) -> 29F_A16
- R104 pad 1: (no net) -> 29F_A14
- R106 pad 1: (no net) -> 29F_A10
- R107 pad 1: (no net) -> 29F_A8
- R108 pad 1: IC11_19 -> 29F_A6
- R109 pad 1: (no net) -> 29F_A4
- R110 pad 1: (no net) -> 29F_A2
- R111 pad 1: (no net) -> 29F_A0
- R114 pad 1: (no net) -> 29F_A17
- R115 pad 1: (no net) -> 29F_A15
- R116 pad 1: (no net) -> 29F_A13
- R117 pad 1: (no net) -> 29F_A11
- R118 pad 1: (no net) -> 29F_A9
- R119 pad 1: (no net) -> 29FA7
- R120 pad 1: (no net) -> 29F_A5
- R121 pad 1: (no net) -> 29F_A3
- R122 pad 1: (no net) -> 29F_A1
- R123 pad 1: (no net) -> 29F_OE#
- R124 pad 1: (no net) -> 29F_WE#
- R124 pad 1: (no net) -> 29F_DQ3
- R125 pad 1: (no net) -> 29F_DQ0
- R126 pad 1: (no net) -> 29F_DQ1
- R127 pad 1: (no net) -> 29F_DQ2
- R129 pad 1: (no net) -> 29F_DQ4
- R130 pad 1: (no net) -> 29F_DQ5
- R131 pad 1: (no net) -> 29F_DQ6
- R132 pad 1: (no net) -> 29F_DQ7
- R19 pad 2: (no net) -> IC10_8
- R28 pad 2: (no net) -> 29F_DQ0
- R29 pad 2: (no net) -> 29F_DQ1
- R30 pad 2: (no net) -> 29F_DQ2
- R31 pad 2: (no net) -> 29F_DQ3
- R32 pad 2: (no net) -> 29F_DQ4
- R36 pad 2: (no net) -> 29F_DQ5
- R37 pad 2: (no net) -> 29F_DQ6
- R38 pad 2: (no net) -> 29F_DQ7
- R98 pad 1: (no net) -> C74_1
Routing:
- net (no net): track 2142.7 -> 1007.1 mm, vias 151 -> 67
- net 29F_DQ6: track 0.00 -> 54.4 mm, vias 0 -> 3
- net 29F_DQ5: track 0.00 -> 52.9 mm, vias 0 -> 3
- net 29F_DQ4: track 0.00 -> 50.3 mm, vias 0 -> 3
- net 29F_A0: track 0.00 -> 49.8 mm, vias 0 -> 3
- net 29F_A3: track 0.00 -> 49.4 mm, vias 0 -> 4
- net 29F_A1: track 0.00 -> 47.9 mm, vias 0 -> 3
- net 29F_A2: track 0.00 -> 47.8 mm, vias 0 -> 3
- net 29F_DQ2: track 0.00 -> 47.8 mm, vias 0 -> 3
- net 29F_DQ3: track 0.00 -> 47.7 mm, vias 0 -> 3
- net 29F_DQ0: track 0.00 -> 46.1 mm, vias 0 -> 3
- net 29F_A10: track 0.00 -> 46.1 mm, vias 0 -> 3
- net 29F_DQ1: track 0.00 -> 45.9 mm, vias 0 -> 3
- net 29F_A4: track 0.00 -> 42.5 mm, vias 0 -> 3
- net 29F_A5: track 0.00 -> 40.9 mm, vias 0 -> 4
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