File: PCB/Modem/Modem.kicad_pcb (KiCad board)
At the start: 6 copper layers, 64.6 x 58.9 mm, 211 parts, among them IC10 AT32 433, IC11 29F040A-12 (I-Reverse, IC12 KM681000BLT-7 (I-Reverse), IC13 EA, IC14 E4, IC15 SOIC-8_5.3x6.2mm_P1.27mm, IC16 E3, IC17 EA, IC18 3L01, IC2 EA, IC3 Line-Module, IC4 E5, IC5 MN195, IC6 54, IC7 EA, IC8 TA31033F, IC9 EA, Q1 CQ, Q2 DA QU, Q3 123, Q4 CQ, Q7 SOT-323_SC-70, Q9 HP, SW2 SW_modem, T1 IsoTransformer

Commit message: Add files via upload
Parts:
- R22, R23, R27: value R_0402_1005Metric -> DNP
Connections:
- net U100_FDC_DIR1#_PC110 renamed FDC_DIR1#_PC110
- net U100_FDC_TXD1_PC110 renamed FDC_TXD1_PC110
- net U102_6A_PC110 renamed MN195_U1RD#_R
- net U110_FDC_RTS1#_PC110 renamed FDC_RTS1#_PC110
- net U54_VCC_PC110 renamed VCC_PC110
- 470nF pad 1: (no net) -> R61_2
- 470nF pad 2: (no net) -> IC15_8
- C1 pad 1: (no net) -> RL1_5
- C1 pad 2: (no net) -> T1_4
- C12 pad 2: (no net) -> IC8_16
- C13 pad 1: (no net) -> IC8_15
- C13 pad 2: (no net) -> R65_2
- C15 pad 1: (no net) -> D1_2
- C15 pad 2: (no net) -> D2_2
- C2 pad 1: (no net) -> IC8_5
- C24 pad 1: (no net) -> OSC1_2
- C26 pad 1: (no net) -> R57_2
- C26 pad 2: (no net) -> R54_2
- C3 pad 1: (no net) -> RL1_5
- C3 pad 2: (no net) -> T1_4
- C32 pad 1: (no net) -> C32_1
- C32 pad 2: (no net) -> C32_2
- C34 pad 1: (no net) -> C34_1
- C37 pad 1: (no net) -> IC13_2
- C38 pad 1: (no net) -> IC8_13
- C38 pad 2: (no net) -> IC8_14
- C39 pad 1: (no net) -> C39_1
- C39 pad 2: (no net) -> R57_2
- C4 pad 1: (no net) -> RL1_5
- C4 pad 2: (no net) -> T1_4
- C40 pad 2: (no net) -> C40_2
- C41 pad 1: (no net) -> IC8_9
- C41 pad 2: (no net) -> IC8_11
- C42 pad 1: (no net) -> L3_1
- C42 pad 2: (no net) -> IC8_10
- C43 pad 2: (no net) -> IC8_7
- C5 pad 2: (no net) -> IC9_2
- C51 pad 1: (no net) -> C51_1
- C52 pad 1: (no net) -> IC15_3
- C54 pad 1: (no net) -> C52_2
- C54 pad 2: (no net) -> D7_1
- C56 pad 1: (no net) -> C52_2
- C56 pad 2: (no net) -> IC15_7
- C58 pad 1: (no net) -> IC18_2
- C59 pad 1: (no net) -> D7_3
- C59 pad 2: (no net) -> R75_1
- C60 pad 1: (no net) -> D7_3
- C60 pad 2: (no net) -> R75_1
- C62 pad 1: (no net) -> RL1_5
- C62 pad 2: (no net) -> R12_2
- C71 pad 1: (no net) -> DA1_2
- C72 pad 1: (no net) -> C72_1
- C73 pad 2: (no net) -> IC17_2
- CNP1 pad 1: (no net) -> TEL_Line
- CNP1 pad 2: (no net) -> TEL_GND
- CNP1 pad 3: (no net) -> TEL_GND
- CNP1 pad 4: (no net) -> TEL_GND
- CNP2 pad 1: (no net) -> L3_2
- CNP2 pad 3: (no net) -> CNP2_3
- CNP2 pad 4: (no net) -> CNP3_1
- CNP2 pad 5: (no net) -> L5_2
- CNP3 pad 1: (no net) -> CNP3_1
- CNP3 pad 5: (no net) -> CNP3_5
- CNP3 pad 6: (no net) -> CNP5_2
- CNP3 pad MP: (no net) -> CNP3_MP1
- CNP5 pad 1: (no net) -> CNP5_1
- CNP5 pad 2: (no net) -> CNP5_2
- CNP5 pad MP: (no net) -> CNP5_MP1
- D1 pad 1: (no net) -> D1_1
- D1 pad 2: (no net) -> D1_2
- D1 pad 3: (no net) -> RL1_5
- D1 pad 4: L1_2 -> L1_1
- D10 pad 2: (no net) -> R56_2
- D2 pad 1: (no net) -> D1_1
- D2 pad 2: (no net) -> D2_2
- D3 pad 1: (no net) -> IC16_1
- D4 pad 1: (no net) -> D4_1
- D4 pad 2: (no net) -> MN195_S3
- D5 pad 1: (no net) -> IC18_2
- D5 pad 2: (no net) -> IC18_2
- D6 pad 1: (no net) -> C52_2
- D6 pad 2: (no net) -> D6_2
- D6 pad 3: (no net) -> D7_1
- D7 pad 1: (no net) -> D7_1
- D7 pad 2: (no net) -> C52_2
- D7 pad 3: (no net) -> D7_3
- D7 pad 4: L1_2 -> L1_1
- D8 pad 1: (no net) -> IC13_4
- D9 pad 4: L1_2 -> L1_1
- DA1 pad 2: (no net) -> DA1_2
- IC10 pad 1: IC10_1 -> GND
- IC10 pad 3: IC10_3 -> R16_1
- IC13 pad 1: (no net) -> IC13_1
- IC13 pad 2: (no net) -> IC13_2
- IC13 pad 4: (no net) -> IC13_4
- IC14 pad 1: (no net) -> IC14_1
- IC14 pad 2: (no net) -> IC16_4
- IC14 pad 4: (no net) -> IC14_4
- IC15 pad 1: (no net) -> D7_1
- IC15 pad 2: (no net) -> IC15_2
- IC15 pad 3: (no net) -> IC15_3
- IC15 pad 4: (no net) -> IC15_4
- IC15 pad 6: (no net) -> IC15_6
- IC15 pad 7: (no net) -> IC15_7
- IC15 pad 8: (no net) -> IC15_8
- IC16 pad 1: (no net) -> IC16_1
- IC16 pad 2: (no net) -> IC13_4
- IC16 pad 4: (no net) -> IC16_4
- IC17 pad 1: (no net) -> IC17_1
- IC17 pad 2: (no net) -> IC17_2
- IC17 pad 3: (no net) -> PNET4
- IC18 pad 2: (no net) -> IC18_2
- IC18 pad 4: (no net) -> IC18_4
- IC18 pad 5: (no net) -> IC18_5
- IC2 pad 1: (no net) -> IC2_1
- IC2 pad 2: (no net) -> R73_2
- IC2 pad 4: (no net) -> D4_1
- IC3 pad 1: (no net) -> IC3_1
- IC3 pad 12: (no net) -> C72_1
- IC3 pad 8: (no net) -> C32_1
- IC4 pad 1: (no net) -> IC4_1
- IC4 pad 4: (no net) -> IC6_2
- IC6 pad 2: (no net) -> IC6_2
- IC6 pad 4: (no net) -> RL1_4
- IC7 pad 1: (no net) -> IC7_1
- IC7 pad 2: (no net) -> D4_1
- IC7 pad 4: (no net) -> IC7_4
- IC8 pad 10: (no net) -> IC8_10
- IC8 pad 11: (no net) -> IC8_11
- IC8 pad 12: (no net) -> IC8_12
- IC8 pad 13: (no net) -> IC8_13
- IC8 pad 14: (no net) -> IC8_14
- IC8 pad 15: (no net) -> IC8_15
- IC8 pad 16: (no net) -> IC8_16
- IC8 pad 2: (no net) -> IC8_2
- IC8 pad 3: (no net) -> IC8_3
- IC8 pad 4: (no net) -> IC8_4
- IC8 pad 5: (no net) -> IC8_5
- IC8 pad 6: (no net) -> IC8_6
- IC8 pad 7: (no net) -> IC8_7
- IC8 pad 9: (no net) -> IC8_9
- IC9 pad 1: (no net) -> IC9_1
- IC9 pad 2: (no net) -> IC9_2
- L1 pad 1: (no net) -> TEL_Line
- L1 pad 2: L1_2 -> L1_1
- L2 pad 1: (no net) -> TEL_GND
- L2 pad 2: L1_1 -> L1_2
- L3 pad 1: (no net) -> L3_1
- L3 pad 2: (no net) -> L3_2
- L4 pad 1: (no net) -> L4_1
- L4 pad 2: (no net) -> CNP2_3
- L5 pad 2: (no net) -> L5_2
- NF1 pad 1: (no net) -> NF1_1
- NF2 pad 1: (no net) -> NF2_1
- NF3 pad 1: (no net) -> OSC1_2
- OSC1 pad 1: (no net) -> OSC1_1
- OSC1 pad 2: (no net) -> OSC1_2
- OSC1 pad 3: (no net) -> OSC1_3
- PC2 pad 1: (no net) -> PC2_1
- Q1 pad 1: (no net) -> D2_2
- Q1 pad 2: (no net) -> Q2_1
- Q1 pad 3: (no net) -> D1_1
- Q2 pad 1: (no net) -> Q2_1
- Q2 pad 2: (no net) -> D1_1
- Q2 pad 3: (no net) -> Q2_1
- Q3 pad 1: (no net) -> MN195_S11
- Q3 pad 3: (no net) -> Q3_3
- Q4 pad 1: (no net) -> Q3_3
- Q7 pad 1: (no net) -> Q7_1
- Q7 pad 3: (no net) -> IC14_1
- Q9 pad 1: (no net) -> Q9_1
- Q9 pad 3: (no net) -> R55_1
- R1 pad 1: (no net) -> Q3_3
- R100 pad 2: (no net) -> IC17_2
- R105 pad 1: (no net) -> 29F_A12
- R112 pad 2: (no net) -> MN195_UC0
- R12 pad 1: (no net) -> L1_2
- R12 pad 2: (no net) -> R12_2
- R13 pad 1: (no net) -> IC8_12
- R13 pad 2: (no net) -> IC8_16
- R133 pad 2: (no net) -> MN195_S11
- R14 pad 1: (no net) -> IC7_4
- R14 pad 2: (no net) -> IC9_2
- R15 pad 1: (no net) -> IC15_6
- R15 pad 2: (no net) -> IC15_7
- R16 pad 1: (no net) -> R16_1
- R17 pad 1: (no net) -> IC10_6
- R18 pad 2: (no net) -> RL1_3
- R2 pad 2: (no net) -> IC16_1
- R20 pad 1: (no net) -> D1_1
- R20 pad 2: (no net) -> D2_2
- R24 pad 1: (no net) -> IC13_2
- R25 pad 2: (no net) -> IC13_2
- R26 pad 2: (no net) -> NF2_1
- R33 pad 2: (no net) -> NF2_1
- R34 pad 2: (no net) -> NF2_1
- R35 pad 1: (no net) -> NF1_1
- R4 pad 2: (no net) -> IC8_15
- R42 pad 1: (no net) -> IC15_2
- R44 pad 2: (no net) -> OSC1_1
- R46 pad 1: (no net) -> IC14_4
- R46 pad 2: (no net) -> RL1_2
- R49 pad 2: (no net) -> IC18_2
- R5 pad 1: (no net) -> R6_2
- R50 pad 2: (no net) -> R57_2
- R53 pad 1: (no net) -> R57_2
- R53 pad 2: (no net) -> R54_2
- R54 pad 2: (no net) -> R54_2
- R55 pad 1: (no net) -> R55_1
- R55 pad 2: (no net) -> IC8_3
- R56 pad 1: (no net) -> IC8_3
- R57 pad 1: (no net) -> IC8_3
- R57 pad 2: (no net) -> R57_2
- R58 pad 1: (no net) -> IC8_16
- R59 pad 1: (no net) -> IC8_13
- R59 pad 2: (no net) -> IC8_14
- R6 pad 1: (no net) -> Q9_1
- R6 pad 2: (no net) -> R6_2
- R60 pad 1: (no net) -> IC8_13
- R60 pad 2: (no net) -> C39_1
- R61 pad 2: (no net) -> R61_2
- R62 pad 1: (no net) -> IC8_11
- R62 pad 2: (no net) -> C40_2
- R63 pad 1: (no net) -> IC8_10
- R63 pad 2: (no net) -> IC8_7
- R65 pad 1: (no net) -> L4_1
- R65 pad 2: (no net) -> R65_2
- R68 pad 1: (no net) -> IC8_9
- R68 pad 2: (no net) -> IC8_11
- R68 pad 1: (no net) -> IC15_8
- R68 pad 2: (no net) -> PC2_1
- R7 pad 1: (no net) -> Q2_1
- R7 pad 2: (no net) -> D1_2
- R70 pad 1: (no net) -> C51_1
- R70 pad 2: (no net) -> IC8_16
- R71 pad 1: (no net) -> L3_1
- R71 pad 2: (no net) -> C51_1
- R73 pad 2: (no net) -> R73_2
- R75 pad 1: (no net) -> R75_1
- R75 pad 2: L1_1 -> L1_2
- R76 pad 1: (no net) -> C32_2
- R76 pad 2: (no net) -> Q3_3
- R77 pad 1: (no net) -> IC15_4
- R77 pad 2: (no net) -> IC15_3
- R78 pad 1: (no net) -> IC15_8
- R78 pad 2: (no net) -> CNP3_5
- R8 pad 2: (no net) -> Q3_3
- R81 pad 2: (no net) -> R73_2
- R82 pad 1: (no net) -> C52_2
- R9 pad 1: (no net) -> D1_2
- R9 pad 2: (no net) -> D2_2
- R90 pad 2: (no net) -> IC14_1
- R92 pad 2: (no net) -> Q7_1
- R99 pad 1: (no net) -> DA1_2
- R99 pad 2: (no net) -> C72_1
- RL1 pad 2: (no net) -> RL1_2
- RL1 pad 3: (no net) -> RL1_3
- RL1 pad 4: (no net) -> RL1_4
- RL1 pad 5: (no net) -> RL1_5
- RL1 pad 6: L1_1 -> L1_2
- RL1 pad 8: L1_1 -> L1_2
- SW2 pad 1: (no net) -> SW2_1
- SW2 pad 2: (no net) -> R82_2
- SW2 pad 3: (no net) -> CNP5_1
- SW2 pad MP: (no net) -> SW2_MP4
- T1 pad 1: L1_2 -> L1_1
- T1 pad 4: (no net) -> T1_4
- VA1 pad 1: L1_2 -> L1_1
- VA1 pad 2: L1_1 -> L1_2
Routing:
- net (no net): track 1007.1 -> 0.00 mm, vias 67 -> 0
- net CNP5_1: track 0.00 -> 70.4 mm, vias 0 -> 2
- net IC8_16: track 0.00 -> 59.9 mm, vias 0 -> 4
- net C72_1: track 0.00 -> 48.2 mm, vias 0 -> 1
- net CNP3_5: track 0.00 -> 43.2 mm, vias 0 -> 2
- net IC8_10: track 0.00 -> 38.7 mm, vias 0 -> 3
- net D7_1: track 0.00 -> 38.6 mm, vias 0 -> 3
- net IC15_8: track 0.00 -> 33.1 mm, vias 0 -> 2
- net CNP3_1: track 0.00 -> 29.8 mm, vias 0 -> 1
- net IC8_3: track 0.00 -> 29.1 mm, vias 0 -> 1
- net RL1_5: track 0.00 -> 28.7 mm, vias 0 -> 2
- net D1_1: track 0.00 -> 28.3 mm, vias 0 -> 1
- net IC8_13: track 0.00 -> 22.9 mm, vias 0 -> 2
- net PC2_1: track 0.00 -> 22.4 mm, vias 0 -> 2
- net IC8_15: track 0.00 -> 22.2 mm, vias 0 -> 2
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
Commit message: finished
Parts:
- C12, C45: value C_1812_4532Metric -> 47uF 16v
- C56: renamed from 470nF; value C_0603_1608Metric -> 470nF
- IC15: value SOIC-8_5.3x6.2mm_P1.27mm -> 8206 5877
- OSC1: value Oscillator_SMD_Fordahl_DFAS2-4Pin_7.3x5.1mm -> 41.472
- R61: value R_0402_1005Metric -> 3.6k
- R90: value R_0402_1005Metric -> 470k
- R92: value R_0402_1005Metric -> 47k
Connections:
- IC3 pad 1: IC3_1 -> MN195_PLSD
- R109 pad 2: (no net) -> MN195_A4
Routing:
- net MN195_HDRES#: track 14.8 -> 24.6 mm
- net MN195_MOD1,3: track 11.8 -> 10.9 mm
- net GND: track 239.8 -> 239.1 mm
