File: PCB/Modem/Modem.kicad_sch (KiCad schematic)
At the start: 0 parts

Commit message: Add files via upload
Parts:
- added C31: 230nF, symbol PCM_Elektuur:C
- added C5: 250nF, symbol PCM_Elektuur:C
- added CNP4: ~, symbol Modem:M_Conn
- added IC11: ~, symbol Modem:EN29F040A
- added IC12: ~, symbol Modem:681000ALP
- added IC2, IC7, IC9: EA, symbol 74xGxx:74AHC1G14
- added IC5: ~, symbol Modem:MN195001
- added Q4: CQ, symbol Simulation_SPICE:NPN
- added R14: 560k, symbol PCM_Elektuur:R
- added R27: DNP, symbol PCM_Elektuur:R
- added R52: 1k, symbol PCM_Elektuur:R
- added R73: 120, symbol PCM_Elektuur:R
- added R81: 100k, symbol PCM_Elektuur:R
Connections:
- new net: IC2.4, IC7.2
- new net: IC7.4, R14.1 (+)
- new net: C5.1 (+), IC9.2, R14.2 (-)
- new net: IC2.2, R73.2 (-), R81.2 (-)
- new net: CNP4.11 (FDC_TXD#), IC9.4
- new net: CNP4.2 (VCC_STNDBY), CNP4.25 (VCC_STNDBY)
- new net: CNP4.3 (U1RD), R27.2 (-)
- new net: IC5.113 (DVDD3), IC5.13 (DVDD1), IC5.25 (DVDD4), IC5.77 (DVDD2)
- new net: IC5.42 (MOD0), IC5.45 (MOD3)
- new net: Q4.2 (B), R52.2 (-)
- new net GND: C31.2 (-), C5.2 (-), CNP4.1 (GND), CNP4.13 (GND), CNP4.14 (GND), CNP4.26 (GND), IC2.3 (GND), IC5.10 (SCX2), IC5.112 (DVSS3), IC5.14 (DVSS1), IC5.19 (HALT), IC5.24 (DVSS4), IC5.43 (MOD1), IC5.44 (MOD2), IC5.76 (DVSS2), IC7.3 (GND), IC9.3 (GND), R81.1 (+)
- new net MN195_ADCK#: CNP4.21 (ADCK#), IC5.21 (ADCK#)
- new net MN195_IRQ1#: CNP4.20 (IRQ1#), IC5.67 (IRQ1#)
- new net MN195_S11: CNP4.22 (S11)
- new net MN195_S5#: CNP4.7 (DSR1), IC5.51 (S5)
- new net MN195_S6#: CNP4.10 (FDC_RXD#), IC5.52 (S6)
- new net MN195_S7#: CNP4.9 (FDC_RTS#), IC5.53 (S7)
- new net MN195_S8#: CNP4.6 (DIR1#), IC5.54 (S8)
- new net MN195_U1RD: IC5.63 (U1RD#), R27.1 (+)
- new net MN195_U1SD: CNP4.4 (DCD1), IC5.65 (U1SD#)
- new net MN195_VPCK#: CNP4.18 (VPCK#), IC5.87 (VPCK#)
- new net MN195_VPDA#: CNP4.19 (VPDA#), IC5.88 (VPDA#)
- new net MN195_VSDA#: CNP4.17 (VSDA#), IC5.96 (VSDA#)
- new net MN195_VSEN#: CNP4.16 (VSEN#), IC5.98 (VSEN#)
- new net PNET1: Q4.1 (C)
- new net PNET4: R52.1 (+)
- new net VCC: C31.1 (+), CNP4.12 (VCC), CNP4.15 (VCC), IC2.5 (VCC), IC7.5 (VCC), IC9.5 (VCC)
- no-connect marks 0 -> 40
Other:
- note removed: "Making this a reality can be your contribution!"
- company: (none) -> Recreated by: Ahmad Byagowi
- title: (none) -> PC110 Internal Modem Module

Commit message: Add files via upload
Parts:
- added C32: 1.2uF, symbol PCM_Elektuur:C
- added D4: 5, symbol PCM_Elektuur:D
- added IC3: Line Module, symbol Connector_Generic:Conn_01x18
- added PC2: TLS124, OptoDevice:Sharp_GP2S700HCP, symbol Sensor_Proximity:GP2S700HCP
- added Q3: 123, symbol Simulation_SPICE:NPN
- added R1: 12k, symbol PCM_Elektuur:R
- added R16, R17, R18: 10k, symbol PCM_Elektuur:R
- added R22, R23: DNP, symbol PCM_Elektuur:R
- added R76: 2.4k, symbol PCM_Elektuur:R
- added R8: 22k, symbol PCM_Elektuur:R
- added U10: AT32, symbol 74xx:74LS32
Connections:
- net GND: now also IC3.14 (Pin_14), U10.1, U10.12, U10.13, U10.4, U10.7 (GND), U10.9
- net MN195_ADCK#: now also IC5.95 (VSCK#)
- net MN195_S11: now also IC5.57 (S11); no longer CNP4.22 (S11)
- net MN195_U1RD: now also R18.1 (+)
- net PNET1: now also R1.1 (+)
- net PNET4: now also Q3.3 (E), R8.2 (-)
- net VCC: now also PC2.2, U10.14 (VCC)
- net at IC2.4, IC7.2: now also D4.1 (K-)
- net at CNP4.3 (U1RD), R27.2 (-): now also U10.10
- net at CNP4.5 (RI1): now also R22.2 (-), U10.2
- net at CNP4.8 (FDC_CTS#): now also R23.2 (-), U10.5
- net MN195_S3: now reaches IC5.49 (S3)
- net MN195_S9: now reaches IC5.55 (S9)
- net MN195_S9: now also R16.1 (+), R22.1 (+)
- net MN195_S10: now reaches IC5.56 (S10)
- net MN195_S10: now also Q3.2 (B), R17.1 (+), R23.1 (+)
- net Line_Module_11: now reaches IC5.92 (MTA1)
- net at R73.1 (+): now also PC2.1
- net at Q4.2 (B): now also Q3.1 (C), R1.2 (-), R76.2 (-), R8.1 (+); no longer R52.2 (-)
- net at Q4.3 (E): now also CNP4.22 (S11), R52.2 (-)
- net MN195_S5# renamed MN195_S5
- net MN195_S6# renamed MN195_S6
- net MN195_S7# renamed MN195_S7
- net MN195_S8# renamed MN195_S8
- new net: C32.2 (-), R76.1 (+)
- new net: R17.2 (-), U10.6
- new net: R18.2 (-), U10.8
- new net: R16.2 (-), U10.3
- new net Line_Module_10: IC3.10 (Pin_10)
- new net Line_Module_12: IC3.12 (Pin_12)
- new net Line_Module_16: IC3.16 (Pin_16)
- new net Line_Module_17: IC3.17 (Pin_17)
- new net Line_Module_18: IC3.18 (Pin_18)
- new net Line_Module_2: IC3.2 (Pin_2)
- new net Line_Module_3: IC3.3 (Pin_3)
- new net Line_Module_4: IC3.4 (Pin_4)
- new net Line_Module_5: IC3.5 (Pin_5)
- new net Line_Module_6: IC3.6 (Pin_6)
- new net Line_Module_7: IC3.7 (Pin_7)
- new net Line_Module_8: C32.1 (+), IC3.8 (Pin_8)
- new net Line_Module_9: IC3.9 (Pin_9)
- new net MN195_S3#: D4.2 (A+)
- no-connect marks 40 -> 46
Other:
- moved on the sheet: C31, C5, CNP4, IC11, IC12, IC2, IC5, IC7, IC9, Q4, R14, R27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

Commit message: Add files via upload
Parts:
- added C30: 1.5uF, symbol PCM_Elektuur:C
- added R101, R102, R103, R104, R105, R106, R107, R108, R109, R110, R111, R112, R114, R115, R116, R117, R118, R119, R120, R121, R122, R123, R124 (x2), R125, R126, R127, R129, R130, R131, R132: 100, symbol PCM_Elektuur:R
- renumbered U10 to IC10
Connections:
- net GND: now also IC11.9 (VSS), IC12.24 (VSS), C30.2 (-)
- net VCC: now also IC11.25 (VCC), IC12.6 (CS2#), IC12.8 (VCC), C30.1 (+)
- net at IC5.1 (MD7): now also R132.1 (+)
- net at IC5.100 (UC1#): now also R112.1 (+)
- net at IC5.108 (A18): now also R102.1 (+)
- net at IC5.109 (A17): now also R114.1 (+)
- net at IC5.110 (A16): now also R103.1 (+)
- net at IC5.111 (A15): now also R115.1 (+)
- net at IC5.114 (A14): now also R104.1 (+)
- net at IC5.115 (A13): now also R116.2 (-)
- net at IC5.116 (A12): now also R105.2 (-)
- net at IC5.117 (A11): now also R117.2 (-)
- net at IC5.118 (A10): now also R106.2 (-)
- net at IC5.119 (A9): now also R118.2 (-)
- net at IC5.120 (A8): now also R107.2 (-)
- net at IC5.121 (A7): now also R119.2 (-)
- net at IC5.122 (A6): now also R108.2 (-)
- net at IC5.123 (A5): now also R120.2 (-)
- net at IC5.124 (A4): now also R109.2 (-)
- net at IC5.125 (A3): now also R121.2 (-)
- net at IC5.126 (A2): now also R110.2 (-)
- net at IC5.127 (A1): now also R122.2 (-)
- net at IC5.128 (A0): now also R111.2 (-)
- net at IC5.15 (WR#): now also R124.1 (+)
- net at IC5.16 (RD#): now also R123.1 (+)
- net at IC5.2 (MD6): now also R131.1 (+)
- net at IC5.3 (MD5): now also R130.1 (+)
- net at IC5.4 (MD4): now also R129.1 (+)
- net at IC5.5 (MD3): now also R124.1 (+)
- net at IC5.6 (MD2): now also R127.1 (+)
- net at IC5.7 (MD1): now also R126.1 (+)
- net at IC5.8 (MD0): now also R125.1 (+)
- net at IC5.99 (UC0#): now also R101.1 (+)
- net 29F_A11: now reaches IC12.1 (A11)
- net 29F_A11: now also IC11.32 (A11), R117.1 (+)
- net 29F_A16: now reaches IC12.10 (A16)
- net 29F_A16: now also IC11.23 (A16), R103.2 (-)
- net 29F_A14: now reaches IC12.11 (A14)
- net 29F_A14: now also IC11.28 (A14), R104.2 (-)
- net 29F_A12: now reaches IC12.12 (A12)
- net 29F_A12: now also IC11.21 (A12), R105.1 (+)
- net 29F_A7: now reaches IC12.13 (A7)
- net 29F_A7: now also IC11.20 (A7), R119.1 (+)
- net 29F_A6: now reaches IC12.14 (A6)
- net 29F_A6: now also IC11.19 (A6), R108.1 (+)
- net 29F_A5: now reaches IC12.15 (A5)
- net 29F_A5: now also IC11.18 (A5), R120.1 (+)
- net 29F_A4: now reaches IC12.16 (A4)
- net 29F_A4: now also IC11.17 (A4), R109.1 (+)
- net 29F_A3: now reaches IC12.17 (A3)
- net 29F_A3: now also IC11.16 (A3), R121.1 (+)
- net 29F_A2: now reaches IC12.18 (A2)
- net 29F_A2: now also IC11.15 (A2), R110.1 (+)
- net 29F_A1: now reaches IC12.19 (A1)
- net 29F_A1: now also IC11.14 (A1), R122.1 (+)
- net 29F_A9: now reaches IC12.2 (A9)
- net 29F_A9: now also R118.1 (+)
- net 29F_A0: now reaches IC12.20 (A0)
- net 29F_A0: now also IC11.13 (A0), R111.1 (+)
- net 29F_DQ0: now reaches IC12.21 (DQ0)
- net 29F_DQ0: now also IC11.12 (DQ0), R125.2 (-)
- net 29F_DQ1: now reaches IC12.22 (DQ1)
- net 29F_DQ1: now also IC11.11 (DQ1), R126.2 (-)
- net 29F_DQ2: now reaches IC12.23 (DQ2)
- net 29F_DQ2: now also IC11.10 (DQ2), R127.2 (-)
- net 29F_DQ3: now reaches IC12.25 (DQ3)
- net 29F_DQ3: now also IC11.8 (DQ3), R124.2 (-)
- net 29F_DQ4: now reaches IC12.26 (DQ4)
- net 29F_DQ4: now also IC11.7 (DQ4), R129.2 (-)
- net 29F_DQ5: now reaches IC12.27 (DQ5)
- net 29F_DQ5: now also IC11.6 (DQ5), R130.2 (-)
- net 29F_DQ6: now reaches IC12.28 (DQ6)
- net 29F_DQ6: now also IC11.5 (DQ6), R131.2 (-)
- net 29F_DQ7: now reaches IC12.29 (DQ7)
- net 29F_DQ7: now also IC11.4 (DQ7), R132.2 (-)
- net 29F_A8: now reaches IC12.3 (A8)
- net 29F_A8: now also IC11.30 (A8), R107.1 (+)
- net 68_CS1#: now reaches IC12.30 (CS1#)
- net 68_CS1#: now also R112.2 (-)
- net 29F_A10: now reaches IC12.31 (A10)
- net 29F_A10: now also IC11.2 (A10), R106.1 (+)
- net 29F_A13: now reaches IC12.4 (A13)
- net 29F_A13: now also IC11.29 (A13), R116.1 (+)
- net 29F_WE#: now reaches IC12.5 (WE#)
- net 29F_WE#: now also IC11.26 (WE#), R124.2 (-)
- net 29F_A15: now reaches IC12.7 (A15)
- net 29F_A15: now also IC11.22 (A15), R115.2 (-)
- net 29F_OE#: now reaches IC11.1 (OE#)
- net 29F_OE#: now also IC12.32 (OE#), R123.2 (-)
- net 29F_A18: now reaches IC11.24 (A18)
- net 29F_A18: now also R102.2 (-)
- net 29F_A17: now reaches IC11.27 (A17)
- net 29F_A17: now also R114.2 (-)
- net 29F_CE#: now reaches IC11.3 (CE#)
- net 29F_CE#: now also R101.2 (-)
- no-connect marks 46 -> 48
Other:
- moved on the sheet: C31, C32, C5, CNP4, D4, IC10A, IC10B, IC10C, IC10D, IC10E, IC11, IC12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

Commit message: Add files via upload
Parts:
- added C1, C3, C4: 330nF, symbol PCM_Elektuur:C
- added C45: 47uF, symbol PCM_Elektuur:C
- added C59, C60, C62: 280nF, symbol PCM_Elektuur:C
- added C70, C72: 1.8uF, symbol PCM_Elektuur:C
- added C71: 1.3uF, symbol PCM_Elektuur:C
- added C73: 100pF, symbol PCM_Elektuur:C
- added C74: 220nF, symbol PCM_Elektuur:C
- added D1, D7, D9: TO-269AA, Package_SO:TSSOP-4_4.4x5mm_P4mm, symbol Diode_Bridge:MDB6S
- added DA1: M1T, symbol Device:D_Dual_CommonAnode_AKK_Split
- added IC17: EA, symbol 74xGxx:74AHC1G14
- added JCNP1: Tel Line, symbol Connector:4P4C
- added L1, L2: 1.2uH, symbol PCM_Elektuur:L
- added NF4: 4.5nH, symbol PCM_Elektuur:L
- added R10, R11: 38k, symbol PCM_Elektuur:R
- added R100: 470k, symbol PCM_Elektuur:R
- added R75: 2.2k, symbol PCM_Elektuur:R
- added R98, R99: 100, symbol PCM_Elektuur:R
- added T1: Iso Trans, Transformer_SMD:Transformer_ED8_4-Lead_10.5x8mm_P5mm, symbol Transformer:ED8_4
- added VA1: R-nonlin, symbol PCM_Elektuur:R-nonlin
- renumbered R124 to R128
Connections:
- net Line_Module_10 is gone; now on net MN195_TXOUT: IC3.10 (Pin_10)
- net Line_Module_11 is gone; now on net MN195_MTA1: IC5.92 (MTA1)
- net Line_Module_16 is gone; now on net MN195_SHIN: IC3.16 (Pin_16)
- net Line_Module_17 is gone; now on net MN195_AGCOUT: IC3.17 (Pin_17)
- net Line_Module_18 is gone; now on net MN195_AGCIN: IC3.18 (Pin_18)
- net Line_Module_2 is gone; now on net MN195_HVDD: IC3.2 (Pin_2)
- net Line_Module_3 is gone; now on net MN195_RXL: IC3.3 (Pin_3)
- net Line_Module_4 is gone; now on net MN195_S1: IC3.4 (Pin_4)
- net Line_Module_5 is gone; now on net MN195_S4: IC3.5 (Pin_5)
- net Line_Module_6 is gone; now on net MN195_HPOUT: IC3.6 (Pin_6)
- net Line_Module_7 is gone; now on net AGND: IC3.7 (Pin_7)
- net Line_Module_9 is gone; now on net MN195_TXLPIN: IC3.9 (Pin_9)
- net PNET4 is gone; now on net AGND: Q3.3 (E), R52.1 (+), R8.2 (-)
- net 29F_A9: now also IC11.31 (A9)
- net GND: now also NF4.2 (-), T1.2
- net Line_Module_12: now also C72.1 (+), R99.1 (+)
- net VCC: now also IC3.13 (Pin_13), R98.2 (-)
- net MN195_PLSD: now reaches IC5.23 (PLSD)
- net MN195_PLSD: now also IC3.1 (Pin_1)
- net MN195_SHIN: now reaches IC5.26 (SHIN)
- net MN195_AGCOUT: now reaches IC5.27 (AGCOUT)
- net MN195_AGCIN: now reaches IC5.28 (AGCIN)
- net MN195_HPOUT: now reaches IC5.29 (HPOUT)
- net MN195_IREF2: now reaches IC5.31 (IREF2)
- net MN195_RXL: now reaches IC5.32 (RXL)
- net MN195_HVDD: now reaches IC5.33 (HVDD)
- net MN195_TXOUT: now reaches IC5.34 (TXOUT)
- net AGND: now reaches IC5.35 (AVSS)
- net AGND: now also IC5.41 (VREFL), C45.2 (-), C71.2 (-), C72.2 (-), C73.2 (-), C74.2 (-), DA1.3 (K), IC17.3 (GND), NF4.1 (+)
- net MN195_TXLPIN: now reaches IC5.36 (TXLPIN)
- net MN195_TXLPIN: now also R11.1 (+)
- net MN195_IREF1: now reaches IC5.37 (IREF1)
- net MN195_IREF1: now also R10.1 (+), R11.2 (-)
- net MN195_IREF0: now reaches IC5.38 (IREF0)
- net MN195_IREF0: now also R10.2 (-)
- net MN195_VREEH: now reaches IC5.39 (AVDD)
- net MN195_VREEH: now also IC5.40 (VREFH), C45.1 (+)
- net MN195_S1: now reaches IC5.47 (S1)
- net MN195_S4: now reaches IC5.50 (S4)
- net MN195_MTA1: now reaches IC3.11 (Pin_11)
- net Line_Module_15: now reaches IC3.15 (Pin_15)
- net Line_Module_15: now also T1.3
- new net: C1.1 (+), C3.1 (+), C4.1 (+), T1.4
- new net: C1.2 (-), C3.2 (-), C4.2 (-), C62.1 (+)
- new net: JCNP1.1, L1.1 (+)
- new net: D7.4, L1.2 (-)
- new net: C59.2 (-), C60.2 (-), R75.1 (+)
- new net: L2.2 (-), R75.2 (-), VA1.1 (+)
- new net: C73.1 (+), IC17.2, R100.1 (+)
- new net: C74.1 (+), IC17.5 (VCC), R98.1 (+)
- new net: C71.1 (+), DA1.1 (A), R99.2 (-)
- new net: C70.1 (+), DA1.1 (A), DA1.2 (K)
- new net: JCNP1.2, JCNP1.3, JCNP1.4, L2.1 (+)
- new net: C70.2 (-), IC17.4, R100.2 (-)
- new net: D1.4, D9.4, T1.1, VA1.2 (-)
- new net: C59.1 (+), C60.1 (+), D7.3
- no-connect marks 48 -> 39
Other:
- moved on the sheet: C30, C31, C32, C5, CNP4, D4, IC10A, IC10B, IC10C, IC10D, IC10E, IC11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
