File: PCB/RAM-16MB/RAM-Module.kicad_pcb (KiCad board)
At the start: 2 copper layers, 41.5 x 41.6 mm, 21 parts, among them J15 RAM Module

Commit message: Add files via upload
Other:
- copper layers 2 -> 4
Changed lines of the file:
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@@
 	(layers
 		(0 "F.Cu" signal)
+		(4 "In1.Cu" signal)
+		(6 "In2.Cu" signal)
 		(2 "B.Cu" signal)
 		(9 "F.Adhes" user "F.Adhesive")
@@
 	)
 	(setup
+		(stackup
+			(layer "F.SilkS"
+				(type "Top Silk Screen")
+			)
+			(layer "F.Paste"
+				(type "Top Solder Paste")
+			)
+			(layer "F.Mask"
+				(type "Top Solder Mask")
+				(thickness 0.01)
+			)
+			(layer "F.Cu"
+				(type "copper")
+				(thickness 0.035)
+			)
+			(layer "dielectric 1"
+				(type "prepreg")
+				(thickness 0.1)
+				(material "FR4")
+				(epsilon_r 4.5)
+				(loss_tangent 0.02)
+			)
+			(layer "In1.Cu"
+				(type "copper")
+				(thickness 0.035)
+			)
+			(layer "dielectric 2"
+				(type "core")
+				(thickness 1.24)
+				(material "FR4")
+				(epsilon_r 4.5)
+				(loss_tangent 0.02)
+			)
+			(layer "In2.Cu"
+				(type "copper")
+				(thickness 0.035)
+			)
+			(layer "dielectric 3"
+				(type "prepreg")
+				(thickness 0.1)
+				(material "FR4")
+				(epsilon_r 4.5)
+				(loss_tangent 0.02)
+			)
+			(layer "B.Cu"
+				(type "copper")
+				(thickness 0.035)
+			)
+			(layer "B.Mask"
+				(type "Bottom Solder Mask")
+				(thickness 0.01)
+			)
+			(layer "B.Paste"
+				(type "Bottom Solder Paste")
+			)
+			(layer "B.SilkS"
+				(type "Bottom Silk Screen")
+			)
+			(copper_finish "None")
+			(dielectric_constraints no)
+		)
 		(pad_to_mask_clearance 0)
 		(allow_soldermask_bridges_in_footprints no)

Commit message: Add files via upload
Parts:
- added G***: LOGO, PC110:logo, B.Cu at (117.0, 114.5)
- U1, U2, U3, U4, U5, U6, U7, U8: renamed from REF**; value SOJ-28_10.16x18.415mm_P1.27mm -> 51W17800TT6
- moved C4 0.72 mm to (116.1, 84.0)
- moved R2 0.62 mm to (116.1, 86.5)
- moved C9 0.61 mm to (120.5, 84.0)
- moved C5 0.56 mm to (116.1, 81.5)
- moved C2 0.55 mm to (112.3, 84.6)
- moved C1 0.48 mm to (112.2, 113.2)
- moved C10 0.46 mm to (120.5, 81.5)
- moved R1 0.46 mm to (116.0, 112.6)
- moved J15 0.45 mm to (119.2, 99.9)
- moved C8 0.43 mm to (120.4, 86.5)
- moved C7 0.43 mm to (120.3, 112.6)
- moved C3 0.43 mm to (116.0, 115.1)
- moved C6 0.37 mm to (120.4, 115.1)
- renumbered REF** to C1, REF** to C10, REF** to C3, REF** to C4, REF** to C5, REF** to C6, REF** to C7, REF** to C8, REF** to C9, REF** to R1, REF** to R2
Connections:
- net J1_1 renamed CPU_D23
- net J1_19 renamed RAM_LCASU#
- net J1_2 renamed CPU_D22
- net J1_22 renamed CPU_D7
- net J1_23 renamed CPU_D6
- net J1_27 renamed CPU_D3
- net J1_28 renamed CPU_D2
- net J1_29 renamed CPU_D1
- net J1_3 renamed CPU_D21
- net J1_30 renamed CPU_D0
- net J1_4 renamed CPU_D20
- net J1_60 renamed RAM_ID1
- net J1_9 renamed CPU_D16
- C1 pad 1: (no net) -> PNET1
- C1 pad 2: (no net) -> GND
- C10 pad 2: (no net) -> GND
- C2 pad 1: (no net) -> PNET1
- C2 pad 2: (no net) -> GND
- C3 pad 1: (no net) -> PNET1
- C3 pad 2: (no net) -> GND
- C4 pad 1: (no net) -> GND
- C5 pad 1: (no net) -> GND
- C6 pad 1: (no net) -> GND
- C6 pad 2: (no net) -> PNET1
- C7 pad 1: (no net) -> GND
- C7 pad 2: (no net) -> PNET1
- C8 pad 2: (no net) -> GND
- C9 pad 2: (no net) -> GND
- J15 pad 10: J1_10 -> PNET1
- J15 pad 11: J1_11 -> RAM_A3
- J15 pad 12: J1_12 -> RAM_A2
- J15 pad 13: J1_13 -> RAM_A1
- J15 pad 14: J1_14 -> RAM_A0
- J15 pad 15: J1_15 -> RAM_A10
- J15 pad 16: J1_16 -> RAM_A11
- J15 pad 17: J1_17 -> PNET1
- J15 pad 18: J1_18 -> RAM_UCASU#
- J15 pad 20: J1_20 -> RAM_RAS2
- J15 pad 21: J1_21 -> GND
- J15 pad 24: J1_24 -> CPU_D5
- J15 pad 25: J1_25 -> CPU_D4
- J15 pad 26: J1_26 -> PNET1
- J15 pad 31: J1_31 -> RAM_ID0
- J15 pad 32: J1_32 -> CPU_D15
- J15 pad 33: J1_33 -> CPU_D14
- J15 pad 34: J1_34 -> CPU_D13
- J15 pad 35: J1_35 -> CPU_D12
- J15 pad 36: J1_36 -> GND
- J15 pad 37: J1_37 -> CPU_D11
- J15 pad 38: J1_38 -> CPU_D10
- J15 pad 39: J1_39 -> CPU_D9
- J15 pad 40: J1_40 -> CPU_D8
- J15 pad 41: J1_41 -> RAM_WE#
- J15 pad 42: J1_42 -> RAM_RAS3
- J15 pad 43: J1_43 -> RAM_LCASL#
- J15 pad 44: J1_44 -> RAM_UCASL#
- J15 pad 45: J1_45 -> RAM_A9
- J15 pad 46: J1_46 -> RAM_A8
- J15 pad 47: J1_47 -> RAM_A7
- J15 pad 48: J1_48 -> RAM_A6
- J15 pad 49: J1_49 -> RAM_A5
- J15 pad 5: J1_5 -> GND
- J15 pad 50: J1_50 -> RAM_A4
- J15 pad 51: J1_51 -> CPU_D31
- J15 pad 52: J1_52 -> CPU_D30
- J15 pad 53: J1_53 -> CPU_D29
- J15 pad 54: J1_54 -> CPU_D28
- J15 pad 55: J1_55 -> GND
- J15 pad 56: J1_56 -> CPU_D27
- J15 pad 57: J1_57 -> CPU_D26
- J15 pad 58: J1_58 -> CPU_D25
- J15 pad 59: J1_59 -> CPU_D24
- J15 pad 6: J1_6 -> CPU_D19
- J15 pad 7: J1_7 -> CPU_D18
- J15 pad 8: J1_8 -> CPU_D17
- R1 pad 1: (no net) -> RAM_ID0
- R1 pad 2: (no net) -> GND
- R2 pad 1: (no net) -> GND
- U1 pad 1: (no net) -> PNET1
- U1 pad 10: J1_14 -> RAM_A0
- U1 pad 11: J1_13 -> RAM_A1
- U1 pad 12: J1_12 -> RAM_A2
- U1 pad 13: J1_11 -> RAM_A3
- U1 pad 14: J1_10 -> PNET1
- U1 pad 15: (no net) -> GND
- U1 pad 16: (no net) -> RAM_A4
- U1 pad 17: (no net) -> RAM_A5
- U1 pad 18: (no net) -> RAM_A6
- U1 pad 19: (no net) -> RAM_A7
- U1 pad 20: (no net) -> RAM_A8
- U1 pad 21: (no net) -> RAM_A9
- U1 pad 22: (no net) -> GND
- U1 pad 24: (no net) -> CPU_D4
- U1 pad 25: (no net) -> CPU_D5
- U1 pad 28: (no net) -> GND
- U1 pad 6: (no net) -> RAM_WE#
- U1 pad 7: (no net) -> RAM_RAS3
- U1 pad 8: J1_16 -> RAM_A11
- U1 pad 9: J1_15 -> RAM_A10
- U2 pad 1: J1_10 -> PNET1
- U2 pad 10: (no net) -> RAM_A0
- U2 pad 11: (no net) -> RAM_A1
- U2 pad 12: (no net) -> RAM_A2
- U2 pad 13: (no net) -> RAM_A3
- U2 pad 14: (no net) -> PNET1
- U2 pad 15: (no net) -> GND
- U2 pad 16: J1_50 -> RAM_A4
- U2 pad 17: J1_49 -> RAM_A5
- U2 pad 18: J1_48 -> RAM_A6
- U2 pad 19: J1_47 -> RAM_A7
- U2 pad 20: J1_46 -> RAM_A8
- U2 pad 21: J1_45 -> RAM_A9
- U2 pad 22: (no net) -> GND
- U2 pad 23: (no net) -> RAM_LCASL#
- U2 pad 28: (no net) -> GND
- U2 pad 3: (no net) -> CPU_D17
- U2 pad 4: (no net) -> CPU_D18
- U2 pad 5: (no net) -> CPU_D19
- U2 pad 6: J1_41 -> RAM_WE#
- U2 pad 7: (no net) -> RAM_RAS3
- U2 pad 8: (no net) -> RAM_A11
- U2 pad 9: (no net) -> RAM_A10
- U3 pad 1: (no net) -> PNET1
- U3 pad 10: J1_14 -> RAM_A0
- U3 pad 11: J1_13 -> RAM_A1
- U3 pad 12: J1_12 -> RAM_A2
- U3 pad 13: J1_11 -> RAM_A3
- U3 pad 14: J1_10 -> PNET1
- U3 pad 15: (no net) -> GND
- U3 pad 16: (no net) -> RAM_A4
- U3 pad 17: (no net) -> RAM_A5
- U3 pad 18: (no net) -> RAM_A6
- U3 pad 19: (no net) -> RAM_A7
- U3 pad 2: (no net) -> CPU_D8
- U3 pad 20: (no net) -> RAM_A8
- U3 pad 21: (no net) -> RAM_A9
- U3 pad 22: (no net) -> GND
- U3 pad 23: (no net) -> RAM_UCASU#
- U3 pad 24: (no net) -> CPU_D12
- U3 pad 25: (no net) -> CPU_D13
- U3 pad 26: (no net) -> CPU_D14
- U3 pad 27: (no net) -> CPU_D15
- U3 pad 28: (no net) -> GND
- U3 pad 3: (no net) -> CPU_D9
- U3 pad 4: (no net) -> CPU_D10
- U3 pad 5: (no net) -> CPU_D11
- U3 pad 6: (no net) -> RAM_WE#
- U3 pad 7: (no net) -> RAM_RAS3
- U3 pad 8: J1_16 -> RAM_A11
- U3 pad 9: J1_15 -> RAM_A10
- U4 pad 1: J1_10 -> PNET1
- U4 pad 10: (no net) -> RAM_A0
- U4 pad 11: (no net) -> RAM_A1
- U4 pad 12: (no net) -> RAM_A2
- U4 pad 13: (no net) -> RAM_A3
- U4 pad 14: (no net) -> PNET1
- U4 pad 15: (no net) -> GND
- U4 pad 16: J1_50 -> RAM_A4
- U4 pad 17: J1_49 -> RAM_A5
- U4 pad 18: J1_48 -> RAM_A6
- U4 pad 19: J1_47 -> RAM_A7
- U4 pad 2: (no net) -> CPU_D24
- U4 pad 20: J1_46 -> RAM_A8
- U4 pad 21: J1_45 -> RAM_A9
- U4 pad 22: (no net) -> GND
- U4 pad 23: (no net) -> RAM_UCASL#
- U4 pad 24: (no net) -> CPU_D28
- U4 pad 25: (no net) -> CPU_D29
- U4 pad 26: (no net) -> CPU_D30
- U4 pad 27: (no net) -> CPU_D31
- U4 pad 28: (no net) -> GND
- U4 pad 3: (no net) -> CPU_D25
- U4 pad 4: (no net) -> CPU_D26
- U4 pad 5: (no net) -> CPU_D27
- U4 pad 6: J1_41 -> RAM_WE#
- U4 pad 7: (no net) -> RAM_RAS3
- U4 pad 8: (no net) -> RAM_A11
- U4 pad 9: (no net) -> RAM_A10
- U5 pad 1: (no net) -> PNET1
- U5 pad 10: J1_14 -> RAM_A0
- U5 pad 11: J1_13 -> RAM_A1
- U5 pad 12: J1_12 -> RAM_A2
- U5 pad 13: J1_11 -> RAM_A3
- U5 pad 14: J1_10 -> PNET1
- U5 pad 15: J1_10 -> GND
- U5 pad 16: (no net) -> RAM_A4
- U5 pad 17: (no net) -> RAM_A5
- U5 pad 18: (no net) -> RAM_A6
- U5 pad 19: (no net) -> RAM_A7
- U5 pad 20: (no net) -> RAM_A8
- U5 pad 21: (no net) -> RAM_A9
- U5 pad 22: (no net) -> GND
- U5 pad 24: J1_25 -> CPU_D4
- U5 pad 25: J1_24 -> CPU_D5
- U5 pad 28: (no net) -> GND
- U5 pad 6: (no net) -> RAM_WE#
- U5 pad 7: J1_18 -> RAM_RAS2
- U5 pad 8: J1_16 -> RAM_A11
- U5 pad 9: J1_15 -> RAM_A10
- U6 pad 1: J1_10 -> PNET1
- U6 pad 10: (no net) -> RAM_A0
- U6 pad 11: (no net) -> RAM_A1
- U6 pad 12: (no net) -> RAM_A2
- U6 pad 13: (no net) -> RAM_A3
- U6 pad 14: (no net) -> PNET1
- U6 pad 15: (no net) -> GND
- U6 pad 16: J1_50 -> RAM_A4
- U6 pad 17: J1_49 -> RAM_A5
- U6 pad 18: J1_48 -> RAM_A6
- U6 pad 19: J1_47 -> RAM_A7
- U6 pad 20: J1_46 -> RAM_A8
- U6 pad 21: J1_45 -> RAM_A9
- U6 pad 22: (no net) -> GND
- U6 pad 23: (no net) -> RAM_LCASL#
- U6 pad 28: J1_10 -> GND
- U6 pad 3: J1_8 -> CPU_D17
- U6 pad 4: J1_7 -> CPU_D18
- U6 pad 5: J1_6 -> CPU_D19
- U6 pad 6: J1_41 -> RAM_WE#
- U6 pad 7: (no net) -> RAM_RAS2
- U6 pad 8: (no net) -> RAM_A11
- U6 pad 9: (no net) -> RAM_A10
- U7 pad 1: (no net) -> PNET1
- U7 pad 10: J1_14 -> RAM_A0
- U7 pad 11: J1_13 -> RAM_A1
- U7 pad 12: J1_12 -> RAM_A2
- U7 pad 13: J1_11 -> RAM_A3
- U7 pad 14: J1_10 -> PNET1
- U7 pad 15: (no net) -> GND
- U7 pad 16: (no net) -> RAM_A4
- U7 pad 17: (no net) -> RAM_A5
- U7 pad 18: (no net) -> RAM_A6
- U7 pad 19: (no net) -> RAM_A7
- U7 pad 2: J1_40 -> CPU_D8
- U7 pad 20: (no net) -> RAM_A8
- U7 pad 21: (no net) -> RAM_A9
- U7 pad 22: (no net) -> GND
- U7 pad 23: (no net) -> RAM_UCASU#
- U7 pad 24: (no net) -> CPU_D12
- U7 pad 25: (no net) -> CPU_D13
- U7 pad 26: (no net) -> CPU_D14
- U7 pad 27: J1_32 -> CPU_D15
- U7 pad 28: (no net) -> GND
- U7 pad 3: (no net) -> CPU_D9
- U7 pad 4: (no net) -> CPU_D10
- U7 pad 5: (no net) -> CPU_D11
- U7 pad 6: (no net) -> RAM_WE#
- U7 pad 7: J1_18 -> RAM_RAS2
- U7 pad 8: J1_16 -> RAM_A11
- U7 pad 9: J1_15 -> RAM_A10
- U8 pad 1: J1_10 -> PNET1
- U8 pad 10: (no net) -> RAM_A0
- U8 pad 11: (no net) -> RAM_A1
- U8 pad 12: (no net) -> RAM_A2
- U8 pad 13: (no net) -> RAM_A3
- U8 pad 14: (no net) -> PNET1
- U8 pad 15: (no net) -> GND
- U8 pad 16: J1_50 -> RAM_A4
- U8 pad 17: J1_49 -> RAM_A5
- U8 pad 18: J1_48 -> RAM_A6
- U8 pad 19: J1_47 -> RAM_A7
- U8 pad 2: (no net) -> CPU_D24
- U8 pad 20: J1_46 -> RAM_A8
- U8 pad 21: J1_45 -> RAM_A9
- U8 pad 22: (no net) -> GND
- U8 pad 23: (no net) -> RAM_UCASL#
- U8 pad 24: (no net) -> CPU_D28
- U8 pad 25: (no net) -> CPU_D29
- U8 pad 26: (no net) -> CPU_D30
- U8 pad 27: (no net) -> CPU_D31
- U8 pad 28: J1_10 -> GND
- U8 pad 3: (no net) -> CPU_D25
- U8 pad 4: (no net) -> CPU_D26
- U8 pad 5: (no net) -> CPU_D27
- U8 pad 6: J1_41 -> RAM_WE#
- U8 pad 7: (no net) -> RAM_RAS2
- U8 pad 8: (no net) -> RAM_A11
- U8 pad 9: (no net) -> RAM_A10
Routing:
- net (no net): track 728.7 -> 0.00 mm, vias 55 -> 0
- net GND: track 0.00 -> 226.3 mm, vias 0 -> 24
- net J1_10: track 177.6 -> 0.00 mm, vias 15 -> 0
- net PNET1: track 0.00 -> 140.5 mm, vias 0 -> 15
- net RAM_A4: track 0.00 -> 123.8 mm, vias 0 -> 3
- net RAM_A5: track 0.00 -> 121.1 mm, vias 0 -> 3
- net RAM_A6: track 0.00 -> 118.6 mm, vias 0 -> 3
- net RAM_A8: track 0.00 -> 117.0 mm, vias 0 -> 3
- net RAM_A7: track 0.00 -> 114.9 mm, vias 0 -> 3
- net RAM_WE#: track 0.00 -> 108.1 mm, vias 0 -> 4
- net RAM_A9: track 0.00 -> 103.6 mm, vias 0 -> 4
- net RAM_A11: track 0.00 -> 102.0 mm, vias 0 -> 3
- net RAM_A10: track 0.00 -> 100.1 mm, vias 0 -> 2
- net RAM_A0: track 0.00 -> 96.1 mm, vias 0 -> 3
- net RAM_A2: track 0.00 -> 94.6 mm, vias 0 -> 3
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- added copper zone on B.Cu, net GND
- added copper zone on F.Cu, net GND
- added copper zone on In2.Cu, net GND
- added copper zone on B.Cu, net PNET1
- added copper zone on F.Cu, net PNET1
- added copper zone on In1.Cu, net PNET1
- added copper zone on F.Cu, net RAM_ID1
Other:
- outline, holes or cut-outs redrawn
