File: PCB/RAM-16MB/RAM-Module.kicad_pcb (KiCad board)
At the start: 4 copper layers, 41.5 x 41.6 mm, 22 parts, among them J15 RAM Module, U1 51W17800TT6, U2 51W17800TT6, U3 51W17800TT6, U4 51W17800TT6, U5 51W17800TT6, U6 51W17800TT6, U7 51W17800TT6, U8 51W17800TT6

Commit message: Add files via upload
Parts:
- C1, C10, C2, C3, C4, C5, C6, C7, C8, C9: value C_0805_2012Metric -> 100nF
- R1, R2: value R_0805_2012Metric -> 0
Routing:
- net PNET1: track 140.5 -> 145.3 mm
Changed lines of the file:
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@@
 			)
 		)
-		(property "Value" "C_0805_2012Metric"
+		(property "Value" "100nF"
 			(at 0 1.68 0)
 			(layer "F.Fab")
@@
 			)
 		)
-		(property "Value" "R_0805_2012Metric"
+		(property "Value" "0"
 			(at 0 1.65 0)
 			(layer "F.Fab")
@@
 			)
 		)
-		(property "Value" "C_0805_2012Metric"
+		(property "Value" "100nF"
 			(at 0 1.68 0)
 			(layer "F.Fab")
@@
 			)
 		)
-		(property "Value" "C_0805_2012Metric"
+		(property "Value" "100nF"
 			(at 0 1.68 90)
 			(layer "F.Fab")
@@
 			)
 		)
-		(property "Value" "C_0805_2012Metric"
+		(property "Value" "100nF"
 			(at 0 1.68 0)
 			(layer "F.Fab")
@@
 			)
 		)
-		(property "Value" "C_0805_2012Metric"
+		(property "Value" "100nF"
 			(at 0 1.68 90)
 			(layer "F.Fab")
@@
 			)
 		)
-		(property "Value" "C_0805_2012Metric"
+		(property "Value" "100nF"
 			(at 0 1.68 0)
 			(layer "F.Fab")
@@
 			)
 		)
-		(property "Value" "R_0805_2012Metric"
+		(property "Value" "0"
 			(at 0 1.65 0)
 			(layer "F.Fab")
@@
 			)
 		)
-		(property "Value" "C_0805_2012Metric"
+		(property "Value" "100nF"
 			(at 0 1.68 0)
 			(layer "F.Fab")
@@
 			)
 		)
-		(property "Value" "C_0805_2012Metric"
+		(property "Value" "100nF"
 			(at 0 1.68 0)
 			(layer "F.Fab")
@@
 			)
 		)
-		(property "Value" "C_0805_2012Metric"
+		(property "Value" "100nF"
 			(at 0 1.68 0)
 			(layer "F.Fab")
@@
 			)
 		)
-		(property "Value" "C_0805_2012Metric"
+		(property "Value" "100nF"
 			(at 0 1.68 0)
 			(layer "F.Fab")
@@
 	)
 	(segment
-		(start 129.36 97.61)
-		(end 129.56 97.61)
-		(width 0.2)
-		(layer "F.Cu")
-		(net 22)
-	)
-	(segment
 		(start 135.345 79.75)
 		(end 135.35 79.745)
@@
 	)
 	(segment
-		(start 143.31 98.39)
-		(end 143.38 98.46)
-		(width 0.2)
-		(layer "F.Cu")
-		(net 22)
-	)
-	(segment
 		(start 145.75 115.41)
 		(end 145.91 115.25)
@@
 	)
 	(segment
-		(start 135.76 97.67)
-		(end 135.8 97.63)
-		(width 0.2)
-		(layer "F.Cu")
-		(net 22)
-	)
-	(segment
-		(start 129.35 97.6)
-		(end 129.36 97.61)
+		(start 142.16 98.46)
+		(end 143.31 97.31)
 		(width 0.2)
 		(layer "F.Cu")
@@
 	)
 	(segment
+		(start 145.43 96.36)
+		(end 145 96.36)
+		(width 0.2)
+		(layer "F.Cu")
+		(net 22)
+	)
+	(segment
 		(start 145.74 96.05)
 		(end 145.84 96.05)
@@
 	)
 	(segment
-		(start 140.94 96.36)
-		(end 143.31 96.36)
-		(width 0.5)
+		(start 140.87 98.46)
+		(end 142.16 98.46)
+		(width 0.2)
 		(layer "F.Cu")
 		(net 22)
@@
 	)
 	(segment
-		(start 129.97 97.61)
-		(end 129.98 97.6)
+		(start 145 96.36)
+		(end 143.31 96.36)
 		(width 0.2)
 		(layer "F.Cu")
@@
 	)
 	(segment
-		(start 134.25 97.41)
-		(end 135.5 97.41)
+		(start 143.39 115.75)
+		(end 143.73 115.41)
 		(width 0.2)
 		(layer "F.Cu")
@@
 	)
 	(segment
-		(start 132.63 97.61)
-		(end 129.56 97.61)
+		(start 144.92 117.77)
+		(end 145.91 116.78)
 		(width 0.2)
 		(layer "F.Cu")
@@
 	)
 	(segment
-		(start 143.39 115.75)
-		(end 143.73 115.41)
+		(start 140.87 98.46)
+		(end 140.25 98.46)
 		(width 0.2)
 		(layer "F.Cu")
@@
 	)
 	(segment
-		(start 144.92 117.77)
-		(end 145.91 116.78)
+		(start 145.89 80.03)
+		(end 146.175 79.745)
 		(width 0.2)
 		(layer "F.Cu")
@@
 	)
 	(segment
-		(start 145.89 80.03)
-		(end 146.175 79.745)
+		(start 139.2 97.41)
+		(end 134.25 97.41)
 		(width 0.2)
 		(layer "F.Cu")
@@
 	)
 	(segment
-		(start 135.8 97.63)
-		(end 139.26 97.63)
-		(width 0.2)
+		(start 121.33 112.61)
+		(end 121.29 112.57)
+		(width 0.5)
 		(layer "F.Cu")
 		(net 22)
 	)
 	(segment
-		(start 133.67 96.57)
-		(end 132.63 97.61)
+		(start 128.23 99.61)
+		(end 127.46 99.61)
 		(width 0.2)
 		(layer "F.Cu")
@@
 	)
 	(segment
-		(start 121.33 112.61)
-		(end 121.29 112.57)
-		(width 0.5)
+		(start 143.31 97.31)
+		(end 143.31 96.36)
+		(width 0.2)
 		(layer "F.Cu")
 		(net 22)
 	)
 	(segment
-		(start 129.56 97.61)
-		(end 129.97 97.61)
+		(start 145.79 98.15)
+		(end 145 97.36)
 		(width 0.2)
 		(layer "F.Cu")
@@
 	)
 	(segment
+		(start 131.75 98.49)
+		(end 129.35 98.49)
+		(width 0.2)
+		(layer "F.Cu")
+		(net 22)
+	)
+	(segment
 		(start 121.33 115.12)
 		(end 121.33 117.77)
@@
 	)
 	(segment
-		(start 133.67 96.54)
-		(end 133.67 96.57)
-		(width 0.2)
-		(layer "F.Cu")
-		(net 22)
-	)
-	(segment
-		(start 133.67 96.83)
-		(end 134.25 97.41)
+		(start 145.79 98.38)
+		(end 145.87 98.46)
 		(width 0.2)
 		(layer "F.Cu")
@@
 	)
 	(segment
-		(start 145.79 98.38)
-		(end 145.87 98.46)
+		(start 129.35 98.49)
+		(end 128.23 99.61)
 		(width 0.2)
 		(layer "F.Cu")
@@
 	)
 	(segment
+		(start 133.67 96.83)
+		(end 133.67 96.54)
+		(width 0.2)
+		(layer "F.Cu")
+		(net 22)
+	)
+	(segment
 		(start 119.745 100.495)
 		(end 119.53 100.28)
@@
 	)
 	(segment
+		(start 143.31 96.36)
+		(end 140.94 96.36)
+		(width 0.2)
+		(layer "F.Cu")
+		(net 22)
+	)
+	(segment
 		(start 121.33 117.77)
 		(end 144.92 117.77)
@@
 	)
 	(segment
-		(start 135.39 98.7)
-		(end 135.4 98.69)
+		(start 133.67 96.57)
+		(end 131.75 98.49)
 		(width 0.2)
 		(layer "F.Cu")
@@
 	)
 	(segment
-		(start 146.06 97.88)
-		(end 145.79 98.15)
+		(start 135.39 98.7)
+		(end 135.4 98.69)
 		(width 0.2)
 		(layer "F.Cu")
@@
 	)
 	(segment
-		(start 143.31 96.36)
-		(end 143.31 98.39)
+		(start 146.06 97.88)
+		(end 145.79 98.15)
 		(width 0.2)
 		(layer "F.Cu")
@@
 	)
 	(segment
-		(start 135.5 97.41)
-		(end 135.76 97.67)
-		(width 0.2)
-		(layer "F.Cu")
-		(net 22)
-	)
-	(segment
-		(start 129.35 98.49)
-		(end 129.35 97.6)
+		(start 134.25 97.41)
+		(end 133.67 96.83)
 		(width 0.2)
 		(layer "F.Cu")
@@
 	)
 	(segment
-		(start 127.46 99.61)
-		(end 128.23 99.61)
+		(start 145 97.36)
+		(end 145 96.36)
 		(width 0.2)
 		(layer "F.Cu")
@@
 	)
 	(segment
-		(start 133.67 96.54)
-		(end 133.67 96.83)
+		(start 140.25 98.46)
+		(end 139.2 97.41)
 		(width 0.2)
 		(layer "F.Cu")
@@
 	)
 	(segment
-		(start 143.31 96.36)
-		(end 145.43 96.36)
-		(width 0.5)
-		(layer "F.Cu")
-		(net 22)
-	)
-	(segment
 		(start 141.11 115.57)
 		(end 141.29 115.75)
@@
 	)
 	(segment
-		(start 148.145 115.25)
-		(end 148.15 115.255)
+		(start 133.67 96.54)
+		(end 133.67 96.57)
 		(width 0.2)
 		(layer "F.Cu")
@@
 	)
 	(segment
-		(start 128.23 99.61)
-		(end 129.35 98.49)
+		(start 148.145 115.25)
+		(end 148.15 115.255)
 		(width 0.2)
 		(layer "F.Cu")
