File: PCB/RAM-16MB/RAM-Module.kicad_pcb (KiCad board)
At the start: 4 copper layers, 41.5 x 41.6 mm, 22 parts, among them J15 RAM Module, U1 51W17800TT6, U2 51W17800TT6, U3 51W17800TT6, U4 51W17800TT6, U5 51W17800TT6, U6 51W17800TT6, U7 51W17800TT6, U8 51W17800TT6

Commit message: Add files via upload
Other:
- board text added: "Recreated by: Ahmad Byagowi"
Changed lines of the file:
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@@
 		(layer "Edge.Cuts")
+	)
+	(gr_text "Recreated by:\nAhmad Byagowi"
+		(at 122.78 118.82 0)
+		(layer "B.Cu" knockout)
+		(effects
+			(font
+				(size 0.8 0.8)
+				(thickness 0.175)
+				(bold yes)
+			)
+			(justify left bottom mirror)
+		)
 	)
 	(segment

Commit message: Add files via upload
Parts:
- moved G*** 2.22 mm to (116.0, 112.6)

Commit message: Add files via upload
Parts:
- J15: footprint Library:RAM Module -> RAM:RAM Module
Connections:
- C10 pad 1: RAM_ID1 -> PNET1
- C4 pad 2: RAM_ID1 -> PNET1
- C5 pad 2: RAM_ID1 -> PNET1
- C8 pad 1: RAM_ID1 -> PNET1
- C9 pad 1: RAM_ID1 -> PNET1
- J15 pad 1: CPU_D23 -> CPU_D0
- J15 pad 10: PNET1 -> GND
- J15 pad 11: RAM_A3 -> RAM_RAS2
- J15 pad 12: RAM_A2 -> RAM_LCASU#
- J15 pad 13: RAM_A1 -> RAM_UCASU#
- J15 pad 14: RAM_A0 -> PNET1
- J15 pad 15: RAM_A10 -> RAM_A11
- J15 pad 16: RAM_A11 -> RAM_A10
- J15 pad 17: PNET1 -> RAM_A0
- J15 pad 18: RAM_UCASU# -> RAM_A1
- J15 pad 19: RAM_LCASU# -> RAM_A2
- J15 pad 2: CPU_D22 -> CPU_D1
- J15 pad 20: RAM_RAS2 -> RAM_A3
- J15 pad 21: GND -> PNET1
- J15 pad 22: CPU_D7 -> CPU_D16
- J15 pad 23: CPU_D6 -> CPU_D17
- J15 pad 24: CPU_D5 -> CPU_D18
- J15 pad 25: CPU_D4 -> CPU_D19
- J15 pad 26: PNET1 -> GND
- J15 pad 27: CPU_D3 -> CPU_D20
- J15 pad 28: CPU_D2 -> CPU_D21
- J15 pad 29: CPU_D1 -> CPU_D22
- J15 pad 3: CPU_D21 -> CPU_D2
- J15 pad 30: CPU_D0 -> CPU_D23
- J15 pad 31: RAM_ID0 -> RAM_ID1
- J15 pad 32: CPU_D15 -> CPU_D24
- J15 pad 33: CPU_D14 -> CPU_D25
- J15 pad 34: CPU_D13 -> CPU_D26
- J15 pad 35: CPU_D12 -> CPU_D27
- J15 pad 37: CPU_D11 -> CPU_D28
- J15 pad 38: CPU_D10 -> CPU_D29
- J15 pad 39: CPU_D9 -> CPU_D30
- J15 pad 4: CPU_D20 -> CPU_D3
- J15 pad 40: CPU_D8 -> CPU_D31
- J15 pad 41: RAM_WE# -> RAM_A4
- J15 pad 42: RAM_RAS3 -> RAM_A5
- J15 pad 43: RAM_LCASL# -> RAM_A6
- J15 pad 44: RAM_UCASL# -> RAM_A7
- J15 pad 45: RAM_A9 -> RAM_A8
- J15 pad 46: RAM_A8 -> RAM_A9
- J15 pad 47: RAM_A7 -> RAM_UCASL#
- J15 pad 48: RAM_A6 -> RAM_LCASL#
- J15 pad 49: RAM_A5 -> RAM_RAS3
- J15 pad 5: GND -> PNET1
- J15 pad 50: RAM_A4 -> RAM_WE#
- J15 pad 51: CPU_D31 -> CPU_D8
- J15 pad 52: CPU_D30 -> CPU_D9
- J15 pad 53: CPU_D29 -> CPU_D10
- J15 pad 54: CPU_D28 -> CPU_D11
- J15 pad 56: CPU_D27 -> CPU_D12
- J15 pad 57: CPU_D26 -> CPU_D13
- J15 pad 58: CPU_D25 -> CPU_D14
- J15 pad 59: CPU_D24 -> CPU_D15
- J15 pad 6: CPU_D19 -> CPU_D4
- J15 pad 60: RAM_ID1 -> RAM_ID0
- J15 pad 7: CPU_D18 -> CPU_D5
- J15 pad 8: CPU_D17 -> CPU_D6
- J15 pad 9: CPU_D16 -> CPU_D7
Routing:
- net RAM_ID1: track 27.8 -> 6.50 mm, vias 2 -> 0
- net PNET1: track 145.3 -> 164.2 mm, vias 15 -> 17
- removed copper zone on F.Cu, net RAM_ID1
