File: PCB/Keyboard/Membrane/PC110_membrance.kicad_pcb (KiCad board)
At the start: 2 copper layers, 259.5 x 153.2 mm, 0 parts

Commit message: Add files via upload
Other:
- board size 259.5 x 153.2 mm -> 261.9 x 153.2 mm

Commit message: Add files via upload
Routing:
- net (no net): track 3222.2 -> 3244.8 mm, vias 0 -> 32
Other:
- board size 261.9 x 153.2 mm -> 250.4 x 158.7 mm
- board text added: "Esc"
- board text added: "F1"
- board text added: "F2"
- board text added: "F3"
- board text added: "F4"

Commit message: Add files via upload
Parts:
- added G1: LOGO, Keyboard:logo, B.Cu at (147.0, 167.6)
Other:
- board text added: "'"
- board text added: "*"
- board text added: "+"
- board text added: "-"
- board text added: "0"
- board text added: "1"
- board text added: "2"
- board text added: "3"
- board text added: "4"
- board text added: "5"
- board text added: "6"
- board text added: "7"
- board text added: "8"
- board text added: "9"
- board text added: "<"
- board text added: "="
- board text added: ">"
- board text added: "?"
- board text added: "A"
- board text added: "Alt"
- board text added: "B"
- board text added: "Back Space"
- board text added: "C"
- board text added: "Caps Lock"
- board text added: "Ctrl"
- board text added: "D"
- board text added: "Del"
- board text added: "E"
- board text added: "End"
- board text added: "Enter ↵"
- board text added: "F"
- board text added: "F10"
- board text added: "F11"
- board text added: "F12"
- board text added: "F5"
- board text added: "F6"
- board text added: "F7"
- board text added: "F8"
- board text added: "F9"
- board text added: "Fn"
- board text added: "G"
- board text added: "H"
- board text added: "Home"
- board text added: "I"
- board text added: "Ins"
- board text added: "J"
- board text added: "K"
- board text added: "L"
- board text added: "Left Click"
- board text added: "M"
- board text added: "N"
- board text added: "NmLk ScLk"
- board text added: "O"
- board text added: "P"
- board text added: "Pause Break"
- board text added: "PgDn"
- board text added: "PgUp"
- board text added: "PrtScn"
- board text added: "Q"
- board text added: "R"
- board text added: "Right Click"
- board text added: "S"
- board text added: "Shift"
- board text added: "Space"
- board text added: "T"
- board text added: "Tab"
- board text added: "U"
- board text added: "V"
- board text added: "W"
- board text added: "X"
- board text added: "Y"
- board text added: "Z"
- board text added: "_"
- board text added: "{"
- board text added: "|"
- board text added: "}"
- board text added: "←"
- board text added: "↑"
- board text added: "→"
- board text added: "↓"
- board text added: "カタカナ ひらローマ"
- board text added: "前候補 変換 全候"
- board text added: "半/全"
- board text added: "無変換"

Commit message: Add files via upload
Parts:
- moved G1 19.9 mm to (138.1, 149.7)
Other:
- board size 250.4 x 158.7 mm -> 227 x 152.9 mm
