File: PCB/Keyboard/Membrane/PC110_membrance.kicad_sch (KiCad schematic)
At the start: 0 parts

Commit message: Add files via upload
Other:
- note added: "Making this a reality can be your contribution!"
Changed lines of the file:
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@@
 	(generator_version "9.0")
 	(paper "A4")
+	(text "Making this a reality can be your contribution!"
+		(exclude_from_sim no)
+		(at 149.606 98.298 0)
+		(effects
+			(font
+				(size 6.35 6.35)
+			)
+		)
+	)
 	(sheet_instances
 		(path "/"

Commit message: Add files via upload
Parts:
- added J1: Keyboard Conn 1, symbol Connector:Conn_01x08_Pin
- added J2: Keyboard Conn 2, symbol Connector:Conn_01x20_Pin
- added SW1: ESC, symbol Switch:SW_Push_45deg
- added SW10: F9, symbol Switch:SW_Push_45deg
- added SW11: PrtScn, symbol Switch:SW_Push_45deg
- added SW12: NmLk, symbol Switch:SW_Push_45deg
- added SW13: Pause, symbol Switch:SW_Push_45deg
- added SW14: Ins, symbol Switch:SW_Push_45deg
- added SW15: Home, symbol Switch:SW_Push_45deg
- added SW16: PgUp, symbol Switch:SW_Push_45deg
- added SW17: F10, symbol Switch:SW_Push_45deg
- added SW18: F11, symbol Switch:SW_Push_45deg
- added SW19: F12, symbol Switch:SW_Push_45deg
- added SW2: F1, symbol Switch:SW_Push_45deg
- added SW20: Del, symbol Switch:SW_Push_45deg
- added SW21: End, symbol Switch:SW_Push_45deg
- added SW22: PgDn, symbol Switch:SW_Push_45deg
- added SW23: 半/全, symbol Switch:SW_Push_45deg
- added SW24: 1, symbol Switch:SW_Push_45deg
- added SW25: 2, symbol Switch:SW_Push_45deg
- added SW26: 3, symbol Switch:SW_Push_45deg
- added SW27: 4, symbol Switch:SW_Push_45deg
- added SW28: 5, symbol Switch:SW_Push_45deg
- added SW29: 6, symbol Switch:SW_Push_45deg
- added SW3: F2, symbol Switch:SW_Push_45deg
- added SW30: 7, symbol Switch:SW_Push_45deg
- added SW31: 8, symbol Switch:SW_Push_45deg
- added SW32: 9, symbol Switch:SW_Push_45deg
- added SW33: 0, symbol Switch:SW_Push_45deg
- added SW34: =, symbol Switch:SW_Push_45deg
- added SW35: -, symbol Switch:SW_Push_45deg
- added SW36: |, symbol Switch:SW_Push_45deg
- added SW37: BkSp, symbol Switch:SW_Push_45deg
- added SW38: Tab, symbol Switch:SW_Push_45deg
- added SW39: Q, symbol Switch:SW_Push_45deg
- added SW4: F3, symbol Switch:SW_Push_45deg
- added SW40: W, symbol Switch:SW_Push_45deg
- added SW41: E, symbol Switch:SW_Push_45deg
- added SW42: R, symbol Switch:SW_Push_45deg
- added SW43: T, symbol Switch:SW_Push_45deg
- added SW44: Y, symbol Switch:SW_Push_45deg
- added SW45: U, symbol Switch:SW_Push_45deg
- added SW46: I, symbol Switch:SW_Push_45deg
- added SW47: O, symbol Switch:SW_Push_45deg
- added SW48: P, symbol Switch:SW_Push_45deg
- added SW49: ', symbol Switch:SW_Push_45deg
- added SW5: F4, symbol Switch:SW_Push_45deg
- added SW50: {, symbol Switch:SW_Push_45deg
- added SW51: Enter, symbol Switch:SW_Push_45deg
- added SW52: CapsLk, symbol Switch:SW_Push_45deg
- added SW53: A, symbol Switch:SW_Push_45deg
- added SW54: S, symbol Switch:SW_Push_45deg
- added SW55: D, symbol Switch:SW_Push_45deg
- added SW56: F, symbol Switch:SW_Push_45deg
- added SW57: G, symbol Switch:SW_Push_45deg
- added SW58: H, symbol Switch:SW_Push_45deg
- added SW59: J, symbol Switch:SW_Push_45deg
- added SW6: F5, symbol Switch:SW_Push_45deg
- added SW60: K, symbol Switch:SW_Push_45deg
- added SW61: L, symbol Switch:SW_Push_45deg
- added SW62: +, symbol Switch:SW_Push_45deg
- added SW63: *, symbol Switch:SW_Push_45deg
- added SW64: }, symbol Switch:SW_Push_45deg
- added SW65, SW77: Shift, symbol Switch:SW_Push_45deg
- added SW66: Z, symbol Switch:SW_Push_45deg
- added SW67: X, symbol Switch:SW_Push_45deg
- added SW68: C, symbol Switch:SW_Push_45deg
- added SW69: V, symbol Switch:SW_Push_45deg
- added SW7: F6, symbol Switch:SW_Push_45deg
- added SW70: B, symbol Switch:SW_Push_45deg
- added SW71: N, symbol Switch:SW_Push_45deg
- added SW72: M, symbol Switch:SW_Push_45deg
- added SW73: <, symbol Switch:SW_Push_45deg
- added SW74: >, symbol Switch:SW_Push_45deg
- added SW75: ?, symbol Switch:SW_Push_45deg
- added SW76: _, symbol Switch:SW_Push_45deg
- added SW78: ↑, symbol Switch:SW_Push_45deg
- added SW79, SW87: Ctrl, symbol Switch:SW_Push_45deg
- added SW8: F7, symbol Switch:SW_Push_45deg
- added SW80: Fn, symbol Switch:SW_Push_45deg
- added SW81, SW86: Alt, symbol Switch:SW_Push_45deg
- added SW82: 無変換, symbol Switch:SW_Push_45deg
- added SW83: Space, symbol Switch:SW_Push_45deg
- added SW84: 前候補, symbol Switch:SW_Push_45deg
- added SW85: カタカナ, symbol Switch:SW_Push_45deg
- added SW88: ←, symbol Switch:SW_Push_45deg
- added SW89: ↓, symbol Switch:SW_Push_45deg
- added SW9: F8, symbol Switch:SW_Push_45deg
- added SW90: →, symbol Switch:SW_Push_45deg
- added SW91: Left ClicK, symbol Switch:SW_Push_45deg
- added SW92: Right Clock, symbol Switch:SW_Push_45deg
Connections:
- new net GND: J2.2 (Pin_2), SW91.1, SW92.1
- new net KB1_0: J1.8 (Pin_8), SW10.1, SW14.1, SW15.1, SW16.1, SW2.1, SW20.1, SW23.1, SW28.1, SW29.1, SW3.1, SW34.1, SW35.1, SW79.1, SW9.1
- new net KB1_1: J1.7 (Pin_7), SW11.1, SW17.1, SW18.1, SW19.1, SW21.1, SW22.1, SW24.1, SW25.1, SW26.1, SW27.1, SW30.1, SW31.1, SW32.1, SW33.1
- new net KB1_2: J1.1 (Pin_1), SW12.1, SW36.1, SW39.1, SW40.1, SW41.1, SW42.1, SW45.1, SW46.1, SW47.1, SW48.1
- new net KB1_3: J1.6 (Pin_6), SW37.1, SW38.1, SW4.1, SW43.1, SW44.1, SW49.1, SW50.1, SW52.1, SW65.1, SW8.1
- new net KB1_4: J1.2 (Pin_2), SW53.1, SW54.1, SW55.1, SW56.1, SW59.1, SW60.1, SW61.1, SW62.1
- new net KB1_5: J1.5 (Pin_5), SW1.1, SW5.1, SW57.1, SW58.1, SW6.1, SW63.1, SW7.1, SW78.1, SW81.1, SW84.1
- new net KB1_6: J1.3 (Pin_3), SW13.1, SW51.1, SW64.1, SW66.1, SW67.1, SW68.1, SW69.1, SW72.1, SW73.1, SW74.1, SW77.1, SW87.1
- new net KB1_7: J1.4 (Pin_4), SW70.1, SW71.1, SW75.1, SW76.1, SW80.1, SW82.1, SW83.1, SW85.1, SW86.1, SW88.1, SW89.1, SW90.1
- new net KB2_1: J2.18 (Pin_18)
- new net KB2_10: J2.11 (Pin_11), SW32.2, SW47.2, SW61.2, SW74.2, SW79.2, SW8.2, SW84.2, SW85.2, SW87.2, SW9.2
- new net KB2_11: J2.7 (Pin_7), SW31.2, SW35.2, SW46.2, SW50.2, SW60.2, SW7.2, SW73.2, SW76.2
- new net KB2_12: J2.12 (Pin_12), SW29.2, SW30.2, SW44.2, SW45.2, SW58.2, SW59.2, SW71.2, SW72.2
- new net KB2_13: J2.13 (Pin_13), SW27.2, SW28.2, SW42.2, SW43.2, SW56.2, SW57.2, SW69.2, SW70.2
- new net KB2_14: J2.15 (Pin_15), SW26.2, SW3.2, SW4.2, SW41.2, SW5.2, SW55.2, SW68.2
- new net KB2_15: J2.20 (Pin_20), SW2.2, SW25.2, SW40.2, SW52.2, SW54.2, SW67.2
- new net KB2_16: J2.19 (Pin_19), SW1.2, SW23.2, SW24.2, SW38.2, SW39.2, SW53.2, SW66.2, SW82.2
- new net KB2_2: J2.6 (Pin_6), SW65.2, SW77.2, SW90.2
- new net KB2_3: J2.17 (Pin_17), SW11.2, SW12.2, SW81.2, SW86.2
- new net KB2_4: J2.14 (Pin_14), SW13.2, SW15.2, SW21.2, SW78.2, SW88.2
- new net KB2_5: J2.16 (Pin_16), SW16.2, SW22.2, SW80.2
- new net KB2_6: J2.9 (Pin_9), SW18.2, SW20.2, SW89.2
- new net KB2_7: J2.5 (Pin_5), SW14.2, SW19.2
- new net KB2_8: J2.10 (Pin_10), SW10.2, SW17.2, SW36.2, SW37.2, SW51.2, SW6.2, SW83.2
- new net KB2_9: J2.8 (Pin_8), SW33.2, SW34.2, SW48.2, SW49.2, SW62.2, SW63.2, SW64.2, SW75.2
- new net TRKPD_Lclick: J2.4 (Pin_4), SW91.2
- new net TRKPD_Rclick: J2.3 (Pin_3), SW92.2
- no-connect marks 0 -> 1
Other:
- note removed: "Making this a reality can be your contribution!"
- company: (none) -> Recreated by: Ahmad Byagowi
- title: (none) -> Keyboard Membrane
