File: PCB/Mainboard/Buffers.kicad_sch (KiCad schematic)
At the start: 17 parts, among them U10 74F08, U11 74F32, U3 74LS14, U5 74LS157, U6 74LS07, U7 74F245, U9 74F138

Commit message: Add files via upload
Parts:
- removed JP39: Green Pwr, My_Components:Conn_Pin_Header_2x1_2.54mm, symbol Jumper:Jumper_2_Open
- removed JP41: Jumper_2_Open, My_Components:Conn_Pin_Header_2x1_2.54mm, symbol Jumper:Jumper_2_Open
- removed JP46: CPU Select 4, My_Components:Conn_Pin_Header_3x1_2.54mm, symbol Jumper:Jumper_3_Open
- removed R15: 330, Resistor_SMD:R_0612_1632Metric_Pad1.18x3.40mm_HandSolder, symbol Device:R
- removed R43, R48, R50, R77: 10k, Resistor_SMD:R_0612_1632Metric_Pad1.18x3.40mm_HandSolder, symbol Device:R
- removed R67, R70: 1k, Resistor_SMD:R_0612_1632Metric_Pad1.18x3.40mm_HandSolder, symbol Device:R
- removed U10: 74F08, My_Components:IC_DIP14_300, symbol 74xx:74LS08
- removed U11: 74F32, My_Components:IC_DIP14_300, symbol 74xx:74LS32
- removed U3: 74LS14, My_Components:IC_DIP14_300, symbol 74xx:74LS14
- removed U5: 74LS157, My_Components:IC_DIP16_300, symbol 74xx:74LS157
- removed U6: 74LS07, My_Components:IC_DIP14_300, symbol 74xx:74LS07
- removed U7: 74F245, My_Components:IC_DIP20_300, symbol 74xx:74LS245
- removed U9: 74F138, My_Components:IC_DIP16_300, symbol 74xx:74LS138
Connections:
- no-connect marks 9 -> 0
Other:
- note removed: "U6A is used for Turbo SW to Turbo LED buffer C7, R27, R64, JP36, JP34 are parts of Turbo circuit"
- note removed: "U6C is unused"
- note removed: "U6D is used for KBD CO to KBD CI buffer"
