File: PCB/Mainboard/Decoup_caps.kicad_sch (KiCad schematic)
At the start: 70 parts

Commit message: Add files via upload
Parts:
- removed BC1, BC10, BC11, BC12, BC13, BC14, BC15, BC16, BC17, BC18, BC19, BC2, BC20, BC21, BC22, BC23, BC24, BC25, BC26, BC27, BC28, BC29, BC3, BC30, BC31, BC32, BC33, BC36, BC37, BC38, BC4, BC5, BC6, BC7, BC8, BC9, C11, C12, C13, C14, C15, C16, C17, C18, C19, C20, C21, C22, C23, C24, C25, C29, C30, C31, C32, C33, C34, C35, C36: 0.1uF, Capacitor_SMD:C_0603_1608Metric_Pad1.08x0.95mm_HandSolder, symbol Device:C
- removed TC1, TC10, TC11, TC12, TC2, TC3, TC4, TC6, TC7, TC8, TC9: 10uF, symbol Device:C_Polarized_US
Other:
- note removed: "(7407)"
- note removed: "(74F08)"
- note removed: "(74F244)"
- note removed: "(74LS138)"
- note removed: "(74LS14)"
- note removed: "(74LS157)"
- note removed: "(74LS255)"
- note removed: "(82C42)"
- note removed: "(82C602A)"
- note removed: "(82C895)"
- note removed: "(Add filter for 3.3V)"
- note removed: "(BIOSROM)"
- note removed: "(DIMMS)"
- note removed: "(ISA)"
- note removed: "(Keyboard)"
- note removed: "(No decoup for 74F32)"
- note removed: "(SIMM30)"
- note removed: "(SIMM72)"
- note removed: "(VLB)"
- note removed: "Bypass"
- note removed: "CPU"
- note removed: "Cache"
- note removed: "Chipset"
- note removed: "Logic"
- note removed: "SIMMs/DIMMs"
