File: PCB/Mainboard/Keyboard_BIOS.kicad_sch (KiCad schematic)
At the start: 21 parts, among them J1 Keyboard, J2 Mouse, J22 Keylock: Unlocked/Locked, U1 8242KBD, U14 SST39SF010A, U61 74LS06, Y3 8MHz

Commit message: Add files via upload
Parts:
- removed C221, C222, C223, C224: 47pF, Capacitor_SMD:C_0603_1608Metric_Pad1.08x0.95mm_HandSolder, symbol Device:C
- removed C225, C226: 20pF, Capacitor_SMD:C_0603_1608Metric_Pad1.08x0.95mm_HandSolder, symbol Device:C
- removed F1: 1.1A, Fuse:Fuse_Littelfuse_395Series, symbol Device:Polyfuse_Small
- removed FB1, FB2, FB3, FB4: Ferrite_Bead, Inductor_SMD:L_0603_1608Metric_Pad1.05x0.95mm_HandSolder, symbol Device:FerriteBead_Small
- removed J1: Keyboard, My_Components:Conn_Mini_DIN_6pin, symbol Connector:Mini-DIN-6
- removed J2: Mouse, My_Components:Conn_Mini_DIN_6pin, symbol Connector:Mini-DIN-6
- removed J22: Keylock: Unlocked/Locked, My_Components:Conn_Pin_Header_3x1_2.54mm, symbol my_components:Jumper_3_Bridged12_Passive
- removed JP1: Display Select, My_Components:Conn_Pin_Header_2x1_2.54mm, symbol Jumper:Jumper_2_Open
- removed JP101: Flash ROM Write Protect, My_Components:Conn_Pin_Header_3x1_2.54mm, symbol my_components:Jumper_3_Bridged12_Passive
- removed JP102: IRQ12: Mouse/ISA, My_Components:Conn_Pin_Header_3x1_2.54mm, symbol my_components:Jumper_3_Bridged12_Passive
- removed U1: 8242KBD, My_Components:IC_DIP40_600, symbol my_components:8242KBD
- removed U14: SST39SF010A, My_Components:IC_DIP32_600, symbol my_components:SST39SF010A
- removed U61: 74LS06, My_Components:IC_DIP14_300, symbol 74xx:74LS06
- removed Y3: 8MHz, My_Components:Crystal_32K_Horiz, symbol Device:Crystal_Small
Connections:
- no-connect marks 15 -> 0
Other:
- note removed: "(KBCO)"
