File: PCB/Mainboard/Pull-ups.kicad_sch (KiCad schematic)
At the start: 45 parts

Commit message: Add files via upload
Parts:
- removed JP31: 0WS#/LRDY#, My_Components:Conn_Pin_Header_3x1_2.54mm, symbol Jumper:Jumper_3_Open
- removed JP33: Jumper_3_Bridged12, My_Components:Conn_Pin_Header_3x1_2.54mm, symbol Jumper:Jumper_3_Bridged12
- removed JP35: No wait / 1 wait, My_Components:Conn_Pin_Header_2x1_2.54mm, symbol Jumper:Jumper_2_Open
- removed JP37: <= 33.3 MHz / > 33.3 MHz, My_Components:Conn_Pin_Header_2x1_2.54mm, symbol Jumper:Jumper_2_Open
- removed JP6: EMPI, My_Components:Conn_Pin_Header_2x1_2.54mm, symbol Jumper:Jumper_2_Open
- removed JP7: OWS#/LRDYI#, My_Components:Conn_Pin_Header_2x1_2.54mm, symbol Jumper:Jumper_2_Bridged
- removed R11, R22, R24, R25: 330, Resistor_SMD:R_0612_1632Metric_Pad1.18x3.40mm_HandSolder, symbol Device:R
- removed R21, R32, R36, R46, R49, R61: 10k, Resistor_SMD:R_0612_1632Metric_Pad1.18x3.40mm_HandSolder, symbol Device:R
- removed R31, R33: 1k, Resistor_SMD:R_0612_1632Metric_Pad1.18x3.40mm_HandSolder, symbol Device:R
- removed R51, R59, R73, R74, R8: 4.7k, Resistor_SMD:R_0612_1632Metric_Pad1.18x3.40mm_HandSolder, symbol Device:R
- removed R6, R7: 2.2k, Resistor_SMD:R_0612_1632Metric_Pad1.18x3.40mm_HandSolder, symbol Device:R
- removed RA5: 75, Resistor_THT:R_Array_SIP8, symbol Device:R_Pack04
- removed RA9: 22, Resistor_THT:R_Array_SIP8, symbol Device:R_Pack04_SIP
- removed RN10: 10k, Resistor_THT:R_Array_SIP9, symbol Device:R_Network08
- removed RP1, RP12: 10k, Resistor_THT:R_Array_SIP10, symbol Device:R_Network09
- removed RP10, RP11, RP13, RP9: 4.7k, Resistor_THT:R_Array_SIP9, symbol Device:R_Network08
- removed RP14: 1k, Resistor_THT:R_Array_SIP10, symbol Device:R_Network09
- removed RP15: 4.7k, Resistor_THT:R_Array_SIP10, symbol Device:R_Network09
- removed RP16, RP7: 4.7k, Resistor_THT:R_Array_SIP8, symbol Device:R_Network07
- removed RP17, RP2, RP3, RP4, RP5, RP6, RP8: 10k, Resistor_THT:R_Array_SIP8, symbol Device:R_Network07
Connections:
- no-connect marks 16 -> 0
Other:
- note removed: "Chipset Straps: MP0 = 0 (JP7 closed, default): Pin 50 = LRDY# MP0 = 1 (JP7 open): Pin 50 = 0WS# MP1 = 0 (hardwired): Pin 192 = LREQ1#, Pin 193 = LGNT1# MP2 = 1 (hardwired): Pin 108 = D/C#, Pin 47 = HITM# MP3 = 1 (hardwired): Pin 62 = EPMI# XD7 = 0, XD6 = 1 (hardwired/pull-down resistors): Chipset 82C802G XD4 = 0 (hardwired): RTC enabled"
- note removed: "VLB ID4 (A56) - GND ID0 = 0, ID1 = 1, ID4 = 0 - 486, Burst possible ID2 = 0 - 1 wait cycle; 1 - no wait ID3 = 0 - > 33.3 MHz; 1 <= 33.3 MHz"
