File: PCB/Mainboard/VLB_IDE.kicad_sch (KiCad schematic)
At the start: 9 parts, among them J16 Secondary IDE, U15 OPTI_82C611A

Commit message: Add files via upload
Parts:
- removed F3: 1.1A, Fuse:Fuse_Littelfuse_395Series, symbol Device:Polyfuse_Small
- removed J16: Secondary IDE, My_Components:Conn_Pin_Header_20x2_2.54mm, symbol Connector_Generic:Conn_02x20_Odd_Even
- removed JP15: IDE2 CFG, My_Components:Conn_Pin_Header_2x3_2.54mm, symbol Connector_Generic:Conn_02x03_Counter_Clockwise
- removed JP16: 82C611A Straps, My_Components:Conn_Pin_Header_8x2_2.54mm, symbol Connector_Generic:Conn_02x08_Odd_Even
- removed JP17: 82C611A Straps, My_Components:Conn_Pin_Header_8x1_2.54mm, symbol Connector_Generic:Conn_01x08
- removed R201: 4.7k, Resistor_SMD:R_0612_1632Metric_Pad1.18x3.40mm_HandSolder, symbol Device:R
- removed RN19, RN20: 4.7k, Resistor_THT:R_Array_SIP8, symbol Device:R_Pack04
- removed U15: OPTI_82C611A, My_Components:IC_PQFP-100_14x20mm_P0.65mm_Hand_Soldering, symbol my_components:OPTI_82C611A
Connections:
- no-connect marks 3 -> 0
Other:
- note removed: "(CSEL)"
- note removed: "(DACK)"
- note removed: "(PDIAG)"
- note removed: "(~{ACTIVE})"
- note removed: "(~{IDE_DRQ})"
- note removed: "0/Tied Low -------------------------- Compatibility Mode Secondary IDE, 17x and 37x Port 3F7 read from local bus ID = 0, IDE disabled on reset SPD[1:0]: 00 - 50MHz; 01 - 40 MHz SPD[1:0]: 10 - 33 MHz; 11 - 25 MHz MODE[1:0]: 00 >= 480 ns; 01 >= 383 ns MODE[1:0]: 10 >= 240 ns; 11 >= 180 ns Disable prefetch"
- note removed: "1/Tied High ----------------- Enhanced Mode Primary IDE, 1Fx and 3Fx Port 3F7 read from ISA bus ID=1, IDE enabled on reset VLB Bus frequency, bit 0 VLB Bus frequency, bit 1 Cycle time, bit 0 Cycle time, bit 1 Enable prefetch"
- note removed: "82C611A Straps ---------- SMI/ENMODE: PRIM: DCS3/ISA3F7: DA2/VICID0: DCS1/SPD0: SPD1: DA0/MODE0: DA1/MODE1: DINTR/ENPREF:"
