File: PCB/Mainboard/Power.kicad_sch (KiCad schematic)
At the start: 53 parts, among them J11 ATX_POWER_20, J12 Front Panel, SW1 POWER, SW2 RESET, U11 74F32, U28 LT1086-ADJ, U3 74LS14, U6 74LS07, U603 74HCT74, U604 74HCT14, U606 LM7905_TO220, U607 IDT514, X1 14.31818MHz, X2 33.333MHz, X3 8MHz, Y2 14.31818MHz

Commit message: Add files via upload
Parts:
- removed C40, C41: 0.1uF, symbol Device:C
- removed C601: 10uF, Capacitor_THT:CP_Radial_D5.0mm_P2.00mm, symbol Device:C_Polarized_US
- removed C602, C603: 1uF, Capacitor_THT:CP_Radial_D5.0mm_P2.00mm, symbol Device:C_Polarized_US
- removed C640, C641: ?pF, Capacitor_SMD:C_0603_1608Metric_Pad1.08x0.95mm_HandSolder, symbol Device:C
- removed D1, D2, D5: 1N4148, Diode_THT:D_DO-35_SOD27_P7.62mm_Horizontal, symbol Device:D
- removed J11: ATX_POWER_20, My_Components:Conn_Power_ATX_20pin, symbol my_components:ATX_POWER_20
- removed J12: Front Panel, Connector_PinHeader_2.54mm:PinHeader_2x10_P2.54mm_Vertical, symbol Connector_Generic:Conn_02x10_Odd_Even
- removed JP117: CPU Frequency, symbol Connector_Generic:Conn_02x03_Odd_Even
- removed JP29: 5V / Low CPU Voltage, symbol Connector_Generic:Conn_02x03_Odd_Even
- removed JP4: 5V / 3.3V CPU Voltage, symbol Connector_Generic:Conn_02x03_Odd_Even
- removed JP45: Low Voltage Select: 3.3V/3.45V/4V, symbol Connector_Generic:Conn_02x03_Odd_Even
- removed JP609: -5V Source, My_Components:Conn_Pin_Header_3x1_2.54mm, symbol Jumper:Jumper_3_Bridged12
- removed LS1: AT-1224TWTR, My_Components:Speaker_12mm, symbol Device:Speaker
- removed R17: 330, Resistor_SMD:R_0612_1632Metric_Pad1.18x3.40mm_HandSolder, symbol Device:R
- removed R18: 51, Resistor_SMD:R_0612_1632Metric_Pad1.18x3.40mm_HandSolder, symbol Device:R
- removed R19, R26, R44, R45, R9: 33, Resistor_SMD:R_0612_1632Metric_Pad1.18x3.40mm_HandSolder, symbol Device:R
- removed R5, R610, R611: 10k, Resistor_SMD:R_0612_1632Metric_Pad1.18x3.40mm_HandSolder, symbol Device:R
- removed R57: 243, symbol Device:R
- removed R58: 150, symbol Device:R
- removed R612: 470, symbol Device:R
- removed R64: 1k, Resistor_SMD:R_0612_1632Metric_Pad1.18x3.40mm_HandSolder, symbol Device:R
- removed R75: 75, symbol Device:R
- removed R76: 22, symbol Device:R
- removed SW1: POWER, My_Components:Switch_Tactile_6mm, symbol my_components:Switch_Tactile
- removed SW2: RESET, My_Components:Switch_Tactile_6mm, symbol my_components:Switch_Tactile
- removed TC13: 22uF, Capacitor_THT:CP_Radial_D5.0mm_P2.00mm, symbol Device:C_Polarized_US
- removed TC14: 220uF, Capacitor_THT:CP_Radial_D5.0mm_P2.00mm, symbol Device:C_Polarized_US
- removed TP1: GPCS#, symbol Connector:TestPoint
- removed TP2: DOZE#, symbol Connector:TestPoint
- removed U11: 74F32, My_Components:IC_DIP14_300, symbol 74xx:74LS32
- removed U28: LT1086-ADJ, symbol Regulator_Linear:LT1086-ADJ
- removed U3: 74LS14, My_Components:IC_DIP14_300, symbol 74xx:74LS14
- removed U6: 74LS07, My_Components:IC_DIP14_300, symbol 74xx:74LS07
- removed U603: 74HCT74, My_Components:IC_DIP14_300, symbol 74xx:74LS74
- removed U604: 74HCT14, My_Components:IC_DIP14_300, symbol 74xx:74LS14
- removed U606: LM7905_TO220, Package_TO_SOT_THT:TO-220-3_Vertical, symbol Regulator_Linear:LM7905_TO220
- removed U607: IDT514, Package_SO:SOIC-8_3.9x4.9mm_P1.27mm, symbol Oscillator:NB3N502
- removed X1: 14.31818MHz, Oscillator:Oscillator_DIP-8, symbol Oscillator:CXO_DIP8
- removed X2: 33.333MHz, Oscillator:Oscillator_DIP-8, symbol Oscillator:CXO_DIP8
- removed X3: 8MHz, Oscillator:Oscillator_DIP-8, symbol Oscillator:CXO_DIP8
- removed Y2: 14.31818MHz, My_Components:Crystal_32K_Horiz, symbol Device:Crystal_Small
- added C137, C138: 1nF, symbol Device:C
- added C139, C55, C56, C57, C58, C60, C63: 100nF, symbol Device:C
- added C27, C28: 18pF, symbol Device:C
- added C59: 10nF, symbol Device:C
- added C62: 120nF, symbol Device:C
- added D4, D5: K, symbol Device:D_Dual_Series_KAC
- added D6, D7: N, symbol Device:D_Dual_CommonCathode_AKA
- added D8, D9: 3D, symbol Device:D_Dual_CommonCathode_AKA
- added J18: Flat-4, symbol Connector_Generic:Conn_01x04
- added J4: connector-4, symbol Connector_Generic:Conn_01x04
- added J5: PSU_Conn, symbol Connector_Generic:Conn_02x20_Counter_Clockwise
- added Q17, Q18: 8C, Package_TO_SOT_SMD:SOT-23, symbol Transistor_BJT:MMBTA44
- added Q19, Q22: IS6, symbol Transistor_BJT:MMBTA56
- added Q72, Q75: HQ, symbol Transistor_BJT:MMBTA56
- added Q73, Q74: QC, symbol Transistor_BJT:BC847W
- added R100: 220, symbol Device:R
- added R107: 33k, symbol Device:R
- added R108, R283, R328, R330, R331, R336, R339, R351, R354, R355, R38, R42, R86, R89, R98: 4.7k, symbol Device:R
- added R109, R110, R41, R97: 10k, symbol Device:R
- added R167, R209, R210, R212, R214, R390, R407, R413: 100k, symbol Device:R
- added R171, R288, R356, R385, R39, R40, R408, R411, R93, R95: 47k, symbol Device:R
- added R207, R208, R211, R213, R52: 120k, symbol Device:R
- added R384, R386: 1k, symbol Device:R
- added R43, R62: 68k, symbol Device:R
- added R60: 50k, symbol Device:R
- added R79, R84, R88: 0, symbol Device:R
- added R83, R91: 470k, symbol Device:R
- added R99: 470, symbol Device:R
- added U13: 8C01, symbol PC110:QC01
- added U15, U17: EA, symbol 74xGxx:74AHC1G14
- added U16: QC01, symbol PC110:QC01
- added U17: 3E00, symbol PC110:QC01
- added U43: Front LCD, symbol Connector_Generic:Conn_01x14
- added U44: NJM2904M, symbol Amplifier_Operational:LM2904
- added U6: M38224M6HP, symbol PC110:M38223E4HP
- added X1: 245759, symbol PCM_Elektuur:X-crystal
- R63: value 1k -> 68k; footprint Resistor_SMD:R_0612_1632Metric_Pad1.18x3.40mm_HandSolder -> (none)
Connections:
- net PLED+ is gone; now on net GND: R63.2
- net GND: now also C139.1, C27.1, C28.1, C55.1, C56.1, C57.1, C58.1, C59.1, C62.1, C63.1, J4.2 (Pin_2), J5.24 (Pin_24), J5.29 (Pin_29), J5.32 (Pin_32), J5.7 (Pin_7), J5.9 (Pin_9), Q73.2 (E), Q74.2 (E), R108.1, R209.1, R210.1, R211.1, R213.1, R408.1, R411.1, R60.2, R83.2, R91.2, R98.1, U13.3 (GND), U15.3 (GND), U16.3 (GND), U17.3 (GND), U17.3 (GND), U44.4 (V-), U6.16 (P50), U6.30 (GND), U6.73 (GND)
- net VCC: now also D5.2 (A), J5.16 (Pin_16), R288.2, R356.1, R52.1, U6.71 (VCC); no longer R63.1
- new net: R83.1, U13.1 (OUT), U15.2
- new net: R331.2, U6.54 (SEG00)
- new net: C28.2, U6.28 (Xin), X1.1 (+)
- new net: Q17.1 (B), R107.2
- new net: Q72.3 (C), R384.2
- new net: C57.2, U17.5 (CD)
- new net: C137.1, R211.2, R214.1, U44.2 (-)
- new net: D7.1 (A), Q18.2 (E)
- new net: D7.3 (A), R95.1
- new net: C27.2, R40.1, X1.2 (-)
- new net: D6.3 (A), R93.1
- new net: Q19.1 (B), R93.2, R99.1
- new net: C58.2, D4.1 (K), U15.5 (VCC), U17.5 (VCC)
- new net: D4.2 (A), D5.1 (K)
- new net: R52.2, R62.1, U6.78 (VL3)
- new net: R43.1, R62.2, U6.79 (VL2)
- new net: C56.2, R79.2, U16.2 (VDD)
- new net: C59.2, U16.5 (CD)
- new net: C55.2, R84.2, U13.2 (VDD)
- new net: D6.1 (A), Q17.2 (E)
- new net: Q17.3 (C), R99.2
- new net: R328.2, U6.50 (P04)
- new net: Q18.1 (B), R97.2
- new net: C60.1, C63.2
- new net: C60.2, U13.5 (CD)
- new net: C62.2, R88.2, U17.2 (VDD)
- new net: R208.1, R209.2, U44.5 (+)
- new net: C138.1, R212.1, R213.2, U44.6 (-)
- new net: Q75.3 (C), R386.2
- new net: R339.2, U6.51 (P03)
- new net: R167.2, U6.45 (P11)
- new net: Q22.1 (B), R100.1, R95.2
- new net: R38.1, U6.19 (P45)
- new net: D9.2 (K), U15.4, U17.2
- new net: R86.2, U6.40 (P16)
- new net: R354.2, U6.49 (P05)
- new net: R39.1, U6.15 (P51)
- new net: R42.2, U6.24 (P40)
- new net: R40.2, U6.29 (Xout)
- new net: R283.2, U6.35 (P23)
- new net: R89.2, U6.36 (P22)
- new net: R390.2, U6.43 (P13)
- new net: R407.2, U6.44 (P12)
- new net: R413.2, U6.46 (P10)
- new net: R330.2, U6.47 (SEG07)
- new net: R355.2, U6.48 (P06)
- new net: R336.2, U6.52 (P02)
- new net: R351.2, U6.53 (SEG01)
- new net: R43.2, R63.1, U6.80 (VL1)
- new net: R207.1, R210.2, U44.3 (+)
- new net: D8.2 (K), U17.4
- new net: Q18.3 (C), R100.2
- new net AV9_FS2: R79.1
- new net AV9_OE: R91.1, U16.1 (OUT)
- new net CMOS_BATT+: J4.3 (Pin_3)
- new net CMOS_BATT_Sense: J4.4 (Pin_4), R41.2, U6.6 (P62)
- new net D18_2_3: J5.21 (Pin_21)
- new net D28_1: J5.12 (Pin_12)
- new net D2_3: J5.35 (Pin_35)
- new net F65_ENAVEE: J5.26 (Pin_26)
- new net J13_53: J5.36 (Pin_36), J5.37 (Pin_37), J5.5 (Pin_5)
- new net J5_6_Yellow: J5.6 (Pin_6)
- new net KB_RESET#: D8.1 (A), D8.3 (A), R109.2
- new net M38_21: U6.55 (21)
- new net M38_COM0: U43.14 (Pin_14), U6.77 (COM0)
- new net M38_COM1: U43.13 (Pin_13), U6.76 (COM1)
- new net M38_COM2: U43.12 (Pin_12), U6.75 (COM2)
- new net M38_COM3: U43.11 (Pin_11), U6.74 (COM3)
- new net M38_P10_R413: Q74.1 (B), R411.2, R413.1
- new net M38_P11_R167: Q75.1 (B), R167.1, R171.1
- new net M38_P12_R407: Q73.1 (B), R407.1, R408.2
- new net M38_P13_R390: Q72.1 (B), R385.1, R390.1
- new net M38_P14: U6.42 (P14)
- new net M38_P15: U6.41 (P15)
- new net M38_P16_R86: R86.1
- new net M38_P17: U6.39 (P17)
- new net M38_P20: J5.19 (Pin_19), U6.38 (P20)
- new net M38_P21: J5.22 (Pin_22), U6.37 (P21)
- new net M38_P22_R88: R89.1
- new net M38_P27_KB_SPKDN: U6.31 (P27)
- new net M38_P34: R356.2, U6.58 (P34)
- new net M38_P35: U6.57 (P35)
- new net M38_P36: U6.56 (P36)
- new net M38_P41: U6.23 (P41)
- new net M38_P43: U6.21 (P43)
- new net M38_P44: U6.20 (P44)
- new net M38_P46: R288.1, U6.18 (P46)
- new net M38_P52: J5.18 (Pin_18), U6.14 (P52)
- new net M38_P53: J5.23 (Pin_23), U6.13 (P53)
- new net M38_P57: U6.9 (P57)
- new net M38_P60: J5.1 (Pin_1), U6.8 (P60)
- new net M38_P61: J5.2 (Pin_2), U6.7 (P61)
- new net M38_P63: J5.40 (Pin_40), U6.5 (P63)
- new net M38_P64: J5.34 (Pin_34), U6.4 (P64)
- new net M38_P65: C137.2, R214.2, U44.1, U6.3 (P65)
- new net M38_P66: C138.2, R212.2, U44.7, U6.2 (P66)
- new net M38_P67: R60.1, U6.1 (P67)
- new net M38_P71: U6.26 (P71)
- new net M38_RESET: U6.25 (RESET)
- new net M38_SEG0: U43.1 (Pin_1), U6.70 (SEG0)
- new net M38_SEG1: U43.2 (Pin_2), U6.69 (SEG1)
- new net M38_SEG2: U43.3 (Pin_3), U6.68 (SEG2)
- new net M38_SEG3: U43.4 (Pin_4), U6.67 (SEG3)
- new net M38_SEG4: U43.5 (Pin_5), U6.66 (SEG4)
- new net M38_SEG5: U43.6 (Pin_6), U6.65 (SEG5)
- new net M38_SEG6: U43.7 (Pin_7), U6.64 (SEG6)
- new net M38_SEG7: U43.8 (Pin_8), U6.63 (SEG7)
- new net M38_SEG8: U43.9 (Pin_9), U6.62 (SEG8)
- new net M38_SEG9: U43.10 (Pin_10), U6.61 (SEG9)
- new net M38_VREF: J5.31 (Pin_31), R41.1, U6.72 (VREF)
- new net MIC_J17: J4.1 (Pin_1)
- new net PNET1: J5.33 (Pin_33), J5.8 (Pin_8), Q22.2 (E), R109.1, R110.1, R84.1
- new net PNET2: Q19.3 (C), R107.1, R108.2, R354.1
- new net PNET4: J5.3 (Pin_3), J5.38 (Pin_38), J5.4 (Pin_4)
- new net PNET5: J5.10 (Pin_10), J5.11 (Pin_11), J5.30 (Pin_30), Q19.2 (E), R39.2, R88.1
- new net PNET7: Q22.3 (C), R97.1, R98.2
- new net PNET8: C139.2, Q72.2 (E), Q75.2 (E), R171.2, R385.2, U44.8 (V+)
- new net PSU_AUX_SW1: J5.28 (Pin_28), R42.1
- new net PWRGD_shift_buff: D6.2 (K), D7.2 (K), U6.27 (PWRGD)
- new net Q43_2: J5.13 (Pin_13)
- new net Q49_1: J5.39 (Pin_39)
- new net R284_2: J5.14 (Pin_14)
- new net R412_1: J5.20 (Pin_20)
- new net R73_2: J5.15 (Pin_15)
- new net RESET: D9.1 (A), D9.3 (A), R110.2
- new net Touch_X+: J18.2 (Pin_2), R207.2, R384.1
- new net Touch_X-: J18.3 (Pin_3), Q73.3 (C)
- new net Touch_Y+: J18.1 (Pin_1), R208.2, R386.1
- new net Touch_Y-: J18.4 (Pin_4), Q74.3 (C)
- new net U106_1CLK: U6.11 (1CLK)
- new net U21_101: R328.1
- new net U21_102: R339.1
- new net U21_103: R336.1
- new net U21_104: R351.1
- new net U21_105: R331.1
- new net U21_131: J5.27 (Pin_27)
- new net U21_97: R330.1
- new net U21_98: R355.1
- new net U54_1D: J5.17 (Pin_17)
- new net U54_1Q: J5.25 (Pin_25)
- new net U8_1A3_KB_TP139: R283.1
- new net U8_2A1_KB_RXD: R38.2
- new net to_ESS_RESET: U17.1 (OUT)
- no-connect marks 21 -> 14
Other:
- note added: "5v"
- note added: "5v switched on via PWRGD"
- note removed: "(16V)"
- note removed: "(check 3.3V pinout)"
- note removed: "Buffer OSC for ISA?"
- note removed: "Buffer clocks separately for CPU/Chipset/Local Bus Chips"
- note removed: "CPU Voltage Regulator (Optional)"
- note removed: "HDD_LED-"
- note removed: "No pin"

Commit message: Add files via upload
Parts:
- added C61: 180nF, symbol Device:C
- added C96: 150nF, symbol Device:C
- added C98: 330pF, symbol Device:C
- added C99: 100pF, symbol Device:C
- added D20, D21, D9: N, symbol Device:D_Dual_CommonCathode_AKA
- added Q14, Q21, Q40: 8C, Package_TO_SOT_SMD:SOT-23, symbol Transistor_BJT:MMBTA44
- added R128, R146, R156, R248, R80, R82, R90: 470k, symbol Device:R
- added R254, R85: 47k, symbol Device:R
- added U29: E2, symbol 74xGxx:SN74LVC1G00DBV
- added U30, U32: 74LVT74, symbol 74xx:74LS74
- added U5: 74HC14, symbol 74xx:74LS14
- renumbered D9 to D10
Connections:
- net GND: now also C61.1, C96.1, C98.1, C99.1, Q21.2 (E), Q40.2 (E), R80.1, R82.1, R90.1, U29.3 (GND), U30.7 (GND), U32.7 (GND), U5.7 (GND)
- net M38_RESET: now also C99.2, U30.4 (~{S})
- net PNET1: now also R156.1
- net U106_1CLK: now also R80.2, U32.3 (C)
- net VCC: now also C61.2, C96.2, R128.2, U29.5 (VCC), U30.1 (~{R}), U30.10 (~{S}), U30.12 (D), U30.14 (VCC), U32.10 (~{S}), U32.12 (D), U32.14 (VCC), U32.2 (D), U5.14 (VCC)
- new net: D20.2 (K), U32.5 (Q)
- new net: D21.2 (K), U32.9 (Q)
- new net: U29.1, U30.8 (~{Q})
- new net: U29.2, U32.6 (~{Q})
- new net: D9.2 (K), R254.1
- new net: Q40.1 (B), R254.2
- new net: D9.1 (A), U30.9 (Q), U32.11 (C)
- new net: U30.11 (C), U5.12
- new net: C98.2, Q14.3 (C), R146.2, U30.13 (~{R})
- new net: Q21.1 (B), R85.1
- new net: Q21.3 (C), U32.1 (~{R}), U32.13 (~{R})
- new net: R146.1, U30.6 (~{Q})
- new net MN195_U1RD#: R128.1, U5.13
- new net Pluto_52: R85.2
- new net Pluto_72: D20.1 (A), D20.3 (A), R156.2
- new net Pluto_73: D21.1 (A), D21.3 (A)
- new net RTCBAT: R248.2
- new net U103_NAND_of_U53_1CLK_and_U53_1Q#: D9.3 (A)
- new net U30_D0: R90.2, U30.2 (D)
- new net U53_2CLK: R82.2, U30.3 (C)
- new net U54_1PRE#: U29.4
- new net U61_RTCBAT_470K: Q40.3 (C), R248.1
- no-connect marks 14 -> 17

Commit message: Add files via upload
Parts:
- added C245, C46: 10nF, symbol PCM_Elektuur:C
- added C47: 5.6uF, symbol PCM_Elektuur:C
- added C49: 2.2uF, symbol PCM_Elektuur:C
- added C51: 10uF, symbol PCM_Elektuur:C
- added D22: 3D, symbol Device:D_Dual_CommonCathode_AKA
- added D6, D7: Q, Package_TO_SOT_SMD:SOT-323_SC-70, symbol Diode:BAT54W
- added F1: 0.5A, symbol Device:Fuse
- added J6: BridgeBattery, symbol Connector_Generic:Conn_01x02
- added L4: 68uH, symbol Device:L_Ferrite
- added Q15: 8B, symbol Simulation_SPICE:NPN
- added Q3: 582 B74, Package_TO_SOT_THT:TO-92_Inline, symbol Regulator_Linear:MCP1700x-120xxTO
- added Q4: YQ, symbol Simulation_SPICE:NPN
- added Q5: HQ, symbol Transistor_BJT:MMBTA56
- added R111: 100, symbol Device:R
- added R313: 300, symbol Device:R
- added R68: 56, symbol Device:R
- added R76: 1k, symbol Device:R
- renumbered D4 to D10, D5 to D13, D6 to D14, D7 to D15, D8 to D16, D9 to D17, D10 to D18, D21 to D31, Q18 to Q10, Q19 to Q11, Q21 to Q12, Q22 to Q13, Q40 to Q26, Q14 to Q7, Q17 to Q9
Connections:
- net GND: now also C245.2 (-), C47.2 (-), C49.1 (+), C51.2 (-), J6.2 (Pin_2), Q15.3 (E), Q3.1 (GND), Q4.3 (E)
- net PNET4: now also D6.3 (K)
- net PNET7: now also R313.2
- new net: Q5.1 (B), R111.1
- new net: Q15.1 (C), R111.2
- new net: C49.2 (-), Q3.2 (VI), R68.1
- new net: C46.1 (+), Q3.3 (VO), R76.1
- new net: C51.1 (+), D6.1 (A), D7.3 (K), R68.2
- new net: D22.1 (A), D22.3 (A), R313.1
- new net: C245.1 (+), D22.2 (K), F1.2, Q5.2 (E)
- new net: D7.1 (A), L4.1, Q4.1 (C)
- new net: C46.2 (-), Q4.2 (B), R76.2
- new net: C47.1 (+), L4.2, Q5.3 (C)
- new net: F1.1, J6.1 (Pin_1)
- new net YellowWire1_2: Q15.2 (B)
Other:
- note added: "10.5v"
- moved on the sheet: C137, C138, C139, C27, C28, C55, C56, C57, C58, C59, C60, C61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

Commit message: Add files via upload
Parts:
- added C228: 100pF, symbol PCM_Elektuur:C
- added C229: 1uF, symbol PCM_Elektuur:C
- added C231: 150nF, symbol Device:C
- added D4, D42, D43, D46: N, symbol Device:D_Dual_CommonCathode_AKA
- added Q27: 8C, Package_TO_SOT_SMD:SOT-23, symbol Transistor_BJT:MMBTA44
- added R235, R262, R278, R282, R287: 470k, symbol Device:R
- added R268, R44: 100k, symbol Device:R
- added R277: 200k, symbol Device:R
- added R280: 47k, symbol Device:R
- added R286: 22k, symbol Device:R
- added SW1: Power Switch, symbol Switch:SW_SPST
- added U52: EA, symbol 74xGxx:74AHC1G14
- added U54: 74HC74, symbol 74xx:74HC74
Connections:
- net GND: now also C228.2 (-), C229.2 (-), C231.1, Q27.2 (E), R280.2, U52.3 (GND), U54.7 (GND)
- net M38_P71: now also U5.3, D4.1 (A), R44.2
- net M38_RESET: now also R282.1
- net PNET1: now also R287.1, U52.5 (VCC)
- net PSU_AUX_SW1: now also U5.1
- net U54_1D: now also U54.2 (D), U54.6 (~{Q})
- net U54_1PRE#: now also U54.4 (~{S})
- net U54_1Q: now also C229.1 (+), R235.2, U54.5 (Q)
- net VCC: now also C231.2, R278.2, R44.1, SW1.1 (A), U54.10 (~{S}), U54.12 (D), U54.14 (VCC)
- net at U5.10: now also U54.3 (C)
- net MN192_VSEN#: now reaches U5.11
- net MN192_VSEN#: now also R277.2
- net at U5.4: now also D42.2 (K)
- net at U5.2: now also D43.2 (K)
- net at U5.8: now also U54.11 (C)
- net at U5.9: now also R278.1
- net D2_3 renamed D4_3
- net D4_3: now also D4.2 (K)
- new net: D42.1 (A), D42.3 (A), D43.1 (A), D43.3 (A), R287.2, U52.2
- new net: C228.1 (+), R282.2, U54.1 (~{R})
- new net: D46.1 (A), R286.1
- new net: R286.2, U54.9 (Q)
- new net: R268.1, U52.4
- new net: Q27.1 (B), R262.1
- new net: R277.1, R280.1, SW1.2 (B)
- new net: R235.1, U54.13 (~{R})
- new net KB_SPKUP: Q27.3 (C), R268.2
- new net R262_1: R262.2
- no-connect marks 17 -> 19
Other:
- moved on the sheet: U5A, U5B, U5D

Commit message: Add files via upload
Parts:
- removed J4: connector-4, symbol Connector_Generic:Conn_01x04
- removed unit 3 of U5
Other:
- moved on the sheet: C137, C138, C139, C228, C229, C231, C245, C27, C28, C46, C47, C49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

Commit message: Add files via upload
Parts:
- D20: value N -> 3D
- Q11, Q13, Q5, Q72, Q75: footprint (none) -> Package_TO_SOT_SMD:SOT-23
- Q73, Q74: footprint (none) -> Package_TO_SOT_SMD:SOT-323_SC-70
- U29: footprint (none) -> Package_TO_SOT_SMD:SOT-23-5

Commit message: Add files via upload
Parts:
- removed D17: N, symbol Device:D_Dual_CommonCathode_AKA
- removed R248: 470k, symbol Device:R
- added D34: N, symbol Device:D_Dual_CommonCathode_AKA
- added U39: 7W00, symbol 74xGxx:74AHC2G00
Connections:
- net D4_3: now also D4.3 (K); no longer D4.2 (K)
- net M38_P71: now also D4.2 (A); no longer D4.1 (A)
- net PNET1: now also U39.5
- net U103_NAND_of_U53_1CLK_and_U53_1Q#: now also D34.3 (A), U39.3
- net at R254.1: now also D34.2 (K)
- net at U30.9 (Q), U32.11 (C): now also D34.1 (A)
- net at D46.1 (A): no longer R286.1
- net at D46.2 (A): now also R286.1
- new net RIOUT#: U39.6
Other:
- moved on the sheet: C231, C61, U30C, U32C, U54C, U5G

Commit message: Add files via upload
Parts:
- renumbered D20 to D30
Connections:
- net KB_RESET#: now also D16.2 (A); no longer D16.3 (A)
- net Pluto_72: now also D30.2 (A); no longer D30.3 (A)
- net RESET: now also D18.2 (A); no longer D18.3 (A)
- net at C245.1 (+), F1.2, Q5.2 (E): now also D22.3 (K); no longer D22.2 (K)
- net at U17.4: now also D16.3 (K); no longer D16.2 (K)
- net at D22.1 (A), R313.1: now also D22.2 (A); no longer D22.3 (A)
- net at U32.5 (Q): now also D30.3 (K); no longer D30.2 (K)
- net at U15.4, U17.2: now also D18.3 (K); no longer D18.2 (K)
Changed lines of the file:
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@@
 	)
 	(symbol
+		(lib_name "D_Dual_CommonCathode_AKA_5")
 		(lib_id "Device:D_Dual_CommonCathode_AKA")
 		(at 742.95 92.71 270)
@@
 	)
 	(symbol
+		(lib_name "D_Dual_CommonCathode_AKA_2")
 		(lib_id "Device:D_Dual_CommonCathode_AKA")
 		(at 218.44 469.9 0)
@@
 		(on_board yes)
 		(dnp no)
-		(property "Reference" "D20"
+		(property "Reference" "D30"
 			(at 218.44 463.55 0)
 			(effects
@@
 			(project "PC110"
 				(path "/45c7911f-b027-440e-9e3e-77a146b41944/00000000-0000-0000-0000-0000638712fb"
-					(reference "D20")
+					(reference "D30")
 					(unit 1)
 				)
@@
 	)
 	(symbol
+		(lib_name "D_Dual_CommonCathode_AKA_3")
 		(lib_id "Device:D_Dual_CommonCathode_AKA")
 		(at 317.5 176.53 0)
@@
 	)
 	(symbol
+		(lib_name "D_Dual_CommonCathode_AKA_4")
 		(lib_id "Device:D_Dual_CommonCathode_AKA")
 		(at 742.95 120.65 270)
