File: PCB/Mainboard/Power.kicad_sch (KiCad schematic)
At the start: 157 parts, among them J18 Flat-4, J5 PSU_Conn, J6 BridgeBattery, Q10 8C, Q11 IS6, Q12 8C, Q13 IS6, Q15 8B, Q26 8C, Q27 8C, Q3 582 B74, Q4 YQ, Q5 HQ, Q7 8C, Q72 HQ, Q73 QC, Q74 QC, Q75 HQ, Q9 8C, SW1 Power Switch, U13 8C01, U15 EA, U16 QC01, U17 3E00, U17 EA, U29 E2, U30 74LVT74, U32 74LVT74, U39 7W00, U43 Front LCD, U44 NJM2904M, U5 74HC14, U52 EA, U54 74HC74, U6 M38224M6HP, X1 245759

Commit message: Add files via upload
Parts:
- added C226: 1uF, symbol PCM_Elektuur:C
Connections:
- net GND: now also C226.2 (-)
- net MN192_VSEN#: now also C226.1 (+)
- net R262_1 renamed KB_SPKUP_DN
Changed lines of the file:
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@@
 	)
 	(junction
+		(at 636.27 336.55)
+		(diameter 0)
+		(color 0 0 0 0)
+	)
+	(junction
 		(at 190.5 140.97)
 		(diameter 0)
@@
 	(wire
 		(pts
-			(xy 631.19 332.74) (xy 631.19 346.71)
+			(xy 604.52 340.36) (xy 631.19 340.36)
 		)
 		(stroke
@@
 	(wire
 		(pts
+			(xy 226.06 133.35) (xy 236.22 133.35)
+		)
+		(stroke
+			(width 0)
+			(type default)
+		)
+	)
+	(wire
+		(pts
 			(xy 142.24 158.75) (xy 152.4 158.75)
 		)
@@
 	(wire
 		(pts
+			(xy 118.11 186.69) (xy 118.11 189.23)
+		)
+		(stroke
+			(width 0)
+			(type default)
+		)
+	)
+	(wire
+		(pts
 			(xy 558.8 435.61) (xy 579.12 435.61)
 		)
@@
 	(wire
 		(pts
+			(xy 118.11 172.72) (xy 118.11 176.53)
+		)
+		(stroke
+			(width 0)
+			(type default)
+		)
+	)
+	(wire
+		(pts
 			(xy 692.15 219.71) (xy 692.15 237.49)
 		)
@@
 	(wire
 		(pts
+			(xy 631.19 340.36) (xy 631.19 346.71)
+		)
+		(stroke
+			(width 0)
+			(type default)
+		)
+	)
+	(wire
+		(pts
 			(xy 180.34 436.88) (xy 184.15 436.88)
 		)
@@
 	(wire
 		(pts
-			(xy 636.27 328.93) (xy 636.27 346.71)
-		)
-		(stroke
-			(width 0)
-			(type default)
-		)
-	)
-	(wire
-		(pts
 			(xy 671.83 237.49) (xy 675.64 237.49)
 		)
@@
 	(wire
 		(pts
+			(xy 604.52 336.55) (xy 636.27 336.55)
+		)
+		(stroke
+			(width 0)
+			(type default)
+		)
+	)
+	(wire
+		(pts
 			(xy 322.58 196.85) (xy 317.5 196.85)
 		)
@@
 	(wire
 		(pts
-			(xy 228.6 146.05) (xy 234.95 146.05)
+			(xy 228.6 146.05) (xy 236.22 146.05)
 		)
 		(stroke
@@
 	(wire
 		(pts
-			(xy 226.06 133.35) (xy 234.95 133.35)
-		)
-		(stroke
-			(width 0)
-			(type default)
-		)
-	)
-	(wire
-		(pts
 			(xy 689.61 398.78) (xy 708.66 398.78)
 		)
@@
 	(wire
 		(pts
+			(xy 636.27 336.55) (xy 636.27 346.71)
+		)
+		(stroke
+			(width 0)
+			(type default)
+		)
+	)
+	(wire
+		(pts
 			(xy 459.74 449.58) (xy 468.63 449.58)
 		)
@@
 	(wire
 		(pts
+			(xy 636.27 328.93) (xy 636.27 336.55)
+		)
+		(stroke
+			(width 0)
+			(type default)
+		)
+	)
+	(wire
+		(pts
 			(xy 673.1 464.82) (xy 695.96 464.82)
 		)
@@
 	)
 	(label "GND"
-		(at 229.87 146.05 0)
+		(at 231.14 146.05 0)
 		(effects
 			(font
@@
 	)
 	(label "M38_P44"
-		(at 631.19 334.01 270)
+		(at 604.52 340.36 0)
 		(effects
 			(font
 				(size 1.27 1.27)
 			)
-			(justify right bottom)
+			(justify left bottom)
 		)
 	)
@@
 	)
 	(label "J13_53"
-		(at 227.33 133.35 0)
+		(at 228.6 133.35 0)
 		(effects
 			(font
@@
 		)
 	)
-	(label "R262_1"
+	(label "KB_SPKUP_DN"
 		(at 340.36 227.33 180)
 		(effects
@@
 	)
 	(label "M38_P46"
-		(at 636.27 334.01 270)
+		(at 604.52 336.55 0)
 		(effects
 			(font
 				(size 1.27 1.27)
 			)
-			(justify right bottom)
+			(justify left bottom)
 		)
 	)
@@
 	)
 	(symbol
+		(lib_id "power:GND")
+		(at 118.11 189.23 0)
+		(unit 1)
+		(exclude_from_sim no)
+		(in_bom yes)
+		(on_board yes)
+		(dnp no)
+		(fields_autoplaced yes)
+		(property "Reference" "#PWR0248"
+			(at 118.11 195.58 0)
+			(effects
+				(font
+					(size 1.27 1.27)
+				)
+				(hide yes)
+			)
+		)
+		(property "Value" "GND"
+			(at 118.11 194.31 0)
+			(effects
+				(font
+					(size 1.27 1.27)
+				)
+			)
+		)
+		(property "Footprint" ""
+			(at 118.11 189.23 0)
+			(effects
+				(font
+					(size 1.27 1.27)
+				)
+				(hide yes)
+			)
+		)
+		(property "Datasheet" ""
+			(at 118.11 189.23 0)
+			(effects
+				(font
+					(size 1.27 1.27)
+				)
+				(hide yes)
+			)
+		)
+		(property "Description" "Power symbol creates a global label with name \"GND\" , ground"
+			(at 118.11 189.23 0)
+			(effects
+				(font
+					(size 1.27 1.27)
+				)
+				(hide yes)
+			)
+		)
+		(pin "1"
+		)
+		(instances
+			(project "PC110"
+				(path "/45c7911f-b027-440e-9e3e-77a146b41944/00000000-0000-0000-0000-0000638712fb"
+					(reference "#PWR0248")
+					(unit 1)
+				)
+			)
+		)
+	)
+	(symbol
 		(lib_id "Device:R")
 		(at 673.1 309.88 270)
@@
 		(dnp no)
 		(property "Reference" "U6"
-			(at 689.61 350.4498 0)
+			(at 681.99 345.694 0)
 			(effects
 				(font
@@
 		)
 		(property "Value" "M38224M6HP"
-			(at 654.05 379.222 0)
+			(at 686.816 347.726 0)
 			(effects
 				(font
@@
 					(unit 1)
 				)
+			)
+		)
+	)
+	(symbol
+		(lib_id "PCM_Elektuur:C")
+		(at 118.11 181.61 0)
+		(unit 1)
+		(exclude_from_sim no)
+		(in_bom yes)
+		(on_board yes)
+		(dnp no)
+		(fields_autoplaced yes)
+		(property "Reference" "C226"
+			(at 121.92 180.3399 0)
+			(effects
+				(font
+					(size 1.27 1.27)
+				)
+				(justify left)
+			)
+		)
+		(property "Value" "1uF"
+			(at 121.92 182.8799 0)
+			(effects
+				(font
+					(size 1.27 1.27)
+				)
+				(justify left)
+			)
+		)
+		(property "Footprint" ""
+			(at 118.11 181.61 0)
+			(effects
+				(font
+					(size 1.27 1.27)
+				)
+				(hide yes)
+			)
+		)
+		(property "Datasheet" ""
+			(at 118.11 181.61 0)
+			(effects
+				(font
+					(size 1.27 1.27)
+				)
+				(hide yes)
+			)
+		)
+		(property "Description" "capacitor, non-polarized/bipolar"
+			(at 118.11 181.61 0)
+			(effects
+				(font
+					(size 1.27 1.27)
+				)
+				(hide yes)
+			)
+		)
+		(property "Indicator" "+"
+			(at 116.84 178.435 0)
+			(effects
+				(font
+					(size 1.27 1.27)
+				)
+				(hide yes)
+			)
+		)
+		(property "Rating" "V"
+			(at 117.475 184.785 0)
+			(effects
+				(font
+					(size 1.27 1.27)
+				)
+				(justify right)
+				(hide yes)
+			)
+		)
+		(pin "1"
+		)
+		(pin "2"
+		)
+		(instances
+			(project "PC110"
+				(path "/45c7911f-b027-440e-9e3e-77a146b41944/00000000-0000-0000-0000-0000638712fb"
+					(reference "C226")
+					(unit 1)
+				)

Commit message: Add files via upload
Parts:
- removed C56, C57: 100nF, symbol Device:C
- removed C59: 10nF, symbol Device:C
- removed C62: 120nF, symbol Device:C
- removed D14, D15, D31, D34, D42, D43: N, symbol Device:D_Dual_CommonCathode_AKA
- removed D16, D18, D22, D30: 3D, symbol Device:D_Dual_CommonCathode_AKA
- removed R79, R88: 0, symbol Device:R
- removed R91: 470k, symbol Device:R
- removed U16: QC01, symbol PC110:QC01
- removed U17: 3E00, symbol PC110:QC01
- added D14, D15, D17, D31, D42, D43: N, symbol PC110:3D_Diode
- added D16, D18, D22: 3D, symbol PC110:D3_PC110
- added D30: 3D, symbol PC110:3D_Diode
- added R87: 100k, symbol Device:R
- added U20: 7W14, symbol 74xGxx:74LVC3G14
Connections:
- net D4_3: now also D4.2 (K); no longer D4.3 (K)
- net GND: now also Q7.2 (E)
- net KB_RESET#: now also D16.1 (A), D16.3 (A)
- net M38_P71: now also D4.3 (A); no longer D4.2 (A)
- net PWRGD_shift_buff: now also D14.3, D15.3, U20.7
- net Pluto_72: now also D30.1, D30.2
- net Pluto_73: now also D31.1, D31.2
- net RESET: now also D18.1 (A), D18.3 (A)
- net U103_NAND_of_U53_1CLK_and_U53_1Q#: now also D17.2
- net at D46.2 (K): no longer R286.1
- net at D46.3 (A): now also R286.1
- net at U32.9 (Q): now also D31.3
- net YellowWire2_1: now reaches C51.1 (+), D6.1 (A), D7.3 (K), R68.2
- net at R287.2, U52.2: now also D42.1, D42.2, D43.1, D43.2
- net at R254.1: now also D17.3
- net at Q10.2 (E): now also D15.1
- net at R95.1: now also D15.2
- net at R93.1: now also D14.1
- net at Q9.2 (E): now also D14.2
- net at U5.4: now also D42.3
- net at C245.1 (+), F1.2, Q5.2 (E): now also D22.2 (K)
- net at U17.4: now also D16.2 (K)
- net at U30.9 (Q), U32.11 (C): now also D17.1
- net at R313.1: now also D22.1 (A), D22.3 (A)
- net at Q7.1 (B): now also R87.1
- net at U32.5 (Q): now also D30.3
- net at U15.4, U17.2: now also D18.2 (K)
- net at U5.2: now also D43.3
- net J5_6_Yellow renamed YellowWire2_3
- net YellowWire1_2 renamed YellowWire1_1
- new net PWRGD_shift: R87.2, U20.1
- no-connect marks 19 -> 17
Other:
- moved on the sheet: C231, C61, C96, C98, C99, Q10, Q11, Q12, Q13, Q26, Q7, Q9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

Commit message: Add files via upload
Parts:
- removed D4, D46: N, symbol Device:D_Dual_CommonCathode_AKA
- added C218: 150nF, symbol PCM_Elektuur:C
- added C224: 10nF, symbol PCM_Elektuur:C
- added D4, D45, D46, D49: N, symbol PC110:3D_Diode
- added D41, D47: 24, symbol Device:D
- added Q28: 8LR, symbol Simulation_SPICE:NPN
- added R260: 133k, symbol Device:R
- added R266: 50k, symbol Device:R
- added R271: DNP, symbol Device:R
- added R276: 33k, symbol Device:R
- added R281: 10k, symbol Device:R
- added U50, U55: ~, symbol PC110:3T01
Connections:
- net D4_3: now also D4.3
- net GND: now also C218.2 (-), C224.2 (-), D41.1 (K), D47.1 (K), Q28.3 (E), R271.2, U50.3 (GND), U55.3 (GND)
- net M38_P71: now also D4.2
- net R284_2: now also C218.1 (+), R266.2, R281.1
- net YellowWire1_1: now also Q28.1 (C)
- net at R286.1: now also D46.2
- net at R278.1, U5.9: now also U55.1 (OUT)
- net Q49_1 renamed D46_1
- net D46_1: now also D46.1
- new net: D41.2 (A), R260.2, R266.1, R271.1, U50.2 (VDD)
- new net: C224.1 (+), D47.2 (A), R281.2, U55.2 (VDD)
- new net: Q28.2 (B), R260.1, U50.1 (OUT)
- new net: D45.3, D46.3, D49.3, R276.1
- new net Pluto_50: R276.2
- no-connect marks 17 -> 21
Other:
- moved on the sheet: C226, C228, C229, C231, C245, C46, C47, C49, C51, C55, C58, C60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

Commit message: Add files via upload
Parts:
- added C179: 1nF, symbol PCM_Elektuur:C
- added C190, C222: 10nF, symbol PCM_Elektuur:C
- added C221: 150nF, symbol PCM_Elektuur:C
- added D37: N, symbol PC110:3D_Diode
- added D38: 40, symbol Device:D
- added D44: 83, symbol Device:D
- added D48: A2, symbol Device:D
- added D50: 26, symbol Device:D
- added D51: C6, symbol Device:D
- added L15: 1.5uH, symbol PCM_Elektuur:L
- added Q20: 7C, symbol Simulation_SPICE:PNP
- added Q21, Q23: 8B, symbol Simulation_SPICE:NPN
- added Q22: YQ, symbol Simulation_SPICE:NPN
- added R232, R237: 10k, symbol Device:R
- added R239: 56, symbol Device:R
- added R240, R397: 47k, symbol Device:R
Connections:
- net D18_2_3: now also D37.1, D37.2, R397.2
- net D28_1: now also C221.1 (+), D50.2 (A)
- net F65_ENAVEE: now also D37.3, R237.1
- net GND: now also C179.2 (-), C190.2 (-), C221.2 (-), C222.2 (-), Q21.3 (E), Q22.3 (E), Q23.3 (E)
- net PNET1: now also D44.2 (A)
- net PNET5: now also D48.2 (A)
- net Q43_2: now also C222.1 (+), D51.2 (A), Q20.3 (E)
- net at D49.1: now also D50.1 (K)
- net at D49.2: now also D51.1 (K)
- net at D45.1: now also D44.1 (K)
- net at D45.2: now also D48.1 (K)
- net YellowWire1_1 renamed YellowWire1
- new net: Q22.1 (C), R239.1
- new net: Q22.2 (B), Q23.1 (C), R240.1
- new net: D38.2 (A), R232.1
- new net: Q20.2 (B), R232.2
- new net: D38.1 (K), Q21.1 (C)
- new net: Q21.2 (B), Q23.2 (B), R237.2
- new net: L15.1 (+), Q20.1 (C), R239.2, R240.2
- new net EN_LCD_VAA: R397.1
- new net LCD_VAA: C179.1 (+), C190.1 (+), L15.2 (-)
Other:
- moved on the sheet: D45, R276

Commit message: Add files via upload
Parts:
- renumbered Q75 to Q39, Q72 to Q40, Q73 to Q41, Q74 to Q42, R384 to R386, R386 to R388
Changed lines of the file:
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@@
 		(on_board yes)
 		(dnp no)
-		(property "Reference" "R384"
+		(property "Reference" "R386"
 			(at 532.638 437.896 90)
 			(effects
@@
 			(project "PC110"
 				(path "/45c7911f-b027-440e-9e3e-77a146b41944/00000000-0000-0000-0000-0000638712fb"
-					(reference "R384")
+					(reference "R386")
 					(unit 1)
 				)
@@
 		(on_board yes)
 		(dnp no)
-		(property "Reference" "R386"
+		(property "Reference" "R388"
 			(at 532.638 491.236 90)
 			(effects
@@
 			(project "PC110"
 				(path "/45c7911f-b027-440e-9e3e-77a146b41944/00000000-0000-0000-0000-0000638712fb"
-					(reference "R386")
+					(reference "R388")
 					(unit 1)
 				)
@@
 		(on_board yes)
 		(dnp no)
-		(property "Reference" "Q73"
+		(property "Reference" "Q41"
 			(at 548.64 452.1199 0)
 			(effects
@@
 			(project ""
 				(path "/45c7911f-b027-440e-9e3e-77a146b41944/00000000-0000-0000-0000-0000638712fb"
-					(reference "Q73")
+					(reference "Q41")
 					(unit 1)
 				)
@@
 		(on_board yes)
 		(dnp no)
-		(property "Reference" "Q75"
+		(property "Reference" "Q39"
 			(at 548.64 490.2201 0)
 			(effects
@@
 			(project "PC110"
 				(path "/45c7911f-b027-440e-9e3e-77a146b41944/00000000-0000-0000-0000-0000638712fb"
-					(reference "Q75")
+					(reference "Q39")
 					(unit 1)
 				)
@@
 		(on_board yes)
 		(dnp no)
-		(property "Reference" "Q74"
+		(property "Reference" "Q42"
 			(at 548.64 505.4599 0)
 			(effects
@@
 			(project "PC110"
 				(path "/45c7911f-b027-440e-9e3e-77a146b41944/00000000-0000-0000-0000-0000638712fb"
-					(reference "Q74")
+					(reference "Q42")
 					(unit 1)
 				)
@@
 		(on_board yes)
 		(dnp no)
-		(property "Reference" "Q72"
+		(property "Reference" "Q40"
 			(at 548.64 436.8801 0)
 			(effects
@@
 			(project ""
 				(path "/45c7911f-b027-440e-9e3e-77a146b41944/00000000-0000-0000-0000-0000638712fb"
-					(reference "Q72")
+					(reference "Q40")
 					(unit 1)
 				)

Commit message: Add files via upload
Other:
- company: (none) -> Recreated by: Ahmad Byagowi
Changed lines of the file:
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@@
 	(title_block
 		(title "PC110")
+		(company "Recreated by: Ahmad Byagowi")
 	)
 	(text "5v switched on via PWRGD"

Commit message: Add files via upload
Connections:
- net J13_53 renamed Dock_PWR_IN-
- net Dock_PWR_IN-: no longer J5.5 (Pin_5)
- new net Dock_PWR_IN: J5.5 (Pin_5)
Changed lines of the file:
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@@
 	(wire
 		(pts
-			(xy 260.35 128.27) (xy 270.51 128.27)
+			(xy 260.35 128.27) (xy 276.86 128.27)
 		)
 		(stroke
@@
 	(wire
 		(pts
-			(xy 229.87 130.81) (xy 238.76 130.81)
+			(xy 219.71 130.81) (xy 238.76 130.81)
 		)
 		(stroke
@@
 		)
 	)
-	(label "J13_53"
-		(at 229.87 130.81 0)
+	(label "Dock_PWR_IN"
+		(at 219.71 130.81 0)
 		(effects
 			(font
@@
 		)
 	)
-	(label "J13_53"
+	(label "Dock_PWR_IN-"
 		(at 262.89 128.27 0)
 		(effects

Commit message: Add part numbers to some SMT parts
Parts:
- removed D16, D18, D22: 3D, symbol PC110:D3_PC110
- removed D30: 3D, symbol PC110:3D_Diode
- removed D38: 40, symbol Device:D
- removed D41, D47: 24, symbol Device:D
- removed D44: 83, symbol Device:D
- removed D48: A2, symbol Device:D
- removed D50: 26, symbol Device:D
- removed D51: C6, symbol Device:D
- added D16, D18, D22, D30: RB715F, symbol Device:D_Schottky_Dual_CommonCathode_AKA
- added D38, D41, D44, D47, D48, D50, D51: ?, symbol Device:D_Zener_Small_Filled
- D10, D13: value K -> DA204U; Topmark (none) -> K
- D14, D15, D17, D31, D37, D4, D42, D43, D45, D46, D49: value N -> DAN222; Topmark (none) -> N
- D6, D7: value Q -> SB05-03; Topmark (none) -> Q
- Q11, Q13: value IS6 -> 2SA1881-6; Topmark (none) -> IS6
- U13: value 8C01 -> RN5VD? 8C01
- X1: value 245759 -> 2.45759MHz
Connections:
- net D28_1: now also D50.1 (K)
- net GND: now also D41.2 (A), D47.2 (A)
- net KB_RESET#: now also D16.1 (A), D16.3 (A)
- net PNET1: now also D44.1 (K)
- net PNET5: now also D48.1 (K)
- net Pluto_72: now also D30.1 (A), D30.3 (A)
- net Q43_2: now also D51.1 (K)
- net RESET: now also D18.1 (A), D18.3 (A)
- net at R260.2, R266.1, R271.1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: now also D41.1 (K)
- net at C224.1 (+), R281.2, U55.2 (VDD): now also D47.1 (K)
- net at C245.1 (+), F1.2, Q5.2 (E): now also D22.2 (K)
- net at R232.1: now also D38.1 (K)
- net at U15.4, U17.2: now also D18.2 (K)
- net at Q21.1 (C): now also D38.2 (A)
- net at D49.1: now also D50.2 (A)
- net at R313.1: now also D22.1 (A), D22.3 (A)
- net at D49.2: now also D51.2 (A)
- net at U17.4: now also D16.2 (K)
- net at U32.5 (Q): now also D30.2 (K)
- net at D45.1: now also D44.2 (A)
- net at D45.2: now also D48.2 (A)
