File: PCB/Mainboard/Chipset.kicad_sch (KiCad schematic)
At the start: 9 parts, among them U13 OPTi_82C895, U4 OPTi_82C602, Y1 32768Hz

Commit message: Add files via upload
Parts:
- removed BT1: CR2032, My_Components:Battery_Holder_CR2032_Universal, symbol Device:Battery_Cell
- removed C8, C9: 5pF, Capacitor_SMD:C_0603_1608Metric_Pad1.08x0.95mm_HandSolder, symbol Device:C
- removed R12: 51, Resistor_SMD:R_0612_1632Metric_Pad1.18x3.40mm_HandSolder, symbol Device:R
- removed R13: 1k, Resistor_SMD:R_0612_1632Metric_Pad1.18x3.40mm_HandSolder, symbol Device:R
- removed R30: 33, Resistor_SMD:R_0612_1632Metric_Pad1.18x3.40mm_HandSolder, symbol Device:R
- removed U13: OPTi_82C895, Package_QFP:PQFP-208_28x28mm_P0.5mm, symbol my_components:OPTi_82C895
- removed U4: OPTi_82C602, Package_QFP:PQFP-100_14x20mm_P0.65mm, symbol my_components:OPTi_82C602
- removed Y1: 32768Hz, My_Components:Crystal_32K_Horiz, symbol Device:Crystal_Small
Connections:
- no-connect marks 3 -> 0

Commit message: Add files via upload
Parts:
- added U1: ~, symbol PC110:VL82C420

Commit message: Add files via upload
Parts:
- removed U1: ~, symbol PC110:VL82C420
- added J4: connector-4, symbol Connector_Generic:Conn_01x04
- added U61: VL82C420FC5, symbol PC110:VL82C420
Connections:
- new net CMOS_BATT+: J4.3 (Pin_3)
- new net CMOS_BATT_Sense: J4.4 (Pin_4)
- new net GND: J4.2 (Pin_2)
- new net MIC_J17: J4.1 (Pin_1)

Commit message: Add files via upload
Parts:
- added C35: 100F, symbol Device:C
- added C69: 1nF, symbol Device:C
- added C70, C82: 100nF, symbol Device:C
- added C8: 150nF, symbol Device:C
- added C80: 1uF, symbol Device:C
- added D21: 3D, symbol Device:D_Dual_CommonCathode_AKA
- added D23: 92, symbol Device:D
- added D58: K, symbol Device:D_Dual_Series_KAC
- added R116: 100k, symbol Device:R
- added R248: 470k, symbol Device:R
- added R308: 10, symbol Device:R
- added R31: 300, symbol Device:R
- added R96: 47k, symbol Device:R
- added U19: 74W126, symbol 74xGxx:74AUC2G126
- added U7: HD151015, symbol PC110:HD151015
Connections:
- net CMOS_BATT+: now also C8.2, R31.1
- net GND: now also C35.1, C69.1, C70.1, C8.1, C80.1, C82.1, D23.2 (A), U19.4 (GND), U19.5, U19.7, U7.12 (GND), U7.13 (GND), U7.23 (G#)
- net at U61.M11 (PS/RCLR#): now also R116.1
- net UNKNOWN2: now reaches U61.N12 (UNKNOWN2)
- net UNKNOWN2: now also U7.5 (A2)
- net Bowman1: now reaches U61.N9 (Bowman1)
- net Bowman2: now reaches U61.P9 (Bowman2)
- net at U61.R10 (PWRGD): now also R96.2, U19.2
- net UNKNOWN1: now reaches U61.R13 (UNKNOWN1)
- net UNKNOWN1: now also U7.4 (A1)
- net Bowman3: now reaches U61.R9 (Bowman3)
- net RTCBAT: now reaches U61.T11 (RTCBAT)
- net RTCBAT: now also C70.2, C80.2, C82.2, D21.2 (K), R116.2, R248.1, U19.8 (VCC)
- net Bowman5: now reaches U61.T13 (Bowman5)
- net Bowman5: now also U7.3 (A0)
- net Bowman4: now reaches U61.T9 (Bowman4)
- new net: D21.1 (A), D23.1 (K), R308.1
- new net: D58.1 (K), R308.2
- new net: D21.3 (A), R31.2
- new net PNET1: R96.1, U7.1 (VCCA), U7.2 (DIR)
- new net PNET5: C35.2, U7.24 (VCCB)
- new net PWRGD: U19.6
- new net VCC: C69.2, D58.2 (A), U19.1
- no-connect marks 0 -> 4
Other:
- moved on the sheet: J4

Commit message: Add files via upload
Parts:
- added R258: 33, symbol Device:R
Connections:
- net U61_RTCBAT_470K: now reaches R248.2
- net U61_RTCBAT_470K: now also U61.P10 (RTCBAT_Sense)
- net CPU_STPCLK#: now reaches U61.E1 (CPUSTPCLK#)
- net CPU_SMIACT#: now reaches U61.F1 (CPUSMIACT#)
- net CPU_SMI#: now reaches U61.F2 (CPUSMI#)
- net Chipset_CPU_CLK_Sense: now reaches U61.J1 (CPUCLKSENS)
- net at U61.J3 (CPUCLK33): now also R258.1
- net Chipset_CPU_CLK: now reaches U61.K1 (CPUCLK)
- net Chipset_CPU_CLK: now also R258.2
- net YMF_VSS_Res: now reaches U61.P12 (PCMCIA_RELATED)
- net PCMCIA_CS: now reaches U61.R14 (PCMCIA_CS)
Other:
- moved on the sheet: R248

Commit message: Add files via upload
Parts:
- added R49: 100k, symbol Device:R
Connections:
- net GND: now also R49.2
- net at U61.P13 (PWRGD_P13): now also U7.6 (A3), R49.1
- net U71_OR1_IN2: now reaches U7.19 (B3)
- net Bowman5_Buff: now reaches U7.22 (B0)
Other:
- moved on the sheet: C35, U7

Commit message: Add files via upload
Connections:
- net KB_SRDY#_shift: now reaches U7.18 (B4)
- net KB_SRDY#: now reaches U7.7 (A4)
- net KB_SCLK#: now reaches U7.8 (A5)
Changed lines of the file:
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@@
+	(wire
+		(pts
+			(xy 143.51 358.14) (xy 160.02 358.14)
+		)
+		(stroke
+			(width 0)
+			(type default)
+		)
+	)
 	(wire
 		(pts
@@
 	(wire
 		(pts
+			(xy 143.51 360.68) (xy 160.02 360.68)
+		)
+		(stroke
+			(width 0)
+			(type default)
+		)
+	)
+	(wire
+		(pts
 			(xy 39.37 242.57) (xy 55.88 242.57)
 		)
@@
 		(pts
 			(xy 152.4 337.82) (xy 161.29 337.82)
+		)
+		(stroke
+			(width 0)
+			(type default)
+		)
+	)
+	(wire
+		(pts
+			(xy 93.98 358.14) (xy 114.3 358.14)
 		)
 		(stroke
@@
 		)
 	)
+	(label "KB_SRDY#_shift"
+		(at 95.25 358.14 0)
+		(effects
+			(font
+				(size 1.27 1.27)
+			)
+			(justify left bottom)
+		)
+	)
+	(label "KB_SRDY#"
+		(at 149.86 358.14 0)
+		(effects
+			(font
+				(size 1.27 1.27)
+			)
+			(justify left bottom)
+		)
+	)
 	(label "U61_RTCBAT_470K"
 		(at 187.96 260.35 0)
@@
 		)
 	)
+	(label "KB_SCLK#"
+		(at 149.86 360.68 0)
+		(effects
+			(font
+				(size 1.27 1.27)
+			)
+			(justify left bottom)
+		)
+	)

Commit message: Add files via upload
Parts:
- added J14: ~, symbol PC110:Debug1
- added R323: 1k, symbol Device:R
- added U58: EA, symbol 74xGxx:74AHC1G14
Connections:
- net GND: now also U58.3 (GND)
- net SA0: now reaches U61.E15 (SA0)
- net SA0: now also U7.11 (A8)
- net SA1: now reaches U61.E16 (SA1)
- net CPU_FLUSH#: now reaches U61.G1 (CPUFLUSH#)
- net CPU_INTR: now reaches U61.G2 (CPUINTR)
- net CPU_NMI: now reaches U61.G3 (CPUNMI)
- net FCS_IOCHRDY: now reaches U61.H14 (IOCHRDY)
- net FCS_IOCHRDY: now also R323.2
- net PCMCIA_ZEROWS#: now reaches U61.H15 (ZEROWS#)
- net PCMCIA_CLK: now reaches U61.H16 (PCMCIA_CLK)
- net CPU_EADS#: now reaches U61.H2 (CPUEADS#)
- net CPU_A20M#: now reaches U61.H3 (CPUA20M#)
- net CPU_MIO#: now reaches U61.H4 (CPUMIO#)
- net CPU_BE3#: now reaches U61.K2 (CPUBE3#)
- net CPU_BE2#: now reaches U61.K3 (CPUBE2#)
- net CPU_BE0#: now reaches U61.L1 (CPUBE0#)
- net CPU_WR#: now reaches U61.L2 (CPUWR#)
- net CPU_HLDA: now reaches U61.L3 (CPUHLDA)
- net CPU_BE1#: now reaches U61.L4 (CPUBE1#)
- net CPU_AHOLD: now reaches U61.L5 (CPUAHOLD)
- net CPU_HOLD: now reaches U61.M1 (CPUHOLD)
- net CPU_KEN#: now reaches U61.M2 (CPUKEN#)
- net CPU_BRDY#: now reaches U61.M3 (CPUBRDY#)
- net CPU_A10: now reaches U61.M6 (CPUA10)
- net CPU_BLAST#: now reaches U61.N1 (CPUBLAST#)
- net at U61.N13 (RESET): now also U58.2
- net CPU_ADS#: now reaches U61.N2 (CPUADS#)
- net CPU_A31: now reaches U61.N3 (CPUA31)
- net CPU_A23: now reaches U61.N4 (CPUA23)
- net CPU_A16: now reaches U61.N5 (CPUA16)
- net CPU_A6: now reaches U61.N6 (CPUA6)
- net CPU_A2: now reaches U61.N7 (CPUA2)
- net CPU_A25: now reaches U61.P1 (CPUA25)
- net CPU_A24: now reaches U61.P2 (CPUA24)
- net CPU_A20: now reaches U61.P3 (CPUA20)
- net CPU_A17: now reaches U61.P4 (CPUA17)
- net CPU_A13: now reaches U61.P5 (CPUA13)
- net CPU_A9: now reaches U61.P6 (CPUA9)
- net CPU_A5: now reaches U61.P7 (CPUA5)
- net CPU_A22: now reaches U61.R1 (CPUA22)
- net Chipset_CLK: now reaches U61.R15 (CLOCK_IN)
- net Chipset_2XCPU_CLK: now reaches U61.R2 (CPU2XCLK)
- net CPU_A19: now reaches U61.R3 (CPUA19)
- net CPU_A15: now reaches U61.R4 (CPUA15)
- net CPU_A12: now reaches U61.R5 (CPUA12)
- net CPU_A8: now reaches U61.R6 (CPUA8)
- net CPU_A4: now reaches U61.R7 (CPUA4)
- net at U61.T14 (TP1): now also J14.1
- net CPU_A21: now reaches U61.T2 (CPUA21)
- net CPU_A18: now reaches U61.T3 (CPUA18)
- net CPU_A14: now reaches U61.T4 (CPUA14)
- net CPU_A11: now reaches U61.T5 (CPUA11)
- net CPU_A7: now reaches U61.T6 (CPUA7)
- net CPU_A3: now reaches U61.T7 (CPUA3)
- net Pluto_EN_IRDA: now reaches U7.10 (A7)
- net YMF_SA0_A0: now reaches U7.14 (B8)
- net Enable_IRDA_Buf: now reaches U7.15 (B7)
- net PWRGD_shift: now reaches U7.16 (B6)
- new net FCS_RESET: U58.4
- new net PNET7: R323.1, U58.5 (VCC)
- no-connect marks 4 -> 35
Other:
- moved on the sheet: C35, C69, C70, C8, C80, C82, D21, D23, D58, J4, R116, R248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
