File: PCB/Mainboard/Chipset.kicad_sch (KiCad schematic)
At the start: 23 parts, among them J4 connector-4, U19 74W126, U58 EA, U61 VL82C420FC5, U7 HD151015

Commit message: Add files via upload
Connections:
- net KB_SPKDN: now reaches U61.T12 (KBSPKDN)
Changed lines of the file:
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@@
+	(wire
+		(pts
+			(xy 482.6 302.26) (xy 504.19 302.26)
+		)
+		(stroke
+			(width 0)
+			(type default)
+		)
+	)
 	(wire
 		(pts
@@
 		(effects
 			(font
+				(size 1.27 1.27)
+			)
+			(justify left bottom)
+		)
+	)
+	(label "KB_SPKDN"
+		(at 492.76 302.26 0)
+		(effects
+			(font

Commit message: Add files via upload
Other:
- moved on the sheet: J14
Changed lines of the file:
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@@
 	(wire
 		(pts
-			(xy 209.55 273.05) (xy 212.09 273.05)
+			(xy 184.15 273.05) (xy 212.09 273.05)
 		)
 		(stroke
@@
 	(symbol
 		(lib_id "PC110:Debug1")
-		(at 204.47 273.05 180)
+		(at 179.07 273.05 180)
 		(unit 1)
 		(exclude_from_sim no)
@@
 		(dnp no)
 		(property "Reference" "J14"
-			(at 204.47 269.24 0)
+			(at 179.07 269.24 0)
 			(effects
 				(font
@@
 		)
 		(property "Value" "~"
-			(at 204.47 269.24 0)
+			(at 179.07 269.24 0)
 			(effects
 				(font
@@
 		)
 		(property "Footprint" ""
-			(at 204.47 273.05 0)
+			(at 179.07 273.05 0)
 			(effects
 				(font
@@
 		)
 		(property "Datasheet" ""
-			(at 204.47 273.05 0)
+			(at 179.07 273.05 0)
 			(effects
 				(font
@@
 		)
 		(property "Description" ""
-			(at 204.47 273.05 0)
+			(at 179.07 273.05 0)
 			(effects
 				(font

Commit message: Add files via upload
Parts:
- added R318, R322, R324, R326: 33, symbol Device:R
Connections:
- net PWRGD: now also U7.9 (A6)
- net at U61.F13 (MEMR#): now also R322.2
- net at U61.G14 (MEMW#): now also R324.2
- net AEN: now reaches U61.G16 (AEN)
- net at U61.J14 (IOW#): now also R318.2
- net at U61.J15 (IOR#): now also R326.2
- net IOCS16#: now reaches U61.J16 (IOCS16#)
- net KB_SCLK_shift: now reaches U7.17 (B5)
- new net IOR#: R326.1
- new net IOW#: R318.1
- new net MEMR#: R322.1
- new net MEMW#: R324.1

Commit message: Add files via upload
Parts:
- added R329, R333, R334, R335, R337, R338, R342, R343, R345, R346, R347, R352: 33, symbol Device:R
Connections:
- net at U61.A10 (RAMA9): now also R329.1
- net at U61.A11 (RAMA6): now also R343.1
- net CPU_D11: now reaches U61.A2 (D11)
- net CPU_D14: now reaches U61.A3 (D14)
- net CPU_D18: now reaches U61.A4 (D18)
- net CPU_D22: now reaches U61.A5 (D22)
- net CPU_D26: now reaches U61.A6 (D26)
- net CPU_D30: now reaches U61.A7 (D30)
- net CPU_D10: now reaches U61.B1 (D10)
- net at U61.B10 (RAMA8): now also R347.1
- net at U61.B11 (RAMA5): now also R333.1
- net at U61.B12 (RAMA2): now also R342.1
- net CPU_D13: now reaches U61.B3 (D13)
- net CPU_D17: now reaches U61.B4 (D17)
- net CPU_D21: now reaches U61.B5 (D21)
- net CPU_D25: now reaches U61.B6 (D25)
- net CPU_D29: now reaches U61.B7 (D29)
- net CPU_D7: now reaches U61.C1 (D7)
- net at U61.C11 (RAMA4): now also R334.1
- net at U61.C12 (RAMA0): now also R346.1
- net CPU_D8: now reaches U61.C2 (D8)
- net CPU_D9: now reaches U61.C3 (D9)
- net CPU_D15: now reaches U61.C4 (D15)
- net CPU_D19: now reaches U61.C5 (D19)
- net CPU_D24: now reaches U61.C6 (D24)
- net CPU_D28: now reaches U61.C7 (D28)
- net at U61.C9 (RAMA11): now also R335.1
- net CPU_D3: now reaches U61.D1 (D3)
- net at U61.D10 (RAMA10): now also R345.1
- net at U61.D11 (RAMA7): now also R352.1
- net CPU_D4: now reaches U61.D2 (D4)
- net CPU_D6: now reaches U61.D3 (D6)
- net CPU_D12: now reaches U61.D4 (D12)
- net CPU_D16: now reaches U61.D5 (D16)
- net CPU_D27: now reaches U61.D6 (D27)
- net CPU_D31: now reaches U61.D7 (D31)
- net at U61.E11 (RAMA3): now also R337.1
- net at U61.E12 (RAMA1): now also R338.1
- net CPU_D0: now reaches U61.E2 (D0)
- net CPU_D2: now reaches U61.E3 (D2)
- net CPU_D5: now reaches U61.E4 (D5)
- net CPU_D1: now reaches U61.E5 (D1)
- net CPU_D23: now reaches U61.E6 (D23)
- net CPU_D20: now reaches U61.F6 (D20)
- net SD4_Bus: now reaches U61.L12 (SD4)
- net SD0_Bus: now reaches U61.L13 (SD0)
- net SD3_Bus: now reaches U61.L14 (SD3)
- net SD2_Bus: now reaches U61.L15 (SD2)
- net SD1_Bus: now reaches U61.L16 (SD1)
- net SD7_Bus: now reaches U61.M12 (SD7)
- net SD10_Bus: now reaches U61.M13 (SD10)
- net SD6_Bus: now reaches U61.M15 (SD6)
- net SD5_Bus: now reaches U61.M16 (SD5)
- net SD11_Bus: now reaches U61.N14 (SD11)
- net SD9_Bus: now reaches U61.N15 (SD9)
- net SD8_Bus: now reaches U61.N16 (SD8)
- net SD15_Bus: now reaches U61.P14 (SD14)
- net SD15_Bus: now also U61.R16 (SD15)
- net SD13_Bus: now reaches U61.P15 (SD13)
- net SD12_Bus: now reaches U61.P16 (SD12)
- new net RAM_A0: R346.2
- new net RAM_A1: R338.2
- new net RAM_A10: R345.2
- new net RAM_A11: R335.2
- new net RAM_A2: R342.2
- new net RAM_A3: R337.2
- new net RAM_A4: R334.2
- new net RAM_A5: R333.2
- new net RAM_A6: R343.2
- new net RAM_A7: R352.2
- new net RAM_A8: R347.2
- new net RAM_A9: R329.2
Other:
- moved on the sheet: C35, C69, C70, C8, C80, C82, D21, D23, D58, J14, J4, R116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

Commit message: Add files via upload
Parts:
- added R400, R402, R403, R405: DNP, symbol Device:R
- added R401, R404, R406: 100k, symbol Device:R
Connections:
- net GND: now also R402.1, R404.1, R405.1, R406.1
- net PNET1: now also R400.2, R401.2, R403.2
- net RAM_A0: now also R400.1, R404.2
- net RAM_A1: now also R403.1, R406.2
- net RAM_A2: now also R401.1, R402.2
- net RAM_A3: now also R405.2
- net RAM_RAS3: now reaches U61.A13 (RAS3)
- net RAM_UCASL#: now reaches U61.A8 (UCASL#)
- net RAM_LCASU#: now reaches U61.A9 (LCASU#)
- net RAM_RAS2: now reaches U61.B13 (RAS2)
- net RAM_RAMWE#: now reaches U61.B8 (RAMWE#)
- net RAM_RAS1: now reaches U61.C13 (RAS1)
- net RAM_LCASL#: now reaches U61.D8 (LCASL#)
- net RAM_UCASU#: now reaches U61.D9 (UCASU#)

Commit message: Add files via upload
Parts:
- added C250, C251: 18pF, symbol Device:C
- added R246, R249: 47k, symbol Device:R
- added X3: 32768, symbol Device:Crystal_GND23
- renumbered R258 to R251
Connections:
- net GND: now also U61.A1 (GND), U61.A16 (GND), U61.C10 (GND), U61.C8 (GND), U61.F11 (GND), U61.H13 (GND), U61.J2 (GND), U61.K14 (GND), U61.P8 (GND), U61.T1 (GND), U61.T16 (GND), C250.2, C251.2
- net PNET1: now also R246.1, R249.1
- net Chipset_SA16: now reaches U61.B16 (SA16)
- net LA18: now reaches U61.C15 (LA18)
- net LA19: now reaches U61.C16 (LA19)
- net LA17: now reaches U61.D13 (LA17)
- net LA20: now reaches U61.D14 (LA20)
- net LA22: now reaches U61.D15 (LA22)
- net LA23: now reaches U61.D16 (LA23)
- net LA21: now reaches U61.E13 (LA21)
- net PCMCIA_REFRESH: now reaches U61.E14 (REFRESH#)
- net PCMCIA_SBHE#: now reaches U61.F12 (SBHE#)
- net CPU_SRESET: now reaches U61.F4 (CPUSRESET#)
- net Chipset_FDC_TC: now reaches U61.G13 (FDCTC)
- net Chipset_BIOS_CE#: now reaches U61.G15 (BIOS_CE#)
- net CPU_RESET: now reaches U61.G4 (CPURESET)
- net CPU_DC#: now reaches U61.H1 (CPUDC#)
- net MEMCS16#: now reaches U61.J13 (MEMCS16#)
- net PCMCIA_BALE: now reaches U61.K15 (PCMCIA_BALE)
- net CPU_RDY#: now reaches U61.L6 (CPURDY#)
- net CPU_LDEV#: now reaches U61.M4 (CPULDEV#)
- net KB_RESET#: now reaches U61.N11 (KBRESET#)
- net at U61.N8 (PullDN): now also R249.2
- net at U61.P11 (RTCOSCO): now also C250.1, X3.4
- net at U61.R11 (RTCOSCI): now also C251.1, X3.1
- net at U61.R8 (PullDN): now also R246.2
- net Chipset_32KHz: now reaches U61.T10 (32KHz)
- net Chipset_Sound: now reaches U61.T15 (SPKR)
- no-connect marks 35 -> 37
Other:
- moved on the sheet: R251, R96

Commit message: Add files via upload
Parts:
- added C73: 120nF, symbol PCM_Elektuur:C
- added C75: 100nF, symbol PCM_Elektuur:C
- added C77, C81: 1nF, symbol PCM_Elektuur:C
Connections:
- net GND: now also C73.1 (+), C75.1 (+), C77.1 (+), C81.2 (-)
- net PNET1: now also U61.A12 (VCC), U61.B15 (VCC), U61.B2 (VCC), U61.B9 (VCC), U61.F14 (VCC), U61.J4 (VCC), U61.K4 (VCC), U61.M14 (VCC), U61.M5 (VCC), C73.2 (-), C75.2 (-), C77.2 (-)
- net PNET7: now also C81.1 (+)
- no-connect marks 37 -> 69
Other:
- moved on the sheet: C250, C251, C35, C69, C70, C8, C80, C82, D21, D23, D58, J14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

Commit message: Add files via upload
Other:
- company: (none) -> Recreated by: Ahmad Byagowi
Changed lines of the file:
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@@
 	(title_block
 		(title "PC110")
+		(company "Recreated by: Ahmad Byagowi")
 	)
 	(junction
