File: PCB/Mainboard/ASIC.kicad_sch (KiCad schematic)
At the start: 0 parts

Commit message: Add files via upload
Parts:
- added U21: Bowman, symbol PC110:Bowman
- added U35: Pluto, symbol PC110:Pluto

Commit message: Add files via upload
Connections:
- net PWRGD: now reaches U35.67 (PWRGD)
- net PWRGD: now also U21.47 (PWRGD)
- net Bowman5: now reaches U21.130 (Chipset_IO5)
- net Bowman2: now reaches U21.140 (Chipset_IO2)
- net Bowman3: now reaches U21.39 (Chipset_IO3)
- net Bowman1: now reaches U21.45 (Chipset_IO1)
- net Bowman4: now reaches U21.52 (Chipset_IO4)
Other:
- moved on the sheet: U21, U35
Changed lines of the file:
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@@
 		(title "PC110")
+	)
+	(wire
+		(pts
+			(xy 177.8 194.31) (xy 203.2 194.31)
+		)
+		(stroke
+			(width 0)
+			(type default)
+		)
+	)
+	(wire
+		(pts
+			(xy 248.92 107.95) (xy 270.51 107.95)
+		)
+		(stroke
+			(width 0)
+			(type default)
+		)
+	)
+	(wire
+		(pts
+			(xy 177.8 102.87) (xy 198.12 102.87)
+		)
+		(stroke
+			(width 0)
+			(type default)
+		)
+	)
+	(wire
+		(pts
+			(xy 177.8 95.25) (xy 198.12 95.25)
+		)
+		(stroke
+			(width 0)
+			(type default)
+		)
+	)
+	(wire
+		(pts
+			(xy 177.8 92.71) (xy 198.12 92.71)
+		)
+		(stroke
+			(width 0)
+			(type default)
+		)
+	)
+	(wire
+		(pts
+			(xy 177.8 97.79) (xy 198.12 97.79)
+		)
+		(stroke
+			(width 0)
+			(type default)
+		)
+	)
+	(wire
+		(pts
+			(xy 177.8 100.33) (xy 198.12 100.33)
+		)
+		(stroke
+			(width 0)
+			(type default)
+		)
+	)
+	(label "PWRGD"
+		(at 257.81 107.95 180)
+		(effects
+			(font
+				(size 1.27 1.27)
+			)
+			(justify right bottom)
+		)
+	)
+	(label "Bowman5"
+		(at 196.85 102.87 180)
+		(effects
+			(font
+				(size 1.27 1.27)
+			)
+			(justify right bottom)
+		)
+	)
+	(label "Bowman3"
+		(at 196.85 97.79 180)
+		(effects
+			(font
+				(size 1.27 1.27)
+			)
+			(justify right bottom)
+		)
+	)
+	(label "Bowman4"
+		(at 196.85 100.33 180)
+		(effects
+			(font
+				(size 1.27 1.27)
+			)
+			(justify right bottom)
+		)
+	)
+	(label "Bowman2"
+		(at 196.85 95.25 180)
+		(effects
+			(font
+				(size 1.27 1.27)
+			)
+			(justify right bottom)
+		)
+	)
+	(label "Bowman1"
+		(at 196.85 92.71 180)
+		(effects
+			(font
+				(size 1.27 1.27)
+			)
+			(justify right bottom)
+		)
+	)
+	(label "PWRGD"
+		(at 201.93 194.31 180)
+		(effects
+			(font
+				(size 1.27 1.27)
+			)
+			(justify right bottom)
+		)
 	)
 	(symbol
@@
 	(symbol
 		(lib_id "PC110:Bowman")
-		(at 153.67 138.43 0)
+		(at 128.27 146.05 0)
 		(unit 1)
 		(exclude_from_sim no)
@@
 		(on_board yes)
 		(dnp no)
-		(fields_autoplaced yes)
 		(property "Reference" "U21"
-			(at 169.7833 223.52 0)
+			(at 159.766 56.642 0)
 			(effects
 				(font
@@
 		)
 		(property "Value" "Bowman"
-			(at 169.7833 224.79 0)
+			(at 159.766 58.42 0)
 			(effects
 				(font
@@
 		)
 		(property "Footprint" ""
-			(at 153.67 138.43 0)
+			(at 128.27 146.05 0)
 			(effects
 				(font
@@
 		)
 		(property "Datasheet" ""
-			(at 153.67 138.43 0)
+			(at 128.27 146.05 0)
 			(effects
 				(font
@@
 		)
 		(property "Description" ""
-			(at 153.67 138.43 0)
-			(effects
-				(font
+			(at 128.27 146.05 0)
+			(effects
+				(font

Commit message: Add files via upload
Connections:
- net CF_CD2_Pluto: now reaches U35.26 (CF_CD2#)
- net CF_CD1_Pluto: now reaches U35.27 (CF_CD1#)
Other:
- moved on the sheet: U35
Changed lines of the file:
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@@
+	(wire
+		(pts
+			(xy 356.87 110.49) (xy 374.65 110.49)
+		)
+		(stroke
+			(width 0)
+			(type default)
+		)
+	)
 	(wire
 		(pts
 			(xy 177.8 102.87) (xy 198.12 102.87)
+		)
+		(stroke
+			(width 0)
+			(type default)
+		)
+	)
+	(wire
+		(pts
+			(xy 356.87 107.95) (xy 374.65 107.95)
 		)
 		(stroke
@@
 		)
 	)
+	(label "CF_CD1_Pluto"
+		(at 373.38 110.49 180)
+		(effects
+			(font
+				(size 1.27 1.27)
+			)
+			(justify right bottom)
+		)
+	)
 	(label "Bowman2"
 		(at 196.85 95.25 180)
@@
 		(effects
 			(font
+				(size 1.27 1.27)
+			)
+			(justify right bottom)
+		)
+	)
+	(label "CF_CD2_Pluto"
+		(at 373.38 107.95 180)
+		(effects
+			(font

Commit message: Add files via upload
Parts:
- added C111, C125: 1nF, symbol Device:C
- added C117, C121, C127, C280: 100nF, symbol Device:C
- added C123, C128: 150nF, symbol Device:C
- added C130, C140, C277: 1uF, symbol Device:C
- added D33: N, symbol Device:D_Dual_CommonCathode_AKA
- added Q14, Q38: 8C, Package_TO_SOT_SMD:SOT-23, symbol Transistor_BJT:MMBTA44
- added R114, R393: 47k, symbol Device:R
- added R119, R182, R186, R215, R216: 470k, symbol Device:R
- added R257: 33, symbol Device:R
- added R382, R383: 50k, symbol Device:R
- added SW2: LidSwitch, symbol Switch:SW_SPST
- added U38: 7W14, symbol 74xGxx:74LVC3G14
- added U39: 7W00, symbol 74xGxx:74AHC2G00
- added U40: 74HC74, symbol 74xx:74HC74
- added U45: 74HC123, symbol 74xx:74HC123
- added U9: E4, symbol 74xGxx:74AHC1G32
Connections:
- net PWRGD: now also U38.3
- net GND: now reaches U35.13 (GND)
- net GND: now also U21.100 (GND), U21.116 (GND), U21.136 (GND), U21.28 (GND), U21.44 (GND), U21.64 (GND), U21.8 (GND), U21.80 (GND), U35.37 (GND), U35.4 (GND), U35.63 (GND), U35.87 (GND), C111.2, C117.2, C121.1, C123.1, C125.1, C127.1, C128.1, C277.2, C280.2, Q14.2 (E), Q38.2 (E), R186.1, R383.2, U38.4 (GND), U39.4 (GND), U40.7 (GND), U45.8 (GND), U45.9 (A), U9.3 (GND)
- net PNET1: now reaches U35.14 (VCC)
- net PNET1: now also U21.1 (VCC), U21.108 (VCC), U21.109 (VCC), U21.126 (VCC), U21.144 (VCC), U21.18 (VCC), U21.36 (VCC), U21.37 (VCC), U21.54 (VCC), U21.72 (VCC), U21.73 (VCC), U21.90 (VCC), U21.99 (VCC), U35.38 (VCC), U35.64 (VCC), U35.7 (VCC), U35.88 (VCC), U35.95 (VCC), U35.97 (VCC), C111.1, C117.1, C121.2, C123.2, C127.2, C128.2, C140.2, C280.1, R182.1, R215.1, R216.2, R393.1, SW2.1 (A), U38.8 (VCC), U39.8 (VCC), U40.13 (~{R}), U40.14 (VCC), U40.2 (D), U45.16 (VCC), U45.2 (B), U45.6 (Cext), U9.5 (VCC)
- net at U35.2 (FF_2D): now also R186.2, U40.12 (D)
- net U53_2CLK: now reaches U35.3 (FF_2CLK)
- net U53_2CLK: now also U40.11 (C)
- net at U35.45 (FF_1CLK): now also Q38.3 (C), R216.1, U38.1
- net FF_1A: now reaches U35.46 (FF_1A)
- net FF_1A: now also U35.78 (FF_1A), U45.1 (A)
- net CPU_STPCLK#: now reaches U35.62 (CPU_STPCLK#)
- net KB_RESET#: now reaches U35.66 (KB_RESET#)
- net KB_RESET#: now also U21.48 (KB_RESET#), U40.10 (~{S}), U40.4 (~{S}), U45.3 (Clr)
- net at U35.90 (FF_2Q#): now also U40.1 (~{R}), U45.12 (~{Q})
- net LCD_STNDBY#: now reaches U35.93 (LCD_STNDBY)
- net LCD_STNDBY#: now also R393.2
- net CPU_A2: now reaches U21.10 (CPUA2)
- net CPU_A3: now reaches U21.11 (CPUA3)
- net CPU_A4: now reaches U21.12 (CPUA4)
- net CPU_A5: now reaches U21.13 (CPUA5)
- net CPU_A6: now reaches U21.14 (CPUA6)
- net at U21.141 (PWRGD_IN): now also U9.4
- net CPU_A7: now reaches U21.15 (CPUA7)
- net CPU_A8: now reaches U21.16 (CPUA8)
- net CPU_A9: now reaches U21.17 (CPUA9)
- net CPU_A10: now reaches U21.19 (CPUA10)
- net CPU_A11: now reaches U21.20 (CPUA11)
- net CPU_A12: now reaches U21.21 (CPUA12)
- net CPU_A13: now reaches U21.22 (CPUA13)
- net CPU_A14: now reaches U21.23 (CPUA14)
- net CPU_A15: now reaches U21.24 (CPUA15)
- net CPU_A16: now reaches U21.25 (CPUA16)
- net CPU_A18: now reaches U21.26 (CPUA18)
- net CPU_A19: now reaches U21.29 (CPUA19)
- net CPU_A20: now reaches U21.30 (CPUA20)
- net CPU_A21: now reaches U21.31 (CPUA21)
- net CPU_A22: now reaches U21.32 (CPUA22)
- net CPU_A23: now reaches U21.33 (CPUA23)
- net CPU_A24: now reaches U21.34 (CPUA24)
- net CPU_A25: now reaches U21.35 (CPUA25)
- net at U21.38 (CPUCLK): now also R257.1
- net CPU_RESET: now reaches U21.46 (CPU_RESET)
- new net: R382.1, R383.1, SW2.2 (B)
- new net: C277.1, Q38.1 (B), R382.2
- new net: D33.1 (A), U45.5 (Q)
- new net: D33.2 (A), U45.13 (Q)
- new net: D33.3 (K), R114.2
- new net: C130.1, R182.2, U45.15 (RCext)
- new net: Q14.1 (B), R114.1
- new net: C130.2, U45.14 (Cext)
- new net: C140.1, R215.2, U45.7 (RCext)
- new net: C125.2, U39.1, U40.6 (~{Q})
- new net: U38.7, U39.2, U40.3 (C)
- new net: U39.7, U45.10 (B)
- new net: U38.5, U9.2
- new net: U40.8 (~{Q}), U45.11 (Clr)
- new net CPU_A17: U21.26 (CPUA18)
- new net CPU_SMIACT#: U9.1
- new net Chipset_CPU_CLK: R257.2
- new net RTCBAT: R119.1
- new net YMF_VSS_Res: Q14.3 (C), R119.2
- no-connect marks 0 -> 6
Other:
- moved on the sheet: U21, U35

Commit message: Add files via upload
Parts:
- added D32: K, symbol Device:D_Dual_Series_KAC
- added Q16: IS6, symbol Simulation_SPICE:PNP
- added Q18: 8C, Package_TO_SOT_SMD:SOT-23, symbol Transistor_BJT:MMBTA44
- added R129: 133k, symbol Device:R
- added R180: 180k, symbol Device:R
- added R185: 4.7k, symbol Device:R
Connections:
- net GND: now also Q18.2 (E)
- net Pluto_Dock_IO1: now reaches U35.28 (Dock_IO1)
- net Pluto_Dock_IO2: now reaches U35.29 (Dock_IO2)
- net at U35.76 (Dev_OE): now also D32.1 (K), R180.2
- net Pluto_Dock_IO3: now reaches U35.77 (Dock_IO3)
- new net: D32.3 (common), Q18.1 (B), R180.1
- new net: Q18.3 (C), R185.1
- new net: Q16.2 (B), R185.2
- new net: D32.2 (A), R129.2
- new net PNET5: Q16.1 (C)
- new net Pluto_Switched_PNET5: Q16.3 (E), R129.1

Commit message: Add files via upload
Parts:
- added D26, D27, D28, D29: 3D, symbol Device:D_Dual_CommonCathode_AKA
- added R304: 4.7k, symbol Device:R
- added RA1: 47k, symbol Device:R_Pack04
Connections:
- net PS2_L1_Pluto: now reaches U35.30 (PS2_IO)
- net at U35.68 (FDD_IO1): now also D28.1 (A), D28.3 (A), RA1.2 (R2.1)
- net at U35.69 (FDD_IO2): now also D26.1 (A), D26.3 (A), RA1.1 (R1.1)
- net at U35.70 (FDD_IO3): now also D29.1 (A), D29.3 (A), RA1.4 (R4.1)
- net at U35.71 (FDD_IO4): now also D27.1 (A), D27.3 (A), RA1.3 (R3.1)
- net at U35.74 (PNET7_SENSE): now also R304.2
- net Modem_VSDA#: now reaches U35.75 (NM192_VDSA#)
- net FDC_MTR3#: now reaches U21.117 (PDRQ)
- net FDC_MTR2#: now reaches U21.121 (PDACK#)
- net FDD_Bowman: now reaches U21.125 (FDD_IO)
- new net FDD_Pluto1: D28.2 (K)
- new net FDD_Pluto2: D26.2 (K)
- new net FDD_Pluto3: D29.2 (K)
- new net FDD_Pluto4: D27.2 (K)
- new net PNET7: R304.1, RA1.5 (R4.2), RA1.6 (R3.2), RA1.7 (R2.2), RA1.8 (R1.2)
Other:
- moved on the sheet: R257, U21, U38C, U9

Commit message: Add files via upload
Parts:
- removed C128: 150nF, symbol Device:C
Connections:
- net SA2: now reaches U35.10 (SA2)
- net SA2: now also U21.57 (SA2)
- net Pluto_EN_IRDA: now reaches U35.48 (IRDA_EN)
- net Pluto_CLK: now reaches U35.65 (CLK)
- net SA0: now reaches U35.8 (SA0)
- net SA0: now also U21.55 (SA0)
- net Pluto_IRDA_OUT: now reaches U35.81 (IRDA_O)
- net SA1: now reaches U35.9 (SA1)
- net SA1: now also U21.56 (SA1)
- net at D33.2 (K): now also R114.2; no longer U45.13 (Q)
- net at D33.3 (A): now also U45.13 (Q); no longer R114.2
- net CPU_INTR: now reaches U21.133 (CPU_INTR)
- net Bowman_CLK: now reaches U21.40 (24MHz)
- net CPU_DC#: now reaches U21.41 (CPU_DC#)
- net CPU_WR#: now reaches U21.42 (CPU_WR#)
- net CPU_ADS#: now reaches U21.49 (CPU_ADS#)
- net CPU_MIO#: now reaches U21.50 (CPU_MIO#)
Other:
- moved on the sheet: C127, U40C

Commit message: Add files via upload
Connections:
- net KB_SPKDN: now reaches U35.43 (KB_SPKDN)
- net KB_SPKUP: now reaches U35.44 (KB_SPKUP)
- net Pluto_50: now reaches U35.50 (PWR_ON_SENSE)
- net Pluto_51: now reaches U35.51 (Bowman_IO1)
- net Pluto_51: now also U21.129 (Pluto_IO)
- net Pluto_52: now reaches U35.52 (Bowman_IO2)
- net KB_SCRLED#: now reaches U21.53 (KB_SCRLED#)
- net KB_IRQ1: now reaches U21.86 (KB_IRQ1)
Changed lines of the file:
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@@
 	(wire
 		(pts
+			(xy 184.15 260.35) (xy 209.55 260.35)
+		)
+		(stroke
+			(width 0)
+			(type default)
+		)
+	)
+	(wire
+		(pts
 			(xy 124.46 127) (xy 121.92 127)
 		)
@@
 	(wire
 		(pts
+			(xy 588.01 266.7) (xy 605.79 266.7)
+		)
+		(stroke
+			(width 0)
+			(type default)
+		)
+	)
+	(wire
+		(pts
 			(xy 549.91 187.96) (xy 549.91 198.12)
 		)
@@
 	(wire
 		(pts
+			(xy 480.06 208.28) (xy 501.65 208.28)
+		)
+		(stroke
+			(width 0)
+			(type default)
+		)
+	)
+	(wire
+		(pts
 			(xy 588.01 234.95) (xy 605.79 234.95)
 		)
@@
 	(wire
 		(pts
+			(xy 588.01 264.16) (xy 605.79 264.16)
+		)
+		(stroke
+			(width 0)
+			(type default)
+		)
+	)
+	(wire
+		(pts
 			(xy 679.45 304.8) (xy 679.45 313.69)
 		)
@@
 		)
 	)
+	(wire
+		(pts
+			(xy 480.06 210.82) (xy 501.65 210.82)
+		)
+		(stroke
+			(width 0)
+			(type default)
+		)
+	)
 	(bus
 		(pts
@@
 	(wire
 		(pts
+			(xy 63.5 297.18) (xy 86.36 297.18)
+		)
+		(stroke
+			(width 0)
+			(type default)
+		)
+	)
+	(wire
+		(pts
 			(xy 63.5 205.74) (xy 86.36 205.74)
 		)
@@
 	(wire
 		(pts
+			(xy 184.15 278.13) (xy 209.55 278.13)
+		)
+		(stroke
+			(width 0)
+			(type default)
+		)
+	)
+	(wire
+		(pts
 			(xy 457.2 219.71) (xy 457.2 237.49)
 		)
@@
 	(wire
 		(pts
+			(xy 588.01 260.35) (xy 605.79 260.35)
+		)
+		(stroke
+			(width 0)
+			(type default)
+		)
+	)
+	(wire
+		(pts
 			(xy 607.06 95.25) (xy 623.57 95.25)
 		)
@@
 		)
 	)
+	(label "KB_SPKDN"
+		(at 482.6 208.28 0)
+		(effects
+			(font
+				(size 1.27 1.27)
+			)
+			(justify left bottom)
+		)
+	)
 	(label "PWRGD"
 		(at 487.68 232.41 180)
@@
 		)
 	)
+	(label "KB_IRQ1"
+		(at 72.39 297.18 180)
+		(effects
+			(font
+				(size 1.27 1.27)
+			)
+			(justify right bottom)
+		)
+	)
 	(label "Pluto_Dock_IO3"
 		(at 590.55 243.84 0)
@@
 		)
 	)
+	(label "Pluto_50"
+		(at 595.63 260.35 0)
+		(effects
+			(font
+				(size 1.27 1.27)
+			)
+			(justify left bottom)
+		)
+	)
 	(label "CPU_A22"
 		(at 66.04 191.77 0)
@@
 		)
 	)
+	(label "KB_SPKUP"
+		(at 482.6 210.82 0)
+		(effects
+			(font
+				(size 1.27 1.27)
+			)
+			(justify left bottom)
+		)
+	)
 	(label "SA2"
 		(at 64.77 208.28 0)
@@
 		)
 	)
+	(label "KB_SCRLED#"
+		(at 196.85 278.13 0)
+		(effects
+			(font
+				(size 1.27 1.27)
+			)
+			(justify left bottom)
+		)
+	)
 	(label "CPU_A19"
 		(at 66.04 184.15 0)
@@
 		)
 	)
+	(label "Pluto_51"
+		(at 595.63 264.16 0)
+		(effects
+			(font
+				(size 1.27 1.27)
+			)
+			(justify left bottom)
+		)
+	)
 	(label "FDC_MTR2#"
 		(at 196.85 245.11 0)
@@
 		)
 	)
+	(label "Pluto_51"
+		(at 199.39 260.35 0)
+		(effects
+			(font
+				(size 1.27 1.27)
+			)
+			(justify left bottom)
+		)
+	)
 	(label "CPU_RESET"
 		(at 198.12 292.1 0)
@@
 		(effects
 			(font
+				(size 1.27 1.27)
+			)
+			(justify left bottom)
+		)
+	)
+	(label "Pluto_52"
+		(at 595.63 266.7 0)
+		(effects
+			(font
