File: PCB/Mainboard/ASIC.kicad_sch (KiCad schematic)
At the start: 59 parts, among them Q14 8C, Q16 2SA1881-6, Q18 8C, Q19 8B, Q38 8C, Q43 8B, Q44 8B, SW2 LidSwitch, U21 Bowman, U35 Pluto, U37 E8, U38 7W14, U39 7W00, U40 74HC74, U45 74HC123, U9 E4

Commit message: Add files via upload
Parts:
- added C66: 1uF, symbol Device:C
- added R104: 47k, symbol Device:R
Connections:
- net CPU_A18: now also U21.27 (CPUA18); no longer U21.26 (CPUA18)
- net GND: now also C66.2
- net M38_P14_Buf: now also U21.107 (M38_IO9); no longer U21.105 (M38_IO7)
- net U21_101: now reaches U21.101 (M38_IO3)
- net U21_102: now reaches U21.102 (M38_IO4)
- net U21_103: now reaches U21.103 (M38_IO5)
- net U21_104: now reaches U21.104 (M38_IO6)
- net M38_P43: now reaches U21.110 (M38_IO10)
- net M38_P41: now reaches U21.111 (M38_IO11)
- net U21_131: now reaches U21.131 (PSU_IO1)
- net CPU_RDY#: now reaches U21.134 (CPU_RDY#)
- net at U21.138 (PSU_IO2): now also R104.1
- net U21_139: now reaches U21.139 (M38_IO12)
- net U21_97: now reaches U21.97 (M38_IO1)
- net U21_98: now reaches U21.98 (M38_IO2)
- net FF_1A: no longer names the net of U35.46 (FF_1A), U35.78 (FF_1A), U45.1 (A)
- net SD0_Bus renamed SD0
- net SD1_Bus renamed SD1
- net SD2_Bus renamed SD2
- net SD3_Bus renamed SD3
- net SD4_Bus renamed SD4
- net SD5_Bus renamed SD5
- net SD6_Bus renamed SD6
- net SD7_Bus renamed SD7
- new net R73_2: C66.1, R104.2
- new net U21_105: U21.105 (M38_IO7)
- no-connect marks 6 -> 3
Other:
- note added: "CPU_ADDRESS_BUS"
- note added: "Device_Address_BUS"
- note added: "Device_Data_BUS"
- note added: "OKI_Extra_Address"

Commit message: Add files via upload
Connections:
- net FDC_UART1_EN: now reaches D32.1 (K), R180.2, U35.76 (Dev_OE)
Changed lines of the file:
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@@
 	)
 	(junction
+		(at 457.2 345.44)
+		(diameter 0)
+		(color 0 0 0 0)
+	)
+	(junction
 		(at 497.84 345.44)
 		(diameter 0)
@@
 	(wire
 		(pts
-			(xy 363.22 345.44) (xy 497.84 345.44)
+			(xy 363.22 345.44) (xy 457.2 345.44)
 		)
 		(stroke
@@
 	(wire
 		(pts
+			(xy 457.2 345.44) (xy 497.84 345.44)
+		)
+		(stroke
+			(width 0)
+			(type default)
+		)
+	)
+	(wire
+		(pts
 			(xy 453.39 220.98) (xy 461.01 220.98)
 		)
@@
 	(wire
 		(pts
+			(xy 457.2 353.06) (xy 457.2 345.44)
+		)
+		(stroke
+			(width 0)
+			(type default)
+		)
+	)
+	(wire
+		(pts
 			(xy 165.1 176.53) (xy 171.45 176.53)
 		)
@@
 	(wire
 		(pts
+			(xy 466.09 353.06) (xy 457.2 353.06)
+		)
+		(stroke
+			(width 0)
+			(type default)
+		)
+	)
+	(wire
+		(pts
 			(xy 44.45 135.89) (xy 67.31 135.89)
 		)
@@
 			(effects
 				(font
+					(size 1.27 1.27)
+				)
+				(justify left)
+				(hide yes)
+			)
+		)
+	)
+	(global_label "FDC_UART1_EN"
+		(shape input)
+		(at 466.09 353.06 0)
+		(fields_autoplaced yes)
+		(effects
+			(font
+				(size 1.27 1.27)
+			)
+			(justify left)
+		)
+		(property "Intersheetrefs" "${INTERSHEET_REFS}"
+			(at 482.9847 353.06 0)
+			(effects
+				(font

Commit message: Add files via upload
Parts:
- added C255: 120nF, symbol Device:C
- added C71, C78: 1nF, symbol Device:C
- added C74: 180nF, symbol Device:C
- added R149: 33, symbol Device:R
Connections:
- net Bowman3: now also R149.2; no longer U21.39 (Chipset_IO3)
- net GND: now also C255.2, C71.2, C74.2, C78.2
- net PNET1: now also C255.1, C71.1, C74.1, C78.1
- new net: R149.1, U21.39 (Chipset_IO3)
Other:
- moved on the sheet: C111, C117

Commit message: Add files via upload
Parts:
- C108, C109, C110, C111, C113, C117, C121, C123, C125, C127, C255, C280, C64, C71, C72, C74, C78: footprint (none) -> Capacitor_SMD:C_0402_1005Metric
- C130, C140, C277, C66: footprint (none) -> Capacitor_SMD:C_0603_1608Metric
- D26, D27, D28, D29: footprint (none) -> PC110:3D
- D32: footprint (none) -> PC110:SOT-416L
- D33: footprint (none) -> Package_TO_SOT_SMD:SOT-416
- Q14, Q18, Q19, Q38: footprint Package_TO_SOT_SMD:SOT-23 -> Package_TO_SOT_SMD:SOT-416
- Q16: footprint (none) -> PCM_Package_TO_SOT_SMD_AKL:TSOT-23
- Q43, Q44: footprint Package_TO_SOT_SMD:SOT-23 -> Package_TO_SOT_SMD:SOT-523
- R104, R114, R119, R129, R149, R180, R182, R185, R186, R215, R216: footprint (none) -> PCM_Resistor_SMD_AKL:R_0402_1005Metric
- R257, R304, R382, R383, R392, R393, R398, R399, R409, R410, R412: footprint (none) -> Resistor_SMD:R_0402_1005Metric
- RA1: footprint (none) -> PC110:R-array
- SW2: footprint (none) -> PC110:LidSwitch
- U21: footprint (none) -> PC110:Bowman
- U35: footprint (none) -> PC110:Pluto
- U37, U9: footprint (none) -> PC110:SOT-353
- U38, U39: footprint (none) -> PC110:sso-8
- U40: footprint (none) -> Package_SO:TSSOP-14_4.4x5mm_P0.65mm
- U45: footprint (none) -> Package_SO:TSSOP-16_4.4x5mm_P0.65mm
Connections:
- net GND: now also C117.1, C121.2, C123.2, C255.1, C277.1, C280.1, C66.1, C71.1, C74.1, C78.1, R186.2, R383.1; no longer C117.2, C121.1, C123.1, C255.2, C277.2, C280.2, C66.2, C71.2, C74.2, C78.2, R186.1, R383.2
- net PNET1: now also C117.2, C121.1, C123.1, C255.2, C280.2, C71.2, C74.2, C78.2, R215.2; no longer C117.1, C121.2, C123.2, C255.1, C280.1, C71.1, C74.1, C78.1, R215.1
- net PNET7: now also R304.2; no longer R304.1
- net Pluto_Switched_PNET5: now also R129.2; no longer R129.1
- net R73_2: now also C66.2; no longer C66.1
- net RTCBAT: now also R119.2; no longer R119.1
- net YMF_VSS_Res: now also R119.1; no longer R119.2
- net at U35.2 (FF_2D), U40.12 (D): now also R186.1; no longer R186.2
- net at U35.74 (PNET7_SENSE): now also R304.1; no longer R304.2
- net at R382.1, SW2.2 (B): now also R383.2; no longer R383.1
- net at Q38.1 (B), R382.2: now also C277.2; no longer C277.1
- net at D32.2 (A): now also R129.1; no longer R129.2
- net at C140.1, U45.7 (RCext): now also R215.1; no longer R215.2
Other:
- moved on the sheet: C121, C123, C255, C71, C74, C78, R129, R186

Commit message: Add files via upload
Parts:
- removed Q16: 2SA1881-6, PCM_Package_TO_SOT_SMD_AKL:TSOT-23, symbol Simulation_SPICE:PNP
- added Q16: 2SA1881-6, symbol PCM_Transistor_BJT_AKL:Q_PNP_Generic_BEC
Connections:
- net PNET5: now also Q16.2 (E)
- net Pluto_Switched_PNET5: now also Q16.3 (C)
- net at R185.2: now also Q16.1 (B)
Changed lines of the file:
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@@
+	)
+	(symbol
+		(lib_id "PCM_Transistor_BJT_AKL:Q_PNP_Generic_BEC")
+		(at 553.72 347.98 270)
+		(mirror x)
+		(unit 1)
+		(exclude_from_sim no)
+		(in_bom yes)
+		(on_board yes)
+		(dnp no)
+		(property "Reference" "Q16"
+			(at 553.72 339.09 90)
+			(effects
+				(font
+					(size 1.27 1.27)
+				)
+			)
+		)
+		(property "Value" "2SA1881-6"
+			(at 553.72 341.63 90)
+			(effects
+				(font
+					(size 1.27 1.27)
+				)
+			)
+		)
+		(property "Footprint" ""
+			(at 551.18 342.9 0)
+			(effects
+				(font
+					(size 1.27 1.27)
+				)
+				(hide yes)
+			)
+		)
+		(property "Datasheet" "~"
+			(at 553.72 347.98 0)
+			(effects
+				(font
+					(size 1.27 1.27)
+				)
+				(hide yes)
+			)
+		)
+		(property "Description" "PNP transistor, generic symbol, Alternate KiCAD Library"
+			(at 553.72 347.98 0)
+			(effects
+				(font
+					(size 1.27 1.27)
+				)
+				(hide yes)
+			)
+		)
+		(pin "1"
+		)
+		(pin "2"
+		)
+		(pin "3"
+		)
+		(instances
+			(project "PC110"
+				(path "/45c7911f-b027-440e-9e3e-77a146b41944/00000000-0000-0000-0000-000064523075"
+					(reference "Q16")
+					(unit 1)
+				)
+			)
+		)
 	)
 	(symbol
@@
 					(unit 1)
 				)
-			)
-		)
-	)
-	(symbol
-		(lib_id "Simulation_SPICE:PNP")
-		(at 553.72 347.98 270)
-		(mirror x)
-		(unit 1)
-		(exclude_from_sim no)
-		(in_bom yes)
-		(on_board yes)
-		(dnp no)
-		(property "Reference" "Q16"
-			(at 553.72 336.55 90)
-			(effects
-				(font
-					(size 1.27 1.27)
-				)
-			)
-		)
-		(property "Value" "2SA1881-6"
-			(at 553.72 339.09 90)
-			(effects
-				(font
-					(size 1.27 1.27)
-				)
-			)
-		)
-		(property "Footprint" "PCM_Package_TO_SOT_SMD_AKL:TSOT-23"
-			(at 553.72 312.42 0)
-			(effects
-				(font
-					(size 1.27 1.27)
-				)
-				(hide yes)
-			)
-		)
-		(property "Datasheet" "https://ngspice.sourceforge.io/docs/ngspice-html-manual/manual.xhtml#cha_BJTs"
-			(at 553.72 312.42 0)
-			(effects
-				(font
-					(size 1.27 1.27)
-				)
-				(hide yes)
-			)
-		)
-		(property "Description" "Bipolar transistor symbol for simulation only, substrate tied to the emitter"
-			(at 553.72 347.98 0)
-			(effects
-				(font
-					(size 1.27 1.27)
-				)
-				(hide yes)
-			)
-		)
-		(property "Sim.Device" "PNP"
-			(at 553.72 347.98 0)
-			(effects
-				(font
-					(size 1.27 1.27)
-				)
-				(hide yes)
-			)
-		)
-		(property "Sim.Type" "GUMMELPOON"
-			(at 553.72 347.98 0)
-			(effects
-				(font
-					(size 1.27 1.27)
-				)
-				(hide yes)
-			)
-		)
-		(property "Sim.Pins" "1=C 2=B 3=E"
-			(at 553.72 347.98 0)
-			(effects
-				(font
-					(size 1.27 1.27)
-				)
-				(hide yes)
-			)
-		)
-		(property "Topmark" "IS6"
-			(at 553.72 347.98 90)
-			(effects
-				(font
-					(size 1.27 1.27)
-				)
-				(hide yes)
-			)
-		)
-		(pin "2"
-		)
-		(pin "1"
-		)
-		(pin "3"
-		)
-		(instances
-			(project ""
-				(path "/45c7911f-b027-440e-9e3e-77a146b41944/00000000-0000-0000-0000-000064523075"
-					(reference "Q16")
-					(unit 1)
-				)

Commit message: Add files via upload
Parts:
- Q16: footprint (none) -> PCM_Package_TO_SOT_SMD_AKL:TSOT-23
Changed lines of the file:
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@@
 			)
 		)
-		(property "Footprint" ""
+		(property "Footprint" "PCM_Package_TO_SOT_SMD_AKL:TSOT-23"
 			(at 551.18 342.9 0)
 			(effects

Commit message: Add files via upload
Parts:
- removed D33: DAN222, Package_TO_SOT_SMD:SOT-416, symbol Device:D_Dual_CommonCathode_AKA
- added D33: N, Package_TO_SOT_SMD:SOT-416, symbol PC110:3D_Diode
- C108, C109, C110, C113, C64, C72: Indicator + -> (none); Rating V -> (none)
- D26, D27, D28, D29: value RB715F -> 3D; Topmark 3D -> (none)
- D32: value DA204U -> K; Topmark K -> (none)
- Q16: value 2SA1881-6 -> IS6
- R383: value 50k -> 33k
- U40: value 74HC74 -> SN74LS74a
- U45: value 74HC123 -> SN74LS123A
Connections:
- net PNET1: now also R216.1; no longer R216.2
- net at Q38.3 (C), U35.45 (FF_1CLK), U38.1: now also R216.2; no longer R216.1
- net at U45.5 (Q): now also D33.1
- net at R114.2: now also D33.3
- net at U45.13 (Q): now also D33.2
Other:
- moved on the sheet: R216

Commit message: Add files via upload
Connections:
- net PNET1: no longer U21.99 (VCC)
- new net PNET2: U21.99 (VCC)
Changed lines of the file:
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@@
 	)
 	(junction
-		(at 110.49 46.99)
-		(diameter 0)
-		(color 0 0 0 0)
-	)
-	(junction
 		(at 518.16 354.33)
 		(diameter 0)
@@
 	(wire
 		(pts
-			(xy 110.49 46.99) (xy 110.49 55.88)
-		)
-		(stroke
-			(width 0)
-			(type default)
-		)
-	)
-	(wire
-		(pts
 			(xy 335.28 381) (xy 332.74 381)
 		)
@@
 	(wire
 		(pts
-			(xy 113.03 46.99) (xy 110.49 46.99)
-		)
-		(stroke
-			(width 0)
-			(type default)
-		)
-	)
-	(wire
-		(pts
 			(xy 223.52 283.21) (xy 223.52 267.97)
 		)
@@
 	(wire
 		(pts
-			(xy 110.49 46.99) (xy 107.95 46.99)
+			(xy 107.95 46.99) (xy 113.03 46.99)
 		)
 		(stroke
@@
 	(wire
 		(pts
+			(xy 110.49 41.91) (xy 110.49 55.88)
+		)
+		(stroke
+			(width 0)
+			(type default)
+		)
+	)
+	(wire
+		(pts
 			(xy 351.79 187.96) (xy 356.87 187.96)
 		)
@@
 					(unit 1)
 				)
+			)
+		)
+	)
+	(symbol
+		(lib_id "power:VCC")
+		(at 110.49 41.91 0)
+		(unit 1)
+		(exclude_from_sim no)
+		(in_bom yes)
+		(on_board yes)
+		(dnp no)
+		(fields_autoplaced yes)
+		(property "Reference" "#PWR0708"
+			(at 110.49 45.72 0)
+			(effects
+				(font
+					(size 1.27 1.27)
+				)
+				(hide yes)
+			)
+		)
+		(property "Value" "PNET2"
+			(at 110.49 36.83 0)
+			(effects
+				(font
+					(size 1.27 1.27)
+				)
+			)
+		)
+		(property "Footprint" ""
+			(at 110.49 41.91 0)
+			(effects
+				(font
+					(size 1.27 1.27)
+				)
+				(hide yes)
+			)
+		)
+		(property "Datasheet" ""
+			(at 110.49 41.91 0)
+			(effects
+				(font
+					(size 1.27 1.27)
+				)
+				(hide yes)
+			)
+		)
+		(property "Description" "Power symbol creates a global label with name \"VCC\""
+			(at 110.49 41.91 0)
+			(effects
+				(font
+					(size 1.27 1.27)
+				)
+				(hide yes)
+			)
+		)
+		(pin "1"
+		)
+		(instances
+			(project "PC110"
+				(path "/45c7911f-b027-440e-9e3e-77a146b41944/00000000-0000-0000-0000-000064523075"
+					(reference "#PWR0708")
+					(unit 1)
+				)
