File: PCB/Mainboard/PC110.kicad_sch (KiCad schematic)
At the start: 0 parts

Commit message: Add files via upload
Other:
- sheet Pull-ups renamed PCMCIA
- sheet PCMCIA: file Pull-ups.kicad_sch -> PCMCIA.kicad_sch
Changed lines of the file:
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@@
 			(color 0 0 0 0.0000)
 		)
-		(property "Sheetname" "Pull-ups"
+		(property "Sheetname" "PCMCIA"
 			(at 64.77 99.6184 0)
 			(effects
@@
 			)
 		)
-		(property "Sheetfile" "Pull-ups.kicad_sch"
+		(property "Sheetfile" "PCMCIA.kicad_sch"
 			(at 64.77 113.6146 0)
 			(effects

Commit message: Add files via upload
Other:
- sheet Audio Controller renamed Audio
- sheet Buffers renamed ASIC
- sheet Decoupling Dapacitors renamed ROM
- sheet Keyboard and BIOS renamed Keyboard and Trackpoint
- sheet Local Bus IDE renamed Storage
- sheet ASIC: file Buffers.kicad_sch -> ASIC.kicad_sch
- sheet Keyboard and Trackpoint: file Keyboard_BIOS.kicad_sch -> Keyboard.kicad_sch
- sheet ROM: file Decoup_caps.kicad_sch -> ROM.kicad_sch
- sheet Storage: file VLB_IDE.kicad_sch -> Storage.kicad_sch
- note removed: "TODO - Schematic: - update all the schematics to be compatible with the PC110"

Commit message: Add files via upload
Changed lines of the file:
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@@
 	)
 	(sheet
-		(at 25.4 25.4)
+		(at 54.61 48.26)
 		(size 25.4 12.7)
 		(exclude_from_sim no)
@@
 		)
 		(property "Sheetname" "Processor"
-			(at 25.4 24.6884 0)
+			(at 54.61 47.5484 0)
 			(effects
 				(font
@@
 		)
 		(property "Sheetfile" "Processor.kicad_sch"
-			(at 25.4 38.6846 0)
+			(at 54.61 61.5446 0)
 			(effects
 				(font
@@
 	)
 	(sheet
-		(at 63.5 78.74)
+		(at 93.98 100.33)
 		(size 25.4 12.7)
 		(exclude_from_sim no)
@@
 		)
 		(property "Sheetname" "Power"
-			(at 63.5 78.0284 0)
+			(at 93.98 99.6184 0)
 			(effects
 				(font
@@
 		)
 		(property "Sheetfile" "Power.kicad_sch"
-			(at 63.5 92.0246 0)
+			(at 93.98 113.6146 0)
 			(effects
 				(font
@@
 	)
 	(sheet
-		(at 101.6 78.74)
+		(at 132.08 100.33)
 		(size 25.4 12.7)
 		(exclude_from_sim no)
@@
 		)
 		(property "Sheetname" "PCMCIA"
-			(at 101.6 78.0284 0)
+			(at 132.08 99.6184 0)
 			(effects
 				(font
@@
 		)
 		(property "Sheetfile" "PCMCIA.kicad_sch"
-			(at 101.6 92.0246 0)
+			(at 132.08 113.6146 0)
 			(effects
 				(font
@@
 	)
 	(sheet
-		(at 25.4 52.07)
+		(at 54.61 73.66)
 		(size 25.4 12.7)
 		(exclude_from_sim no)
@@
 		)
 		(property "Sheetname" "Memory"
-			(at 25.4 51.3584 0)
+			(at 54.61 72.9484 0)
 			(effects
 				(font
@@
 		)
 		(property "Sheetfile" "Memory.kicad_sch"
-			(at 25.4 65.3546 0)
+			(at 54.61 86.9446 0)
 			(effects
 				(font
@@
 	)
 	(sheet
-		(at 63.5 25.4)
+		(at 93.98 48.26)
 		(size 25.4 12.7)
 		(exclude_from_sim no)
@@
 		)
 		(property "Sheetname" "Chipset"
-			(at 63.5 24.6884 0)
+			(at 93.98 47.5484 0)
 			(effects
 				(font
@@
 		)
 		(property "Sheetfile" "Chipset.kicad_sch"
-			(at 63.5 38.6846 0)
+			(at 93.98 61.5446 0)
 			(effects
 				(font
@@
 	)
 	(sheet
-		(at 101.6 52.07)
+		(at 132.08 73.66)
 		(size 25.4 12.7)
 		(exclude_from_sim no)
@@
 		)
 		(property "Sheetname" "ASIC"
-			(at 101.6 51.3584 0)
+			(at 132.08 72.9484 0)
 			(effects
 				(font
@@
 		)
 		(property "Sheetfile" "ASIC.kicad_sch"
-			(at 101.6 65.3546 0)
+			(at 132.08 86.9446 0)
 			(effects
 				(font
@@
 	)
 	(sheet
-		(at 101.6 101.6)
+		(at 132.08 125.73)
 		(size 25.4 12.7)
 		(exclude_from_sim no)
@@
 		)
 		(property "Sheetname" "Keyboard and Trackpoint"
-			(at 101.6 100.8884 0)
+			(at 132.08 125.0184 0)
 			(effects
 				(font
@@
 		)
 		(property "Sheetfile" "Keyboard.kicad_sch"
-			(at 101.6 114.8846 0)
+			(at 132.08 139.0146 0)
 			(effects
 				(font
@@
 	)
 	(sheet
-		(at 101.6 25.4)
+		(at 132.08 48.26)
 		(size 25.4 12.7)
 		(exclude_from_sim no)
@@
 		)
 		(property "Sheetname" "VGA Controller"
-			(at 101.6 24.6884 0)
+			(at 132.08 47.5484 0)
 			(effects
 				(font
@@
 		)
 		(property "Sheetfile" "VGA.kicad_sch"
-			(at 101.6 38.6846 0)
+			(at 132.08 61.5446 0)
 			(effects
 				(font
@@
 	)
 	(sheet
-		(at 25.4 78.74)
+		(at 54.61 100.33)
 		(size 25.4 12.7)
 		(exclude_from_sim no)
@@
 		)
 		(property "Sheetname" "Super I/O"
-			(at 25.4 78.0284 0)
+			(at 54.61 99.6184 0)
 			(effects
 				(font
@@
 		)
 		(property "Sheetfile" "Super_IO.kicad_sch"
-			(at 25.4 92.0246 0)
+			(at 54.61 113.6146 0)
 			(effects
 				(font
@@
 	)
 	(sheet
-		(at 63.5 101.6)
+		(at 93.98 125.73)
 		(size 25.4 12.7)
 		(exclude_from_sim no)
@@
 		)
 		(property "Sheetname" "Storage"
-			(at 63.5 100.8884 0)
+			(at 93.98 125.0184 0)
 			(effects
 				(font
@@
 		)
 		(property "Sheetfile" "Storage.kicad_sch"
-			(at 63.5 114.8846 0)
+			(at 93.98 139.0146 0)
 			(effects
 				(font
@@
 	)
 	(sheet
-		(at 25.4 101.6)
+		(at 54.61 125.73)
 		(size 25.4 12.7)
 		(exclude_from_sim no)
@@
 		)
 		(property "Sheetname" "Audio"
-			(at 25.4 100.8884 0)
+			(at 54.61 125.0184 0)
 			(effects
 				(font
@@
 		)
 		(property "Sheetfile" "Audio.kicad_sch"
-			(at 25.4 114.8846 0)
+			(at 54.61 139.0146 0)
 			(effects
 				(font
@@
 	)
 	(sheet
-		(at 63.5 52.07)
+		(at 93.98 73.66)
 		(size 25.4 12.7)
 		(exclude_from_sim no)
@@
 		)
 		(property "Sheetname" "ROM"
-			(at 63.5 51.3584 0)
+			(at 93.98 72.9484 0)
 			(effects
 				(font
@@
 		)
 		(property "Sheetfile" "ROM.kicad_sch"
-			(at 63.5 65.3546 0)
-			(effects
-				(font
+			(at 93.98 86.9446 0)
+			(effects
+				(font

Commit message: Add files via upload
Other:
- added sheet Docking Station (DockStation.kicad_sch)
Changed lines of the file:
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@@
+		)
+	)
+	(sheet
+		(at 54.61 152.4)
+		(size 25.4 12.7)
+		(exclude_from_sim no)
+		(in_bom yes)
+		(on_board yes)
+		(dnp no)
+		(fields_autoplaced yes)
+		(stroke
+			(width 0)
+			(type solid)
+		)
+		(fill
+			(color 0 0 0 0.0000)
+		)
+		(property "Sheetname" "Docking Station"
+			(at 54.61 151.6884 0)
+			(effects
+				(font
+					(size 1.27 1.27)
+				)
+				(justify left bottom)
+			)
+		)
+		(property "Sheetfile" "DockStation.kicad_sch"
+			(at 54.61 165.6846 0)
+			(effects
+				(font
+					(size 1.27 1.27)
+				)
+				(justify left top)
+			)
+		)
+		(instances
+			(project "PC110"
+				(path "/45c7911f-b027-440e-9e3e-77a146b41944"
+					(page "14")
+				)
+			)
 		)
 	)

Commit message: Add files via upload
Other:
- sheet Docking Station renamed Docking Station and Modem
Changed lines of the file:
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@@
 			(color 0 0 0 0.0000)
 		)
-		(property "Sheetname" "Docking Station"
+		(property "Sheetname" "Docking Station and Modem"
 			(at 54.61 151.6884 0)
 			(effects

Commit message: Add files via upload
Other:
- added sheet Clock (Clock.kicad_sch)

Commit message: Add files via upload
Other:
- sheet Clock renamed Clock Tree
Changed lines of the file:
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@@
 	)
 	(sheet
-		(at 100.33 41.91)
+		(at 101.6 38.1)
 		(size 25.4 12.7)
 		(exclude_from_sim no)
@@
 		)
 		(property "Sheetname" "Processor"
-			(at 100.33 41.1984 0)
+			(at 101.6 37.3884 0)
 			(effects
 				(font
@@
 		)
 		(property "Sheetfile" "Processor.kicad_sch"
-			(at 100.33 55.1946 0)
+			(at 101.6 51.3846 0)
 			(effects
 				(font
@@
 	)
 	(sheet
-		(at 151.13 93.98)
+		(at 152.4 88.9)
 		(size 25.4 12.7)
 		(exclude_from_sim no)
@@
 		)
 		(property "Sheetname" "Power"
-			(at 151.13 93.2684 0)
+			(at 152.4 88.1884 0)
 			(effects
 				(font
@@
 		)
 		(property "Sheetfile" "Power.kicad_sch"
-			(at 151.13 107.2646 0)
+			(at 152.4 102.1846 0)
 			(effects
 				(font
@@
 	)
 	(sheet
-		(at 52.07 120.65)
+		(at 50.8 114.3)
 		(size 25.4 12.7)
 		(exclude_from_sim no)
@@
 		)
 		(property "Sheetname" "PCMCIA"
-			(at 52.07 119.9384 0)
+			(at 50.8 113.5884 0)
 			(effects
 				(font
@@
 		)
 		(property "Sheetfile" "PCMCIA.kicad_sch"
-			(at 52.07 133.9346 0)
+			(at 50.8 127.5846 0)
 			(effects
 				(font
@@
 	)
 	(sheet
-		(at 100.33 67.31)
+		(at 101.6 63.5)
 		(size 25.4 12.7)
 		(exclude_from_sim no)
@@
 		)
 		(property "Sheetname" "Memory"
-			(at 100.33 66.5984 0)
+			(at 101.6 62.7884 0)
 			(effects
 				(font
@@
 		)
 		(property "Sheetfile" "Memory.kicad_sch"
-			(at 100.33 80.5946 0)
+			(at 101.6 76.7846 0)
 			(effects
 				(font
@@
 	)
 	(sheet
-		(at 151.13 41.91)
+		(at 152.4 38.1)
 		(size 25.4 12.7)
 		(exclude_from_sim no)
@@
 		)
 		(property "Sheetname" "Chipset"
-			(at 151.13 41.1984 0)
+			(at 152.4 37.3884 0)
 			(effects
 				(font
@@
 		)
 		(property "Sheetfile" "Chipset.kicad_sch"
-			(at 151.13 55.1946 0)
+			(at 152.4 51.3846 0)
 			(effects
 				(font
@@
 	)
 	(sheet
-		(at 52.07 93.98)
+		(at 50.8 88.9)
 		(size 25.4 12.7)
 		(exclude_from_sim no)
@@
 		)
 		(property "Sheetname" "ASIC"
-			(at 52.07 93.2684 0)
+			(at 50.8 88.1884 0)
 			(effects
 				(font
@@
 		)
 		(property "Sheetfile" "ASIC.kicad_sch"
-			(at 52.07 107.2646 0)
+			(at 50.8 102.1846 0)
 			(effects
 				(font
@@
 	)
 	(sheet
-		(at 52.07 146.05)
+		(at 50.8 139.7)
 		(size 25.4 12.7)
 		(exclude_from_sim no)
@@
 		)
 		(property "Sheetname" "Keyboard and Trackpoint"
-			(at 52.07 145.3384 0)
+			(at 50.8 138.9884 0)
 			(effects
 				(font
@@
 		)
 		(property "Sheetfile" "Keyboard.kicad_sch"
-			(at 52.07 159.3346 0)
+			(at 50.8 152.9846 0)
 			(effects
 				(font
@@
 	)
 	(sheet
-		(at 52.07 67.31)
+		(at 50.8 63.5)
 		(size 25.4 12.7)
 		(exclude_from_sim no)
@@
 		)
 		(property "Sheetname" "VGA Controller"
-			(at 52.07 66.5984 0)
+			(at 50.8 62.7884 0)
 			(effects
 				(font
@@
 		)
 		(property "Sheetfile" "VGA.kicad_sch"
-			(at 52.07 80.5946 0)
+			(at 50.8 76.7846 0)
 			(effects
 				(font
@@
 	)
 	(sheet
-		(at 100.33 93.98)
+		(at 101.6 88.9)
 		(size 25.4 12.7)
 		(exclude_from_sim no)
@@
 		)
 		(property "Sheetname" "Super I/O"
-			(at 100.33 93.2684 0)
+			(at 101.6 88.1884 0)
 			(effects
 				(font
@@
 		)
 		(property "Sheetfile" "Super_IO.kicad_sch"
-			(at 100.33 107.2646 0)
+			(at 101.6 102.1846 0)
 			(effects
 				(font
@@
 	)
 	(sheet
-		(at 151.13 120.65)
+		(at 152.4 114.3)
 		(size 25.4 12.7)
 		(exclude_from_sim no)
@@
 		)
 		(property "Sheetname" "Storage"
-			(at 151.13 119.9384 0)
+			(at 152.4 113.5884 0)
 			(effects
 				(font
@@
 		)
 		(property "Sheetfile" "Storage.kicad_sch"
-			(at 151.13 133.9346 0)
+			(at 152.4 127.5846 0)
 			(effects
 				(font
@@
 	)
 	(sheet
-		(at 100.33 120.65)
+		(at 101.6 114.3)
 		(size 25.4 12.7)
 		(exclude_from_sim no)
@@
 		)
 		(property "Sheetname" "Audio"
-			(at 100.33 119.9384 0)
+			(at 101.6 113.5884 0)
 			(effects
 				(font
@@
 		)
 		(property "Sheetfile" "Audio.kicad_sch"
-			(at 100.33 133.9346 0)
+			(at 101.6 127.5846 0)
 			(effects
 				(font
@@
 	)
 	(sheet
-		(at 151.13 67.31)
+		(at 152.4 63.5)
 		(size 25.4 12.7)
 		(exclude_from_sim no)
@@
 		)
 		(property "Sheetname" "ROM"
-			(at 151.13 66.5984 0)
+			(at 152.4 62.7884 0)
 			(effects
 				(font
@@
 		)
 		(property "Sheetfile" "ROM.kicad_sch"
-			(at 151.13 80.5946 0)
+			(at 152.4 76.7846 0)
 			(effects
 				(font
@@
 	)
 	(sheet
-		(at 100.33 146.05)
+		(at 101.6 139.7)
 		(size 25.4 12.7)
 		(exclude_from_sim no)
@@
 		)
 		(property "Sheetname" "Docking Station and Modem"
-			(at 100.33 145.3384 0)
+			(at 101.6 138.9884 0)
 			(effects
 				(font
@@
 		)
 		(property "Sheetfile" "DockStation.kicad_sch"
-			(at 100.33 159.3346 0)
+			(at 101.6 152.9846 0)
 			(effects
 				(font
@@
 	)
 	(sheet
-		(at 52.07 41.91)
-		(size 25.4 12.7)
-		(exclude_from_sim no)
-		(in_bom yes)
-		(on_board yes)
-		(dnp no)
-		(fields_autoplaced yes)
-		(stroke
-			(width 0)
-			(type solid)
-		)
-		(fill
-			(color 0 0 0 0.0000)
-		)
-		(property "Sheetname" "Clock"
-			(at 52.07 41.1984 0)
+		(at 50.8 38.1)
+		(size 25.4 12.7)
+		(exclude_from_sim no)
+		(in_bom yes)
+		(on_board yes)
+		(dnp no)
+		(fields_autoplaced yes)
+		(stroke
+			(width 0)
+			(type solid)
+		)
+		(fill
+			(color 0 0 0 0.0000)
+		)
+		(property "Sheetname" "Clock Tree"
+			(at 50.8 37.3884 0)
 			(effects
 				(font
@@
 		)
 		(property "Sheetfile" "Clock.kicad_sch"
-			(at 52.07 55.1946 0)
-			(effects
-				(font
+			(at 50.8 51.3846 0)
+			(effects
+				(font
