File: PCB/Mainboard/PC110.kicad_sch (KiCad schematic)
At the start: 0 parts

Commit message: Add files via upload
Other:
- company: (none) -> Recreated by: Ahmad Byagowi
Changed lines of the file:
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@@
 	(title_block
 		(title "PC110 Motherboard")
+		(company "Recreated by: Ahmad Byagowi")
 	)
 	(sheet
