File: PCB/Mainboard/Keyboard.kicad_sch (KiCad schematic)
At the start: 0 parts

Commit message: Add files via upload
Parts:
- added U67: ~, symbol PC110:M38813
- added U75: ~, symbol PC110:D17137

Commit message: Add files via upload
Parts:
- renumbered U75 to U?, U67 to U?
Changed lines of the file:
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@@
 		(on_board yes)
 		(dnp no)
-		(property "Reference" "U75"
+		(property "Reference" "U?"
 			(at 91.694 70.866 0)
 			(effects
@@
 		)
 		(instances
-			(project ""
+			(project "PC110"
 				(path "/45c7911f-b027-440e-9e3e-77a146b41944/00000000-0000-0000-0000-0000655ddd04"
-					(reference "U75")
+					(reference "U?")
 					(unit 1)
 				)
@@
 		(on_board yes)
 		(dnp no)
-		(property "Reference" "U67"
+		(property "Reference" "U?"
 			(at 202.692 59.436 0)
 			(effects
@@
 		)
 		(instances
-			(project ""
+			(project "PC110"
 				(path "/45c7911f-b027-440e-9e3e-77a146b41944/00000000-0000-0000-0000-0000655ddd04"
-					(reference "U67")
+					(reference "U?")
 					(unit 1)
 				)

Commit message: Add files via upload
Parts:
- added J16: Keyboard Conn 2, symbol Connector_Generic:Conn_01x20
- added J17: Keyboard Conn 1, symbol Connector_Generic:Conn_01x08
- added R78: 10K, symbol Device:R
- gave numbers to parts that had none: 2
Connections:
- net TRKPD_Lclick: now reaches U75.4 (P0C1/ADC1)
- net TRKPD_Lclick: now also J16.4 (Pin_4)
- net TRKPD_Rclick: now reaches U75.5 (P0C0/ADC0)
- net TRKPD_Rclick: now also J16.3 (Pin_3)
- net SD2_Bus: now reaches U67.1 (DQ2)
- net SD1_Bus: now reaches U67.2 (DQ1)
- net SD0_Bus: now reaches U67.3 (DQ0)
- net KB2_1: now reaches U67.33 (P17/AD15)
- net KB2_1: now also J16.18 (Pin_18)
- net KB2_2: now reaches U67.34 (P16/AD14)
- net KB2_2: now also J16.6 (Pin_6)
- net KB2_3: now reaches U67.35 (P15/AD13)
- net KB2_3: now also J16.17 (Pin_17)
- net KB2_4: now reaches U67.36 (P14/AD12)
- net KB2_4: now also J16.14 (Pin_14)
- net KB2_5: now reaches U67.37 (P13/AD11)
- net KB2_5: now also J16.16 (Pin_16)
- net KB2_6: now reaches U67.38 (P12/AD10)
- net KB2_6: now also J16.9 (Pin_9)
- net KB2_7: now reaches U67.39 (P11/AD9)
- net KB2_7: now also J16.5 (Pin_5)
- net KB2_8: now reaches U67.40 (P10/AD8)
- net KB2_8: now also J16.10 (Pin_10)
- net KB2_9: now reaches U67.41 (P07/AD7)
- net KB2_9: now also J16.8 (Pin_8)
- net KB2_10: now reaches U67.42 (P06/AD6)
- net KB2_10: now also J16.11 (Pin_11)
- net KB2_11: now reaches U67.43 (P05/AD5)
- net KB2_11: now also J16.7 (Pin_7)
- net KB2_12: now reaches U67.44 (P04/AD4)
- net KB2_12: now also J16.12 (Pin_12)
- net KB2_13: now reaches U67.45 (P03/AD3)
- net KB2_13: now also J16.13 (Pin_13)
- net KB2_14: now reaches U67.46 (P02/AD2)
- net KB2_14: now also J16.15 (Pin_15)
- net KB2_15: now reaches U67.47 (P01/AD1)
- net KB2_15: now also J16.20 (Pin_20)
- net KB2_16: now reaches U67.48 (P00/AD0)
- net KB2_16: now also J16.19 (Pin_19)
- net KB1_7: now reaches U67.49 (P37/RD#)
- net KB1_7: now also J17.5 (Pin_5)
- net KB1_6: now reaches U67.50 (P36/WR#)
- net KB1_6: now also J17.6 (Pin_6)
- net KB1_5: now reaches U67.51 (P35/SYNC)
- net KB1_5: now also J17.4 (Pin_4)
- net KB1_4: now reaches U67.52 (P34)
- net KB1_4: now also J17.7 (Pin_7)
- net KB1_3: now reaches U67.53 (P33)
- net KB1_3: now also J17.3 (Pin_3)
- net KB1_2: now reaches U67.54 (P32/ONW#)
- net KB1_2: now also J17.8 (Pin_8)
- net KB1_1: now reaches U67.55 (P31/DA2)
- net KB1_1: now also J17.2 (Pin_2)
- net KB1_0: now reaches U67.56 (P30/DA1)
- net KB1_0: now also J17.1 (Pin_1)
- net PNET1: now reaches U67.57 (VCC)
- net KB_INT5: now reaches U67.58 (P61)
- net KB_INT5: now also R78.2
- net KB_CNTR#_Pluto: now reaches U67.59 (PC60)
- net SD7_Bus: now reaches U67.60 (DQ7)
- net SD6_Bus: now reaches U67.61 (DQ6)
- net SD5_Bus: now reaches U67.62 (DQ5)
- net SD4_Bus: now reaches U67.63 (DQ4)
- net SD3_Bus: now reaches U67.64 (DQ3)
- new net GND: J16.2 (Pin_2)
- new net KB_SOUND: R78.1
- no-connect marks 0 -> 1
Other:
- moved on the sheet: U67, U75

Commit message: Add files via upload
Parts:
- added C136: 150nF, symbol PCM_Elektuur:C
- added Q8: 6D, symbol Simulation_SPICE:PNP
- added R196, R206: 47k, symbol Device:R
- added R203: 10k, symbol Device:R
- added R45, R59: 100k, symbol Device:R
Connections:
- net GND: now also C136.2 (-)
- net PNET1: now also R45.1, R59.1
- net TRKPD_Lclick: now also R206.2
- net TRKPD_Rclick: now also R196.2
- net PNET3: now reaches U75.1 (VADC)
- net PNET3: now also U75.28 (VDD), C136.1 (+), Q8.1 (C), R196.1, R203.1, R206.1
- net at U75.24 (P0D1/SO): now also U75.25 (P0D0/SCK#), R203.2
- net KB_INIT1: now reaches U67.17 (P42/INT1)
- net KB_SRDY#: now reaches U67.8 (P53/SRDY2)
- net KB_SRDY#: now also R59.2
- net KB_SCLK#: now reaches U67.9 (P52/SCLK2)
- net KB_SCLK#: now also Q8.2 (B), R45.2
- new net PNET5: Q8.3 (E)
Other:
- moved on the sheet: J16, J17, R78, U67, U75

Commit message: Add files via upload
Parts:
- added C128: 150nF, symbol Device:C
- added R372: 100k, symbol Device:R
- added U72: ~, symbol PC110:HD151015
Connections:
- net GND: now also U75.14 (GND), C128.1, U72.12 (GND), U72.13 (GND), U72.23 (G#)
- net PNET1: now also C128.2, R372.2, U72.1 (VCCA), U72.2 (DIR)
- net PNET5: now also U72.24 (VCCB)
- new net: R372.1, U72.10 (A7)
- new net ESS_DACK1#: U72.15 (B7)
- new net FCS_RESET: U72.11 (A8)
- no-connect marks 1 -> 2

Commit message: Add files via upload
Parts:
- added C281, C283: 39pF, symbol PCM_Elektuur:C
- added R198: 10k, symbol Device:R
- added U73: SN74LVT244B, symbol 74xx:74LS244
- added X6: 8.00, symbol Device:Crystal_GND3
Connections:
- net GND: now also U67.18 (CNVSS), C281.2 (-), C283.2 (-), U73.10 (GND), X6.3
- net PNET1: now also U73.20 (VCC)
- net PNET3: now also R198.1
- net D171_GPDATA: now reaches R203.2, U75.24 (P0D1/SO), U75.25 (P0D0/SCK#)
- net D171_GPDATA: now also U67.21 (P40/INT4)
- net D171_GPCLK: now reaches U75.22 (P0D3/TM0OUT#)
- net D171_GPCLK: now also U67.20 (P41/INT0), U75.23 (P0D2/SI), R198.2
- net at U75.26 (Xout): now also C283.1 (+), X6.1
- net at U75.27 (Xin): now also C281.1 (+), X6.2
- net KB_IRQ1: now reaches U67.15 (P44/RxD)
- net KB_INIT2: now reaches U67.16 (P43/INT2)
- net KB_RESET#: now reaches U67.19 (RESET)
- net KB_SCRLED#: now reaches U67.25 (P27/DB7)
- net KB_NUMLED#: now reaches U67.26 (P26/DB6)
- net KB_NUMLED#: now also U73.3 (O3b)
- net KB_CAPLED#: now reaches U67.27 (P25/DB5)
- net KB_CAPLED#: now also U73.4 (I1a)
- net KB_PADLED#: now reaches U67.28 (P24/DB4)
- net KB_PADLED#: now also U73.5 (O2b)
- net KB_SPKUP: now reaches U67.29 (P23/DB3)
- net KB_SPKDN: now reaches U67.30 (P22/DB2)
- net KB_SPKDN: now also U73.16 (O1a)
- net KB_TP139: now reaches U67.31 (P21/DB1)
- net KB_TP139: now also U73.14 (O2a)
- net KB_KBCSMI: now reaches U67.32 (P20/DB0)
- net KB_KBCSMI: now also U73.12 (O3a)
Other:
- moved on the sheet: C128, R203, R372, U72

Commit message: Add files via upload
Parts:
- added C135: 2.7uF, symbol PCM_Elektuur:C
- added C264, C268: 56pF, symbol PCM_Elektuur:C
- added D35: 3D, symbol Device:D_Dual_CommonCathode_AKA
- added J19: Trackpoint, symbol Connector_Generic:Conn_01x18
- added R197, R200, R204: 47k, symbol Device:R
- added R199, R202: DNP, symbol Device:R
- added R201, R205: 100k, symbol Device:R
- added U69: SN74LVC2G32, symbol 74xGxx:74LVC2G32
- added X5: 4.00, symbol Device:Crystal_GND3
Connections:
- net GND: now also U67.24 (VSS), U73.1 (OEa), U73.19 (OEb), C135.2 (-), C264.2 (-), C268.2 (-), J19.9 (Pin_9), R199.2, R202.2, U69.4 (GND), X5.3
- net KB_CAPLED#: now also U72.4 (A1); no longer U73.4 (I1a)
- net KB_NUMLED#: now also U72.3 (A0); no longer U73.3 (O3b)
- net KB_PADLED#: now also U72.5 (A2); no longer U73.5 (O2b)
- net PNET1: now also U69.8 (VCC)
- net PNET3: now also D35.2 (K), R197.1, R200.1, R201.1, R204.1, R205.1
- net TRKPD_Lclick: now also J19.10 (Pin_10)
- net TRKPD_Rclick: now also J19.11 (Pin_11)
- net ESS_AEN: now reaches U72.16 (B6)
- net YMF_WR#_Buf: now reaches U72.17 (B5)
- net YMF_RD#_Buf: now reaches U72.18 (B4)
- net M38_P44: now reaches U72.19 (B3)
- net M38_P35: now reaches U72.20 (B2)
- net M38_21: now reaches U72.21 (B1)
- net M38_P36: now reaches U72.22 (B0)
- net KB_TXD: now reaches U72.6 (A3)
- net KB_TXD: now also U67.10 (P51/SOUT2)
- net IOR#: now reaches U72.7 (A4)
- net IOR#: now also U67.5 (R#)
- net IOW#: now reaches U72.8 (A5)
- net IOW#: now also U67.4 (W#)
- net at U72.9 (A6): now also U69.3
- net D171_P0A3: now reaches U75.10 (P0A3)
- net D171_P0A3: now also J19.3 (Pin_3)
- net D171_P0A2: now reaches U75.11 (P0A2)
- net D171_P0A2: now also J19.4 (Pin_4)
- net D171_P0A1: now reaches U75.12 (P0A1)
- net D171_P0A1: now also J19.5 (Pin_5)
- net D171_P0A0: now reaches U75.13 (P0A0)
- net D171_P0A0: now also J19.6 (Pin_6)
- net at U75.15 (INT): now also R199.1, R204.2
- net at U75.16 (RESET#): now also C135.1 (+), D35.1 (A), D35.3 (A), R200.2
- net at U75.17 (P1B0): now also R197.2, R202.1
- net D171_P1A3: now reaches U75.18 (P1A3)
- net D171_P1A3: now also J19.7 (Pin_7)
- net D171_P1A2: now reaches U75.19 (P1A2)
- net D171_P1A2: now also J19.17 (Pin_17)
- net D171_P0C3: now reaches U75.2 (P0C3/ADC3)
- net D171_P0C3: now also J19.16 (Pin_16), R201.2
- net D171_P1A1: now reaches U75.20 (P1A1)
- net D171_P1A1: now also J19.8 (Pin_8)
- net D171_P1A0: now reaches U75.21 (P1A0)
- net D171_P1A0: now also J19.18 (Pin_18)
- net D171_P0C2: now reaches U75.3 (P0C2/ADC2)
- net D171_P0C2: now also J19.2 (Pin_2), R205.2
- net D171_P0B3: now reaches U75.6 (P0B3)
- net D171_P0B3: now also J19.12 (Pin_12)
- net D171_P0B2: now reaches U75.7 (P0B2)
- net D171_P0B2: now also J19.13 (Pin_13)
- net D171_P0B1: now reaches U75.8 (P0B1)
- net D171_P0B1: now also J19.14 (Pin_14)
- net D171_P0B0: now reaches U75.9 (P0B0)
- net D171_P0B0: now also J19.15 (Pin_15)
- net KB_RXD: now reaches U67.11 (P50/SIN2)
- net KB_RXD: now also U73.9 (O0b)
- net KB_INIT4: now reaches U67.12 (P47/SRDY1)
- net KB_INIT3: now reaches U67.13 (P46/SCLK1)
- net KB_IRQ12: now reaches U67.14 (P45/TxD)
- net at U67.22 (Xin): now also C264.1 (+), X5.2
- net at U67.23 (Xout): now also C268.1 (+), X5.1
- net KBCCS#: now reaches U67.6 (S#)
- net SA2: now reaches U67.7 (A0)
- net U8_2A1_KB_RXD: now reaches U73.11 (I0b)
- net ESS_IRQ1: now reaches U73.13 (I1b)
- net ESS_IRQ2: now reaches U73.15 (I2b)
- net M38_P14: now reaches U73.17 (I3b)
- net M38_P15_Buf: now reaches U73.18 (O0a)
- net M38_P15: now reaches U73.2 (I0a)
- net U8_1A3_KB_TP139: now reaches U73.6 (I2a)
- net ESS_IRQ1_Buf: now reaches U73.7 (O1b)
- net M38_P22_R88: now reaches U73.8 (I3a)
- net KB_CNTR#_Pluto renamed KB_CNTR#
- new net: U69.5, U69.7
- new net AEN: U69.6
- new net ESS_IRQ2_Buf: U73.5 (O2b)
- new net FDC_DS3: U69.1
- new net M38_P14_Buf: U73.3 (O3b)
- new net M38_P27_KB_SPKDN: U73.4 (I1a)
- new net Pluto_ESS_AEN: U69.2
- no-connect marks 2 -> 3
Other:
- moved on the sheet: C128, C136, C281, C283, J16, J17, Q8, R196, R198, R203, R206, R372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
