File: PCB/Mainboard/Keyboard.kicad_sch (KiCad schematic)
At the start: 33 parts, among them J16 Keyboard Conn 2, J17 Keyboard Conn 1, J19 Trackpoint, Q8 MUN2114, U69 SN74LVC2G32, U73 SN74LVT244B, X5 4.00, X6 8.00

Commit message: Add files via upload
Connections:
- net KB_SCLK#: no longer Q8.1 (B)
- net SD0_Bus renamed SD0
- net SD1_Bus renamed SD1
- net SD2_Bus renamed SD2
- net SD3_Bus renamed SD3
- net SD4_Bus renamed SD4
- net SD5_Bus renamed SD5
- net SD6_Bus renamed SD6
- net SD7_Bus renamed SD7
- new net KB_SCLK_shift: Q8.1 (B)
Other:
- note added: "Device_Address_BUS"
- note added: "Device_Data_BUS"
- moved on the sheet: C136, Q8, R45

Commit message: Add files via upload
Parts:
- added C267: DNP, symbol Device:C
- added C274, C275: 100nF, symbol Device:C
Connections:
- net GND: now also C267.2, C274.2, C275.2
- net KB_RESET#: now also C267.1
- net PNET1: now also C274.1, C275.1

Commit message: Add files via upload
Parts:
- C128, C136, C264, C267, C268, C274, C275, C281, C283: footprint (none) -> Capacitor_SMD:C_0402_1005Metric
- C135: footprint (none) -> Capacitor_SMD:C_0805_2012Metric
- D35, Q8: footprint (none) -> PC110:3D
- J16: footprint (none) -> PC110:Flat-20
- J17: footprint (none) -> PC110:Flat-8
- J19: footprint (none) -> PC110:Flat-18
- R196, R197, R198, R199, R200, R201, R202, R203, R204, R205, R206, R45, R59: footprint (none) -> PCM_Resistor_SMD_AKL:R_0402_1005Metric
- R372: footprint (none) -> Resistor_SMD:R_0402_1005Metric
- U67: footprint (none) -> PC110:QFN64
- U69: footprint (none) -> Package_SO:SSOP-8_2.95x2.8mm_P0.65mm
- U72: footprint (none) -> Package_SO:SSOP-24_5.3x8.2mm_P0.65mm
- U73: footprint (none) -> Package_SO:TSSOP-20_4.4x6.5mm_P0.65mm
- U75: footprint (none) -> PC110:SSOP-28
- X5: footprint (none) -> PC110:XTAL-5
- X6: footprint (none) -> PC110:XTAL-4
Connections:
- net Bowman_ESS_DACK1#: now also R372.2; no longer R372.1
- net D171_GPCLK: now also R198.1; no longer R198.2
- net D171_GPDATA: now also R203.1; no longer R203.2
- net D171_P0C2: now also R205.1; no longer R205.2
- net D171_P0C3: now also R201.1; no longer R201.2
- net GND: now also C128.2, C264.1 (+), C267.1, C268.1 (+), C281.1 (+), R199.1, R202.1; no longer C128.1, C264.2 (-), C267.2, C268.2 (-), C281.2 (-), R199.2, R202.2
- net KB_RESET#: now also C267.2; no longer C267.1
- net KB_SCLK#: now also R45.1; no longer R45.2
- net KB_SRDY#: now also R59.1; no longer R59.2
- net PNET1: now also C128.1, R372.1, R45.2, R59.2; no longer C128.2, R372.2, R45.1, R59.1
- net PNET3: now also R196.2, R197.2, R198.2, R200.2, R201.2, R203.2, R204.2, R205.2, R206.2; no longer R196.1, R197.1, R198.1, R200.1, R201.1, R203.1, R204.1, R205.1, R206.1
- net TRKPD_Lclick: now also R206.1; no longer R206.2
- net TRKPD_Rclick: now also R196.1; no longer R196.2
- net at C135.1 (+), D35.1 (A), D35.3 (A)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: now also R200.1; no longer R200.2
- net at U75.27 (Xin), X6.2: now also C281.2 (-); no longer C281.1 (+)
- net at U67.22 (Xin), X5.2: now also C264.2 (-); no longer C264.1 (+)
- net at U67.23 (Xout), X5.1: now also C268.2 (-); no longer C268.1 (+)
- new net: R197.1, R202.2, U75.17 (P1B0)
- new net: R199.2, R204.1, U75.15 (INT)
Other:
- moved on the sheet: C264, C268, C281, R196, R197, R198, R199, R200, R201, R202, R203, R204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

Commit message: Add files via upload
Parts:
- removed Q8: MUN2114, PC110:3D, symbol Transistor_BJT:DTA114Y
- added Q8: MUN2114, symbol PCM_Transistor_BJT_AKL:Q_PNP_Generic_ECB
Connections:
- net KB_SCLK_shift: now also Q8.3 (B)
- net PNET3: now also Q8.2 (C)
- net PNET5: now also Q8.1 (E)
Changed lines of the file:
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@@
 	(wire
 		(pts
-			(xy 140.97 241.3) (xy 147.32 241.3)
+			(xy 140.97 241.3) (xy 148.59 241.3)
 		)
 		(stroke
@@
 	)
 	(symbol
-		(lib_id "Transistor_BJT:DTA114Y")
-		(at 153.67 241.3 0)
-		(mirror x)
-		(unit 1)
-		(exclude_from_sim no)
-		(in_bom yes)
-		(on_board yes)
-		(dnp no)
-		(property "Reference" "Q8"
-			(at 159.004 240.2839 0)
-			(effects
-				(font
-					(size 1.27 1.27)
-				)
-				(justify left)
-			)
-		)
-		(property "Value" "MUN2114"
-			(at 158.75 242.57 0)
-			(effects
-				(font
-					(size 1.27 1.27)
-				)
-				(justify left)
-			)
-		)
-		(property "Footprint" "PC110:3D"
-			(at 153.67 241.3 0)
-			(effects
-				(font
-					(size 1.27 1.27)
-				)
-				(justify left)
-				(hide yes)
-			)
-		)
-		(property "Datasheet" ""
-			(at 153.67 241.3 0)
-			(effects
-				(font
-					(size 1.27 1.27)
-				)
-				(justify left)
-				(hide yes)
-			)
-		)
-		(property "Description" "Digital PNP Transistor, 10k/47k, SOT-23"
-			(at 153.67 241.3 0)
-			(effects
-				(font
-					(size 1.27 1.27)
-				)
-				(hide yes)
-			)
-		)
-		(property "Topmark" "6D"
-			(at 153.67 241.3 0)
-			(effects
-				(font
-					(size 1.27 1.27)
-				)
-				(hide yes)
-			)
-		)
-		(pin "2"
-		)
-		(pin "3"
-		)
-		(pin "1"
-		)
-		(instances
-			(project "PC110"
-				(path "/45c7911f-b027-440e-9e3e-77a146b41944/00000000-0000-0000-0000-0000655ddd04"
-					(reference "Q8")
-					(unit 1)
-				)
-			)
-		)
-	)
-	(symbol
 		(lib_id "power:GND")
 		(at 321.31 187.96 0)
@@
 					(unit 1)
 				)
+			)
+		)
+	)
+	(symbol
+		(lib_id "PCM_Transistor_BJT_AKL:Q_PNP_Generic_ECB")
+		(at 153.67 241.3 0)
+		(unit 1)
+		(exclude_from_sim no)
+		(in_bom yes)
+		(on_board yes)
+		(dnp no)
+		(property "Reference" "Q8"
+			(at 158.75 240.0299 0)
+			(effects
+				(font
+					(size 1.27 1.27)
+				)
+				(justify left)
+			)
+		)
+		(property "Value" "MUN2114"
+			(at 158.75 242.5699 0)
+			(effects
+				(font
+					(size 1.27 1.27)
+				)
+				(justify left)
+			)
+		)
+		(property "Footprint" ""
+			(at 158.75 238.76 0)
+			(effects
+				(font
+					(size 1.27 1.27)
+				)
+				(hide yes)
+			)
+		)
+		(property "Datasheet" "~"
+			(at 153.67 241.3 0)
+			(effects
+				(font
+					(size 1.27 1.27)
+				)
+				(hide yes)
+			)
+		)
+		(property "Description" "PNP transistor, generic symbol, Alternate KiCAD Library"
+			(at 153.67 241.3 0)
+			(effects
+				(font
+					(size 1.27 1.27)
+				)
+				(hide yes)
+			)
+		)
+		(pin "2"
+		)
+		(pin "3"
+		)
+		(pin "1"
+		)
+		(instances
+			(project "PC110"
+				(path "/45c7911f-b027-440e-9e3e-77a146b41944/00000000-0000-0000-0000-0000655ddd04"
+					(reference "Q8")
+					(unit 1)
+				)

Commit message: Add files via upload
Parts:
- Q8: footprint (none) -> PC110:3D
Changed lines of the file:
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@@
 			)
 		)
-		(property "Footprint" ""
+		(property "Footprint" "PC110:3D"
 			(at 158.75 238.76 0)
 			(effects

Commit message: Add files via upload
Parts:
- C135, C136, C264, C281, C283: Indicator + -> (none); Rating V -> (none)
- C268: value 56pF -> 56pf; Indicator + -> (none); Rating V -> (none)
- D35: value RB715F -> 3D; Topmark 3D -> (none)
- J16: value Keyboard Conn 2 -> Flat-20
- J17: value Keyboard Conn 1 -> Flat-8
- J19: value Trackpoint -> Flat-18
- Q8: value MUN2114 -> 6D
- R199, R202: now not fitted
- U67: value ~ -> M38813M4
- U72: value ~ -> HD151015
- U75: value ~ -> D17137AGT
Connections:
- net KB1_0: now also J17.8 (Pin_8); no longer J17.1 (Pin_1)
- net KB1_1: now also J17.7 (Pin_7); no longer J17.2 (Pin_2)
- net KB1_2: now also J17.1 (Pin_1); no longer J17.8 (Pin_8)
- net KB1_3: now also J17.6 (Pin_6); no longer J17.3 (Pin_3)
- net KB1_4: now also J17.2 (Pin_2); no longer J17.7 (Pin_7)
- net KB1_5: now also J17.5 (Pin_5); no longer J17.4 (Pin_4)
- net KB1_6: now also J17.3 (Pin_3); no longer J17.6 (Pin_6)
- net KB1_7: now also J17.4 (Pin_4); no longer J17.5 (Pin_5)
Other:
- moved on the sheet: J17

Commit message: Add files via upload
Connections:
- net at U75.26 (Xout), X6.1: now also C281.2 (-); no longer C283.1 (+)
- net at U75.27 (Xin), X6.2: now also C283.1 (+); no longer C281.2 (-)
Other:
- moved on the sheet: C281, C283
Changed lines of the file:
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@@
 	)
 	(junction
-		(at 373.38 101.6)
-		(diameter 0)
-		(color 0 0 0 0)
-	)
-	(junction
 		(at 257.81 217.17)
 		(diameter 0)
@@
 	)
 	(junction
+		(at 373.38 111.76)
+		(diameter 0)
+		(color 0 0 0 0)
+	)
+	(junction
 		(at 251.46 116.84)
 		(diameter 0)
@@
 	)
 	(junction
+		(at 373.38 101.6)
+		(diameter 0)
+		(color 0 0 0 0)
+	)
+	(junction
 		(at 41.91 149.86)
 		(diameter 0)
@@
 	)
 	(junction
-		(at 373.38 111.76)
-		(diameter 0)
-		(color 0 0 0 0)
-	)
-	(junction
 		(at 251.46 91.44)
 		(diameter 0)
@@
 	(wire
 		(pts
+			(xy 392.43 101.6) (xy 392.43 106.68)
+		)
+		(stroke
+			(width 0)
+			(type default)
+		)
+	)
+	(wire
+		(pts
 			(xy 224.79 212.09) (xy 224.79 198.12)
 		)
@@
 	(wire
 		(pts
-			(xy 325.12 105.41) (xy 325.12 121.92)
+			(xy 392.43 111.76) (xy 392.43 106.68)
 		)
 		(stroke
@@
 	(wire
 		(pts
-			(xy 255.27 91.44) (xy 255.27 106.68)
+			(xy 373.38 101.6) (xy 378.46 101.6)
 		)
 		(stroke
@@
 	(wire
 		(pts
-			(xy 251.46 106.68) (xy 251.46 116.84)
+			(xy 325.12 105.41) (xy 325.12 121.92)
 		)
 		(stroke
@@
 	(wire
 		(pts
-			(xy 49.53 234.95) (xy 55.88 234.95)
+			(xy 255.27 91.44) (xy 255.27 106.68)
 		)
 		(stroke
@@
 	(wire
 		(pts
-			(xy 106.68 179.07) (xy 106.68 181.61)
+			(xy 251.46 106.68) (xy 251.46 116.84)
 		)
 		(stroke
@@
 	(wire
 		(pts
-			(xy 334.01 105.41) (xy 334.01 139.7)
+			(xy 49.53 234.95) (xy 55.88 234.95)
 		)
 		(stroke
@@
 	(wire
 		(pts
-			(xy 316.23 116.84) (xy 369.57 116.84)
+			(xy 106.68 179.07) (xy 106.68 181.61)
 		)
 		(stroke
@@
 	(wire
 		(pts
-			(xy 49.53 252.73) (xy 55.88 252.73)
+			(xy 334.01 105.41) (xy 334.01 139.7)
 		)
 		(stroke
@@
 	(wire
 		(pts
-			(xy 219.71 262.89) (xy 219.71 260.35)
+			(xy 316.23 116.84) (xy 369.57 116.84)
 		)
 		(stroke
@@
 	(wire
 		(pts
-			(xy 114.3 39.37) (xy 114.3 54.61)
+			(xy 49.53 252.73) (xy 55.88 252.73)
 		)
 		(stroke
@@
 	(wire
 		(pts
-			(xy 114.3 64.77) (xy 114.3 83.82)
+			(xy 219.71 262.89) (xy 219.71 260.35)
 		)
 		(stroke
@@
 	(wire
 		(pts
-			(xy 156.21 267.97) (xy 156.21 270.51)
+			(xy 114.3 39.37) (xy 114.3 54.61)
 		)
 		(stroke
@@
 	(wire
 		(pts
-			(xy 304.8 119.38) (xy 309.88 119.38)
+			(xy 114.3 64.77) (xy 114.3 83.82)
 		)
 		(stroke
@@
 	(wire
 		(pts
-			(xy 392.43 111.76) (xy 392.43 106.68)
+			(xy 156.21 267.97) (xy 156.21 270.51)
 		)
 		(stroke
@@
 	(wire
 		(pts
-			(xy 325.12 91.44) (xy 316.23 91.44)
+			(xy 304.8 119.38) (xy 309.88 119.38)
 		)
 		(stroke
@@
 	(wire
 		(pts
-			(xy 49.53 250.19) (xy 55.88 250.19)
+			(xy 325.12 91.44) (xy 316.23 91.44)
 		)
 		(stroke
@@
 	(wire
 		(pts
-			(xy 106.68 193.04) (xy 101.6 193.04)
+			(xy 49.53 250.19) (xy 55.88 250.19)
 		)
 		(stroke
@@
 	(wire
 		(pts
-			(xy 392.43 101.6) (xy 392.43 106.68)
+			(xy 106.68 193.04) (xy 101.6 193.04)
 		)
 		(stroke
@@
 	(wire
 		(pts
-			(xy 373.38 101.6) (xy 379.73 101.6)
-		)
-		(stroke
-			(width 0)
-			(type default)
-		)
-	)
-	(wire
-		(pts
 			(xy 134.62 134.62) (xy 134.62 153.67)
 		)
@@
 	(wire
 		(pts
-			(xy 373.38 111.76) (xy 379.73 111.76)
-		)
-		(stroke
-			(width 0)
-			(type default)
-		)
-	)
-	(wire
-		(pts
 			(xy 276.86 219.71) (xy 284.48 219.71)
 		)
@@
 	(wire
 		(pts
-			(xy 389.89 111.76) (xy 392.43 111.76)
+			(xy 388.62 101.6) (xy 392.43 101.6)
 		)
 		(stroke
@@
 	(wire
 		(pts
+			(xy 373.38 111.76) (xy 378.46 111.76)
+		)
+		(stroke
+			(width 0)
+			(type default)
+		)
+	)
+	(wire
+		(pts
 			(xy 88.9 64.77) (xy 88.9 83.82)
 		)
@@
 	(wire
 		(pts
-			(xy 389.89 101.6) (xy 392.43 101.6)
+			(xy 388.62 111.76) (xy 392.43 111.76)
 		)
 		(stroke
@@
 		(on_board yes)
 		(dnp no)
-		(fields_autoplaced yes)
 		(property "Reference" "X6"
 			(at 369.57 105.4099 90)
@@
 	(symbol
 		(lib_id "PCM_Elektuur:C")
-		(at 384.81 111.76 90)
-		(mirror x)
+		(at 383.54 101.6 90)
 		(unit 1)
 		(exclude_from_sim no)
@@
 		(dnp no)
 		(property "Reference" "C283"
-			(at 384.81 115.062 90)
+			(at 383.54 98.298 90)
 			(effects
 				(font
@@
 		)
 		(property "Value" "39pF"
-			(at 385.064 116.84 90)
+			(at 383.794 96.52 90)
 			(effects
 				(font
@@
 		)
 		(property "Footprint" "Capacitor_SMD:C_0402_1005Metric"
-			(at 384.81 111.76 0)
+			(at 383.54 101.6 0)
 			(effects
 				(font
@@
 		)
 		(property "Datasheet" ""
-			(at 384.81 111.76 0)
+			(at 383.54 101.6 0)
 			(effects
 				(font
@@
 		)
 		(property "Description" ""
-			(at 384.81 111.76 0)
+			(at 383.54 101.6 0)
 			(effects
 				(font
@@
 	(symbol
 		(lib_id "PCM_Elektuur:C")
-		(at 384.81 101.6 270)
-		(mirror x)
+		(at 383.54 111.76 270)
 		(unit 1)
 		(exclude_from_sim no)
@@
 		(dnp no)
 		(property "Reference" "C281"
-			(at 384.81 95.25 90)
+			(at 383.54 118.11 90)
 			(effects
 				(font
@@
 		)
 		(property "Value" "39pF"
-			(at 384.81 97.79 90)
+			(at 383.54 115.57 90)
 			(effects
 				(font
@@
 		)
 		(property "Footprint" "Capacitor_SMD:C_0402_1005Metric"
-			(at 384.81 101.6 0)
+			(at 383.54 111.76 0)
 			(effects
 				(font
@@
 		)
 		(property "Datasheet" ""
-			(at 384.81 101.6 0)
+			(at 383.54 111.76 0)
 			(effects
 				(font
@@
 		)
 		(property "Description" ""
-			(at 384.81 101.6 0)
+			(at 383.54 111.76 0)
 			(effects
 				(font
