File: PCB/Mainboard/Super_IO.kicad_sch (KiCad schematic)
At the start: 19 parts, among them J13 Serial2, J14 Floppy, J15 Primary IDE, J4 Serial1, J5 Parallel, U12 FDC37C655GT, U213 GD75232N, U214 GD75232N, U67 74F245, U68 74F245, U69 74F541, Y5 24MHz

Commit message: Add files via upload
Parts:
- removed C61, C62: 22pF, Capacitor_SMD:C_0603_1608Metric_Pad1.08x0.95mm_HandSolder, symbol Device:C
- removed F2: 1.1A, Fuse:Fuse_Littelfuse_395Series, symbol Device:Polyfuse_Small
- removed J13: Serial2, Connector_PinHeader_2.54mm:PinHeader_2x05_P2.54mm_Vertical, symbol Connector_Generic:Conn_02x05_Odd_Even
- removed J14: Floppy, My_Components:Conn_Pin_Header_17x2_2.54mm_Shrouded, symbol Connector_Generic:Conn_02x17_Odd_Even
- removed J15: Primary IDE, My_Components:Conn_Pin_Header_20x2_2.54mm, symbol Connector_Generic:Conn_02x20_Odd_Even
- removed J4: Serial1, My_Components:Conn_Dsub_DE9M, symbol Connector:DB9_Male_MountingHoles
- removed J5: Parallel, My_Components:Conn_Dsub_DB25F, symbol Connector:DB25_Female_MountingHoles
- removed JP14: Super I/O IRQ, My_Components:Conn_Pin_Header_2x3_2.54mm, symbol Connector_Generic:Conn_02x03_Counter_Clockwise
- removed JP213: IDE1 CFG, My_Components:Conn_Pin_Header_2x3_2.54mm, symbol Connector_Generic:Conn_02x03_Counter_Clockwise
- removed RN17: 1k, Resistor_THT:R_Array_SIP6, symbol Device:R_Network05
- removed RN18: 2.2k, Resistor_THT:R_Array_SIP6, symbol Device:R_Network05
- removed U12: FDC37C655GT, My_Components:IC_PQFP-100_14x20mm_P0.65mm_Hand_Soldering, symbol my_components:FDC37C665GT
- removed U213, U214: GD75232N, My_Components:IC_DIP20_300, symbol Interface_UART:GD75232N
- removed U67, U68: 74F245, My_Components:IC_DIP20_300, symbol 74xx:74LS245
- removed U69: 74F541, My_Components:IC_DIP20_300, symbol 74xx:74LS541
- removed Y5: 24MHz, My_Components:Crystal_HC-49U_Vert, symbol Device:Crystal_Small
Connections:
- no-connect marks 18 -> 0
Other:
- note removed: "(CSEL)"
- note removed: "(DACK)"
- note removed: "(IORDY)"
- note removed: "(PDIAG)"
- note removed: "(~{ACTIVE})"
- note removed: "(~{IDE_DRQ})"

Commit message: Add files via upload
Parts:
- added U22: FDC37C665IR, symbol PC110:FDC37C665IR

Commit message: Add files via upload
Connections:
- net PWRGD: now reaches U22.56 (PWRGD)
Changed lines of the file:
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@@
 		(title "PC110")
+	)
+	(wire
+		(pts
+			(xy 62.23 137.16) (xy 88.9 137.16)
+		)
+		(stroke
+			(width 0)
+			(type default)
+		)
+	)
+	(label "PWRGD"
+		(at 71.12 137.16 180)
+		(effects
+			(font
+				(size 1.27 1.27)
+			)
+			(justify right bottom)
+		)
 	)
 	(symbol
@@
 		(on_board yes)
 		(dnp no)
-		(fields_autoplaced yes)
 		(property "Reference" "U22"
-			(at 149.4633 29.21 0)
+			(at 179.832 28.956 0)
 			(effects
 				(font
@@
 		)
 		(property "Value" "FDC37C665IR"
-			(at 149.4633 31.75 0)
+			(at 179.324 31.496 0)
 			(effects
 				(font

Commit message: Add files via upload
Connections:
- net FDD_INDEX#: now reaches U22.10 (INDEX#)
- net FDD_MOTEN: now reaches U22.100 (MTR0#)
- net FDC_TRK0#: now reaches U22.11 (TRK0#)
- net FDC_WRTPRT#: now reaches U22.12 (WRTPRT#)
- net PNET1: now reaches U22.13 (VCC)
- net PNET1: now also U22.70 (VCC)
- net FDC_DSKCHG#: now reaches U22.15 (DSKCHG#)
- net FDC_DRATE1: now reaches U22.16 (DRATE1)
- net FDC_DRATE0: now reaches U22.17 (DRATE0)
- net FDD_DRSEL: now reaches U22.2 (DS0#)
- net FDC_DIR#: now reaches U22.5 (DIR#)
- net FDC_STEP#: now reaches U22.6 (STEP#)
- net FDC_WGATE#: now reaches U22.8 (WGATE#)
- net FDC_HDSEL#: now reaches U22.9 (HDSEL#)
- net PNET5: now reaches U22.96 (VIO)
- no-connect marks 0 -> 3

Commit message: Add files via upload
Parts:
- added D24, D25: 3D, symbol Device:D_Dual_CommonCathode_AKA
- added R132, R133, R137: 2k, symbol Device:R
- added R136, R138, R140, R141, R142: 1k, symbol Device:R
- added R143: 10k, symbol Device:R
- added R310: 100k, symbol Device:R
- added R332: 33, symbol Device:R
Connections:
- net PNET1: now also R310.1
- net PNET5: now also D24.1 (A), D24.2 (A), D25.1 (A), D25.2 (A)
- net FDC_RDATA#: now reaches U22.14 (RDATA#)
- net at U22.18 (X1/CLK1): now also R332.2
- net GND: now reaches U22.4 (VSS)
- net GND: now also U22.45 (VSS), U22.65 (VSS), U22.93 (VSS)
- net FDC_SLCT: now reaches U22.57 (SLCT)
- net FDC_SLCT: now also R140.2
- net FDC_PE: now reaches U22.58 (PE)
- net FDC_PE: now also R138.2
- net FDC_BUSY: now reaches U22.59 (BUSY)
- net FDC_BUSY: now also R143.2
- net FDC_ACK#: now reaches U22.60 (ACK#)
- net FDC_ACK#: now also R136.2
- net FDC_PD7: now reaches U22.61 (PD7)
- net FDC_PD6: now reaches U22.62 (PD6)
- net FDC_PD5: now reaches U22.63 (PD5)
- net FDC_PD4: now reaches U22.64 (PD4)
- net FDC_PD3: now reaches U22.66 (PD3)
- net FDC_PD2: now reaches U22.67 (PD2)
- net FDC_PD1: now reaches U22.68 (PD1)
- net FDC_PD0: now reaches U22.69 (PD0)
- net FDC_WDATA#: now reaches U22.7 (WDATA#)
- net FDC_SLCTIN#: now reaches U22.71 (SLCTIN#)
- net FDC_SLCTIN#: now also R132.2
- net FDC_INIT#: now reaches U22.72 (INIT#)
- net FDC_INIT#: now also R133.2
- net FDC_ERROR#: now reaches U22.73 (ERROR#)
- net FDC_ERROR#: now also R142.2
- net FDC_AUTOFD#: now reaches U22.74 (AUTOFD#)
- net FDC_AUTOFD#: now also R141.2
- net FDC_STROBE#: now reaches U22.75 (STROBE#)
- net FDC_STROBE#: now also R137.2
- net FDC_RXD1: now reaches U22.76 (RXD1)
- net FDC_TXD1: now reaches U22.77 (TXD1)
- net FDC_DSR1: now reaches U22.78 (DSR1)
- net FDC_RTS1#: now reaches U22.79 (RTS1#)
- net FDC_CTS1#: now reaches U22.80 (CTS1#)
- net FDC_DTR1#: now reaches U22.81 (DTR1#)
- net FDC_RI1#: now reaches U22.82 (RI1#)
- net FDC_DCD1#: now reaches U22.83 (DCD1#)
- net FDC_RI2#: now reaches U22.84 (RI2#)
- net FDC_DCD2#: now reaches U22.85 (DCD2#)
- net FDC_DSR2#: now reaches U22.88 (DSR2#)
- net FDC_RTS2#: now reaches U22.89 (RTS2#)
- net FDC_CTS2#: now reaches U22.90 (CTS2#)
- net FDC_DTR2#: now reaches U22.91 (DTR2#)
- net FDC_MTR2#: now reaches U22.94 (MTR2#)
- net FDC_MTR2#: now also R310.2
- net FDC_MTR3#: now reaches U22.97 (MTR3#)
- new net: D25.3 (K), R133.1, R138.1, R140.1, R142.1, R143.1
- new net: D24.3 (K), R132.1, R136.1, R137.1, R141.1
- no-connect marks 3 -> 4
Other:
- moved on the sheet: U22

Commit message: Add files via upload
Parts:
- removed D24, D25: 3D, symbol Device:D_Dual_CommonCathode_AKA
- removed R332: 33, symbol Device:R
- added D24, D25: 3D, symbol PC110:D3_PC110
Connections:
- net PNET5: now also D24.1 (A), D24.3 (A), D25.1 (A), D25.3 (A)
- net at R133.1, R138.1, R140.1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: now also D25.2 (K)
- net at R132.1, R136.1, R137.1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: now also D24.2 (K)
- net FDC_CLK: now reaches U22.18 (X1/CLK1)
- net SA0: now reaches U22.26 (A0)
- net SA1: now reaches U22.27 (A1)
- net SA2: now reaches U22.28 (A2)
- net FDC_IRRX_RXD2: now reaches U22.86 (IRRX/RXD2)
- net FDC_IRTX_TXD2: now reaches U22.87 (IRTX/TXD2)
- net FCS_IOCHRDY: now reaches U22.98 (IOCHRDY)

Commit message: Add files via upload
Parts:
- added R118: 100k, symbol Device:R
Connections:
- net PNET1: now also R118.1
- net FDC_DACK#: now reaches U22.34 (DACK#)
- net FDC_DACK#: now also R118.2
- net FDC_DS3: now reaches U22.95 (A10)
Changed lines of the file:
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@@
+	(wire
+		(pts
+			(xy 36.83 113.03) (xy 36.83 115.57)
+		)
+		(stroke
+			(width 0)
+			(type default)
+		)
+	)
 	(wire
 		(pts
@@
 	(wire
 		(pts
+			(xy 36.83 127) (xy 88.9 127)
+		)
+		(stroke
+			(width 0)
+			(type default)
+		)
+	)
+	(wire
+		(pts
 			(xy 62.23 80.01) (xy 88.9 80.01)
 		)
@@
 	(wire
 		(pts
+			(xy 36.83 123.19) (xy 36.83 127)
+		)
+		(stroke
+			(width 0)
+			(type default)
+		)
+	)
+	(wire
+		(pts
 			(xy 326.39 95.25) (xy 381 95.25)
 		)
@@
 		(pts
 			(xy 113.03 181.61) (xy 111.76 181.61)
+		)
+		(stroke
+			(width 0)
+			(type default)
+		)
+	)
+	(wire
+		(pts
+			(xy 62.23 147.32) (xy 88.9 147.32)
 		)
 		(stroke
@@
 		)
 	)
+	(label "FDC_DACK#"
+		(at 63.5 127 0)
+		(effects
+			(font
+				(size 1.27 1.27)
+			)
+			(justify left bottom)
+		)
+	)
 	(label "FDC_DSR2#"
 		(at 209.55 140.97 0)
@@
 		)
 	)
+	(label "FDC_DS3"
+		(at 63.5 147.32 0)
+		(effects
+			(font
+				(size 1.27 1.27)
+			)
+			(justify left bottom)
+		)
+	)
 	(label "FDC_WDATA#"
 		(at 179.07 218.44 90)
@@
 			)
 			(justify left bottom)
+		)
+	)
+	(symbol
+		(lib_id "Device:R")
+		(at 36.83 119.38 0)
+		(unit 1)
+		(exclude_from_sim no)
+		(in_bom yes)
+		(on_board yes)
+		(dnp no)
+		(fields_autoplaced yes)
+		(property "Reference" "R118"
+			(at 39.37 118.1099 0)
+			(effects
+				(font
+					(size 1.27 1.27)
+				)
+				(justify left)
+			)
+		)
+		(property "Value" "100k"
+			(at 39.37 120.6499 0)
+			(effects
+				(font
+					(size 1.27 1.27)
+				)
+				(justify left)
+			)
+		)
+		(property "Footprint" ""
+			(at 35.052 119.38 90)
+			(effects
+				(font
+					(size 1.27 1.27)
+				)
+				(hide yes)
+			)
+		)
+		(property "Datasheet" "~"
+			(at 36.83 119.38 0)
+			(effects
+				(font
+					(size 1.27 1.27)
+				)
+				(hide yes)
+			)
+		)
+		(property "Description" "Resistor"
+			(at 36.83 119.38 0)
+			(effects
+				(font
+					(size 1.27 1.27)
+				)
+				(hide yes)
+			)
+		)
+		(pin "2"
+		)
+		(pin "1"
+		)
+		(instances
+			(project "PC110"
+				(path "/45c7911f-b027-440e-9e3e-77a146b41944/00000000-0000-0000-0000-00006bbfee6b"
+					(reference "R118")
+					(unit 1)
+				)
+			)
 		)
 	)
@@
 					(unit 1)
 				)
+			)
+		)
+	)
+	(symbol
+		(lib_id "power:VCC")
+		(at 36.83 113.03 0)
+		(unit 1)
+		(exclude_from_sim no)
+		(in_bom yes)
+		(on_board yes)
+		(dnp no)
+		(fields_autoplaced yes)
+		(property "Reference" "#PWR0358"
+			(at 36.83 116.84 0)
+			(effects
+				(font
+					(size 1.27 1.27)
+				)
+				(hide yes)
+			)
+		)
+		(property "Value" "PNET1"
+			(at 36.83 107.95 0)
+			(effects
+				(font
+					(size 1.27 1.27)
+				)
+			)
+		)
+		(property "Footprint" ""
+			(at 36.83 113.03 0)
+			(effects
+				(font
+					(size 1.27 1.27)
+				)
+				(hide yes)
+			)
+		)
+		(property "Datasheet" ""
+			(at 36.83 113.03 0)
+			(effects
+				(font
+					(size 1.27 1.27)
+				)
+				(hide yes)
+			)
+		)
+		(property "Description" "Power symbol creates a global label with name \"VCC\""
+			(at 36.83 113.03 0)
+			(effects
+				(font
+					(size 1.27 1.27)
+				)
+				(hide yes)
+			)
+		)
+		(pin "1"
+		)
+		(instances
+			(project "PC110"
+				(path "/45c7911f-b027-440e-9e3e-77a146b41944/00000000-0000-0000-0000-00006bbfee6b"
+					(reference "#PWR0358")
+					(unit 1)
+				)

Commit message: Add files via upload
Parts:
- added R319: 1k, symbol Device:R
- added U23: EA, symbol 74xGxx:74AHC1G14
- added U25: E4, symbol 74xGxx:74AUP1G02
Connections:
- net GND: now also U23.3 (GND), U25.3 (GND)
- net PNET1: now also U23.5 (VCC), U25.5 (VCC)
- net IOCS16#: now reaches U22.25 (IOCS16#)
- net IOCS16#: now also R319.2
- net IOR#: now reaches U22.42 (IOR#)
- net at U22.43 (IOW#): now also U25.4
- net AEN: now reaches U22.44 (AEN)
- new net: U23.4, U25.1
- new net FDC_IOW: U23.2
- new net IOW#: U25.2
- new net PNET7: R319.1
Other:
- moved on the sheet: D24, D25, R118, R132, R133, R136, R137, R138, R140, R141, R142, R143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
