File: PCB/Mainboard/Super_IO.kicad_sch (KiCad schematic)
At the start: 17 parts, among them U22 FDC37C665IR, U23 EA, U25 E4

Commit message: Add files via upload
Connections:
- net SD0_Bus renamed SD0
- net SD1_Bus renamed SD1
- net SD2_Bus renamed SD2
- net SD3_Bus renamed SD3
- net SD4_Bus renamed SD4
- net SD5_Bus renamed SD5
- net SD6_Bus renamed SD6
- net SD7_Bus renamed SD7
Other:
- note added: "Device_Address_BUS"
- note added: "Device_Data_BUS"

Commit message: Add files via upload
Parts:
- added C120, C83, C84: 100nF, symbol PCM_Elektuur:C
- added C244: 120nF, symbol Device:C
- added C247: 1nF, symbol Device:C
- added R314, R315: 470k, symbol Device:R
Connections:
- net FDC_IRRX_RXD2: now also R315.1
- net GND: now also C120.2 (-), C244.2, C247.2, C83.1 (+), C84.2 (-), R314.2
- net PNET1: now also C247.1, C83.2 (-)
- net PNET5: now also C120.1 (+), C244.1, C84.1 (+), R315.2
- net PWRGD: now also R314.1

Commit message: Add files via upload
Parts:
- C120, C244, C247, C83, C84: footprint (none) -> Capacitor_SMD:C_0402_1005Metric
- D24, D25: footprint (none) -> PC110:3D
- R118, R132, R133, R136, R137, R138, R140, R141, R142, R143, R314, R319: footprint (none) -> PCM_Resistor_SMD_AKL:R_0402_1005Metric
- R310, R315: footprint (none) -> Resistor_SMD:R_0402_1005Metric
- U22: footprint (none) -> PC110:FDC
- U23, U25: footprint (none) -> PC110:SOT-353
Connections:
- net FDC_ACK#: now also R136.1; no longer R136.2
- net FDC_AUTOFD#: now also R141.1; no longer R141.2
- net FDC_DACK#: now also R118.1; no longer R118.2
- net FDC_ERROR#: now also R142.1; no longer R142.2
- net FDC_INIT#: now also R133.1; no longer R133.2
- net FDC_MTR2#: now also R310.1; no longer R310.2
- net FDC_PE: now also R138.1; no longer R138.2
- net FDC_SLCTIN#: now also R132.1; no longer R132.2
- net FDC_STROBE#: now also R137.1; no longer R137.2
- net GND: now also C83.2 (-); no longer C83.1 (+)
- net PNET1: now also C83.1 (+), R118.2, R310.2; no longer C83.2 (-), R118.1, R310.1
- net at D25.2 (K), R140.1, R143.1: now also R133.2, R138.2, R142.2; no longer R133.1, R138.1, R142.1
- new net: D24.2 (K), R132.2, R136.2, R137.2, R141.2
Other:
- moved on the sheet: C83

Commit message: Add files via upload
Parts:
- C120, C83, C84: Indicator + -> (none); Rating V -> (none)
- D24, D25: value RB715F -> 3D; Topmark 3D -> (none)
Changed lines of the file:
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@@
 			)
 		)
-		(property "Datasheet" "http://www.ti.com/lit/sg/scyt129e/scyt129e.pdf"
+		(property "Datasheet" ""
 			(at 100.33 48.26 0)
 			(effects
@@
 			)
 		)
-		(property "Description" "Single OR Gate, Low-Voltage CMOS"
+		(property "Description" ""
 			(at 100.33 48.26 0)
 			(effects
@@
 			)
 		)
-		(property "Description" "Resistor"
+		(property "Description" ""
 			(at 38.1 148.59 0)
 			(effects
@@
 			)
 		)
-		(property "Description" "Resistor"
+		(property "Description" ""
 			(at 121.92 238.76 0)
 			(effects
@@
 			)
 		)
-		(property "Description" "Resistor"
+		(property "Description" ""
 			(at 337.82 110.49 0)
 			(effects
@@
 			)
 		)
-		(property "Description" "Resistor"
+		(property "Description" ""
 			(at 358.14 110.49 0)
 			(effects
@@
 			)
 		)
-		(property "Value" "RB715F"
+		(property "Value" "3D"
 			(at 337.82 86.36 0)
 			(effects
@@
 			)
 		)
-		(property "Description" "Dual Schottky diode, common cathode on pin 2"
-			(at 337.82 90.17 0)
-			(effects
-				(font
-					(size 1.27 1.27)
-				)
-				(hide yes)
-			)
-		)
-		(property "Topmark" "3D"
+		(property "Description" ""
 			(at 337.82 90.17 0)
 			(effects
@@
 			)
 		)
-		(property "Description" "Resistor"
+		(property "Description" ""
 			(at 237.49 156.21 0)
 			(effects
@@
 			)
 		)
-		(property "Value" "RB715F"
+		(property "Value" "3D"
 			(at 287.02 86.36 0)
 			(effects
@@
 			)
 		)
-		(property "Description" "Dual Schottky diode, common cathode on pin 2"
-			(at 287.02 90.17 0)
-			(effects
-				(font
-					(size 1.27 1.27)
-				)
-				(hide yes)
-			)
-		)
-		(property "Topmark" "3D"
+		(property "Description" ""
 			(at 287.02 90.17 0)
 			(effects
@@
 			)
 		)
-		(property "Description" "Resistor"
+		(property "Description" ""
 			(at 327.66 110.49 0)
 			(effects
@@
 			)
 		)
-		(property "Description" "Resistor"
+		(property "Description" ""
 			(at 292.1 110.49 0)
 			(effects
@@
 			)
 		)
-		(property "Description" "Resistor"
+		(property "Description" ""
 			(at 303.53 110.49 0)
 			(effects
@@
 			)
 		)
-		(property "Description" "Resistor"
+		(property "Description" ""
 			(at 270.51 110.49 0)
 			(effects
@@
 			)
 		)
-		(property "Description" "Resistor"
+		(property "Description" ""
 			(at 195.58 219.71 0)
 			(effects
@@
 			)
 		)
-		(property "Description" "Resistor"
+		(property "Description" ""
 			(at 82.55 203.2 0)
 			(effects
@@
 			)
 		)
-		(property "Description" "capacitor, non-polarized/bipolar"
+		(property "Description" ""
 			(at 160.02 82.55 0)
 			(effects
@@
 					(size 1.27 1.27)
 				)
-				(hide yes)
-			)
-		)
-		(property "Indicator" "+"
-			(at 156.845 83.82 0)
-			(effects
-				(font
-					(size 1.27 1.27)
-				)
-				(hide yes)
-			)
-		)
-		(property "Rating" "V"
-			(at 163.195 83.185 0)
-			(effects
-				(font
-					(size 1.27 1.27)
-				)
-				(justify right)
 				(hide yes)
 			)
@@
 			)
 		)
-		(property "Description" "Resistor"
+		(property "Description" ""
 			(at 316.23 110.49 0)
 			(effects
@@
 			)
 		)
-		(property "Description" "Resistor"
+		(property "Description" ""
 			(at 347.98 110.49 0)
 			(effects
@@
 			)
 		)
-		(property "Description" "Unpolarized capacitor"
+		(property "Description" ""
 			(at 312.42 81.28 0)
 			(effects
@@
 			)
 		)
-		(property "Description" "capacitor, non-polarized/bipolar"
+		(property "Description" ""
 			(at 270.51 85.09 0)
 			(effects
@@
 					(size 1.27 1.27)
 				)
-				(hide yes)
-			)
-		)
-		(property "Indicator" "+"
-			(at 273.685 86.36 0)
-			(effects
-				(font
-					(size 1.27 1.27)
-				)
-				(hide yes)
-			)
-		)
-		(property "Rating" "V"
-			(at 267.335 85.725 0)
-			(effects
-				(font
-					(size 1.27 1.27)
-				)
-				(justify right)
 				(hide yes)
 			)
@@
 			)
 		)
-		(property "Datasheet" "https://www.ti.com/lit/ds/symlink/sn74lvc1g14.pdf"
+		(property "Datasheet" ""
 			(at 151.13 52.07 0)
 			(effects
@@
 			)
 		)
-		(property "Description" "Single Schmitt NOT Gate, Low-Voltage CMOS"
+		(property "Description" ""
 			(at 151.13 45.72 0)
 			(effects
@@
 			)
 		)
-		(property "Description" "Unpolarized capacitor"
+		(property "Description" ""
 			(at 195.58 67.31 0)
 			(effects
@@
 			)
 		)
-		(property "Description" "capacitor, non-polarized/bipolar"
+		(property "Description" ""
 			(at 129.54 82.55 0)
 			(effects
@@
 					(size 1.27 1.27)
 				)
-				(hide yes)
-			)
-		)
-		(property "Indicator" "+"
-			(at 132.715 83.82 0)
-			(effects
-				(font
-					(size 1.27 1.27)
-				)
-				(hide yes)
-			)
-		)
-		(property "Rating" "V"
-			(at 126.365 83.185 0)
-			(effects
-				(font
-					(size 1.27 1.27)
-				)
-				(justify right)
 				(hide yes)
 			)
@@
 			)
 		)
-		(property "Description" "Resistor"
+		(property "Description" ""
 			(at 281.94 110.49 0)
 			(effects

Commit message: Add files via upload
Connections:
- net GND: now also C244.1; no longer C244.2
- net PNET5: now also C244.2; no longer C244.1
Other:
- moved on the sheet: C244
Changed lines of the file:
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@@
 	(symbol
 		(lib_id "Device:C")
-		(at 312.42 81.28 0)
-		(mirror y)
+		(at 312.42 81.28 180)
 		(unit 1)
 		(exclude_from_sim no)
@@
 		(dnp no)
 		(property "Reference" "C244"
-			(at 317.754 80.264 0)
+			(at 317.754 82.296 0)
 			(effects
 				(font
@@
 		)
 		(property "Value" "120nF"
-			(at 318.516 82.55 0)
+			(at 318.516 80.01 0)
 			(effects
 				(font
@@
 		)
 		(property "Footprint" "Capacitor_SMD:C_0402_1005Metric"
-			(at 311.4548 85.09 0)
+			(at 311.4548 77.47 0)
 			(effects
 				(font
