File: PCB/Mainboard/Audio.kicad_sch (KiCad schematic)
At the start: 56 parts, among them J10 Game/MIDI, J17 CD In, J18 Wave Table, J7 Line In, J8 Mic In, J9 Line Out, U19 AD1816AJS, Y6 24MHz

Commit message: Add files via upload
Parts:
- removed C140, C141: 18pF, Capacitor_SMD:C_0603_1608Metric_Pad1.08x0.95mm_HandSolder, symbol Device:C
- removed C142, C144, C168: 10uF, Capacitor_THT:CP_Radial_D5.0mm_P2.00mm, symbol Device:C_Polarized_US
- removed C143, C145, C146, C148, C165, C166, C167: 100nF, Capacitor_SMD:C_0603_1608Metric_Pad1.08x0.95mm_HandSolder, symbol Device:C
- removed C147: 47nF, Capacitor_SMD:C_0603_1608Metric_Pad1.08x0.95mm_HandSolder, symbol Device:C
- removed C149, C150: 560pF, Capacitor_SMD:C_0603_1608Metric_Pad1.08x0.95mm_HandSolder, symbol Device:C
- removed C151, C152: 1uF, Capacitor_THT:CP_Radial_D5.0mm_P2.00mm, symbol Device:C
- removed C153, C154, C157, C158: 1nF?, Capacitor_SMD:C_0603_1608Metric_Pad1.08x0.95mm_HandSolder, symbol Device:C
- removed C155, C156, C159, C160, C169, C170: 10nF, Capacitor_SMD:C_0603_1608Metric_Pad1.08x0.95mm_HandSolder, symbol Device:C
- removed C161, C162, C163, C164: 10nF?, Capacitor_SMD:C_0603_1608Metric_Pad1.08x0.95mm_HandSolder, symbol Device:C
- removed J10: Game/MIDI, Connector_Dsub:DSUB-15_Female_Horizontal_P2.77x2.84mm_EdgePinOffset4.94mm_Housed_MountingHolesOffset7.48mm, symbol Connector:DB15_Female
- removed J17: CD In, My_Components:Conn_Pin_Header_4x1_2.54mm, symbol Connector_Generic:Conn_01x04
- removed J18: Wave Table, My_Components:Conn_Pin_Header_13x2_2.54mm, symbol Connector_Generic:Conn_02x13_Odd_Even
- removed J7: Line In, My_Components:Conn_Audio_3.5mm_Stereo_SJ1-352XNG, symbol my_components:JACK_TRS_5PINS
- removed J8: Mic In, My_Components:Conn_Audio_3.5mm_Stereo_SJ1-352XNG, symbol my_components:JACK_TRS_5PINS
- removed J9: Line Out, My_Components:Conn_Audio_3.5mm_Stereo_SJ1-352XNG, symbol my_components:JACK_TRS_5PINS
- removed JP18: Speaker, My_Components:Conn_Pin_Header_2x1_2.54mm, symbol Jumper:Jumper_2_Open
- removed R141: 47k, Resistor_SMD:R_0612_1632Metric_Pad1.18x3.40mm_HandSolder, symbol Device:R
- removed R142: 1.2k, Resistor_SMD:R_0612_1632Metric_Pad1.18x3.40mm_HandSolder, symbol Device:R
- removed R143, R144, R145, R146: 1k, Resistor_SMD:R_0612_1632Metric_Pad1.18x3.40mm_HandSolder, symbol Device:R
- removed R147, R148, R149, R150, R152: 2.2k, Resistor_SMD:R_0612_1632Metric_Pad1.18x3.40mm_HandSolder, symbol Device:R
- removed R151: 4.7k, Resistor_SMD:R_0612_1632Metric_Pad1.18x3.40mm_HandSolder, symbol Device:R
- removed R153, R154: 10k, Resistor_SMD:R_0612_1632Metric_Pad1.18x3.40mm_HandSolder, symbol Device:R
- removed R155, R156: 20k, Resistor_SMD:R_0612_1632Metric_Pad1.18x3.40mm_HandSolder, symbol Device:R
- removed U19: AD1816AJS, My_Components:IC_PQFP-100_14x20mm_P0.65mm_Hand_Soldering, symbol my_components:AD1816AJS
- removed Y6: 24MHz, My_Components:Crystal_HC-49U_Vert, symbol Device:Crystal_Small
Connections:
- no-connect marks 20 -> 0
Other:
- note removed: "TODO: - Level adjustment for speaker input - Filter for analog supply voltage - Decoupling capacitors, including -12V/+12V for Wave Table"

Commit message: Add files via upload
Parts:
- added D19: 3D, symbol Device:D_Dual_CommonCathode_AKA
- added U10: YMF3812, symbol PC110:YM3812
- added U4: ~, symbol PC110:ES488
- added U5: 74HC14, symbol 74xx:74LS14
Connections:
- new net: D19.2 (K), U5.6
- new net: D19.1 (A), D19.3 (A)
- new net Enable_YMF_Bus: U10.3 (IC#), U5.5

Commit message: Add files via upload
Changed lines of the file:
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@@
-	)
-	(symbol
-		(lib_id "Device:D_Dual_CommonCathode_AKA")
-		(at 113.03 170.18 270)
-		(unit 1)
-		(exclude_from_sim no)
-		(in_bom yes)
-		(on_board yes)
-		(dnp no)
-		(fields_autoplaced yes)
-		(property "Reference" "D19"
-			(at 115.57 168.9099 90)
-			(effects
-				(font
-					(size 1.27 1.27)
-				)
-				(justify left)
-			)
-		)
-		(property "Value" "3D"
-			(at 115.57 171.4499 90)
-			(effects
-				(font
-					(size 1.27 1.27)
-				)
-				(justify left)
-			)
-		)
-		(property "Footprint" ""
-			(at 113.03 170.18 0)
-			(effects
-				(font
-					(size 1.27 1.27)
-				)
-				(hide yes)
-			)
-		)
-		(property "Datasheet" "~"
-			(at 113.03 170.18 0)
-			(effects
-				(font
-					(size 1.27 1.27)
-				)
-				(hide yes)
-			)
-		)
-		(property "Description" "Dual diode, common cathode on pin 2"
-			(at 113.03 170.18 0)
-			(effects
-				(font
-					(size 1.27 1.27)
-				)
-				(hide yes)
-			)
-		)
-		(pin "1"
-		)
-		(pin "3"
-		)
-		(pin "2"
-		)
-		(instances
-			(project "PC110"
-				(path "/45c7911f-b027-440e-9e3e-77a146b41944/00000000-0000-0000-0000-00006ffe9bec"
-					(reference "D19")
-					(unit 1)
-				)
-			)
-		)
 	)
 	(symbol
@@
 					(unit 1)
 				)
+			)
+		)
+	)
+	(symbol
+		(lib_id "Device:D_Dual_CommonCathode_AKA")
+		(at 113.03 170.18 270)
+		(mirror x)
+		(unit 1)
+		(exclude_from_sim no)
+		(in_bom yes)
+		(on_board yes)
+		(dnp no)
+		(property "Reference" "D19"
+			(at 119.38 170.18 0)
+			(effects
+				(font
+					(size 1.27 1.27)
+				)
+			)
+		)
+		(property "Value" "3D"
+			(at 116.84 170.18 0)
+			(effects
+				(font
+					(size 1.27 1.27)
+				)
+			)
+		)
+		(property "Footprint" ""
+			(at 113.03 170.18 0)
+			(effects
+				(font
+					(size 1.27 1.27)
+				)
+				(hide yes)
+			)
+		)
+		(property "Datasheet" "~"
+			(at 113.03 170.18 0)
+			(effects
+				(font
+					(size 1.27 1.27)
+				)
+				(hide yes)
+			)
+		)
+		(property "Description" "Dual diode, common cathode on pin 2"
+			(at 113.03 170.18 0)
+			(effects
+				(font
+					(size 1.27 1.27)
+				)
+				(hide yes)
+			)
+		)
+		(pin "1"
+		)
+		(pin "3"
+		)
+		(pin "2"
+		)
+		(instances
+			(project "PC110"
+				(path "/45c7911f-b027-440e-9e3e-77a146b41944/00000000-0000-0000-0000-00006ffe9bec"
+					(reference "D19")
+					(unit 1)
+				)

Commit message: Add files via upload
Parts:
- added U64: 74LV126, symbol 74xx:74LS126
Connections:
- new net PNET1: U64.13
Changed lines of the file:
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@@
+	(wire
+		(pts
+			(xy 53.34 54.61) (xy 92.71 54.61)
+		)
+		(stroke
+			(width 0)
+			(type default)
+		)
+	)
 	(wire
 		(pts
@@
 	(wire
 		(pts
-			(xy 67.31 170.18) (xy 86.36 170.18)
+			(xy 106.68 72.39) (xy 106.68 76.2)
 		)
 		(stroke
@@
 	(wire
 		(pts
-			(xy 34.29 113.03) (xy 57.15 113.03)
+			(xy 67.31 170.18) (xy 86.36 170.18)
 		)
 		(stroke
 			(width 0)
 			(type default)
+		)
+	)
+	(wire
+		(pts
+			(xy 34.29 113.03) (xy 57.15 113.03)
+		)
+		(stroke
+			(width 0)
+			(type default)
+		)
+	)
+	(label "Modem_Audio_Out"
+		(at 54.61 54.61 0)
+		(effects
+			(font
+				(size 1.27 1.27)
+			)
+			(justify left bottom)
 		)
 	)
@@
 					(unit 1)
 				)
+			)
+		)
+	)
+	(symbol
+		(lib_id "74xx:74LS126")
+		(at 106.68 82.55 0)
+		(mirror x)
+		(unit 4)
+		(exclude_from_sim no)
+		(in_bom yes)
+		(on_board yes)
+		(dnp no)
+		(property "Reference" "U64"
+			(at 106.68 91.44 0)
+			(effects
+				(font
+					(size 1.27 1.27)
+				)
+			)
+		)
+		(property "Value" "74LV126"
+			(at 106.68 88.9 0)
+			(effects
+				(font
+					(size 1.27 1.27)
+				)
+			)
+		)
+		(property "Footprint" ""
+			(at 106.68 82.55 0)
+			(effects
+				(font
+					(size 1.27 1.27)
+				)
+				(hide yes)
+			)
+		)
+		(property "Datasheet" "http://www.ti.com/lit/gpn/sn74LS126"
+			(at 106.68 82.55 0)
+			(effects
+				(font
+					(size 1.27 1.27)
+				)
+				(hide yes)
+			)
+		)
+		(property "Description" "Quad buffer 3-State outputs"
+			(at 106.68 82.55 0)
+			(effects
+				(font
+					(size 1.27 1.27)
+				)
+				(hide yes)
+			)
+		)
+		(pin "14"
+		)
+		(pin "9"
+		)
+		(pin "1"
+		)
+		(pin "7"
+		)
+		(pin "13"
+		)
+		(pin "2"
+		)
+		(pin "11"
+		)
+		(pin "6"
+		)
+		(pin "8"
+		)
+		(pin "10"
+		)
+		(pin "5"
+		)
+		(pin "12"
+		)
+		(pin "4"
+		)
+		(pin "3"
+		)
+		(instances
+			(project "PC110"
+				(path "/45c7911f-b027-440e-9e3e-77a146b41944/00000000-0000-0000-0000-00006ffe9bec"
+					(reference "U64")
+					(unit 4)
+				)
+			)
+		)
+	)
+	(symbol
+		(lib_id "power:VCC")
+		(at 106.68 72.39 0)
+		(unit 1)
+		(exclude_from_sim no)
+		(in_bom yes)
+		(on_board yes)
+		(dnp no)
+		(fields_autoplaced yes)
+		(property "Reference" "#PWR0252"
+			(at 106.68 76.2 0)
+			(effects
+				(font
+					(size 1.27 1.27)
+				)
+				(hide yes)
+			)
+		)
+		(property "Value" "PNET1"
+			(at 106.68 67.31 0)
+			(effects
+				(font
+					(size 1.27 1.27)
+				)
+			)
+		)
+		(property "Footprint" ""
+			(at 106.68 72.39 0)
+			(effects
+				(font
+					(size 1.27 1.27)
+				)
+				(hide yes)
+			)
+		)
+		(property "Datasheet" ""
+			(at 106.68 72.39 0)
+			(effects
+				(font
+					(size 1.27 1.27)
+				)
+				(hide yes)
+			)
+		)
+		(property "Description" "Power symbol creates a global label with name \"VCC\""
+			(at 106.68 72.39 0)
+			(effects
+				(font
+					(size 1.27 1.27)
+				)
+				(hide yes)
+			)
+		)
+		(pin "1"
+		)
+		(instances
+			(project "PC110"
+				(path "/45c7911f-b027-440e-9e3e-77a146b41944/00000000-0000-0000-0000-00006ffe9bec"
+					(reference "#PWR0252")
+					(unit 1)
+				)

Commit message: Add files via upload
Parts:
- added C100, C248: 10nF, symbol Device:C
- added C19, C205: 150nF, symbol Device:C
- added C213, C215, C57, C68: 100nF, symbol Device:C
- added C62: 120nF, symbol Device:C
- added R223: 100k, symbol Device:R
- added R243, R244, R245, R77: 470k, symbol Device:R
- added R250, R88: 0, symbol Device:R
- added R47, R48, R50, R54, R55, R56, R64, R65, R70: DNP, symbol Device:R
- added R92: 47, symbol Device:R
- added U18: 74HC74, symbol 74xx:74HC74
- added U20: 7W14, symbol 74xGxx:74LVC3G14
- added U23: 3E00, symbol PC110:QC01
- added U31: 3F01, symbol PC110:QC01
- added U34: 74LV126, symbol 74xx:74LS126
- added U46: ~, symbol PC110:YM3014
- added U49: ~, symbol PC110:HD151015
Connections:
- net Enable_YMF_Bus: now also U31.1 (OUT), U34.1, U34.10, U34.13, U34.4
- net PNET1: now also C215.2, U49.1 (VCCA)
- net PNET5: now reaches U4.20 (VCC)
- net PNET5: now also U4.27 (VCC), C19.2, R47.1, R48.1, R50.1, R54.1, R55.1, R56.1, R64.1, R65.1, R88.1, U34.14 (VCC)
- net GND: now reaches U4.22 (GND)
- net GND: now also U10.12 (GND), U4.26 (GND), U4.33 (GND), U4.5 (GND), C100.1, C19.1, C205.1, C215.1, C57.1, C62.1, C68.1, R223.2, R77.2, U18.7 (GND), U23.3 (GND), U31.3 (GND), U34.7 (GND), U49.12 (GND), U49.13 (GND)
- net at U4.23 (D0): now also U10.10 (D0), R64.2, U49.22 (B0)
- net at U4.24 (D1): now also U10.11 (D1), R54.2, U49.21 (B1)
- net at U4.25 (D2): now also U10.13 (D2), R47.2, U49.20 (B2)
- net at U4.28 (D3): now also U10.14 (D3), R50.2, U49.19 (B3)
- net at U4.29 (D4): now also U10.15 (D4), R65.2, U49.18 (B4)
- net at U4.30 (D5): now also U10.16 (D5), R55.2, U49.17 (B5)
- net at U4.31 (D6): now also U10.17 (D6), R48.2, U49.16 (B6)
- net at U4.32 (D7): now also U10.18 (D7), R56.2, U49.15 (B7)
- net at U4.34 (Xin): now also R70.1
- net ESS_DACK1#: now reaches U4.36 (DACK1#)
- net at U4.39 (RESET): now also U20.5
- net YMF_SA0_A0: now reaches U4.41 (A0)
- net YMF_SA0_A0: now also U34.12
- net at U4.44 (VCC_Bus): now also C213.1, U49.24 (VCCB)
- net PNET2: now reaches U10.1 (VCC)
- net PNET2: now also C205.2, C68.2, R243.1, R244.1, R245.1, U18.1 (~{R}), U18.10 (~{S}), U18.13 (~{R}), U18.14 (VCC), U18.4 (~{S})
- net at U10.23 (SY): now also U46.4 (LOAD)
- net at U10.24 (M): now also R92.2
- net at U10.4 (AO): now also R77.1, U34.11
- net at U10.5 (WR#): now also R245.2, U34.8
- net at U10.6 (RD#): now also R243.2, U34.6
- net at U10.7 (CS#): now also R244.2, U34.3
- new net: C213.2, R250.2
- new net: R223.1, U49.14 (B8)
- new net: C57.2, U23.5 (CD)
- new net: C100.2, U31.5 (CD)
- new net: C62.2, R88.2, U23.2 (VDD)
- new net: R92.1, U18.12 (D), U18.8 (~{Q})
- new net: U20.3, U23.1 (OUT)
- new net: U18.11 (C), U18.2 (D), U18.6 (~{Q})
- new net ESS_CLK: R70.2
- new net PWRGD_shift: C248.1
- new net YMF_CLK: U18.3 (C)
- no-connect marks 0 -> 14
Other:
- moved on the sheet: D19, U10, U4, U5C, U64D

Commit message: Add files via upload
Parts:
- added U66: 74LS02, symbol 74xx:74LS02
- added U68: SN74LV02, symbol 74xx:74LS02
- added U71: SN74LV32, symbol 74xx:74LS32
Connections:
- net YMF_RD#_Buf: now reaches U34.5
- net YMF_RD#_Buf: now also U71.12
- net at U4.37 (IOR): now also U71.11
- net at U4.38 (IOW): now also U71.8
- net YMF_WR#_Buf: now reaches U34.9
- net YMF_WR#_Buf: now also U71.9
- new net PWRGD_shift_buff: U71.10, U71.13
Other:
- moved on the sheet: D19, U5C

Commit message: Add files via upload
Parts:
- removed U68: SN74LV02, symbol 74xx:74LS02
- added R364: DNP, symbol Device:R
- added R370: 0, symbol Device:R
- added unit 1 of U66
- added unit 2 of U66
- renumbered U23 to U17
Connections:
- net at U49.2 (DIR): now also R364.1, R370.2
- net ESS_DRDY: now reaches U4.21 (DRDY)
- net ESS_DRDY: now also U66.6
- net at U66.10: now also R370.1
- net at U66.8: now also U66.1
- net at U66.9: now also U66.4
- new net IOR#: R364.2, U66.3, U66.5
- new net YMF_CS#_Buf: U66.2
Other:
- moved on the sheet: C68, D19, U18C, U34E, U5C, U66C

Commit message: Add files via upload
Parts:
- added R219: 100k, symbol Device:R
Connections:
- net GND: now also R219.2
- net SD7_Bus: now reaches U49.10 (A7)
- net at U49.11 (A8): now also R219.1
- net SD0_Bus: now reaches U49.3 (A0)
- net SD1_Bus: now reaches U49.4 (A1)
- net SD2_Bus: now reaches U49.5 (A2)
- net SD3_Bus: now reaches U49.6 (A3)
- net SD4_Bus: now reaches U49.7 (A4)
- net SD5_Bus: now reaches U49.8 (A5)
- net SD6_Bus: now reaches U49.9 (A6)
