File: PCB/Mainboard/Audio.kicad_sch (KiCad schematic)
At the start: 135 parts, among them J3 Audio-Jack, J7 Speaker, Q6 2SC4452, U10 YMF3812, U11 NJM2904M, U12 LM4861, U17 RN5VD? 3E, U18 VT74, U20 7W14, U31 RN5VD? 3F, U34 74LV126, U47 3414A, U48 DS1669, U5 74HC14, U64 74LV126, U66 74LS02, U71 SN74LV32, X2 89G6821

Commit message: Add files via upload
Parts:
- U17: value RN5VD? 3E -> 3E00
- U18: value 74HC74 -> VT74
Connections:
- net Bowman_Audio_Vol_Dn: now also U48.7 (DnC); no longer U48.3 (DnC)
- net Bowman_Audio_Vol_Up: now also U48.2 (UpC); no longer U48.3 (DnC)
- net SD0_Bus renamed SD0
- net SD1_Bus renamed SD1
- net SD2_Bus renamed SD2
- net SD3_Bus renamed SD3
- net SD4_Bus renamed SD4
- net SD5_Bus renamed SD5
- net SD6_Bus renamed SD6
- net SD7_Bus renamed SD7
- no-connect marks 24 -> 7
Other:
- note added: "Device_Address_BUS"
- note added: "Device_Data_BUS"
Changed lines of the file:
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@@
 		(company "Recreated by: Ahmad Byagowi")
 	)
+	(text "Device_Data_BUS"
+		(exclude_from_sim no)
+		(at 305.816 169.164 0)
+		(effects
+			(font
+				(size 1.27 1.27)
+			)
+		)
+	)
+	(text "Device_Address_BUS"
+		(exclude_from_sim no)
+		(at 347.726 141.224 0)
+		(effects
+			(font
+				(size 1.27 1.27)
+			)
+		)
+	)
 	(junction
 		(at 359.41 335.28)
@@
 	)
 	(no_connect
-		(at 172.72 149.86)
-	)
-	(no_connect
-		(at 185.42 149.86)
-	)
-	(no_connect
-		(at 177.8 149.86)
-	)
-	(no_connect
-		(at 167.64 149.86)
-	)
-	(no_connect
-		(at 436.88 194.31)
-	)
-	(no_connect
-		(at 240.03 118.11)
-	)
-	(no_connect
-		(at 240.03 120.65)
-	)
-	(no_connect
 		(at 173.99 78.74)
 	)
@@
 	)
 	(no_connect
-		(at 240.03 125.73)
-	)
-	(no_connect
 		(at 166.37 43.18)
 	)
 	(no_connect
-		(at 170.18 149.86)
-	)
-	(no_connect
-		(at 180.34 149.86)
-	)
-	(no_connect
-		(at 175.26 149.86)
-	)
-	(no_connect
 		(at 267.97 96.52)
 	)
 	(no_connect
-		(at 439.42 194.31)
-	)
-	(no_connect
 		(at 468.63 146.05)
 	)
 	(no_connect
-		(at 240.03 123.19)
-	)
-	(no_connect
-		(at 431.8 194.31)
-	)
-	(no_connect
 		(at 90.17 353.06)
 	)
@@
 		(at 434.34 248.92)
 	)
-	(no_connect
-		(at 429.26 194.31)
-	)
-	(no_connect
-		(at 434.34 194.31)
-	)
-	(no_connect
-		(at 182.88 149.86)
-	)
 	(bus_entry
 		(at 293.37 194.31)
@@
 	(bus
 		(pts
-			(xy 295.91 168.91) (xy 293.37 168.91)
+			(xy 302.26 166.37) (xy 293.37 166.37)
 		)
 		(stroke
@@
 	(wire
 		(pts
-			(xy 240.03 123.19) (xy 242.57 123.19)
-		)
-		(stroke
-			(width 0)
-			(type default)
-		)
-	)
-	(wire
-		(pts
 			(xy 335.28 207.01) (xy 335.28 209.55)
 		)
@@
 	(wire
 		(pts
-			(xy 240.03 120.65) (xy 242.57 120.65)
-		)
-		(stroke
-			(width 0)
-			(type default)
-		)
-	)
-	(wire
-		(pts
 			(xy 203.2 208.28) (xy 209.55 208.28)
 		)
@@
 	(wire
 		(pts
-			(xy 240.03 118.11) (xy 242.57 118.11)
-		)
-		(stroke
-			(width 0)
-			(type default)
-		)
-	)
-	(wire
-		(pts
 			(xy 280.67 105.41) (xy 280.67 177.8)
 		)
@@
 	(bus
 		(pts
-			(xy 384.81 138.43) (xy 360.68 138.43)
+			(xy 384.81 138.43) (xy 349.25 138.43)
 		)
 		(stroke
@@
 	(bus
 		(pts
-			(xy 293.37 168.91) (xy 293.37 176.53)
+			(xy 293.37 166.37) (xy 293.37 176.53)
 		)
 		(stroke
@@
 	(wire
 		(pts
-			(xy 240.03 125.73) (xy 242.57 125.73)
-		)
-		(stroke
-			(width 0)
-			(type default)
-		)
-	)
-	(wire
-		(pts
 			(xy 448.31 198.12) (xy 449.58 198.12)
 		)
@@
 		)
 	)
-	(label "SD6_Bus"
+	(label "SD6"
 		(at 307.34 194.31 180)
 		(effects
@@
 		)
 	)
-	(label "SD0_Bus"
+	(label "SD0"
 		(at 307.34 179.07 180)
 		(effects
@@
 		)
 	)
-	(label "YMF_CLK"
-		(at 124.46 81.28 0)
-		(effects
-			(font
-				(size 1.27 1.27)
-			)
-			(justify left bottom)
-		)
-	)
-	(label "IOR#"
-		(at 346.71 247.65 180)
-		(effects
-			(font
-				(size 1.27 1.27)
-			)
-			(justify right bottom)
-		)
-	)
-	(label "SD5_Bus"
+	(label "SD5"
 		(at 307.1751 191.77 180)
 		(effects
@@
 		)
 	)
-	(label "SD3_Bus"
+	(label "SD3"
 		(at 307.34 186.69 180)
 		(effects
@@
 		)
 	)
-	(label "SD1_Bus"
+	(label "SD1"
 		(at 307.34 181.61 180)
 		(effects
@@
 		)
 	)
-	(label "SD4_Bus"
+	(label "SD4"
 		(at 307.34 189.23 180)
 		(effects
@@
 		)
 	)
-	(label "SD7_Bus"
+	(label "SD7"
 		(at 307.34 196.85 180)
 		(effects
@@
 		)
 	)
-	(label "SD2_Bus"
+	(label "SD2"
 		(at 307.34 184.15 180)
 		(effects
@@
 		)
 	)
-	(global_label "Device_Data_BUS"
+	(global_label "SD[0..15]"
 		(shape input)
-		(at 295.91 168.91 0)
+		(at 302.26 166.37 0)
 		(fields_autoplaced yes)
 		(effects
@@
 		)
 		(property "Intersheetrefs" "${INTERSHEET_REFS}"
-			(at 315.0423 168.91 0)
+			(at 314.2562 166.37 0)
 			(effects
 				(font
@@
 		)
 	)
-	(global_label "Device_Address_BUS"
+	(global_label "SA[0..15]"
 		(shape input)
-		(at 360.68 138.43 180)
+		(at 349.25 138.43 180)
 		(fields_autoplaced yes)
 		(effects
@@
 		)
 		(property "Intersheetrefs" "${INTERSHEET_REFS}"
-			(at 338.5238 138.43 0)
+			(at 337.4352 138.43 0)
 			(effects
 				(font
@@
 		)
 	)
+	(global_label "IOR#"
+		(shape input)
+		(at 346.71 247.65 0)
+		(fields_autoplaced yes)
+		(effects
+			(font
+				(size 1.27 1.27)
+			)
+			(justify left)
+		)
+		(property "Intersheetrefs" "${INTERSHEET_REFS}"
+			(at 354.1705 247.65 0)
+			(effects
+				(font
+					(size 1.27 1.27)
+				)
+				(justify left)
+				(hide yes)
+			)
+		)
+	)
 	(global_label "PWRGD_shift"
 		(shape input)
@@
 		)
 	)
+	(global_label "YMF_CLK"
+		(shape input)
+		(at 124.46 81.28 180)
+		(fields_autoplaced yes)
+		(effects
+			(font
+				(size 1.27 1.27)
+			)
+			(justify right)
+		)
+		(property "Intersheetrefs" "${INTERSHEET_REFS}"
+			(at 113.3105 81.28 0)
+			(effects
+				(font
+					(size 1.27 1.27)
+				)
+				(justify right)
+				(hide yes)
+			)
+		)
+	)
 	(global_label "ESS_Sound"
 		(shape input)
@@
 		(pin "4"
 		)
-		(pin "2"
+		(pin "3"
 		)
 		(pin "16"
@@
 		(pin "3"
 		)
-		(pin "3"
+		(pin "7"
 		)
 		(pin "5"
 		)
-		(pin "3"
+		(pin "2"
 		)
 		(pin "8"
@@
 			)
 		)
-		(property "Value" "RN5VD? 3E"
+		(property "Value" "3E00"
 			(at 447.04 237.49 0)
 			(effects
@@
 			)
 		)
-		(property "Value" "74HC74"
+		(property "Value" "VT74"
 			(at 509.27 340.3599 0)
 			(effects
@@
 			)
 		)
-		(property "Value" "74HC74"
+		(property "Value" "VT74"
 			(at 196.4533 73.66 0)
 			(effects

Commit message: Add files via upload
Parts:
- removed D34: DNP, symbol PC110:D3_PC110
- added D34: DNP, symbol Device:D_Schottky_Dual_CommonCathode_AKA
- U31: value RN5VD? 3F -> RN5VD
Connections:
- net PNET2: now also D34.2 (K)
- net at C100.2, U31.5 (CD): now also D34.3 (A)
- net at C97.1, R195.2, U31.2 (VDD): now also D34.1 (A)
- no-connect marks 7 -> 5
Changed lines of the file:
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@@
 	)
 	(no_connect
-		(at 166.37 43.18)
-	)
-	(no_connect
 		(at 267.97 96.52)
 	)
@@
 		(at 90.17 353.06)
 	)
-	(no_connect
-		(at 434.34 248.92)
-	)
 	(bus_entry
 		(at 293.37 194.31)
@@
 	(wire
 		(pts
-			(xy 434.34 248.92) (xy 436.88 248.92)
-		)
-		(stroke
-			(width 0)
-			(type default)
-		)
-	)
-	(wire
-		(pts
 			(xy 331.47 147.32) (xy 331.47 152.4)
 		)
@@
 	(wire
 		(pts
-			(xy 166.37 43.18) (xy 167.64 43.18)
-		)
-		(stroke
-			(width 0)
-			(type default)
-		)
-	)
-	(wire
-		(pts
 			(xy 179.07 46.99) (xy 179.07 48.26)
 		)
@@
 	)
 	(symbol
+		(lib_id "Device:D_Schottky_Dual_CommonCathode_AKA")
+		(at 125.73 48.26 0)
+		(mirror x)
+		(unit 1)
+		(exclude_from_sim no)
+		(in_bom yes)
+		(on_board yes)
+		(dnp no)
+		(property "Reference" "D34"
+			(at 125.73 54.61 0)
+			(effects
+				(font
+					(size 1.27 1.27)
+				)
+			)
+		)
+		(property "Value" "DNP"
+			(at 125.73 52.07 0)
+			(effects
+				(font
+					(size 1.27 1.27)
+				)
+			)
+		)
+		(property "Footprint" ""
+			(at 125.73 48.26 0)
+			(effects
+				(font
+					(size 1.27 1.27)
+				)
+				(hide yes)
+			)
+		)
+		(property "Datasheet" "~"
+			(at 125.73 48.26 0)
+			(effects
+				(font
+					(size 1.27 1.27)
+				)
+				(hide yes)
+			)
+		)
+		(property "Description" "Dual Schottky diode, common cathode on pin 2"
+			(at 125.73 48.26 0)
+			(effects
+				(font
+					(size 1.27 1.27)
+				)
+				(hide yes)
+			)
+		)
+		(property "Topmark" "3D"
+			(at 125.73 48.26 0)
+			(effects
+				(font
+					(size 1.27 1.27)
+				)
+				(hide yes)
+			)
+		)
+		(pin "1"
+		)
+		(pin "3"
+		)
+		(pin "2"
+		)
+		(instances
+			(project "PC110"
+				(path "/45c7911f-b027-440e-9e3e-77a146b41944/00000000-0000-0000-0000-00006ffe9bec"
+					(reference "D34")
+					(unit 1)
+				)
+			)
+		)
+	)
+	(symbol
 		(lib_id "power:GND")
 		(at 109.22 274.32 0)
@@
 	)
 	(symbol
+		(lib_name "QC01_1")
 		(lib_id "PC110:QC01")
 		(at 447.04 245.11 0)
@@
 			)
 		)
-		(property "Value" "RN5VD? 3F"
+		(property "Value" "RN5VD"
 			(at 177.8 31.75 0)
 			(effects
@@
 				)
 			)
-		)
-	)
-	(symbol
-		(lib_id "PC110:D3_PC110")
-		(at 125.73 48.26 0)
-		(mirror x)
-		(unit 1)
-		(exclude_from_sim no)
-		(in_bom yes)
-		(on_board yes)
-		(dnp no)
-		(property "Reference" "D34"
-			(at 124.4599 50.8 90)
-			(effects
-				(font
-					(size 1.27 1.27)
-				)
-				(justify left)
-			)
-		)
-		(property "Value" "DNP"
-			(at 126.9999 50.8 90)
-			(effects
-				(font
-					(size 1.27 1.27)
-				)
-				(justify left)
-			)
-		)
-		(property "Footprint" ""
-			(at 125.73 48.26 0)
-			(effects
-				(font
-					(size 1.27 1.27)
-				)
-				(hide yes)
-			)
-		)
-		(property "Datasheet" "~"
-			(at 125.73 48.26 0)
-			(effects
-				(font
-					(size 1.27 1.27)
-				)
-				(hide yes)
-			)
-		)
-		(property "Description" "Dual diode, common cathode on pin 2"
-			(at 125.73 48.26 0)
-			(effects
-				(font
-					(size 1.27 1.27)
-				)
-				(hide yes)
-			)
-		)
-		(pin "1"
-		)
-		(pin "2"
-		)
-		(pin "3"
-		)
-		(instances
-			(project "PC110"
-				(path "/45c7911f-b027-440e-9e3e-77a146b41944/00000000-0000-0000-0000-00006ffe9bec"
-					(reference "D34")
-					(unit 1)
-				)
-			)

Commit message: Add files via upload
Parts:
- added C14, C204, C9: 10uF, symbol Device:C
- added C155, C203, C211, C212: 150nF, symbol Device:C
- added C208: 1nF, symbol Device:C
- added C6: DNP, symbol Device:C
- added D12: DNP, symbol Device:D_Dual_Series_KAC
- added R147: 470k, symbol Device:R
- added R28: 56, symbol Device:R
- added R29: 1k, symbol Device:R
Connections:
- net ESS_IRQ1: now also R29.2
- net Enable_YMF_Bus: now also R147.1
- net GND: now also C14.2, C155.2, C203.2, C204.2, C208.2, C211.2, C212.2, C6.1, C9.2, R147.2, R29.1
- net MIC_in_pin: now also C6.2
- net PNET1: now also C208.1, C211.1, C212.1
- net PNET2: now also C203.1, C204.1, R28.1
- net PNET5: now also D12.3 (common)
- net PNET6: now also C14.1, C9.1, R28.2
- net at C152.1, C161.1, R226.1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: now also C155.1
- net D11_2: now reaches C62.2, R88.2, U17.2 (VDD)
- net D11_2: now also D12.2 (A)
- net at U17.1 (OUT), U20.3: now also D12.1 (K)
Other:
- moved on the sheet: C10, C100, C11, C12, C13, C147, C148, C149, C15, C150, C151, C152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

Commit message: Add files via upload
Parts:
- C10, C14, C152, C160, C161, C162, C204, C209, C214, C23, C9: footprint (none) -> Capacitor_SMD:C_1206_3216Metric
- C100, C11, C12, C13, C147, C150, C153, C158, C164, C166, C18, C207, C21, C22, C248, C25, C57: footprint (none) -> Capacitor_SMD:C_0603_1608Metric
- C148, C149, C15, C151, C154, C155, C157, C159, C16, C165, C19, C20, C203, C205, C208, C211, C212, C213, C215, C24, C270, C44, C50, C52, C53, C6, C62, C68, C85, C97: footprint (none) -> Capacitor_SMD:C_0402_1005Metric
- C54: footprint (none) -> Capacitor_SMD:C_0805_2012Metric
- D12, D3, D34, D5: footprint (none) -> PC110:3D
- D40, Q6: footprint (none) -> PC110:SOT-416L
- J3: footprint (none) -> PC110:Audio-Jack
- J7: footprint (none) -> PC110:SPKR
- L13, L2, L5, L7, L8: footprint (none) -> Inductor_SMD:L_0603_1608Metric
- R120, R121, R147, R195, R217, R218, R219, R220, R221, R222, R223, R224, R225, R227, R23, R24, R25, R258, R26, R27, R29, R30, R32, R33, R34, R35, R36, R37, R47, R48, R50, R54, R55, R56, R64, R65, R67, R69, R70, R71, R72, R73, R74, R75, R77, R78, R88, R92: footprint (none) -> PCM_Resistor_SMD_AKL:R_0402_1005Metric
- R226, R28: footprint (none) -> PCM_Resistor_SMD_AKL:R_1206_3216Metric
- R243, R244, R245, R247, R364, R370: footprint (none) -> Resistor_SMD:R_0402_1005Metric
- R250, R256: footprint (none) -> PCM_Resistor_SMD_AKL:R_0805_2012Metric
- U10: footprint (none) -> PC110:SOP-24
- U11: footprint (none) -> PC110:soic-8-small
- U12: footprint (none) -> PC110:SOIC-8-narrow
- U17, U31: footprint (none) -> Package_TO_SOT_SMD:SOT-23-5
- U18, U34, U5, U64, U66, U71: footprint (none) -> Package_SO:TSSOP-14_4.4x5mm_P0.65mm
- U20: footprint (none) -> PC110:sso-8
- U4: footprint (none) -> PC110:QFN-52
- U46: footprint (none) -> PC110:SOP-16
- U47, U48: footprint (none) -> PC110:SOIC-8
- U49: footprint (none) -> Package_SO:SSOP-24_5.3x8.2mm_P0.65mm
- X2: footprint (none) -> PC110:XTAL-1
Connections:
- net D11_2: now also R88.1; no longer R88.2
- net ESS_CLK: now also R70.1; no longer R70.2
- net ESS_IRQ1: now also R29.1; no longer R29.2
- net GND: now also C100.2, C151.2, C155.1, C165.2, C203.1, C204.1, C205.2, C208.1, C211.1, C215.2, C54.2, C68.2, R219.1, R29.2; no longer C100.1, C151.1, C155.2, C165.1, C203.2, C204.2, C205.1, C208.2, C211.2, C215.1, C54.1, C68.1, R219.2, R29.1
- net PCMCIA_Sound: now also R120.2; no longer R120.1
- net PNET1: now also C208.2, C211.2, C215.1, R120.1; no longer C208.1, C211.1, C215.2, R120.2
- net PNET2: now also C203.2, C204.2, C205.1, C68.1, R28.2; no longer C203.1, C204.1, C205.2, C68.2, R28.1
- net PNET5: now also R48.2, R55.2, R56.2, R88.2; no longer R48.1, R55.1, R56.1, R88.1
- net PNET6: now also C151.1, R28.1, R36.1; no longer C151.2, R28.2, R36.2
- net at U49.11 (A8): now also R219.2; no longer R219.1
- net at U10.18 (D7), U4.32 (D7), U49.15 (B7): now also R56.1; no longer R56.2
- net at U10.17 (D6), U4.31 (D6), U49.16 (B6): now also R48.1; no longer R48.2
- net at U10.16 (D5), U4.30 (D5), U49.17 (B5): now also R55.1; no longer R55.2
- net at C25.1 (+), Q6.1 (C): now also R36.2; no longer R36.1
- net at C152.1, C161.1, R226.1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: now also C155.2; no longer C155.1
- net at R256.1, U11.8 (V+), U46.1 (VDD): now also C157.1, C209.1; no longer C157.2, C209.2
- net at D34.3 (A), U31.5 (CD): now also C100.1; no longer C100.2
- net at C10.1 (+), L7.1 (+): now also C23.1 (+); no longer C23.2 (-)
- net at C10.2 (-), C154.2 (-), R227.2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: now also C23.2 (-); no longer C23.1 (+)
- net at R250.2, U11.4 (V-), U46.12 (GND): now also C157.2, C209.2; no longer C157.1, C209.1
- net at J3.2 (SI), L7.2 (-): now also C165.1; no longer C165.2
- net at C44.2, U46.2 (toBUFF): now also R69.2; no longer R69.1
- net at U11.2 (-), U46.16 (MP): now also R67.2; no longer R67.1
- net at U11.5 (+): now also R69.1; no longer R69.2
- net at U11.6 (-): now also R72.2; no longer R72.1
- net at C11.1 (+), C50.2, U11.7: now also R72.1; no longer R72.2
- net at U12.2 (Bypass), U12.3 (IN+): now also C54.1; no longer C54.2
- net at C52.1, U4.34 (Xin), X2.1: now also R70.2; no longer R70.1
- net at R73.2, U11.1: now also R67.1; no longer R67.2
Other:
- moved on the sheet: C151, C203, C204, C208, C211, C23, C68, R120, R219, R28, R29, R36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

Commit message: Add files via upload
Parts:
- removed Q6: 2SC4452, PC110:SOT-416L, symbol Simulation_SPICE:NPN
- added Q6: 2SC4452, symbol PCM_Transistor_BJT_AKL:Q_NPN_Generic_EBC
Connections:
- net GND: now also Q6.1 (E)
- net at C25.1 (+), R36.2: now also Q6.3 (C)
- net at D5.2 (K), R71.1, R74.1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: now also Q6.2 (B)
Changed lines of the file:
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@@
+	)
+	(symbol
+		(lib_id "PCM_Transistor_BJT_AKL:Q_NPN_Generic_EBC")
+		(at 102.87 264.16 0)
+		(mirror y)
+		(unit 1)
+		(exclude_from_sim no)
+		(in_bom yes)
+		(on_board yes)
+		(dnp no)
+		(property "Reference" "Q6"
+			(at 97.79 262.8899 0)
+			(effects
+				(font
+					(size 1.27 1.27)
+				)
+				(justify left)
+			)
+		)
+		(property "Value" "2SC4452"
+			(at 97.79 265.4299 0)
+			(effects
+				(font
+					(size 1.27 1.27)
+				)
+				(justify left)
+			)
+		)
+		(property "Footprint" ""
+			(at 97.79 261.62 0)
+			(effects
+				(font
+					(size 1.27 1.27)
+				)
+				(hide yes)
+			)
+		)
+		(property "Datasheet" "~"
+			(at 102.87 264.16 0)
+			(effects
+				(font
+					(size 1.27 1.27)
+				)
+				(hide yes)
+			)
+		)
+		(property "Description" "NPN transistor, generic symbol, Alternate KiCAD Library"
+			(at 102.87 264.16 0)
+			(effects
+				(font
+					(size 1.27 1.27)
+				)
+				(hide yes)
+			)
+		)
+		(pin "2"
+		)
+		(pin "3"
+		)
+		(pin "1"
+		)
+		(instances
+			(project ""
+				(path "/45c7911f-b027-440e-9e3e-77a146b41944/00000000-0000-0000-0000-00006ffe9bec"
+					(reference "Q6")
+					(unit 1)
+				)
+			)
+		)
 	)
 	(symbol
@@
 					(unit 1)
 				)
-			)
-		)
-	)
-	(symbol
-		(lib_id "Simulation_SPICE:NPN")
-		(at 102.87 264.16 0)
-		(mirror y)
-		(unit 1)
-		(exclude_from_sim no)
-		(in_bom yes)
-		(on_board yes)
-		(dnp no)
-		(property "Reference" "Q6"
-			(at 97.79 262.8899 0)
-			(effects
-				(font
-					(size 1.27 1.27)
-				)
-				(justify left)
-			)
-		)
-		(property "Value" "2SC4452"
-			(at 97.79 265.4299 0)
-			(effects
-				(font
-					(size 1.27 1.27)
-				)
-				(justify left)
-			)
-		)
-		(property "Footprint" "PC110:SOT-416L"
-			(at 39.37 264.16 0)
-			(effects
-				(font
-					(size 1.27 1.27)
-				)
-				(hide yes)
-			)
-		)
-		(property "Datasheet" "https://ngspice.sourceforge.io/docs/ngspice-html-manual/manual.xhtml#cha_BJTs"
-			(at 39.37 264.16 0)
-			(effects
-				(font
-					(size 1.27 1.27)
-				)
-				(hide yes)
-			)
-		)
-		(property "Description" "Bipolar transistor symbol for simulation only, substrate tied to the emitter"
-			(at 102.87 264.16 0)
-			(effects
-				(font
-					(size 1.27 1.27)
-				)
-				(hide yes)
-			)
-		)
-		(property "Sim.Device" "NPN"
-			(at 102.87 264.16 0)
-			(effects
-				(font
-					(size 1.27 1.27)
-				)
-				(hide yes)
-			)
-		)
-		(property "Sim.Type" "GUMMELPOON"
-			(at 102.87 264.16 0)
-			(effects
-				(font
-					(size 1.27 1.27)
-				)
-				(hide yes)
-			)
-		)
-		(property "Sim.Pins" "1=C 2=B 3=E"
-			(at 102.87 264.16 0)
-			(effects
-				(font
-					(size 1.27 1.27)
-				)
-				(hide yes)
-			)
-		)
-		(property "Topmark" "ST3"
-			(at 102.87 264.16 0)
-			(effects
-				(font
-					(size 1.27 1.27)
-				)
-				(hide yes)
-			)
-		)
-		(pin "2"
-		)
-		(pin "1"
-		)
-		(pin "3"
-		)
-		(instances
-			(project "PC110"
-				(path "/45c7911f-b027-440e-9e3e-77a146b41944/00000000-0000-0000-0000-00006ffe9bec"
-					(reference "Q6")
-					(unit 1)
-				)

Commit message: Add files via upload
Parts:
- Q6: footprint (none) -> PC110:SOT-416L
Changed lines of the file:
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@@
 			)
 		)
-		(property "Footprint" ""
+		(property "Footprint" "PC110:SOT-416L"
 			(at 97.79 261.62 0)
 			(effects

Commit message: Add files via upload
Parts:
- C10, C24: Indicator + -> (none); Rating V -> (none); now not fitted
- C11, C12, C13, C147, C15, C150, C154, C160, C162, C166, C18, C20, C207, C21, C22, C23, C25, C85: Indicator + -> (none); Rating V -> (none)
- C149: value 1uF -> 100nF
- C248: value 10nF -> 1uF
- C270, C50, C6, R47, R48, R50, R54, R55, R56, R64, R65: now not fitted
- D12: Topmark K -> (none); now not fitted
- D3, D5: value RB715F -> 3D; Topmark 3D -> (none)
- D34: Topmark 3D -> (none); now not fitted
- D40: value DAN222 -> N; Topmark N -> (none)
- J7: value Speaker -> SPKR
- L13, L2, L5, L7, L8: Indicator ● -> (none); Rating A -> (none)
- Q6: value 2SC4452 -> ST3
- R71, R78: value 10K -> 10k
- U10: value YMF3812 -> YM3812
- U17: Topmark 3E00 -> (none)
- U31: value RN5VD -> 3F01; Topmark 3F01 -> (none)
- U4: value ~ -> ES488F
- U46: value ~ -> Y3014
- U49: value ~ -> HD151015
- U64: value 74LV126 -> SN74LV126
- U66: value 74LS02 -> SN74LV02
- X2: Frequency 14.318MHz? -> (none)
Connections:
- net IOR#: now also R364.1; no longer R364.2
- net at R370.1: now also R364.2, U49.2 (DIR); no longer U66.10
- new net: R370.2, U66.10
Other:
- moved on the sheet: R364, R370

Commit message: Add files via upload
Parts:
- removed D12: DNP, PC110:3D, symbol Device:D_Dual_Series_KAC
- added D12: DNP, PC110:3D, symbol Device:D_Schottky_Dual_CommonCathode_AKA
Connections:
- net D11_2: now also D12.1 (A)
- net PNET5: now also D12.2 (K)
- net at C57.2, U17.5 (CD): now also D12.3 (A)
- net at C44.2, R69.2: now also U11.5 (+); no longer U46.2 (toBUFF)
- net at R69.1: now also U46.2 (toBUFF); no longer U11.5 (+)
Other:
- moved on the sheet: C44, R69
