File: PCB/Mainboard/PCMCIA.kicad_sch (KiCad schematic)
At the start: 0 parts

Commit message: Add files via upload
Parts:
- added U74: RB5C396, symbol PC110:RB5C396

Commit message: Add files via upload
Parts:
- added J10: PCMCIA Connector, symbol PC110:PCMCIA_Conn

Commit message: Add files via upload
Parts:
- added R160: 470k, symbol Device:R
- added U38: 7W14, symbol 74xGxx:74LVC3G14
Connections:
- net RIOUT#: now reaches U74.C8 (RIOUT#)
- net at U74.M4 (CS#): now also U38.2
- new net GND: R160.1
- new net PCMCIA_CS: R160.2, U38.6

Commit message: Add files via upload
Parts:
- added U70: TPS2201, symbol PC110:TPS2201
- added U71: SN74LV32, symbol 74xx:74LS32
Connections:
- new net PWRGD_shift_buff: U71.10, U71.13
Other:
- moved on the sheet: J10, R160, U38B, U74

Commit message: Add files via upload
Parts:
- added R317: 33, symbol Device:R
Connections:
- net at U74.C1 (SYSCLK): now also R317.2
- net SA1: now reaches U74.D4 (SA1)
- net SA0: now reaches U74.F5 (SA0)
- net FCS_IOCHRDY: now reaches U74.K3 (IOCHRDY)
- net PCMCIA_ZEROWS#: now reaches U74.L3 (ZEROWS#)
- new net PCMCIA_CLK: R317.1
Other:
- moved on the sheet: R160, U38B
Changed lines of the file:
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@@
 	)
 	(junction
-		(at 110.49 374.65)
+		(at 97.79 372.11)
 		(diameter 0)
 		(color 0 0 0 0)
@@
 	(wire
 		(pts
+			(xy 132.08 372.11) (xy 161.29 372.11)
+		)
+		(stroke
+			(width 0)
+			(type default)
+		)
+	)
+	(wire
+		(pts
+			(xy 132.08 374.65) (xy 161.29 374.65)
+		)
+		(stroke
+			(width 0)
+			(type default)
+		)
+	)
+	(wire
+		(pts
+			(xy 132.08 227.33) (xy 161.29 227.33)
+		)
+		(stroke
+			(width 0)
+			(type default)
+		)
+	)
+	(wire
+		(pts
 			(xy 132.08 152.4) (xy 161.29 152.4)
 		)
@@
 	(wire
 		(pts
-			(xy 110.49 374.65) (xy 110.49 377.19)
-		)
-		(stroke
-			(width 0)
-			(type default)
-		)
-	)
-	(wire
-		(pts
-			(xy 110.49 384.81) (xy 110.49 387.35)
+			(xy 97.79 372.11) (xy 97.79 374.65)
+		)
+		(stroke
+			(width 0)
+			(type default)
+		)
+	)
+	(wire
+		(pts
+			(xy 132.08 388.62) (xy 132.08 374.65)
+		)
+		(stroke
+			(width 0)
+			(type default)
+		)
+	)
+	(wire
+		(pts
+			(xy 97.79 382.27) (xy 97.79 384.81)
 		)
 		(stroke
@@
 	(wire
 		(pts
-			(xy 110.49 374.65) (xy 116.84 374.65)
-		)
-		(stroke
-			(width 0)
-			(type default)
-		)
-	)
-	(wire
-		(pts
-			(xy 144.78 374.65) (xy 161.29 374.65)
+			(xy 97.79 372.11) (xy 104.14 372.11)
+		)
+		(stroke
+			(width 0)
+			(type default)
+		)
+	)
+	(wire
+		(pts
+			(xy 81.28 407.67) (xy 132.08 407.67)
+		)
+		(stroke
+			(width 0)
+			(type default)
+		)
+	)
+	(wire
+		(pts
+			(xy 132.08 229.87) (xy 161.29 229.87)
 		)
 		(stroke
@@
 	(wire
 		(pts
+			(xy 132.08 364.49) (xy 161.29 364.49)
+		)
+		(stroke
+			(width 0)
+			(type default)
+		)
+	)
+	(wire
+		(pts
+			(xy 132.08 367.03) (xy 161.29 367.03)
+		)
+		(stroke
+			(width 0)
+			(type default)
+		)
+	)
+	(wire
+		(pts
+			(xy 132.08 396.24) (xy 132.08 407.67)
+		)
+		(stroke
+			(width 0)
+			(type default)
+		)
+	)
+	(wire
+		(pts
 			(xy 680.72 445.77) (xy 676.91 445.77)
 		)
@@
 	(wire
 		(pts
-			(xy 93.98 374.65) (xy 110.49 374.65)
+			(xy 81.28 372.11) (xy 97.79 372.11)
 		)
 		(stroke
@@
 		)
 	)
+	(label "PCMCIA_CLK"
+		(at 83.82 407.67 0)
+		(effects
+			(font
+				(size 1.27 1.27)
+			)
+			(justify left bottom)
+		)
+	)
+	(label "SA0"
+		(at 133.35 227.33 0)
+		(effects
+			(font
+				(size 1.27 1.27)
+			)
+			(justify left bottom)
+		)
+	)
 	(label "PCMCIA_CS"
-		(at 96.52 374.65 0)
+		(at 83.82 372.11 0)
+		(effects
+			(font
+				(size 1.27 1.27)
+			)
+			(justify left bottom)
+		)
+	)
+	(label "PCMCIA_ZEROWS#"
+		(at 133.35 364.49 0)
+		(effects
+			(font
+				(size 1.27 1.27)
+			)
+			(justify left bottom)
+		)
+	)
+	(label "SA1"
+		(at 133.35 229.87 0)
+		(effects
+			(font
+				(size 1.27 1.27)
+			)
+			(justify left bottom)
+		)
+	)
+	(label "FCS_IOCHRDY"
+		(at 133.35 367.03 0)
 		(effects
 			(font
@@
 	(symbol
 		(lib_id "power:GND")
-		(at 110.49 387.35 0)
+		(at 97.79 384.81 0)
 		(unit 1)
 		(exclude_from_sim no)
@@
 		(fields_autoplaced yes)
 		(property "Reference" "#PWR0142"
-			(at 110.49 393.7 0)
+			(at 97.79 391.16 0)
 			(effects
 				(font
@@
 		)
 		(property "Value" "GND"
-			(at 110.49 392.43 0)
+			(at 97.79 389.89 0)
 			(effects
 				(font
@@
 		)
 		(property "Footprint" ""
-			(at 110.49 387.35 0)
+			(at 97.79 384.81 0)
 			(effects
 				(font
@@
 		)
 		(property "Datasheet" ""
-			(at 110.49 387.35 0)
+			(at 97.79 384.81 0)
 			(effects
 				(font
@@
 		)
 		(property "Description" "Power symbol creates a global label with name \"GND\" , ground"
-			(at 110.49 387.35 0)
+			(at 97.79 384.81 0)
 			(effects
 				(font
@@
 	(symbol
 		(lib_id "74xGxx:74LVC3G14")
-		(at 132.08 374.65 0)
+		(at 119.38 372.11 0)
 		(unit 2)
 		(exclude_from_sim no)
@@
 		(dnp no)
 		(property "Reference" "U38"
-			(at 131.064 383.286 0)
+			(at 118.364 380.746 0)
 			(effects
 				(font
@@
 		)
 		(property "Value" "7W14"
-			(at 130.81 381 0)
+			(at 118.11 378.46 0)
 			(effects
 				(font
@@
 		)
 		(property "Footprint" ""
-			(at 130.81 374.65 0)
+			(at 118.11 372.11 0)
 			(effects
 				(font
@@
 		)
 		(property "Datasheet" "https://www.ti.com/lit/ds/symlink/sn74lvc3g14.pdf"
-			(at 132.08 374.65 0)
+			(at 119.38 372.11 0)
 			(effects
 				(font
@@
 		)
 		(property "Description" "Triple NOT Gate Schmitt, Low-Voltage CMOS"
-			(at 132.08 374.65 0)
+			(at 119.38 372.11 0)
 			(effects
 				(font
@@
 	(symbol
 		(lib_id "Device:R")
-		(at 110.49 381 180)
+		(at 132.08 392.43 0)
+		(mirror x)
+		(unit 1)
+		(exclude_from_sim no)
+		(in_bom yes)
+		(on_board yes)
+		(dnp no)
+		(property "Reference" "R317"
+			(at 129.54 391.1599 0)
+			(effects
+				(font
+					(size 1.27 1.27)
+				)
+				(justify right)
+			)
+		)
+		(property "Value" "33"
+			(at 129.54 393.6999 0)
+			(effects
+				(font
+					(size 1.27 1.27)
+				)
+				(justify right)
+			)
+		)
+		(property "Footprint" ""
+			(at 130.302 392.43 90)
+			(effects
+				(font
+					(size 1.27 1.27)
+				)
+				(hide yes)
+			)
+		)
+		(property "Datasheet" "~"
+			(at 132.08 392.43 0)
+			(effects
+				(font
+					(size 1.27 1.27)
+				)
+				(hide yes)
+			)
+		)
+		(property "Description" "Resistor"
+			(at 132.08 392.43 0)
+			(effects
+				(font
+					(size 1.27 1.27)
+				)
+				(hide yes)
+			)
+		)
+		(pin "2"
+		)
+		(pin "1"
+		)
+		(instances
+			(project "PC110"
+				(path "/45c7911f-b027-440e-9e3e-77a146b41944/00000000-0000-0000-0000-0000639b00c7"
+					(reference "R317")
+					(unit 1)
+				)
+			)
+		)
+	)
+	(symbol
+		(lib_id "Device:R")
+		(at 97.79 378.46 180)
 		(unit 1)
 		(exclude_from_sim no)
@@
 		(fields_autoplaced yes)
 		(property "Reference" "R160"
-			(at 113.03 379.7299 0)
+			(at 100.33 377.1899 0)
 			(effects
 				(font
@@
 		)
 		(property "Value" "470k"
-			(at 113.03 382.2699 0)
+			(at 100.33 379.7299 0)
 			(effects
 				(font
@@
 		)
 		(property "Footprint" ""
-			(at 112.268 381 90)
+			(at 99.568 378.46 90)
 			(effects
 				(font
@@
 		)
 		(property "Datasheet" "~"
-			(at 110.49 381 0)
+			(at 97.79 378.46 0)
 			(effects
 				(font
@@
 		)
 		(property "Description" "Resistor"
-			(at 110.49 381 0)
-			(effects
-				(font
+			(at 97.79 378.46 0)
+			(effects
+				(font

Commit message: Add files via upload
Parts:
- removed U71: SN74LV32, symbol 74xx:74LS32
Changed lines of the file:
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@@
-		(color 0 0 0 0)
-	)
-	(junction
-		(at 680.72 440.69)
-		(diameter 0)
 		(color 0 0 0 0)
 	)
 	(wire
 		(pts
-			(xy 680.72 440.69) (xy 708.66 440.69)
+			(xy 132.08 372.11) (xy 161.29 372.11)
 		)
 		(stroke
@@
 	(wire
 		(pts
-			(xy 132.08 372.11) (xy 161.29 372.11)
+			(xy 132.08 374.65) (xy 161.29 374.65)
 		)
 		(stroke
@@
 	(wire
 		(pts
-			(xy 132.08 374.65) (xy 161.29 374.65)
+			(xy 132.08 227.33) (xy 161.29 227.33)
 		)
 		(stroke
@@
 	(wire
 		(pts
-			(xy 132.08 227.33) (xy 161.29 227.33)
+			(xy 132.08 152.4) (xy 161.29 152.4)
 		)
 		(stroke
@@
 	(wire
 		(pts
-			(xy 132.08 152.4) (xy 161.29 152.4)
+			(xy 97.79 372.11) (xy 97.79 374.65)
 		)
 		(stroke
@@
 	(wire
 		(pts
-			(xy 97.79 372.11) (xy 97.79 374.65)
+			(xy 132.08 388.62) (xy 132.08 374.65)
 		)
 		(stroke
@@
 	(wire
 		(pts
-			(xy 132.08 388.62) (xy 132.08 374.65)
+			(xy 97.79 382.27) (xy 97.79 384.81)
 		)
 		(stroke
@@
 	(wire
 		(pts
-			(xy 97.79 382.27) (xy 97.79 384.81)
+			(xy 97.79 372.11) (xy 104.14 372.11)
 		)
 		(stroke
@@
 	(wire
 		(pts
-			(xy 680.72 435.61) (xy 676.91 435.61)
+			(xy 81.28 407.67) (xy 132.08 407.67)
 		)
 		(stroke
@@
 	(wire
 		(pts
-			(xy 97.79 372.11) (xy 104.14 372.11)
+			(xy 132.08 229.87) (xy 161.29 229.87)
 		)
 		(stroke
@@
 	(wire
 		(pts
-			(xy 81.28 407.67) (xy 132.08 407.67)
+			(xy 132.08 364.49) (xy 161.29 364.49)
 		)
 		(stroke
@@
 	(wire
 		(pts
-			(xy 132.08 229.87) (xy 161.29 229.87)
+			(xy 132.08 367.03) (xy 161.29 367.03)
 		)
 		(stroke
@@
 	(wire
 		(pts
-			(xy 680.72 440.69) (xy 680.72 445.77)
+			(xy 132.08 396.24) (xy 132.08 407.67)
 		)
 		(stroke
@@
 	(wire
 		(pts
-			(xy 132.08 364.49) (xy 161.29 364.49)
-		)
-		(stroke
-			(width 0)
-			(type default)
-		)
-	)
-	(wire
-		(pts
-			(xy 132.08 367.03) (xy 161.29 367.03)
-		)
-		(stroke
-			(width 0)
-			(type default)
-		)
-	)
-	(wire
-		(pts
-			(xy 132.08 396.24) (xy 132.08 407.67)
-		)
-		(stroke
-			(width 0)
-			(type default)
-		)
-	)
-	(wire
-		(pts
-			(xy 680.72 445.77) (xy 676.91 445.77)
-		)
-		(stroke
-			(width 0)
-			(type default)
-		)
-	)
-	(wire
-		(pts
 			(xy 81.28 372.11) (xy 97.79 372.11)
-		)
-		(stroke
-			(width 0)
-			(type default)
-		)
-	)
-	(wire
-		(pts
-			(xy 680.72 440.69) (xy 680.72 435.61)
 		)
 		(stroke
@@
 			)
 			(justify left bottom)
-		)
-	)
-	(label "PWRGD_shift_buff"
-		(at 707.39 440.69 180)
-		(effects
-			(font
-				(size 1.27 1.27)
-			)
-			(justify right bottom)
 		)
 	)
@@
 				)
 			)
-		)
-	)
-	(symbol
-		(lib_id "74xx:74LS32")
-		(at 669.29 433.07 0)
-		(mirror y)
-		(unit 3)
-		(exclude_from_sim no)
-		(in_bom yes)
-		(on_board yes)
-		(dnp no)
-		(property "Reference" "U71"
-			(at 669.29 424.18 0)
-			(effects
-				(font
-					(size 1.27 1.27)
-				)
-			)
-		)
-		(property "Value" "SN74LV32"
-			(at 669.29 426.72 0)
-			(effects
-				(font
-					(size 1.27 1.27)
-				)
-			)
-		)
-		(property "Footprint" ""
-			(at 669.29 433.07 0)
-			(effects
-				(font
-					(size 1.27 1.27)
-				)
-				(hide yes)
-			)
-		)
-		(property "Datasheet" "http://www.ti.com/lit/gpn/sn74LS32"
-			(at 669.29 433.07 0)
-			(effects
-				(font
-					(size 1.27 1.27)
-				)
-				(hide yes)
-			)
-		)
-		(property "Description" "Quad 2-input OR"
-			(at 669.29 433.07 0)
-			(effects
-				(font
-					(size 1.27 1.27)
-				)
-				(hide yes)
-			)
-		)
-		(pin "1"
-		)
-		(pin "2"
-		)
-		(pin "3"
-		)
-		(pin "4"
-		)
-		(pin "5"
-		)
-		(pin "6"
-		)
-		(pin "9"
-		)
-		(pin "10"
-		)
-		(pin "8"
-		)
-		(pin "12"
-		)
-		(pin "13"
-		)
-		(pin "11"
-		)
-		(pin "14"
-		)
-		(pin "7"
-		)
-		(instances
-			(project "PC110"
-				(path "/45c7911f-b027-440e-9e3e-77a146b41944/00000000-0000-0000-0000-0000639b00c7"
-					(reference "U71")
-					(unit 3)
-				)
-			)
-		)
-	)
-	(symbol
-		(lib_id "74xx:74LS32")
-		(at 669.29 448.31 180)
-		(unit 4)
-		(exclude_from_sim no)
-		(in_bom yes)
-		(on_board yes)
-		(dnp no)
-		(property "Reference" "U71"
-			(at 669.29 457.2 0)
-			(effects
-				(font
-					(size 1.27 1.27)
-				)
-			)
-		)
-		(property "Value" "SN74LV32"
-			(at 669.29 454.66 0)
-			(effects
-				(font
-					(size 1.27 1.27)
-				)
-			)
-		)
-		(property "Footprint" ""
-			(at 669.29 448.31 0)
-			(effects
-				(font
-					(size 1.27 1.27)
-				)
-				(hide yes)
-			)
-		)
-		(property "Datasheet" "http://www.ti.com/lit/gpn/sn74LS32"
-			(at 669.29 448.31 0)
-			(effects
-				(font
-					(size 1.27 1.27)
-				)
-				(hide yes)
-			)
-		)
-		(property "Description" "Quad 2-input OR"
-			(at 669.29 448.31 0)
-			(effects
-				(font
-					(size 1.27 1.27)
-				)
-				(hide yes)
-			)
-		)
-		(pin "1"
-		)
-		(pin "2"
-		)
-		(pin "3"
-		)
-		(pin "4"
-		)
-		(pin "5"
-		)
-		(pin "6"
-		)
-		(pin "9"
-		)
-		(pin "10"
-		)
-		(pin "8"
-		)
-		(pin "12"
-		)
-		(pin "13"
-		)
-		(pin "11"
-		)
-		(pin "14"
-		)
-		(pin "7"
-		)
-		(instances
-			(project "PC110"
-				(path "/45c7911f-b027-440e-9e3e-77a146b41944/00000000-0000-0000-0000-0000639b00c7"
-					(reference "U71")
-					(unit 4)
-				)
-			)

Commit message: Add files via upload
Connections:
- net IOCS16#: now reaches U74.B1 (IOCS16#)
- net IRQ14: now reaches U74.B4 (IRQ14)
- net MEMR#: now reaches U74.B5 (MEMR#)
- net MEMW#: now reaches U74.D6 (MEMW#)
- net AEN: now reaches U74.K1 (AEN)
Changed lines of the file:
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@@
+	(wire
+		(pts
+			(xy 132.08 293.37) (xy 161.29 293.37)
+		)
+		(stroke
+			(width 0)
+			(type default)
+		)
+	)
 	(wire
 		(pts
@@
 	(wire
 		(pts
+			(xy 132.08 354.33) (xy 161.29 354.33)
+		)
+		(stroke
+			(width 0)
+			(type default)
+		)
+	)
+	(wire
+		(pts
 			(xy 97.79 372.11) (xy 104.14 372.11)
 		)
@@
 	(wire
 		(pts
+			(xy 132.08 359.41) (xy 161.29 359.41)
+		)
+		(stroke
+			(width 0)
+			(type default)
+		)
+	)
+	(wire
+		(pts
 			(xy 132.08 367.03) (xy 161.29 367.03)
 		)
@@
 		(pts
 			(xy 132.08 396.24) (xy 132.08 407.67)
+		)
+		(stroke
+			(width 0)
+			(type default)
+		)
+	)
+	(wire
+		(pts
+			(xy 132.08 351.79) (xy 161.29 351.79)
+		)
+		(stroke
+			(width 0)
+			(type default)
+		)
+	)
+	(wire
+		(pts
+			(xy 132.08 219.71) (xy 161.29 219.71)
 		)
 		(stroke
@@
 		)
 	)
+	(label "MEMR#"
+		(at 133.35 351.79 0)
+		(effects
+			(font
+				(size 1.27 1.27)
+			)
+			(justify left bottom)
+		)
+	)
+	(label "AEN"
+		(at 133.35 293.37 0)
+		(effects
+			(font
+				(size 1.27 1.27)
+			)
+			(justify left bottom)
+		)
+	)
 	(label "FCS_IOCHRDY"
 		(at 133.35 367.03 0)
@@
 		)
 	)
+	(label "MEMW#"
+		(at 133.35 354.33 0)
+		(effects
+			(font
+				(size 1.27 1.27)
+			)
+			(justify left bottom)
+		)
+	)
 	(label "RIOUT#"
 		(at 133.35 152.4 0)
 		(effects
 			(font
+				(size 1.27 1.27)
+			)
+			(justify left bottom)
+		)
+	)
+	(label "IOCS16#"
+		(at 133.35 359.41 0)
+		(effects
+			(font
+				(size 1.27 1.27)
+			)
+			(justify left bottom)
+		)
+	)
+	(label "IRQ14"
+		(at 133.35 219.71 0)
+		(effects
+			(font

Commit message: Add files via upload
Parts:
- added R316: 1k, symbol Device:R
Connections:
- net LA22: now reaches U74.A1 (LA22)
- net LA21: now reaches U74.A2 (LA21)
- net LA19: now reaches U74.A3 (LA19)
- net LA17: now reaches U74.A4 (LA17)
- net PCMCIA_SBHE#: now reaches U74.C3 (SBHE#)
- net LA18: now reaches U74.C5 (LA18)
- net PCMCIA_BALE: now reaches U74.D1 (BALE)
- net MEMCS16#: now reaches U74.D3 (MEMCS16#)
- net MEMCS16#: now also R316.2
- net LA23: now reaches U74.E5 (LA23)
- net LA20: now reaches U74.E6 (LA20)
- net PCMCIA_REFRESH: now reaches U74.H1 (REFRESH#)
- net Chipset_SA16: now reaches U74.J1 (SA16)
- net IOW#: now reaches U74.J2 (IOW#)
- net IOR#: now reaches U74.J3 (IOR#)
- net PCMCIA_Sound: now reaches U74.N3 (SPKROUT#)
- net RESET: now reaches U74.T3 (RESETDRV)
- new net PNET7: R316.1
