File: PCB/Mainboard/PCMCIA.kicad_sch (KiCad schematic)
At the start: 26 parts, among them J10 PCMCIA Connector, U38 7W14, U70 TPS2201, U74 RB5C396

Commit message: Add files via upload
Connections:
- net GND: now also U74.P1 (POWERGOOD)
- net PNET10: now also J10.34 (VCC), J10.35 (VCC)
- net PNET9: now also J10.104 (VCC), J10.105 (VCC)
- net SD0_Bus renamed SD0
- net SD10_Bus renamed SD10
- net SD11_Bus renamed SD11
- net SD12_Bus renamed SD12
- net SD13_Bus renamed SD13
- net SD15_Bus renamed SD14
- net SD14: no longer U74.B8 (SD15)
- net SD1_Bus renamed SD1
- net SD2_Bus renamed SD2
- net SD3_Bus renamed SD3
- net SD4_Bus renamed SD4
- net SD5_Bus renamed SD5
- net SD6_Bus renamed SD6
- net SD7_Bus renamed SD7
- net SD8_Bus renamed SD8
- net SD9_Bus renamed SD9
- new net SD15: U74.B8 (SD15)
Other:
- note added: "Device_Address_BUS"
- note added: "Device_Data_BUS"

Commit message: Add files via upload
Parts:
- added C115, C116, C119, C122, C276: 100nF, symbol Device:C
- added R117, R165, R177, R312: 47k, symbol Device:R
- added R163, R164, R166, R168, R169, R170, R172, R174, R175, R176, R178, R179: 10k, symbol Device:R
Connections:
- net ABVD1: now also R163.2
- net ABVD2: now also R176.2
- net ACD1#: now also R117.2
- net ACD2#: now also R177.2
- net AINPACK#: now also R179.2
- net ARDY: now also R174.2
- net AWAIT: now also R164.2
- net AWP: now also R168.2
- net BBVD1: now also R175.2
- net BBVD2: now also R170.2
- net BCD1#: now also R312.2
- net BCD2#: now also R165.2
- net BINPACK#: now also R172.2
- net BRDY: now also R166.2
- net BWAIT: now also R169.2
- net BWP: now also R178.2
- net GND: now also C115.2, C116.1, C119.1, C122.2, C276.2
- net PNET1: now also C115.1, C122.1, R117.1, R165.1, R177.1, R312.1
- net PNET10: now also C119.2, R163.1, R164.1, R168.1, R174.1, R176.1, R179.1
- net PNET5: now also C276.1
- net PNET9: now also C116.2, R166.1, R169.1, R170.1, R172.1, R175.1, R178.1

Commit message: Add files via upload
Parts:
- C114, C115, C116, C119, C122, C126, C276, C278, C279, C87: footprint (none) -> Capacitor_SMD:C_0402_1005Metric
- C124, C273: footprint (none) -> Capacitor_SMD:C_0603_1608Metric
- J10: footprint (none) -> PC110:PCMCIA
- R115, R117, R126, R160, R162, R163, R164, R165, R166, R168, R169, R170, R172, R174, R175, R176, R177, R178, R179, R316, R317: footprint (none) -> PCM_Resistor_SMD_AKL:R_0402_1005Metric
- R312, R325, R363, R379, R384, R387, R389, R391, R394, R396: footprint (none) -> Resistor_SMD:R_0402_1005Metric
- U38: footprint (none) -> PC110:sso-8
- U70: footprint (none) -> Package_SO:TSSOP-30_6.1x9.7mm_P0.65mm
- U74: footprint (none) -> PC110:BGA-256
Connections:
- net AVPP: now also C124.2 (-); no longer C124.1 (+)
- net BBVD1: now also R175.1; no longer R175.2
- net BCD2#: now also R165.1; no longer R165.2
- net BINPACK#: now also R172.1; no longer R172.2
- net BWP: now also R178.1; no longer R178.2
- net GND: now also C116.2, C119.2, C124.1 (+); no longer C116.1, C119.1, C124.2 (-)
- net PCMCIA_CLK: now also R317.2; no longer R317.1
- net PNET1: now also R165.2; no longer R165.1
- net PNET10: now also C119.1; no longer C119.2
- net PNET9: now also C116.1, R172.2, R175.2, R178.2; no longer C116.2, R172.1, R175.1, R178.1
- net at U74.C1 (SYSCLK): now also R317.1; no longer R317.2
Other:
- moved on the sheet: C116, C119

Commit message: Add files via upload
Connections:
- net GND: now also U74.F11 (GND); no longer U74.F100 (GND)
Changed lines of the file:
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@@
 		(pin "E11"
 		)
-		(pin "F100"
+		(pin "F11"
 		)
 		(pin "F10"

Commit message: Add files via upload
Parts:
- C124, C126, C273, C278, C279, C87: Indicator + -> (none); Rating V -> (none)
- J10: value PCMCIA Connector -> PCMCIA
- R394: now not fitted

Commit message: Add files via upload
Connections:
- net ABVD1: now also J10.59 (ABVD1_STSCHG#); no longer J10.57 (ABVD2_SPKR#)
- net ABVD2: now also J10.57 (ABVD2_SPKR#); no longer J10.59 (ABVD1_STSCHG#)
- net BBVD1: now also J10.129 (BBVD1_STSCHG#); no longer J10.127 (BBVD2_SPKR#)
- net BBVD2: now also J10.127 (BBVD2_SPKR#); no longer J10.129 (BBVD1_STSCHG#)
- net BCA10: now also U74.G15 (BCA10); no longer U74.D9 (BCA10)
- net BCD1#: now also U74.K16 (BCD1#); no longer U74.A8 (BCD2#)
- net BCD10: now also U74.D9 (BCD10); no longer U74.G15 (BCD10)
- net BCD2#: now also U74.A8 (BCD2#); no longer U74.K16 (BCD1#)
- net BCE1#: now also U74.G16 (BCE1#); no longer U74.F16 (BCE2#)
- net BCE2#: now also U74.F16 (BCE2#); no longer U74.G16 (BCE1#)
- net GND: now also C115.1; no longer C115.2
- net PNET1: now also C115.2; no longer C115.1
Other:
- moved on the sheet: C115
Changed lines of the file:
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@@
 	(wire
 		(pts
-			(xy 544.83 266.7) (xy 561.34 266.7)
-		)
-		(stroke
-			(width 0)
-			(type default)
-		)
-	)
-	(wire
-		(pts
 			(xy 445.77 90.17) (xy 462.28 90.17)
 		)
@@
 	(wire
 		(pts
-			(xy 445.77 217.17) (xy 462.28 217.17)
-		)
-		(stroke
-			(width 0)
-			(type default)
-		)
-	)
-	(wire
-		(pts
 			(xy 544.83 232.41) (xy 561.34 232.41)
 		)
@@
 	(wire
 		(pts
+			(xy 445.77 214.63) (xy 462.28 214.63)
+		)
+		(stroke
+			(width 0)
+			(type default)
+		)
+	)
+	(wire
+		(pts
 			(xy 332.74 378.46) (xy 334.01 378.46)
 		)
@@
 	(wire
 		(pts
-			(xy 544.83 269.24) (xy 561.34 269.24)
-		)
-		(stroke
-			(width 0)
-			(type default)
-		)
-	)
-	(wire
-		(pts
 			(xy 57.15 35.56) (xy 57.15 33.02)
 		)
@@
 	(wire
 		(pts
+			(xy 487.68 269.24) (xy 504.19 269.24)
+		)
+		(stroke
+			(width 0)
+			(type default)
+		)
+	)
+	(wire
+		(pts
 			(xy 335.28 372.11) (xy 335.28 378.46)
 		)
@@
 	(wire
 		(pts
-			(xy 504.19 269.24) (xy 487.68 269.24)
-		)
-		(stroke
-			(width 0)
-			(type default)
-		)
-	)
-	(wire
-		(pts
 			(xy 307.34 372.11) (xy 307.34 378.46)
 		)
@@
 	(wire
 		(pts
+			(xy 544.83 269.24) (xy 561.34 269.24)
+		)
+		(stroke
+			(width 0)
+			(type default)
+		)
+	)
+	(wire
+		(pts
 			(xy 194.31 181.61) (xy 223.52 181.61)
 		)
@@
 	(wire
 		(pts
-			(xy 281.94 372.11) (xy 281.94 378.46)
+			(xy 487.68 266.7) (xy 504.19 266.7)
 		)
 		(stroke
@@
 	(wire
 		(pts
-			(xy 445.77 240.03) (xy 462.28 240.03)
+			(xy 281.94 372.11) (xy 281.94 378.46)
 		)
 		(stroke
@@
 	(wire
 		(pts
-			(xy 445.77 326.39) (xy 462.28 326.39)
+			(xy 445.77 240.03) (xy 462.28 240.03)
 		)
 		(stroke
@@
 	(wire
 		(pts
-			(xy 530.86 297.18) (xy 533.4 297.18)
+			(xy 445.77 326.39) (xy 462.28 326.39)
 		)
 		(stroke
@@
 	(wire
 		(pts
-			(xy 445.77 339.09) (xy 462.28 339.09)
+			(xy 530.86 297.18) (xy 533.4 297.18)
 		)
 		(stroke
@@
 	(wire
 		(pts
-			(xy 66.04 59.69) (xy 27.94 59.69)
+			(xy 445.77 339.09) (xy 462.28 339.09)
 		)
 		(stroke
@@
 	(wire
 		(pts
-			(xy 534.67 52.07) (xy 534.67 54.61)
+			(xy 66.04 59.69) (xy 27.94 59.69)
 		)
 		(stroke
@@
 	(wire
 		(pts
-			(xy 504.19 266.7) (xy 487.68 266.7)
+			(xy 534.67 52.07) (xy 534.67 54.61)
 		)
 		(stroke
@@
 	(wire
 		(pts
-			(xy 445.77 237.49) (xy 462.28 237.49)
+			(xy 445.77 269.24) (xy 462.28 269.24)
 		)
 		(stroke
@@
 	(wire
 		(pts
-			(xy 445.77 269.24) (xy 462.28 269.24)
+			(xy 297.18 372.11) (xy 297.18 378.46)
 		)
 		(stroke
@@
 	(wire
 		(pts
-			(xy 297.18 372.11) (xy 297.18 378.46)
+			(xy 544.83 266.7) (xy 561.34 266.7)
 		)
 		(stroke
@@
 	(wire
 		(pts
-			(xy 445.77 214.63) (xy 462.28 214.63)
-		)
-		(stroke
-			(width 0)
-			(type default)
-		)
-	)
-	(wire
-		(pts
 			(xy 106.68 48.26) (xy 110.49 48.26)
 		)
@@
 	(wire
 		(pts
+			(xy 445.77 217.17) (xy 462.28 217.17)
+		)
+		(stroke
+			(width 0)
+			(type default)
+		)
+	)
+	(wire
+		(pts
 			(xy 544.83 189.23) (xy 561.34 189.23)
 		)
@@
 	(wire
 		(pts
+			(xy 445.77 234.95) (xy 462.28 234.95)
+		)
+		(stroke
+			(width 0)
+			(type default)
+		)
+	)
+	(wire
+		(pts
 			(xy 217.17 161.29) (xy 223.52 161.29)
 		)
@@
 	(wire
 		(pts
-			(xy 445.77 234.95) (xy 462.28 234.95)
-		)
-		(stroke
-			(width 0)
-			(type default)
-		)
-	)
-	(wire
-		(pts
 			(xy 504.19 154.94) (xy 487.68 154.94)
 		)
@@
 	(wire
 		(pts
+			(xy 445.77 237.49) (xy 462.28 237.49)
+		)
+		(stroke
+			(width 0)
+			(type default)
+		)
+	)
+	(wire
+		(pts
 			(xy 445.77 331.47) (xy 462.28 331.47)
 		)
@@
 	)
 	(label "BBVD2"
-		(at 487.68 269.24 0)
+		(at 487.68 266.7 0)
 		(effects
 			(font
@@
 	)
 	(label "ABVD2"
-		(at 561.34 269.24 180)
+		(at 561.34 266.7 180)
 		(effects
 			(font
@@
 	)
 	(label "BBVD1"
-		(at 487.68 266.7 0)
+		(at 487.68 269.24 0)
 		(effects
 			(font
@@
 	)
 	(label "BCE1#"
-		(at 462.28 214.63 180)
+		(at 462.28 217.17 180)
 		(effects
 			(font
@@
 	)
 	(label "ABVD1"
-		(at 561.34 266.7 180)
+		(at 561.34 269.24 180)
 		(effects
 			(font
@@
 	)
 	(label "BCD2#"
-		(at 462.28 237.49 180)
+		(at 462.28 234.95 180)
 		(effects
 			(font
@@
 	)
 	(label "BCE2#"
-		(at 462.28 217.17 180)
+		(at 462.28 214.63 180)
 		(effects
 			(font
@@
 	)
 	(label "BCD1#"
-		(at 462.28 234.95 180)
+		(at 462.28 237.49 180)
 		(effects
 			(font
@@
 	(symbol
 		(lib_id "Device:C")
-		(at 298.45 36.83 0)
-		(mirror y)
+		(at 298.45 36.83 180)
 		(unit 1)
 		(exclude_from_sim no)
@@
 		(dnp no)
 		(property "Reference" "C115"
-			(at 304.038 35.814 0)
+			(at 304.038 37.846 0)
 			(effects
 				(font
@@
 		)
 		(property "Value" "100nF"
-			(at 304.546 38.1 0)
+			(at 304.546 35.56 0)
 			(effects
 				(font
@@
 		)
 		(property "Footprint" "Capacitor_SMD:C_0402_1005Metric"
-			(at 297.4848 40.64 0)
+			(at 297.4848 33.02 0)
 			(effects
 				(font
