File: PCB/Mainboard/ROM.kicad_sch (KiCad schematic)
At the start: 0 parts

Commit message: Add files via upload
Parts:
- added U36: ~, symbol PC110:M538032C
- added U59: ~, symbol PC110:28F002BX

Commit message: Add files via upload
Connections:
- net GND: now reaches U36.15 (VSS)
Other:
- moved on the sheet: U59
Changed lines of the file:
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@@
 	(generator_version "9.0")
 	(paper "A4")
+	(wire
+		(pts
+			(xy 81.28 128.27) (xy 81.28 132.08)
+		)
+		(stroke
+			(width 0)
+			(type default)
+		)
+	)
 	(symbol
 		(lib_id "PC110:28F002BX")
-		(at 180.34 95.25 0)
+		(at 200.66 92.71 0)
 		(unit 1)
 		(exclude_from_sim no)
@@
 		(dnp no)
 		(property "Reference" "U59"
-			(at 197.104 69.596 0)
+			(at 217.424 67.056 0)
 			(effects
 				(font
@@
 		)
 		(property "Value" "~"
-			(at 190.1033 69.85 0)
+			(at 210.4233 67.31 0)
 			(effects
 				(font
@@
 		)
 		(property "Footprint" ""
-			(at 180.34 95.25 0)
+			(at 200.66 92.71 0)
 			(effects
 				(font
@@
 		)
 		(property "Datasheet" ""
-			(at 180.34 95.25 0)
+			(at 200.66 92.71 0)
 			(effects
 				(font
@@
 		)
 		(property "Description" ""
-			(at 180.34 95.25 0)
+			(at 200.66 92.71 0)
 			(effects
 				(font
@@
 					(unit 1)
 				)
+			)
+		)
+	)
+	(symbol
+		(lib_id "power:GND")
+		(at 81.28 132.08 0)
+		(unit 1)
+		(exclude_from_sim no)
+		(in_bom yes)
+		(on_board yes)
+		(dnp no)
+		(fields_autoplaced yes)
+		(property "Reference" "#PWR0129"
+			(at 81.28 138.43 0)
+			(effects
+				(font
+					(size 1.27 1.27)
+				)
+				(hide yes)
+			)
+		)
+		(property "Value" "GND"
+			(at 81.28 137.16 0)
+			(effects
+				(font
+					(size 1.27 1.27)
+				)
+			)
+		)
+		(property "Footprint" ""
+			(at 81.28 132.08 0)
+			(effects
+				(font
+					(size 1.27 1.27)
+				)
+				(hide yes)
+			)
+		)
+		(property "Datasheet" ""
+			(at 81.28 132.08 0)
+			(effects
+				(font
+					(size 1.27 1.27)
+				)
+				(hide yes)
+			)
+		)
+		(property "Description" "Power symbol creates a global label with name \"GND\" , ground"
+			(at 81.28 132.08 0)
+			(effects
+				(font
+					(size 1.27 1.27)
+				)
+				(hide yes)
+			)
+		)
+		(pin "1"
+		)
+		(instances
+			(project "PC110"
+				(path "/45c7911f-b027-440e-9e3e-77a146b41944/29aeee43-2869-4080-920c-a693b0bc5770"
+					(reference "#PWR0129")
+					(unit 1)
+				)

Commit message: Add files via upload
Parts:
- added C246: 150nF, symbol PCM_Elektuur:C
- added D20: 3D, symbol Device:D_Dual_CommonCathode_AKA
- added Q35: 8C, Package_TO_SOT_SMD:SOT-23, symbol Transistor_BJT:MMBTA44
- added Q36: 7C, symbol Simulation_SPICE:PNP
- added R113, R327: 470k, symbol Device:R
- added R320: 10k, symbol Device:R
- added R321: 100k, symbol Device:R
- added U60: E3, symbol 74xGxx:74AUP1G02
Connections:
- net GND: now also C246.2 (-), Q35.2 (E), R113.1, R327.1, U60.3 (GND)
- net at U59.10 (RP#): now also D20.3 (K), R113.2
- net at U59.11 (VPP): now also C246.1 (+), D20.1 (A), Q36.1 (C), R327.2
- new net: R321.1, U60.4
- new net: Q35.1 (B), R321.2
- new net: Q36.2 (B), R320.2
- new net: Q35.3 (C), R320.1
- new net Bowman5_Buff: U60.1
- new net D28_1: Q36.3 (E)
- new net PNET5: U60.5 (VCC)
- new net PWRGD: D20.2 (A)
- new net PWRGD_shift_buff: U60.2
Other:
- moved on the sheet: U59

Commit message: Add files via upload
Other:
- moved on the sheet: U36
Changed lines of the file:
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@@
 	(wire
 		(pts
-			(xy 81.28 128.27) (xy 81.28 132.08)
+			(xy 90.17 154.94) (xy 90.17 158.75)
 		)
 		(stroke
@@
 	(symbol
 		(lib_id "power:GND")
-		(at 81.28 132.08 0)
+		(at 90.17 158.75 0)
 		(unit 1)
 		(exclude_from_sim no)
@@
 		(fields_autoplaced yes)
 		(property "Reference" "#PWR0129"
-			(at 81.28 138.43 0)
+			(at 90.17 165.1 0)
 			(effects
 				(font
@@
 		)
 		(property "Value" "GND"
-			(at 81.28 137.16 0)
+			(at 90.17 163.83 0)
 			(effects
 				(font
@@
 		)
 		(property "Footprint" ""
-			(at 81.28 132.08 0)
+			(at 90.17 158.75 0)
 			(effects
 				(font
@@
 		)
 		(property "Datasheet" ""
-			(at 81.28 132.08 0)
+			(at 90.17 158.75 0)
 			(effects
 				(font
@@
 		)
 		(property "Description" "Power symbol creates a global label with name \"GND\" , ground"
-			(at 81.28 132.08 0)
+			(at 90.17 158.75 0)
 			(effects
 				(font
@@
 	(symbol
 		(lib_id "PC110:M538032C")
-		(at 88.9 96.52 0)
+		(at 97.79 123.19 0)
 		(unit 1)
 		(exclude_from_sim no)
@@
 		(dnp no)
 		(property "Reference" "U36"
-			(at 101.346 66.04 0)
+			(at 110.236 92.71 0)
 			(effects
 				(font
@@
 		)
 		(property "Value" "~"
-			(at 91.0433 66.04 0)
+			(at 99.9333 92.71 0)
 			(effects
 				(font
@@
 		)
 		(property "Footprint" ""
-			(at 88.9 96.52 0)
+			(at 97.79 123.19 0)
 			(effects
 				(font
@@
 		)
 		(property "Datasheet" ""
-			(at 88.9 96.52 0)
+			(at 97.79 123.19 0)
 			(effects
 				(font
@@
 		)
 		(property "Description" ""
-			(at 88.9 96.52 0)
-			(effects
-				(font
+			(at 97.79 123.19 0)
+			(effects
+				(font

Commit message: Add files via upload
Parts:
- added C282: 150nF, symbol PCM_Elektuur:C
Connections:
- net GND: now also U59.23 (GND), U59.39 (GND), C282.1 (+)
- net PWRGD: now also D20.3 (A); no longer D20.2 (A)
- net at R113.2, U59.10 (RP#): now also D20.2 (K); no longer D20.3 (K)
- net SA2: now reaches U59.19 (A2)
- net SA2: now also U36.12 (A1)
- net SA1: now reaches U59.20 (A1)
- net SA1: now also U36.13 (A0)
- net SA0: now reaches U59.21 (A0)
- net SA3: now reaches U36.11 (A2)
- net PNET7: now reaches U36.25 (VCC)
- net PNET7: now also C282.2 (-)
- no-connect marks 0 -> 10
Other:
- moved on the sheet: C246, D20, Q35, Q36, R113, R320, R321, R327, U36, U59, U60

Commit message: Add files via upload
Parts:
- added U24: E4, symbol 74xGxx:74AUP1G02
Connections:
- net GND: now also U24.3 (GND)
- net PNET5: now also U24.5 (VCC)
- net MEMR#: now reaches U59.24 (OE#)
- net at U59.9 (WE#): now also U24.4
- new net MEMW#: U24.1

Commit message: Add files via upload
Connections:
- net SD0_Bus: now reaches U36.17 (D0)
- net SD8_Bus: now reaches U36.18 (D8)
- net SD1_Bus: now reaches U36.19 (D1)
- net SD9_Bus: now reaches U36.20 (D9)
- net SD2_Bus: now reaches U36.21 (D2)
- net SD10_Bus: now reaches U36.22 (D10)
- net SD3_Bus: now reaches U36.23 (D3)
- net SD11_Bus: now reaches U36.24 (D11)
- net SD4_Bus: now reaches U36.26 (D4)
- net SD12_Bus: now reaches U36.27 (D12)
- net SD5_Bus: now reaches U36.28 (D5)
- net SD13_Bus: now reaches U36.29 (D13)
- net SD6_Bus: now reaches U36.30 (D6)
- net SD15_Bus: now reaches U36.31 (D14)
- net SD15_Bus: now also U36.33 (D15)
- net SD7_Bus: now reaches U36.32 (D7)

Commit message: Add files via upload
Connections:
- net Chipset_SA16: now reaches U59.1 (A16)
- net Chipset_BIOS_CE#: now reaches U59.22 (CE#)
- net BIOS_SA17: now reaches U59.40 (A17)
- no-connect marks 10 -> 11
Changed lines of the file:
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@@
+	)
+	(no_connect
+		(at 290.83 146.05)
 	)
 	(no_connect
@@
 	(wire
 		(pts
+			(xy 210.82 172.72) (xy 234.95 172.72)
+		)
+		(stroke
+			(width 0)
+			(type default)
+		)
+	)
+	(wire
+		(pts
 			(xy 256.54 181.61) (xy 256.54 184.15)
 		)
@@
 	(wire
 		(pts
+			(xy 287.02 146.05) (xy 290.83 146.05)
+		)
+		(stroke
+			(width 0)
+			(type default)
+		)
+	)
+	(wire
+		(pts
+			(xy 210.82 175.26) (xy 234.95 175.26)
+		)
+		(stroke
+			(width 0)
+			(type default)
+		)
+	)
+	(wire
+		(pts
 			(xy 210.82 134.62) (xy 234.95 134.62)
 		)
@@
 		(pts
 			(xy 274.32 93.98) (xy 269.24 93.98)
+		)
+		(stroke
+			(width 0)
+			(type default)
+		)
+	)
+	(wire
+		(pts
+			(xy 287.02 142.24) (xy 311.15 142.24)
 		)
 		(stroke
@@
 		)
 	)
+	(label "Chipset_BIOS_CE#"
+		(at 293.37 142.24 0)
+		(effects
+			(font
+				(size 1.27 1.27)
+			)
+			(justify left bottom)
+		)
+	)
 	(label "SA1"
 		(at 210.82 134.62 0)
@@
 		)
 	)
+	(label "BIOS_SA17"
+		(at 212.09 175.26 0)
+		(effects
+			(font
+				(size 1.27 1.27)
+			)
+			(justify left bottom)
+		)
+	)
 	(label "SD10_Bus"
 		(at 134.62 153.67 0)
@@
 		(effects
 			(font
+				(size 1.27 1.27)
+			)
+			(justify left bottom)
+		)
+	)
+	(label "Chipset_SA16"
+		(at 212.09 172.72 0)
+		(effects
+			(font
