File: PCB/Mainboard/ROM.kicad_sch (KiCad schematic)
At the start: 16 parts, among them Q35 8C, Q36 7C, U24 E4, U60 E3

Commit message: Add files via upload
Connections:
- net SD0_Bus renamed SD0
- net SD10_Bus renamed SD10
- net SD11_Bus renamed SD11
- net SD12_Bus renamed SD12
- net SD13_Bus renamed SD13
- net SD15_Bus renamed SD14
- net SD14: no longer U36.33 (D15)
- net SD1_Bus renamed SD1
- net SD2_Bus renamed SD2
- net SD3_Bus renamed SD3
- net SD4_Bus renamed SD4
- net SD5_Bus renamed SD5
- net SD6_Bus renamed SD6
- net SD7_Bus renamed SD7
- net SD8_Bus renamed SD8
- net SD9_Bus renamed SD9
- new net SD15: U36.33 (D15)
- no-connect marks 11 -> 1
Other:
- note added: "Device_Address_BUS"
- note added: "Device_Data_BUS"
- note added: "OKI_Extra_Address"
Changed lines of the file:
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@@
 		(company "Recreated by: Ahmad Byagowi")
 	)
+	(text "Device_Data_BUS"
+		(exclude_from_sim no)
+		(at 153.162 132.588 0)
+		(effects
+			(font
+				(size 1.27 1.27)
+			)
+		)
+	)
+	(text "Device_Address_BUS"
+		(exclude_from_sim no)
+		(at 188.976 136.398 0)
+		(effects
+			(font
+				(size 1.27 1.27)
+			)
+		)
+	)
+	(text "Device_Data_BUS"
+		(exclude_from_sim no)
+		(at 317.246 159.258 0)
+		(effects
+			(font
+				(size 1.27 1.27)
+			)
+		)
+	)
+	(text "Device_Address_BUS"
+		(exclude_from_sim no)
+		(at 49.276 132.588 0)
+		(effects
+			(font
+				(size 1.27 1.27)
+			)
+		)
+	)
+	(text "OKI_Extra_Address"
+		(exclude_from_sim no)
+		(at 47.752 162.56 0)
+		(effects
+			(font
+				(size 1.27 1.27)
+			)
+		)
+	)
 	(junction
 		(at 246.38 189.23)
@@
 	)
 	(no_connect
-		(at 259.08 186.69)
-	)
-	(no_connect
 		(at 281.94 151.13)
 	)
-	(no_connect
-		(at 100.33 190.5)
-	)
-	(no_connect
-		(at 107.95 190.5)
-	)
-	(no_connect
-		(at 102.87 190.5)
-	)
-	(no_connect
-		(at 97.79 190.5)
-	)
-	(no_connect
-		(at 261.62 186.69)
-	)
-	(no_connect
-		(at 256.54 186.69)
-	)
-	(no_connect
-		(at 105.41 190.5)
-	)
-	(no_connect
-		(at 110.49 190.5)
-	)
-	(no_connect
-		(at 254 186.69)
-	)
 	(bus_entry
 		(at 60.96 166.37)
@@
 	(bus
 		(pts
-			(xy 308.61 156.21) (xy 303.53 156.21)
+			(xy 314.96 156.21) (xy 303.53 156.21)
 		)
 		(stroke
@@
 	(bus
 		(pts
-			(xy 55.88 129.54) (xy 60.96 129.54)
+			(xy 50.8 129.54) (xy 60.96 129.54)
 		)
 		(stroke
@@
 	(bus
 		(pts
-			(xy 138.43 129.54) (xy 143.51 129.54)
+			(xy 138.43 129.54) (xy 149.86 129.54)
 		)
 		(stroke
@@
 	(bus
 		(pts
-			(xy 195.58 133.35) (xy 200.66 133.35)
+			(xy 190.5 133.35) (xy 200.66 133.35)
 		)
 		(stroke
@@
 		)
 	)
-	(label "SD2_Bus"
+	(label "SD2"
 		(at 292.1 165.1 0)
 		(effects
@@
 		)
 	)
-	(label "SD4_Bus"
+	(label "SD4"
 		(at 127 143.51 0)
 		(effects
@@
 		)
 	)
-	(label "SD3_Bus"
+	(label "SD3"
 		(at 292.1 167.64 0)
 		(effects
@@
 		)
 	)
-	(label "SD7_Bus"
+	(label "SD7"
 		(at 292.1 177.8 0)
 		(effects
@@
 		)
 	)
-	(label "SD3_Bus"
+	(label "SD3"
 		(at 127 140.97 0)
 		(effects
@@
 		)
 	)
-	(label "SD13_Bus"
+	(label "SD13"
 		(at 125.73 166.37 0)
 		(effects
@@
 		)
 	)
-	(label "SD9_Bus"
+	(label "SD9"
 		(at 127 156.21 0)
 		(effects
@@
 		)
 	)
-	(label "SD8_Bus"
+	(label "SD8"
 		(at 127 153.67 0)
 		(effects
@@
 		)
 	)
-	(label "SD6_Bus"
+	(label "SD6"
 		(at 292.1 175.26 0)
 		(effects
@@
 		)
 	)
-	(label "SD10_Bus"
+	(label "SD10"
 		(at 125.73 158.75 0)
 		(effects
@@
 		)
 	)
-	(label "SD15_Bus"
+	(label "SD14"
 		(at 125.73 168.91 0)
 		(effects
@@
 		)
 	)
-	(label "SD7_Bus"
+	(label "SD7"
 		(at 127 151.13 0)
 		(effects
@@
 		)
 	)
-	(label "SD6_Bus"
+	(label "SD6"
 		(at 127 148.59 0)
 		(effects
@@
 		)
 	)
-	(label "SD5_Bus"
+	(label "SD5"
 		(at 127.1649 146.05 0)
 		(effects
@@
 		)
 	)
-	(label "SD0_Bus"
+	(label "SD0"
 		(at 127 133.35 0)
 		(effects
@@
 		)
 	)
-	(label "SD2_Bus"
+	(label "SD2"
 		(at 127 138.43 0)
 		(effects
@@
 		)
 	)
-	(label "SD11_Bus"
+	(label "SD11"
 		(at 125.73 161.29 0)
 		(effects
@@
 		)
 	)
-	(label "SD1_Bus"
+	(label "SD1"
 		(at 127 135.89 0)
 		(effects
@@
 		)
 	)
-	(label "SD1_Bus"
+	(label "SD1"
 		(at 292.1 162.56 0)
 		(effects
@@
 		)
 	)
-	(label "SD12_Bus"
+	(label "SD12"
 		(at 125.73 163.83 0)
 		(effects
@@
 		)
 	)
-	(label "SD0_Bus"
+	(label "SD0"
 		(at 292.1 160.02 0)
 		(effects
@@
 		)
 	)
-	(label "SD5_Bus"
+	(label "SD5"
 		(at 292.2649 172.72 0)
 		(effects
@@
 		)
 	)
-	(label "SD15_Bus"
+	(label "SD15"
 		(at 125.73 171.45 0)
 		(effects
@@
 		)
 	)
-	(label "SD4_Bus"
+	(label "SD4"
 		(at 292.1 170.18 0)
 		(effects
@@
 		)
 	)
-	(global_label "Device_Address_BUS"
+	(global_label "SA[0..15]"
 		(shape input)
-		(at 55.88 129.54 180)
+		(at 50.8 129.54 180)
 		(fields_autoplaced yes)
 		(effects
@@
 		)
 		(property "Intersheetrefs" "${INTERSHEET_REFS}"
-			(at 33.7238 129.54 0)
+			(at 38.9852 129.54 0)
 			(effects
 				(font
@@
 		)
 	)
-	(global_label "Device_Data_BUS"
+	(global_label "SD[0..15]"
 		(shape input)
-		(at 308.61 156.21 0)
+		(at 314.96 156.21 0)
 		(fields_autoplaced yes)
 		(effects
@@
 		)
 		(property "Intersheetrefs" "${INTERSHEET_REFS}"
-			(at 327.7423 156.21 0)
+			(at 326.9562 156.21 0)
 			(effects
 				(font
@@
 		)
 	)
-	(global_label "Device_Address_BUS"
+	(global_label "SA[0..15]"
 		(shape input)
-		(at 195.58 133.35 180)
+		(at 190.5 133.35 180)
 		(fields_autoplaced yes)
 		(effects
@@
 		)
 		(property "Intersheetrefs" "${INTERSHEET_REFS}"
-			(at 173.4238 133.35 0)
+			(at 178.6852 133.35 0)
 			(effects
 				(font
@@
 		)
 	)
-	(global_label "OKI_Extra_Address"
+	(global_label "OKI_SA[12..19]"
 		(shape input)
 		(at 55.88 160.02 180)
@@
 		)
 		(property "Intersheetrefs" "${INTERSHEET_REFS}"
-			(at 35.5987 160.02 0)
+			(at 38.6828 160.02 0)
 			(effects
 				(font
@@
 		)
 	)
-	(global_label "Device_Data_BUS"
+	(global_label "SD[0..15]"
 		(shape input)
-		(at 143.51 129.54 0)
+		(at 149.86 129.54 0)
 		(fields_autoplaced yes)
 		(effects
@@
 		)
 		(property "Intersheetrefs" "${INTERSHEET_REFS}"
-			(at 162.6423 129.54 0)
+			(at 161.8562 129.54 0)
 			(effects
 				(font

Commit message: Add files via upload
Parts:
- C246: footprint (none) -> Capacitor_SMD:C_0603_1608Metric
- C249, C282: footprint (none) -> Capacitor_SMD:C_0402_1005Metric
- D19, D20: footprint (none) -> PC110:SOT-416L
- Q35: footprint Package_TO_SOT_SMD:SOT-23 -> Package_TO_SOT_SMD:SOT-523
- Q36: footprint (none) -> Package_TO_SOT_SMD:TSOT-23
- R112, R113, R320, R321, R327: footprint (none) -> PCM_Resistor_SMD_AKL:R_0402_1005Metric
- U24, U60: footprint (none) -> PC110:SOT-353
- U36: footprint (none) -> PC110:SOP48
- U59: footprint (none) -> PC110:Flash-40
Connections:
- net GND: now also C282.2 (-), R327.2; no longer C282.1 (+), R327.1
- net PNET7: now also C282.1 (+); no longer C282.2 (-)
- net at C246.1 (+), D20.1 (A), Q36.1 (C)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: now also R327.1; no longer R327.2
Other:
- moved on the sheet: R327
Changed lines of the file:
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@@
 			)
 		)
-		(property "Footprint" ""
+		(property "Footprint" "PCM_Resistor_SMD_AKL:R_0402_1005Metric"
 			(at 314.96 101.092 90)
 			(effects
@@
 			)
 		)
-		(property "Footprint" ""
+		(property "Footprint" "PC110:Flash-40"
 			(at 252.73 157.48 0)
 			(effects
@@
 			)
 		)
-		(property "Footprint" ""
+		(property "Footprint" "PC110:SOT-416L"
 			(at 245.11 99.06 0)
 			(effects
@@
 			)
 		)
-		(property "Footprint" ""
+		(property "Footprint" "PC110:SOT-353"
 			(at 337.82 102.87 0)
 			(effects
@@
 			)
 		)
-		(property "Footprint" ""
+		(property "Footprint" "Package_TO_SOT_SMD:TSOT-23"
 			(at 227.33 87.63 0)
 			(effects
@@
 		(lib_id "PCM_Elektuur:C")
 		(at 88.9 113.03 0)
-		(mirror x)
 		(unit 1)
 		(exclude_from_sim no)
@@
 		(dnp no)
 		(property "Reference" "C282"
-			(at 85.09 111.7599 0)
+			(at 85.09 114.3001 0)
 			(effects
 				(font
@@
 		)
 		(property "Value" "150nF"
-			(at 85.09 114.2999 0)
+			(at 85.09 111.7601 0)
 			(effects
 				(font
@@
 			)
 		)
-		(property "Footprint" ""
+		(property "Footprint" "Capacitor_SMD:C_0402_1005Metric"
 			(at 88.9 113.03 0)
 			(effects
@@
 		)
 		(property "Indicator" "+"
-			(at 87.63 116.205 0)
+			(at 87.63 109.855 0)
 			(effects
 				(font
@@
 		)
 		(property "Rating" "V"
-			(at 88.265 109.855 0)
+			(at 88.265 116.205 0)
 			(effects
 				(font
@@
 			)
 		)
-		(property "Footprint" ""
+		(property "Footprint" "PCM_Resistor_SMD_AKL:R_0402_1005Metric"
 			(at 229.87 107.442 90)
 			(effects
@@
 			)
 		)
-		(property "Footprint" ""
+		(property "Footprint" "PCM_Resistor_SMD_AKL:R_0402_1005Metric"
 			(at 281.94 85.852 90)
 			(effects
@@
 			)
 		)
-		(property "Footprint" ""
+		(property "Footprint" "PC110:SOP48"
 			(at 100.33 158.75 0)
 			(effects
@@
 			)
 		)
-		(property "Footprint" ""
+		(property "Footprint" "Capacitor_SMD:C_0603_1608Metric"
 			(at 278.13 110.49 0)
 			(effects
@@
 			)
 		)
-		(property "Footprint" "Package_TO_SOT_SMD:SOT-23"
+		(property "Footprint" "Package_TO_SOT_SMD:SOT-523"
 			(at 294.64 104.775 0)
 			(effects
@@
 			)
 		)
-		(property "Footprint" ""
+		(property "Footprint" "Capacitor_SMD:C_0402_1005Metric"
 			(at 223.52 121.92 0)
 			(effects
@@
 			)
 		)
-		(property "Footprint" ""
+		(property "Footprint" "PC110:SOT-416L"
 			(at 375.92 195.58 0)
 			(effects
@@
 	(symbol
 		(lib_id "Device:R")
-		(at 265.43 110.49 180)
-		(unit 1)
-		(exclude_from_sim no)
-		(in_bom yes)
-		(on_board yes)
-		(dnp no)
-		(fields_autoplaced yes)
+		(at 265.43 110.49 0)
+		(mirror y)
+		(unit 1)
+		(exclude_from_sim no)
+		(in_bom yes)
+		(on_board yes)
+		(dnp no)
 		(property "Reference" "R327"
-			(at 267.97 109.2199 0)
+			(at 267.97 111.7601 0)
 			(effects
 				(font
@@
 		)
 		(property "Value" "470k"
-			(at 267.97 111.7599 0)
+			(at 267.97 109.2201 0)
 			(effects
 				(font
@@
 			)
 		)
-		(property "Footprint" ""
+		(property "Footprint" "PCM_Resistor_SMD_AKL:R_0402_1005Metric"
 			(at 267.208 110.49 90)
 			(effects
@@
 			)
 		)
-		(property "Footprint" ""
+		(property "Footprint" "PCM_Resistor_SMD_AKL:R_0402_1005Metric"
 			(at 374.142 168.91 90)
 			(effects
@@
 			)
 		)
-		(property "Footprint" ""
+		(property "Footprint" "PC110:SOT-353"
 			(at 337.82 142.24 0)
 			(effects

Commit message: Add files via upload
Parts:
- removed Q36: 7C, Package_TO_SOT_SMD:TSOT-23, symbol Simulation_SPICE:PNP
- added Q36: 7C, symbol PCM_Transistor_BJT_AKL:Q_PNP_Generic_BEC
Connections:
- net D28_1: now also Q36.2 (E)
- net at C246.1 (+), D20.1 (A), R327.1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: now also Q36.3 (C)
- net at R320.2: now also Q36.1 (B)
Changed lines of the file:
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@@
 	)
 	(symbol
-		(lib_id "Simulation_SPICE:PNP")
-		(at 262.89 87.63 180)
+		(lib_id "PCM_Transistor_BJT_AKL:Q_PNP_Generic_BEC")
+		(at 262.89 87.63 0)
+		(mirror y)
 		(unit 1)
 		(exclude_from_sim no)
@@
 		(dnp no)
 		(property "Reference" "Q36"
-			(at 257.81 88.9001 0)
+			(at 257.81 86.3599 0)
 			(effects
 				(font
@@
 		)
 		(property "Value" "7C"
-			(at 257.81 86.3601 0)
+			(at 257.81 88.8999 0)
 			(effects
 				(font
@@
 			)
 		)
-		(property "Footprint" "Package_TO_SOT_SMD:TSOT-23"
-			(at 227.33 87.63 0)
+		(property "Footprint" ""
+			(at 257.81 90.17 0)
 			(effects
 				(font
@@
 			)
 		)
-		(property "Datasheet" "https://ngspice.sourceforge.io/docs/ngspice-html-manual/manual.xhtml#cha_BJTs"
-			(at 227.33 87.63 0)
-			(effects
-				(font
-					(size 1.27 1.27)
-				)
-				(hide yes)
-			)
-		)
-		(property "Description" "Bipolar transistor symbol for simulation only, substrate tied to the emitter"
+		(property "Datasheet" "~"
 			(at 262.89 87.63 0)
 			(effects
@@
 			)
 		)
-		(property "Sim.Device" "PNP"
+		(property "Description" "PNP transistor, generic symbol, Alternate KiCAD Library"
 			(at 262.89 87.63 0)
 			(effects
@@
 			)
 		)
-		(property "Sim.Type" "GUMMELPOON"
-			(at 262.89 87.63 0)
-			(effects
-				(font
-					(size 1.27 1.27)
-				)
-				(hide yes)
-			)
-		)
-		(property "Sim.Pins" "1=C 2=B 3=E"
-			(at 262.89 87.63 0)
-			(effects
-				(font
-					(size 1.27 1.27)
-				)
-				(hide yes)
-			)
-		)
-		(pin "3"
-		)
 		(pin "1"
 		)
 		(pin "2"
 		)
+		(pin "3"
+		)
 		(instances
-			(project ""
+			(project "PC110"
 				(path "/45c7911f-b027-440e-9e3e-77a146b41944/29aeee43-2869-4080-920c-a693b0bc5770"
 					(reference "Q36")

Commit message: Add files via upload
Parts:
- Q36: footprint (none) -> Package_TO_SOT_SMD:TSOT-23
Changed lines of the file:
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@@
 			)
 		)
-		(property "Footprint" ""
+		(property "Footprint" "Package_TO_SOT_SMD:TSOT-23"
 			(at 257.81 90.17 0)
 			(effects

Commit message: Add files via upload
Parts:
- C246, C249, C282: Indicator + -> (none); Rating V -> (none)
- D19: value DAN222 -> N; Topmark N -> (none)
- D20: value RB715F -> 3D; Topmark 3D -> (none)
- U36: value ~ -> MSM538032E
- U59: value ~ -> 28F002BX
Changed lines of the file:
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@@
 			)
 		)
-		(property "Description" "Resistor"
+		(property "Description" ""
 			(at 314.96 102.87 0)
 			(effects
@@
 			)
 		)
-		(property "Value" "~"
+		(property "Value" "28F002BX"
 			(at 262.4933 132.08 0)
 			(effects
@@
 			)
 		)
-		(property "Value" "RB715F"
+		(property "Value" "3D"
 			(at 245.11 95.25 0)
 			(effects
@@
 			)
 		)
-		(property "Description" "Dual Schottky diode, common cathode on pin 2"
-			(at 245.11 99.06 0)
-			(effects
-				(font
-					(size 1.27 1.27)
-				)
-				(hide yes)
-			)
-		)
-		(property "Topmark" "3D"
+		(property "Description" ""
 			(at 245.11 99.06 0)
 			(effects
@@
 			)
 		)
-		(property "Datasheet" "https://www.ti.com/lit/ds/symlink/sn74aup1g02.pdf"
+		(property "Datasheet" ""
 			(at 337.82 102.87 0)
 			(effects
@@
 			)
 		)
-		(property "Description" "Single NOR Gate, Low-Voltage CMOS"
+		(property "Description" ""
 			(at 337.82 102.87 0)
 			(effects
@@
 			)
 		)
-		(property "Description" "PNP transistor, generic symbol, Alternate KiCAD Library"
+		(property "Description" ""
 			(at 262.89 87.63 0)
 			(effects
@@
 			)
 		)
-		(property "Description" "capacitor, non-polarized/bipolar"
+		(property "Description" ""
 			(at 88.9 113.03 0)
 			(effects
@@
 					(size 1.27 1.27)
 				)
-				(hide yes)
-			)
-		)
-		(property "Indicator" "+"
-			(at 87.63 109.855 0)
-			(effects
-				(font
-					(size 1.27 1.27)
-				)
-				(hide yes)
-			)
-		)
-		(property "Rating" "V"
-			(at 88.265 116.205 0)
-			(effects
-				(font
-					(size 1.27 1.27)
-				)
-				(justify right)
 				(hide yes)
 			)
@@
 			)
 		)
-		(property "Description" "Resistor"
+		(property "Description" ""
 			(at 229.87 109.22 0)
 			(effects
@@
 			)
 		)
-		(property "Description" "Resistor"
+		(property "Description" ""
 			(at 281.94 87.63 0)
 			(effects
@@
 			)
 		)
-		(property "Value" "~"
+		(property "Value" "MSM538032E"
 			(at 102.4733 128.27 0)
 			(effects
@@
 			)
 		)
-		(property "Description" "capacitor, non-polarized/bipolar"
+		(property "Description" ""
 			(at 278.13 110.49 0)
 			(effects
@@
 					(size 1.27 1.27)
 				)
-				(hide yes)
-			)
-		)
-		(property "Indicator" "+"
-			(at 276.86 107.315 0)
-			(effects
-				(font
-					(size 1.27 1.27)
-				)
-				(hide yes)
-			)
-		)
-		(property "Rating" "V"
-			(at 277.495 113.665 0)
-			(effects
-				(font
-					(size 1.27 1.27)
-				)
-				(justify right)
 				(hide yes)
 			)
@@
 			)
 		)
-		(property "Datasheet" "https://diotec.com/request/datasheet/mmbta42.pdf"
+		(property "Datasheet" ""
 			(at 299.72 102.87 0)
 			(effects
@@
 			)
 		)
-		(property "Description" "0.3A Ic, 400V Vce, NPN High Voltage Transistor, SOT-23"
+		(property "Description" ""
 			(at 299.72 102.87 0)
 			(effects
@@
 			)
 		)
-		(property "Description" "capacitor, non-polarized/bipolar"
+		(property "Description" ""
 			(at 223.52 121.92 0)
 			(effects
@@
 					(size 1.27 1.27)
 				)
-				(hide yes)
-			)
-		)
-		(property "Indicator" "+"
-			(at 222.25 125.095 0)
-			(effects
-				(font
-					(size 1.27 1.27)
-				)
-				(hide yes)
-			)
-		)
-		(property "Rating" "V"
-			(at 222.885 118.745 0)
-			(effects
-				(font
-					(size 1.27 1.27)
-				)
-				(justify right)
 				(hide yes)
 			)
@@
 			)
 		)
-		(property "Value" "DAN222"
+		(property "Value" "N"
 			(at 381.508 196.342 90)
 			(effects
@@
 				)
 				(hide yes)
-			)
-		)
-		(property "Topmark" "N"
-			(at 375.92 195.58 0)
-			(effects
-				(font
-					(size 1.27 1.27)
-				)
 			)
 		)
@@
 			)
 		)
-		(property "Description" "Resistor"
+		(property "Description" ""
 			(at 265.43 110.49 0)
 			(effects
@@
 			)
 		)
-		(property "Description" "Resistor"
+		(property "Description" ""
 			(at 375.92 168.91 0)
 			(effects
@@
 			)
 		)
-		(property "Datasheet" "https://www.ti.com/lit/ds/symlink/sn74aup1g02.pdf"
+		(property "Datasheet" ""
 			(at 337.82 142.24 0)
 			(effects
@@
 			)
 		)
-		(property "Description" "Single NOR Gate, Low-Voltage CMOS"
+		(property "Description" ""
 			(at 337.82 142.24 0)
 			(effects

Commit message: Add files via upload
Parts:
- removed D20: 3D, PC110:SOT-416L, symbol Device:D_Schottky_Dual_CommonCathode_AKA
- added D20: 3D, PC110:SOT-416L, symbol PC110:3D_Diode
Connections:
- net PNET5: no longer U24.5 (VCC)
- net PNET7: now also U24.5 (VCC)
- net PWRGD: now also D20.2
- net at R113.2, U59.10 (RP#): now also D20.3
- net at C246.1 (+), Q36.3 (C), R327.1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: now also D20.1
Changed lines of the file:
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@@
-	)
-	(symbol
-		(lib_id "Device:D_Schottky_Dual_CommonCathode_AKA")
-		(at 245.11 99.06 0)
-		(mirror y)
-		(unit 1)
-		(exclude_from_sim no)
-		(in_bom yes)
-		(on_board yes)
-		(dnp no)
-		(property "Reference" "D20"
-			(at 245.11 92.71 0)
-			(effects
-				(font
-					(size 1.27 1.27)
-				)
-			)
-		)
-		(property "Value" "3D"
-			(at 245.11 95.25 0)
-			(effects
-				(font
-					(size 1.27 1.27)
-				)
-			)
-		)
-		(property "Footprint" "PC110:SOT-416L"
-			(at 245.11 99.06 0)
-			(effects
-				(font
-					(size 1.27 1.27)
-				)
-				(hide yes)
-			)
-		)
-		(property "Datasheet" "~"
-			(at 245.11 99.06 0)
-			(effects
-				(font
-					(size 1.27 1.27)
-				)
-				(hide yes)
-			)
-		)
-		(property "Description" ""
-			(at 245.11 99.06 0)
-			(effects
-				(font
-					(size 1.27 1.27)
-				)
-				(hide yes)
-			)
-		)
-		(pin "1"
-		)
-		(pin "3"
-		)
-		(pin "2"
-		)
-		(instances
-			(project "PC110"
-				(path "/45c7911f-b027-440e-9e3e-77a146b41944/29aeee43-2869-4080-920c-a693b0bc5770"
-					(reference "D20")
-					(unit 1)
-				)
-			)
-		)
 	)
 	(symbol
@@
 	)
 	(symbol
+		(lib_id "PC110:3D_Diode")
+		(at 245.11 99.06 0)
+		(mirror y)
+		(unit 1)
+		(exclude_from_sim no)
+		(in_bom yes)
+		(on_board yes)
+		(dnp no)
+		(property "Reference" "D20"
+			(at 245.11 92.71 0)
+			(effects
+				(font
+					(size 1.27 1.27)
+				)
+			)
+		)
+		(property "Value" "3D"
+			(at 245.11 95.25 0)
+			(effects
+				(font
+					(size 1.27 1.27)
+				)
+			)
+		)
+		(property "Footprint" "PC110:SOT-416L"
+			(at 245.11 99.06 0)
+			(effects
+				(font
+					(size 1.27 1.27)
+				)
+				(hide yes)
+			)
+		)
+		(property "Datasheet" ""
+			(at 245.11 99.06 0)
+			(effects
+				(font
+					(size 1.27 1.27)
+				)
+				(hide yes)
+			)
+		)
+		(property "Description" ""
+			(at 245.11 99.06 0)
+			(effects
+				(font
+					(size 1.27 1.27)
+				)
+				(hide yes)
+			)
+		)
+		(pin "3"
+		)
+		(pin "2"
+		)
+		(pin "1"
+		)
+		(instances
+			(project "PC110"
+				(path "/45c7911f-b027-440e-9e3e-77a146b41944/29aeee43-2869-4080-920c-a693b0bc5770"
+					(reference "D20")
+					(unit 1)
+				)
+			)
+		)
+	)
+	(symbol
 		(lib_id "PCM_Elektuur:C")
 		(at 88.9 113.03 0)
@@
 			)
 		)
-		(property "Value" "PNET5"
+		(property "Value" "PNET7"
 			(at 337.82 125.73 0)
 			(effects

Commit message: Personal notes for PSU understanding
Connections:
- net GND: now also U36.34 (VSS)
Changed lines of the file:
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@@
 	)
 	(junction
+		(at 92.71 191.77)
+		(diameter 0)
+		(color 0 0 0 0)
+	)
+	(junction
 		(at 260.35 99.06)
 		(diameter 0)
@@
 	(wire
 		(pts
+			(xy 90.17 190.5) (xy 90.17 191.77)
+		)
+		(stroke
+			(width 0)
+			(type default)
+		)
+	)
+	(wire
+		(pts
 			(xy 120.65 143.51) (xy 135.89 143.51)
 		)
@@
 	(wire
 		(pts
+			(xy 90.17 191.77) (xy 92.71 191.77)
+		)
+		(stroke
+			(width 0)
+			(type default)
+		)
+	)
+	(wire
+		(pts
 			(xy 278.13 115.57) (xy 278.13 119.38)
 		)
@@
 	(wire
 		(pts
-			(xy 92.71 190.5) (xy 92.71 194.31)
+			(xy 92.71 190.5) (xy 92.71 191.77)
+		)
+		(stroke
+			(width 0)
+			(type default)
+		)
+	)
+	(wire
+		(pts
+			(xy 92.71 191.77) (xy 92.71 194.31)
 		)
 		(stroke
@@
 		(pin "35"
 		)
+		(pin "34"
+		)
 		(instances
