File: PCB/Mainboard/VGA.kicad_sch (KiCad schematic)
At the start: 20 parts, among them U101 TGUI9440

Commit message: Add files via upload
Parts:
- removed C120, C125, C126: 10uF, Capacitor_THT:CP_Radial_D5.0mm_P2.00mm, symbol Device:C_Polarized_US
- removed C121: C, Capacitor_SMD:C_0603_1608Metric_Pad1.08x0.95mm_HandSolder, symbol Device:C
- removed C52: 120pF, Capacitor_SMD:C_0603_1608Metric_Pad1.08x0.95mm_HandSolder, symbol Device:C
- removed C53: 100nF, Capacitor_SMD:C_0603_1608Metric_Pad1.08x0.95mm_HandSolder, symbol Device:C
- removed FB5: Ferrite_Bead, Inductor_SMD:L_0603_1608Metric_Pad1.05x0.95mm_HandSolder, symbol Device:FerriteBead_Small
- removed JP51, JP52: Jumper_2_Open, My_Components:Conn_Pin_Header_2x1_2.54mm, symbol Jumper:Jumper_2_Open
- removed JP53: Ready?!, My_Components:Conn_Pin_Header_3x1_2.54mm, symbol my_components:Jumper_3_Bridged12_Passive
- removed L1, L2: 2.7uH, Inductor_SMD:L_0603_1608Metric_Pad1.05x0.95mm_HandSolder, symbol Device:L
- removed R101, R125, R135: 33, Resistor_SMD:R_0612_1632Metric_Pad1.18x3.40mm_HandSolder, symbol Device:R
- removed R106: 510, Resistor_SMD:R_0612_1632Metric_Pad1.18x3.40mm_HandSolder, symbol Device:R
- removed R111: 4.7k, Resistor_SMD:R_0612_1632Metric_Pad1.18x3.40mm_HandSolder, symbol Device:R
- removed R133: 1k, Resistor_SMD:R_0612_1632Metric_Pad1.18x3.40mm_HandSolder, symbol Device:R
- removed RN16: 4.7k, Resistor_THT:R_Array_SIP10, symbol Device:R_Network09
- removed U101: TGUI9440, Package_QFP:PQFP-208_28x28mm_P0.5mm, symbol my_components:TGUI9440
Connections:
- no-connect marks 37 -> 0
Other:
- note removed: "(1x clock for VL BUS)"
- note removed: "(256Kx16 DRAMs)"
- note removed: "(Closed: Interlaced)"
- note removed: "(Closed: VLB Clock > 33 MHz?)"
- note removed: "(On-chip clock synthesizer)"
- note removed: "(ROM on ISA Bus)"
- note removed: "(Two extra ~{RAS} clocks)"
- note removed: "(VLB - LCLK)"
- note removed: "(VLB - LDEV#)"
- note removed: "(VLB - LRDY#)"
- note removed: "(VLB - RDYRTN#)"
- note removed: "(~{CASA0}-~{CASA3})"
- note removed: "RESET Selection: RESSEL = 1 - Active High RESSEL = 0 - Active Low VLB Uses active low"
- note removed: "TGUI94xx Straps"
- note removed: "VLF/MLF values from TKD8001 datasheet should they be connected to AVDD/AVSS?"

Commit message: Add files via upload
Parts:
- added U51: CHIPS65535, symbol PC110:65535
- added U8: ~, symbol PC110:51W4260

Commit message: Add files via upload
Connections:
- net LCD_STNDBY#: now reaches U51.K13 (STNDBY#)
Changed lines of the file:
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@@
 		(title "PC110")
+	)
+	(wire
+		(pts
+			(xy 278.13 195.58) (xy 303.53 195.58)
+		)
+		(stroke
+			(width 0)
+			(type default)
+		)
+	)
+	(label "LCD_STNDBY#"
+		(at 289.56 195.58 0)
+		(effects
+			(font
+				(size 1.27 1.27)
+			)
+			(justify left bottom)
+		)
 	)
 	(symbol

Commit message: Add files via upload
Connections:
- net VGA_HSync: now reaches U51.A10 (HSYNC)
- net VGA_Green: now reaches U51.A12 (VGA_Green)
- net GND: now reaches U51.B10 (GND)
- net GND: now also U51.B12 (GND), U51.B3 (GND), U51.D3 (GND), U51.D7 (GND), U51.E11 (GND), U51.G11 (GND), U51.H10 (GND), U51.J4 (GND), U51.L11 (GND), U51.L7 (GND), U51.N11 (GND)
- net VGA_Blue: now reaches U51.C10 (VGA_Blue)
- net CPU_BS16#: now reaches U51.C11 (BS16#)
- net VGA_VSync: now reaches U51.C9 (VSYNC)
- net CPU_WR#: now reaches U51.D12 (WEA#)
- net VGA_Red: now reaches U51.D9 (VGA_Red)
- net CPU_MIO#: now reaches U51.J11 (MIO#)
- net CPU_BE3#: now reaches U51.J9 (BE3)
- net CPU_ADS#: now reaches U51.K12 (ADS#)
- net VGA_CLK: now reaches U51.K9 (XTALI)
- net CPU_BE1#: now reaches U51.L13 (BE1#)
- net CPU_BE0#: now reaches U51.M5 (BE0#)
- net CPU_BE2#: now reaches U51.N5 (BE2#)
- no-connect marks 0 -> 1

Commit message: Add files via upload
Connections:
- net F65_ENAVEE: now reaches U51.E9 (ENAVEE)
Changed lines of the file:
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@@
+	(wire
+		(pts
+			(xy 229.87 38.1) (xy 229.87 54.61)
+		)
+		(stroke
+			(width 0)
+			(type default)
+		)
+	)
 	(wire
 		(pts
@@
 		)
 	)
-	(label "CPU_MIO#"
-		(at 288.29 187.96 0)
+	(label "F65_ENAVEE"
+		(at 229.87 50.8 90)
 		(effects
 			(font
@@
 		)
 	)
+	(label "CPU_MIO#"
+		(at 288.29 187.96 0)
+		(effects
+			(font
+				(size 1.27 1.27)
+			)
+			(justify left bottom)
+		)
+	)
 	(label "VGA_CLK"
 		(at 289.56 165.1 0)
 		(effects
 			(font
+				(size 1.27 1.27)
+			)
+			(justify left bottom)
+		)
+	)
+	(label "LCD_NC_L11"
+		(at 330.2 227.33 0)
+		(effects
+			(font

Commit message: Add files via upload
Connections:
- net CPU_D17: now reaches U51.B1 (D17)
- net CPU_D16: now reaches U51.B2 (D16)
- net CPU_D20: now reaches U51.C1 (D20)
- net CPU_D18: now reaches U51.C2 (D18)
- net CPU_D23: now reaches U51.D1 (D23)
- net CPU_D0: now reaches U51.D13 (D0)
- net CPU_D21: now reaches U51.D2 (D21)
- net CPU_D26: now reaches U51.E1 (D26)
- net CPU_D2: now reaches U51.E13 (D2)
- net CPU_D25: now reaches U51.E2 (D25)
- net CPU_D22: now reaches U51.E3 (D22)
- net CPU_D19: now reaches U51.E5 (D19)
- net CPU_D30: now reaches U51.F1 (D30)
- net CPU_D1: now reaches U51.F10 (D1)
- net CPU_D3: now reaches U51.F11 (D3)
- net CPU_D5: now reaches U51.F12 (D5)
- net CPU_D6: now reaches U51.F13 (D6)
- net CPU_D28: now reaches U51.F2 (D28)
- net CPU_D27: now reaches U51.F3 (D27)
- net CPU_D24: now reaches U51.F4 (D24)
- net CPU_D29: now reaches U51.F5 (D29)
- net CPU_D4: now reaches U51.F9 (D4)
- net CPU_D9: now reaches U51.G12 (D9)
- net CPU_D8: now reaches U51.G13 (D8)
- net CPU_D31: now reaches U51.G4 (D31)
- net CPU_D7: now reaches U51.G9 (D7)
- net CPU_D13: now reaches U51.H11 (D13)
- net CPU_D12: now reaches U51.H12 (D12)
- net CPU_D10: now reaches U51.H13 (D10)
- net CPU_D11: now reaches U51.H9 (D11)
- net CPU_D15: now reaches U51.J12 (D15)
- net CPU_D14: now reaches U51.J13 (D14)

Commit message: Add files via upload
Parts:
- added C169, C171, C173, C174, C175, C177, C178, C180, C181, C182, C183, C184, C185, C186, C187, C191, C192, C193, C194, C195, C196: 56pF, symbol PCM_Elektuur:C
- added C172, C189: 100nF, symbol PCM_Elektuur:C
- added C176: 470nF, symbol PCM_Elektuur:C
- added C188, C34, C37, C40, C43: 1nF, symbol PCM_Elektuur:C
- added C26, C31, C32, C38, C39, C41, C42: 150nF, symbol PCM_Elektuur:C
- added C30, C36: 10uF, symbol PCM_Elektuur:C
- added C48: 330nF, symbol PCM_Elektuur:C
- added D2: K, symbol Device:D_Dual_Series_KAC
- added D36: 71, symbol Device:D
- added EM1, EM2, EM3, EM4: EMI, symbol Device:Filter_EMI_LLLL_15263748
- added J2: LCD_Connector, symbol Connector_Generic:Conn_01x30
- added L10, L14, L9: 300nH, symbol PCM_Elektuur:L
- added L11, L16, L17, L18, L3: 1.5uH, symbol PCM_Elektuur:L
- added Q1: IS6, symbol Simulation_SPICE:PNP
- added Q2: 8C, Package_TO_SOT_SMD:SOT-23, symbol Transistor_BJT:MMBTA44
- added R1, R10, R11, R13, R15, R18, R19, R2, R22, R229, R233, R259, R269, R5, R6, R61, R7: 470k, symbol Device:R
- added R12: 182k, symbol Device:R
- added R14, R17, R20: 10, symbol Device:R
- added R16, R21, R51, R58: 0, symbol Device:R
- added R234: 100k, symbol Device:R
- added R236: 470, symbol Device:R
- added R255, R46, R53: 33, symbol Device:R
- added R263, R265, R270, R279, R9: 4.7k, symbol Device:R
- added R264, R267, R273: 150, symbol Device:R
- added R3: 131k, symbol Device:R
- added R66: 270, symbol Device:R
Connections:
- net GND: now also U8.21 (GND), U8.27 (OE#), U8.35 (GND), U8.40 (GND), C169.2 (-), C171.2 (-), C172.1 (+), C173.2 (-), C174.2 (-), C175.2 (-), C176.2 (-), C177.2 (-), C178.2 (-), C180.2 (-), C181.2 (-), C182.2 (-), C183.2 (-), C184.2 (-), C185.2 (-), C186.2 (-), C187.2 (-), C188.2 (-), C189.1 (+), C191.2 (-), C192.2 (-), C193.2 (-), C194.2 (-), C195.1 (+), C196.2 (-), C26.2 (-), C30.1 (+), C31.1 (+), C32.2 (-), C34.2 (-), C36.1 (+), C37.2 (-), C38.2 (-), C39.2 (-), C40.2 (-), C41.2 (-), C42.1 (+), C43.2 (-), C48.2 (-), D36.2 (A), L10.2 (-), Q2.2 (E), R1.1, R10.1, R11.2, R13.1, R15.2, R18.2, R19.1, R2.1, R22.1, R233.2, R259.2, R263.2, R264.2, R265.2, R267.2, R269.2, R270.2, R273.2, R279.2, R5.1, R6.1, R61.1, R66.1, R7.1
- net VGA_Blue: now also R264.1
- net VGA_Green: now also R273.1
- net VGA_HSync: now also R53.1; no longer U51.A10 (HSYNC)
- net VGA_Red: now also R267.1
- net VGA_VSync: now also R46.1; no longer U51.C9 (VSYNC)
- net at U51.A11 (ENAVDD): now also D2.1 (K), R12.2
- net at U51.A13 (RSET): now also R66.2
- net at U51.A3 (P15): now also EM4.8
- net at U51.A4 (P12): now also EM4.5
- net at U51.A5 (P9): now also EM2.6
- net at U51.A6 (P5): now also EM3.6
- net at U51.A7 (P3): now also EM1.8
- net at U51.A8 (P1): now also EM1.6
- net at U51.A9 (LP): now also R17.1
- net PNET1: now reaches U51.B11 (VCC)
- net PNET1: now also U51.C7 (VCC), U51.D8 (VCC), U51.E12 (VCC), U51.E4 (VCC), U51.G10 (VCC), U51.K6 (VCC), U51.K7 (VCC), U51.M1 (VCC), U8.1 (VCC), U8.20 (VCC), U8.6 (VCC), C172.2 (-), C26.1 (+), C31.2 (-), C32.1 (+), C34.1 (+), C37.1 (+), C38.1 (+), C39.1 (+), C40.1 (+), C41.1 (+), C42.2 (-), C43.1 (+), L3.1 (+), R229.2
- net at U51.B13 (OEL#): now also R263.1
- net at U51.B4 (P14): now also EM4.7
- net at U51.B5 (P10): now also EM2.7
- net at U51.B6 (P6): now also EM3.7
- net at U51.B7 (P2): now also EM1.7
- net at U51.B8 (SHFCLK): now also R20.1
- net at U51.B9 (FLM): now also R14.1
- net CPU_RDY#: now reaches U51.C12 (RDY#)
- net CPU_RDY#: now also U51.C13 (RDY#)
- net at U51.C5 (P13): now also EM4.6
- net at U51.C6 (P8): now also EM2.5
- net VGA_LDEV#: now reaches U51.D11 (LDEV#)
- net at U51.D6 (P11): now also EM2.8
- net at U51.E10 (CCLK): now also R255.2
- net at U51.E6 (P7): now also EM3.8
- net at U51.E7 (P4): now also EM3.5
- net at U51.E8 (P0): now also EM1.5
- net at U51.G1 (SA1): now also U8.17 (A1)
- net at U51.G2 (SA0): now also U8.16 (A0), R265.1
- net at U51.G3 (SA2): now also U8.18 (A2)
- net at U51.G5 (SA3): now also U8.19 (A3)
- net at U51.H1 (SA4): now also U8.22 (A4)
- net at U51.H2 (SA5): now also U8.23 (A5), R270.1
- net at U51.H3 (SA7): now also U8.25 (A7)
- net at U51.H4 (RASA#): now also R21.2
- net at U51.H5 (SA6): now also U8.24 (A6)
- net at U51.J1 (SA8): now also U8.26 (A8), R279.1
- net VGA_ADDHI: now reaches U51.J10 (ADDHI)
- net Chipset_32KHz: now reaches U51.J2 (32kHz)
- net at U51.J3 (UCAS#): now also R51.1
- net at U51.J5 (IO11): now also U8.34 (DQ11), R18.1
- net CPU_A4: now reaches U51.J6 (A4)
- net CPU_A8: now reaches U51.J7 (A8)
- net CPU_A11: now reaches U51.J8 (A11)
- net at U51.K1 (CASAH#): now also R16.2
- net RESET: now reaches U51.K10 (RESET)
- net CPU_A21: now reaches U51.K11 (A21)
- net at U51.K2 (CASAL#): now also R58.1
- net at U51.K3 (IO1): now also U8.3 (DQ1), R1.2
- net at U51.K4 (IO3): now also U8.5 (DQ3), R6.2
- net at U51.K5 (IO10): now also U8.33 (DQ10), R61.2
- net CPU_A15: now reaches U51.K8 (A15)
- net at U51.L1 (IO0): now also U8.2 (DQ0), R11.1
- net CPU_A23: now reaches U51.L12 (A23)
- net at U51.L2 (IO2): now also U8.4 (DQ2), R10.2
- net at U51.L3 (IO4): now also U8.7 (DQ4), R7.2
- net at U51.L4 (IO7): now also U8.10 (DQ7), R2.2
- net at U51.L5 (IO14): now also U8.38 (DQ14), R233.1
- net CPU_A2: now reaches U51.L6 (A2)
- net CPU_A12: now reaches U51.L8 (A12)
- net CPU_A17: now reaches U51.L9 (A17)
- net CPU_A18: now reaches U51.M10 (A18)
- net PNET5: now reaches U51.M11 (CVCC)
- net PNET5: now also Q1.2 (E)
- net CPU_A20: now reaches U51.M12 (A20)
- net CPU_A22: now reaches U51.M13 (A22)
- net at U51.M2 (IO6): now also U8.9 (DQ6), R5.2
- net at U51.M3 (IO9): now also U8.32 (DQ9), R259.1
- net at U51.M4 (IO13): now also U8.37 (DQ13), R22.2
- net CPU_A3: now reaches U51.M6 (A3)
- net CPU_A6: now reaches U51.M7 (A6)
- net CPU_A10: now reaches U51.M8 (A10)
- net CPU_A14: now reaches U51.M9 (A14)
- net at U51.N1 (IO5): now also U8.8 (DQ5), R13.2
- net CPU_A16: now reaches U51.N10 (A16)
- net at U51.N12 (CVCC2): now also C30.2 (-), C36.2 (-), C48.1 (+), L3.2 (-)
- net CPU_A19: now reaches U51.N13 (A19)
- net at U51.N2 (IO8): now also U8.31 (DQ8), R269.1
- net at U51.N3 (IO12): now also U8.36 (DQ12), R15.1
- net at U51.N4 (IO15): now also U8.39 (DQ15), R19.2
- net CPU_A5: now reaches U51.N6 (A5)
- net CPU_A7: now reaches U51.N7 (A7)
- net CPU_A9: now reaches U51.N8 (A9)
- net CPU_A13: now reaches U51.N9 (A13)
- net at U8.13 (WE#): now also R16.1
- net at U8.14 (RAS#): now also R21.1
- net at U8.28 (UCAS#): now also R51.2
- net at U8.29 (LCAS#): now also R58.2
- new net: C193.1 (+), J2.5 (Pin_5), R234.1
- new net: C189.2 (-), J2.2 (Pin_2), L14.1 (+)
- new net: C177.1 (+), J2.27 (Pin_27), L18.1 (+)
- new net: L18.2 (-), R17.2
- new net: C195.2 (-), J2.29 (Pin_29), L17.2 (-)
- new net: L11.1 (+), R14.2
- new net: D36.1 (K), L14.2 (-), R236.1
- new net: L16.1 (+), R229.1
- new net: C176.1 (+), C188.1 (+), J2.4 (Pin_4), L9.1 (+), R234.2
- new net: L9.2 (-), Q1.3 (C), R236.2, R3.2
- new net: R53.2, U51.A10 (HSYNC)
- new net: R46.2, U51.C9 (VSYNC)
- new net: C192.1 (+), J2.26 (Pin_26), L11.2 (-)
- new net: D2.2 (A), R3.1
- new net: C171.1 (+), J2.6 (Pin_6), L16.2 (-)
- new net: D2.3 (common), Q2.1 (B), R12.1
- new net: J2.1 (Pin_1), J2.16 (Pin_16), J2.25 (Pin_25), J2.28 (Pin_28), J2.30 (Pin_30), J2.7 (Pin_7), L10.1 (+)
- new net: L17.1 (+), R20.2
- new net: Q2.3 (C), R9.1
- new net: Q1.1 (B), R9.2
- new net Chipset_CPU_CLK: R255.1
- new net LCD_24: C174.1 (+), EM4.1, J2.24 (Pin_24)
- new net LCD_B0: C173.1 (+), EM1.4, J2.8 (Pin_8)
- new net LCD_B1: C183.1 (+), EM1.3, J2.9 (Pin_9)
- new net LCD_B2: C194.1 (+), EM1.2, J2.10 (Pin_10)
- new net LCD_B3: C181.1 (+), EM1.1, J2.11 (Pin_11)
- new net LCD_B4: C180.1 (+), EM3.4, J2.17 (Pin_17)
- new net LCD_G0: C182.1 (+), EM3.3, J2.18 (Pin_18)
- new net LCD_G1: C187.1 (+), EM3.2, J2.19 (Pin_19)
- new net LCD_G2: C186.1 (+), EM3.1, J2.20 (Pin_20)
- new net LCD_G3: C191.1 (+), EM2.4, J2.12 (Pin_12)
- new net LCD_G4: C184.1 (+), EM2.3, J2.13 (Pin_13)
- new net LCD_R0: C185.1 (+), EM2.2, J2.14 (Pin_14)
- new net LCD_R1: C169.1 (+), EM2.1, J2.15 (Pin_15)
- new net LCD_R2: C196.1 (+), EM4.4, J2.21 (Pin_21)
- new net LCD_R3: C175.1 (+), EM4.3, J2.22 (Pin_22)
- new net LCD_R4: C178.1 (+), EM4.2, J2.23 (Pin_23)
- new net LCD_VAA: J2.3 (Pin_3)
- no-connect marks 1 -> 22
