File: PCB/Mainboard/VGA.kicad_sch (KiCad schematic)
At the start: 98 parts, among them J2 LCD_Connector, Q1 2SA1881-6, Q2 8C, U51 CHIPS65535

Commit message: Add files via upload
Connections:
- net PNET5: now also Q1.3 (E); no longer Q1.2 (E)
- net LCD_NC_L11: now reaches L16.1 (+), R229.1
- net at L9.2 (-), R236.2, R3.2: now also Q1.1 (C); no longer Q1.3 (C)
- net at R9.2: now also Q1.2 (B); no longer Q1.1 (B)
- net VGA_LDEV# renamed CPU_LDEV#
- no-connect marks 22 -> 9
Other:
- moved on the sheet: R229

Commit message: Add files via upload
Parts:
- added C156: 100nF, symbol PCM_Elektuur:C
- added C17, C5: 150nF, symbol PCM_Elektuur:C
- added C206, C210: 10uF, symbol PCM_Elektuur:C
- added C45: 270nF, symbol PCM_Elektuur:C
- added L6: 1.5uH, symbol PCM_Elektuur:L
Connections:
- net GND: now also C156.1 (+), C17.2 (-), C206.2 (-), C210.2 (-), C45.2 (-), C5.2 (-)
- net PNET1: now also C156.2 (-), C17.1 (+), C5.1 (+), L6.2 (-)
- net PNET5: no longer U51.M11 (CVCC)
- new net: C206.1 (+), C210.1 (+), C45.1 (+), L6.1 (+), U51.M11 (CVCC)

Commit message: Add files via upload
Parts:
- C156, C169, C17, C171, C172, C173, C174, C175, C177, C178, C180, C181, C182, C183, C184, C185, C186, C187, C188, C189, C191, C192, C193, C194, C195, C196, C26, C31, C32, C34, C37, C38, C39, C40, C41, C42, C43, C48, C5: footprint (none) -> Capacitor_SMD:C_0402_1005Metric
- C176, C45: footprint (none) -> Capacitor_SMD:C_0603_1608Metric
- C206, C210, C30, C36: footprint (none) -> Capacitor_SMD:C_1206_3216Metric
- D2: footprint (none) -> PC110:SOT-416L
- D36: footprint (none) -> Diode_SMD:D_0603_1608Metric
- EM1, EM2, EM3, EM4: footprint (none) -> PC110:R-array
- J2: footprint (none) -> PC110:LCD_connector
- L10, L9: footprint (none) -> Inductor_SMD:L_0805_2012Metric
- L11, L14, L16, L17, L18, L3, L6: footprint (none) -> Inductor_SMD:L_0603_1608Metric
- Q1: footprint (none) -> PCM_Package_TO_SOT_SMD_AKL:SOT-23
- Q2: footprint Package_TO_SOT_SMD:SOT-23 -> Package_TO_SOT_SMD:SOT-416
- R1, R10, R11, R12, R13, R14, R15, R16, R17, R18, R19, R2, R20, R21, R22, R229, R233, R234, R236, R255, R259, R263, R265, R269, R270, R279, R3, R46, R5, R51, R53, R58, R6, R61, R66, R7, R9: footprint (none) -> PCM_Resistor_SMD_AKL:R_0402_1005Metric
- R264, R267, R273: footprint (none) -> PCM_Resistor_SMD_AKL:R_0805_2012Metric
- U51: footprint (none) -> PC110:BGA-169
- U8: footprint (none) -> PC110:GRAMchip
Connections:
- net GND: now also C177.1 (+), C206.1 (+), C210.1 (+); no longer C177.2 (-), C206.2 (-), C210.2 (-)
- net LCD_NC_L11: now also L16.2 (-); no longer L16.1 (+)
- net at J2.27 (Pin_27), L18.1 (+): now also C177.2 (-); no longer C177.1 (+)
- net at D36.1 (K), L14.2 (-): now also R236.2; no longer R236.1
- net at L9.2 (-), Q1.1 (C), R3.2: now also R236.1; no longer R236.2
- net at C45.1 (+), L6.1 (+), U51.M11 (CVCC): now also C206.2 (-), C210.2 (-); no longer C206.1 (+), C210.1 (+)
- net at C171.1 (+), J2.6 (Pin_6): now also L16.1 (+); no longer L16.2 (-)
Other:
- moved on the sheet: C189, R236

Commit message: Add files via upload
Parts:
- removed Q1: 2SA1881-6, PCM_Package_TO_SOT_SMD_AKL:SOT-23, symbol Simulation_SPICE:PNP
- added Q1: 2SA1881-6, symbol PCM_Transistor_BJT_AKL:Q_PNP_Generic_BEC
Connections:
- net PNET5: now also Q1.2 (E)
- net at L9.2 (-), R236.1, R3.2: now also Q1.3 (C)
- net at R9.2: now also Q1.1 (B)
Changed lines of the file:
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@@
+	)
+	(symbol
+		(lib_id "PCM_Transistor_BJT_AKL:Q_PNP_Generic_BEC")
+		(at 518.16 33.02 0)
+		(unit 1)
+		(exclude_from_sim no)
+		(in_bom yes)
+		(on_board yes)
+		(dnp no)
+		(fields_autoplaced yes)
+		(property "Reference" "Q1"
+			(at 523.24 31.7499 0)
+			(effects
+				(font
+					(size 1.27 1.27)
+				)
+				(justify left)
+			)
+		)
+		(property "Value" "2SA1881-6"
+			(at 523.24 34.2899 0)
+			(effects
+				(font
+					(size 1.27 1.27)
+				)
+				(justify left)
+			)
+		)
+		(property "Footprint" ""
+			(at 523.24 35.56 0)
+			(effects
+				(font
+					(size 1.27 1.27)
+				)
+				(hide yes)
+			)
+		)
+		(property "Datasheet" "~"
+			(at 518.16 33.02 0)
+			(effects
+				(font
+					(size 1.27 1.27)
+				)
+				(hide yes)
+			)
+		)
+		(property "Description" "PNP transistor, generic symbol, Alternate KiCAD Library"
+			(at 518.16 33.02 0)
+			(effects
+				(font
+					(size 1.27 1.27)
+				)
+				(hide yes)
+			)
+		)
+		(pin "1"
+		)
+		(pin "2"
+		)
+		(pin "3"
+		)
+		(instances
+			(project ""
+				(path "/45c7911f-b027-440e-9e3e-77a146b41944/00000000-0000-0000-0000-000066b27913"
+					(reference "Q1")
+					(unit 1)
+				)
+			)
+		)
 	)
 	(symbol
@@
 					(unit 1)
 				)
-			)
-		)
-	)
-	(symbol
-		(lib_id "Simulation_SPICE:PNP")
-		(at 518.16 33.02 0)
-		(mirror x)
-		(unit 1)
-		(exclude_from_sim no)
-		(in_bom yes)
-		(on_board yes)
-		(dnp no)
-		(property "Reference" "Q1"
-			(at 523.24 29.718 0)
-			(effects
-				(font
-					(size 1.27 1.27)
-				)
-				(justify left)
-			)
-		)
-		(property "Value" "2SA1881-6"
-			(at 523.24 32.258 0)
-			(effects
-				(font
-					(size 1.27 1.27)
-				)
-				(justify left)
-			)
-		)
-		(property "Footprint" "PCM_Package_TO_SOT_SMD_AKL:SOT-23"
-			(at 553.72 33.02 0)
-			(effects
-				(font
-					(size 1.27 1.27)
-				)
-				(hide yes)
-			)
-		)
-		(property "Datasheet" "https://ngspice.sourceforge.io/docs/ngspice-html-manual/manual.xhtml#cha_BJTs"
-			(at 553.72 33.02 0)
-			(effects
-				(font
-					(size 1.27 1.27)
-				)
-				(hide yes)
-			)
-		)
-		(property "Description" "Bipolar transistor symbol for simulation only, substrate tied to the emitter"
-			(at 518.16 33.02 0)
-			(effects
-				(font
-					(size 1.27 1.27)
-				)
-				(hide yes)
-			)
-		)
-		(property "Sim.Device" "PNP"
-			(at 518.16 33.02 0)
-			(effects
-				(font
-					(size 1.27 1.27)
-				)
-				(hide yes)
-			)
-		)
-		(property "Sim.Type" "GUMMELPOON"
-			(at 518.16 33.02 0)
-			(effects
-				(font
-					(size 1.27 1.27)
-				)
-				(hide yes)
-			)
-		)
-		(property "Sim.Pins" "1=C 2=B 3=E"
-			(at 518.16 33.02 0)
-			(effects
-				(font
-					(size 1.27 1.27)
-				)
-				(hide yes)
-			)
-		)
-		(property "Topmark" "IS6"
-			(at 518.16 33.02 0)
-			(effects
-				(font
-					(size 1.27 1.27)
-				)
-				(hide yes)
-			)
-		)
-		(pin "2"
-		)
-		(pin "1"
-		)
-		(pin "3"
-		)
-		(instances
-			(project "PC110"
-				(path "/45c7911f-b027-440e-9e3e-77a146b41944/00000000-0000-0000-0000-000066b27913"
-					(reference "Q1")
-					(unit 1)
-				)

Commit message: Add files via upload
Parts:
- Q1: footprint (none) -> PCM_Package_TO_SOT_SMD_AKL:SOT-23
Changed lines of the file:
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@@
 			)
 		)
-		(property "Footprint" ""
+		(property "Footprint" "PCM_Package_TO_SOT_SMD_AKL:SOT-23"
 			(at 523.24 35.56 0)
 			(effects

Commit message: Add files via upload
Parts:
- removed EM1, EM2, EM3, EM4: EMI, PC110:R-array, symbol Device:Filter_EMI_LLLL_15263748
- added EM1, EM2, EM3, EM4: R-array, PC110:R-array, symbol PC110:EMI_filter_Array
- C156, C169, C17, C171, C172, C173, C174, C175, C176, C177, C178, C180, C181, C182, C183, C184, C185, C186, C187, C188, C189, C191, C192, C193, C194, C195, C196, C206, C210, C26, C30, C31, C32, C34, C36, C37, C39, C40, C42, C43, C45, C48, C5: Indicator + -> (none); Rating V -> (none)
- C38: value 150nF -> 1nF; Indicator + -> (none); Rating V -> (none)
- C41: value 150nF -> 120nF; Indicator + -> (none); Rating V -> (none)
- D2: value DA204U -> K; Topmark K -> (none)
- J2: value LCD_Connector -> LCD_connector
- L10, L11, L16, L17, L18, L3, L6, L9: Indicator ● -> (none); Rating A -> (none)
- L14: value 300nH -> 1.5uH; Indicator ● -> (none); Rating A -> (none)
- Q1: value 2SA1881-6 -> IS6
- U8: value ~ -> 51W4260ATT7
Connections:
- net LCD_24: now also EM4.1
- net LCD_B0: now also EM1.4
- net LCD_B1: now also EM1.3
- net LCD_B2: now also EM1.2
- net LCD_B3: now also EM1.1
- net LCD_B4: now also EM3.4
- net LCD_G0: now also EM3.3
- net LCD_G1: now also EM3.2
- net LCD_G2: now also EM3.1
- net LCD_G3: now also EM2.4
- net LCD_G4: now also EM2.3
- net LCD_R0: now also EM2.2
- net LCD_R1: now also EM2.1
- net LCD_R2: now also EM4.4
- net LCD_R3: now also EM4.3
- net LCD_R4: now also EM4.2
- net at U51.E8 (P0): now also EM1.5
- net at U51.A8 (P1): now also EM1.6
- net at U51.B7 (P2): now also EM1.7
- net at U51.A7 (P3): now also EM1.8
- net at U51.A4 (P12): now also EM4.5
- net at U51.C5 (P13): now also EM4.6
- net at U51.B4 (P14): now also EM4.7
- net at U51.A3 (P15): now also EM4.8
- net at U51.E7 (P4): now also EM3.5
- net at U51.A6 (P5): now also EM3.6
- net at U51.B6 (P6): now also EM3.7
- net at U51.E6 (P7): now also EM3.8
- net at U51.A5 (P9): now also EM2.6
- net at U51.B5 (P10): now also EM2.7
- net at U51.C6 (P8): now also EM2.5
- net at U51.D6 (P11): now also EM2.8
