File: PCB/Mainboard/Storage.kicad_sch (KiCad schematic)
At the start: 0 parts

Commit message: Add files via upload
Parts:
- added U41: SDBL-4, symbol PC110:SDLB-4
- added U42: SC414281PU4, symbol PC110:SC414281PU4

Commit message: Add files via upload
Parts:
- added J11: ~, symbol PC110:CF_Conn
- added U27: AT29LV512, symbol PC110:AT29LV512
Other:
- moved on the sheet: U41, U42

Commit message: Add files via upload
Parts:
- added R161, R173: 470k, symbol Device:R
Connections:
- net GND: now reaches J11.1 (GND)
- net GND: now also J11.15 (GND), J11.16 (GND), J11.17 (GND), J11.19 (GND), J11.21 (GND), J11.23 (GND), J11.27 (GND), J11.29 (GND), J11.31 (GND), J11.33 (GND), J11.50 (GND)
- net SD15_Bus: now reaches J11.10 (SD14)
- net SD15_Bus: now also J11.12 (SD15)
- net SD7_Bus: now reaches J11.11 (SD7)
- net CF_CD1_Pluto: now reaches J11.2 (CD1#)
- net CF_CD1_Pluto: now also R173.2
- net SD3_Bus: now reaches J11.3 (SD3)
- net SD11_Bus: now reaches J11.4 (SD11)
- net SD0_Bus: now reaches J11.41 (SD0)
- net SD1_Bus: now reaches J11.43 (SD1)
- net SD8_Bus: now reaches J11.44 (SD8)
- net SD2_Bus: now reaches J11.45 (SD2)
- net SD9_Bus: now reaches J11.46 (SD9)
- net SD10_Bus: now reaches J11.48 (SD10)
- net CF_CD2_Pluto: now reaches J11.49 (CD2#)
- net CF_CD2_Pluto: now also R161.2
- net SD4_Bus: now reaches J11.5 (SD4)
- net SD12_Bus: now reaches J11.6 (SD12)
- net SD5_Bus: now reaches J11.7 (SD5)
- net SD13_Bus: now reaches J11.8 (SD13)
- net SD6_Bus: now reaches J11.9 (SD6)
- new net PNET1: R161.1, R173.1
Other:
- moved on the sheet: J11, U27, U42

Commit message: Add files via upload
Parts:
- added C272: 150nF, symbol PCM_Elektuur:C
- added F4: 0.5A, symbol Device:Fuse
- added R184: DNP, symbol Device:R
Connections:
- net GND: now also C272.2 (-), R184.2
- net SA2: now reaches U42.33 (SA2)
- net SA2: now also J11.35 (SA2)
- net SA1: now reaches U42.34 (SA1)
- net SA1: now also J11.37 (SA1)
- net SA0: now reaches U42.35 (SA0)
- net SA0: now also J11.39 (SA0)
- net FCS_RESET: now reaches U42.36 (RESET)
- net FCS_RESET: now also J11.32 (RESET), R184.1
- net FCS_IOCHRDY: now reaches U42.47 (WAIT)
- net FCS_IOCHRDY: now also J11.34 (IOCHRDY)
- net FCS_BVD2: now reaches U42.49 (BVD2)
- net FCS_BVD2: now also J11.40 (BVD2)
- net FCS_BVD1: now reaches U42.50 (BVD1)
- net FCS_BVD1: now also J11.42 (BVD1)
- net at J11.25 (VCC): now also J11.26 (VCC), C272.1 (+), F4.1
- new net PNET12: F4.2
Other:
- moved on the sheet: U27, U42

Commit message: Add files via upload
Parts:
- added C236: 100nF, symbol Device:C
- added C271: 150nF, symbol Device:C
- added R145, R290, R296, R298, R301: DNP, symbol Device:R
- added R295, R366, R367: 0, symbol Device:R
- added R360, R361: 470k, symbol Device:R
- added R365: 10k, symbol Device:R
- added U56: SN74LV32, symbol 74xx:74LS32
- added U68: SN74LV08, symbol 74xx:74LS08
Connections:
- net CF_CD1_Pluto: no longer J11.2 (CD1#), R173.2
- net CF_CD2_Pluto: no longer J11.49 (CD2#), R161.2
- net GND: now also U42.10 (GND), U42.20 (GND), U42.32 (GND), U42.44 (GND), U42.61 (GND), U42.70 (GND), U42.82 (GND), U42.94 (GND), C236.1, C271.1, R145.2, U56.7 (GND), U68.7 (GND)
- net PNET12: now also C236.2, C271.2, R360.1, R361.1, U56.14 (VCC), U68.14 (VCC)
- net at U42.37 (CE1): now also J11.13 (CE1#), R361.2, R366.1
- net at U42.39 (CE2): now also J11.14 (CE2#), R360.2, R367.1
- net at U42.42 (IORD): now also R296.2, R301.1, U56.3
- net at U42.43 (IOWR): now also R290.1, R298.1, U56.6
- net IRQ14: now reaches U42.46 (RDY)
- net IRQ14: now also J11.24 (IRQ14), R365.2
- net IOCS16#: now reaches U42.52 (IO16)
- net IOCS16#: now also J11.47 (IOCS16#)
- net at J11.18 (IOR#): now also R295.2, R301.2
- net at J11.20 (IOW#): now also R290.2
- net at J11.28 (CSEL#): now also R145.1
- new net: U56.2, U56.5, U68.3
- new net: R367.2, U68.2
- new net: J11.49 (CD2#), R161.2
- new net: R366.2, U68.1
- new net: J11.2 (CD1#), R173.2
- new net IOR#: R295.1, R296.1, U56.1
- new net IOW#: R298.2, U56.4
- new net PNET7: R365.1
- no-connect marks 0 -> 5
Other:
- moved on the sheet: C272, F4, J11, R161, R173, R184, U27, U41, U42

Commit message: Add files via upload
Parts:
- added C220pF, C266: 180pF, symbol Device:C
- added R362, R371: 2k, symbol Device:R
Connections:
- net GND: now also U42.23 (CSEL), U42.24 (SA10), U42.25 (SA9), U42.26 (SA8), U42.27 (SA7), U42.28 (SA6), U42.29 (SA5), U42.30 (SA4), U42.31 (SA3), U42.40 (OE), C220pF.1
- net PNET12: now also U42.38 (VCC)
- net SD0_Bus: now also U42.22 (HD0)
- net SD10_Bus: now also U42.7 (HD10)
- net SD11_Bus: now also U42.6 (HD11)
- net SD12_Bus: now also U42.4 (HD12)
- net SD13_Bus: now also U42.3 (HD13)
- net SD15_Bus: now also U42.1 (HD15), U42.2 (HD14)
- net SD1_Bus: now also U42.21 (HD1)
- net SD2_Bus: now also U42.19 (HD2)
- net SD3_Bus: now also U42.18 (HD3)
- net SD4_Bus: now also U42.17 (HD4)
- net SD5_Bus: now also U42.16 (HD5)
- net SD6_Bus: now also U42.14 (HD6)
- net SD7_Bus: now also U42.13 (HD7)
- net SD8_Bus: now also U42.9 (HD8)
- net SD9_Bus: now also U42.8 (HD9)
- net at U42.11 (RC_IN): now also R371.1
- net at U42.12 (C_EXT): now also R362.1, R371.2
- new net: C266.2, R362.2
- new net: C220pF.2, C266.1
- no-connect marks 5 -> 8

Commit message: Add files via upload
Parts:
- added C131: 10nF, symbol Device:C
- added C133, C141, C146, C241, C263, C94: 100nF, symbol Device:C
- added C142, C143: 150nF, symbol Device:C
- added C144, C145: 100pF, symbol Device:C
- added C262: 1.5uF, symbol Device:C
- added Q37: BH, symbol PCM_Generic:Q-BJT-Darlington,PNP,IEEE
- added R131: DNP, symbol Device:R
- added R134: 10k, symbol Device:R
- added R368: 1.5k, symbol Device:R
- added U65: E4, symbol 74xGxx:74AHC1G32
Connections:
- net GND: now also U27.24 (GND), U42.51 (WPROTCT), U56.10, U56.12, U56.13, U56.9, U68.10, U68.12, U68.13, U68.4, U68.5, U68.9, C131.1, C133.1, C144.1, C145.1, C241.1, C262.1, C263.1, C94.1, R131.2, U65.2, U65.3 (GND)
- net PNET12: now also U27.8 (VCC), U42.15 (VCC), U42.5 (VCC), U42.56 (VCC), U42.65 (VCC), U42.88 (VCC), C133.2, C241.2, C262.2, C263.2, C94.2, Q37.3 (E), R134.1, U65.5 (VCC)
- net at U42.100 (MD7): now also U27.29 (MD7)
- net at U42.53 (SCLK1): now also U41.5 (SCLK1)
- net at U42.55 (CS): now also U41.7 (CS)
- net at U42.57 (PD): now also U41.4 (PD)
- net at U42.58 (SI1): now also U41.2 (SI1)
- net at U42.59 (SI0): now also U41.1 (SI0)
- net at U42.60 (SO1): now also U41.17 (SO1)
- net at U42.62 (SO0): now also U41.13 (SO0)
- net at U42.66 (IO0): now also U65.1
- net at U42.71 (ROMCEL0): now also U27.30 (ROMCEL0#)
- net at U42.72 (ROMOEL): now also U27.32 (ROMOEL#)
- net at U42.73 (ROMWEL): now also U27.7 (ROMWEL#), R131.1, R134.2
- net at U42.74 (MA0): now also U27.20 (MA0)
- net at U42.75 (MA1): now also U27.19 (MA1)
- net at U42.76 (MA2): now also U27.18 (MA2)
- net at U42.77 (MA3): now also U27.17 (MA3)
- net at U42.78 (MA4): now also U27.16 (MA4)
- net at U42.79 (MA5): now also U27.15 (MA5)
- net at U42.80 (MA6): now also U27.14 (MA6)
- net at U42.81 (MA7): now also U27.13 (MA7)
- net at U42.83 (MA8): now also U27.3 (MA8)
- net at U42.84 (MA9): now also U27.2 (MA9)
- net at U42.85 (MA10): now also U27.31 (MA10)
- net at U42.86 (MA11): now also U27.1 (MA11)
- net at U42.87 (MA12): now also U27.12 (MA12)
- net at U42.89 (MA13): now also U27.4 (MA13)
- net at U42.90 (MA14): now also U27.5 (MA14)
- net at U42.91 (MA15): now also U27.11 (MA15)
- net at U42.92 (MD0): now also U27.21 (MD0)
- net at U42.93 (MD1): now also U27.22 (MD1)
- net at U42.95 (MD2): now also U27.23 (MD2)
- net at U42.96 (MD3): now also U27.25 (MD3)
- net at U42.97 (MD4): now also U27.26 (MD4)
- net at U42.98 (MD5): now also U27.27 (MD5)
- net at U42.99 (MD6): now also U27.28 (MD6)
- net at U41.20 (Cext2): now also C141.2
- net at U41.21 (Cext3): now also C143.2
- net at U41.22 (Cext4): now also C142.2, C144.2
- net at U41.23 (Cext5): now also C141.1, C145.2
- net at U41.24 (Cext6): now also C146.2
- net at U41.25 (Cext7): now also C142.1
- net at U41.26 (Cext8): now also C143.1
- net at U41.27 (Cext9): now also C146.1
- net at U41.28 (VCC): now also C131.2, Q37.1 (C)
- new net: R368.1, U65.4
- new net: Q37.2 (B), R368.2
- no-connect marks 8 -> 22
Other:
- moved on the sheet: C220pF, C236, C266, C271, C272, F4, J11, R145, R161, R173, R184, R290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

Commit message: Add files via upload
Parts:
- added R369: 22k, symbol Device:R
Connections:
- net PNET12: now also R369.1
- net FDC_HDCS1#: now reaches R367.2, U68.2
- net FDC_HDCS0#: now reaches R366.2, U68.1
- net SD7_Bus renamed FDC_IDE7
- net FDC_IDE7: now also R369.2
