File: PCB/Mainboard/Storage.kicad_sch (KiCad schematic)
At the start: 46 parts, among them Q37 BH, U27 AT29LV512, U41 SDBL-4, U42 SC414281PU4, U56 SN74LV32, U65 E4, U68 SN74LV08

Commit message: Add files via upload
Parts:
- added C132: 100nF, symbol Device:C
- added C134: 150nF, symbol Device:C
- renumbered C220pF to C269
Connections:
- net GND: now also U41.12 (GND), U41.15 (GND), U41.16 (GND), U41.18 (GND), U41.19 (GND), U41.3 (GND), U41.6 (GND), U41.8 (GND), C132.1, C134.1
- net SD0_Bus renamed SD0
- net SD10_Bus renamed SD10
- net SD11_Bus renamed SD11
- net SD12_Bus renamed SD12
- net SD13_Bus renamed SD13
- net SD15_Bus renamed SD14
- net SD14: no longer J11.12 (SD15), U42.1 (HD15)
- net SD1_Bus renamed SD1
- net SD2_Bus renamed SD2
- net SD3_Bus renamed SD3
- net SD4_Bus renamed SD4
- net SD5_Bus renamed SD5
- net SD6_Bus renamed SD6
- net SD8_Bus renamed SD8
- net SD9_Bus renamed SD9
- new net: C132.2, C134.2, U41.10 (Cext1)
- new net SD15: J11.12 (SD15), U42.1 (HD15)
- no-connect marks 22 -> 18
Other:
- note added: "Device_Address_BUS"
- note added: "Device_Data_BUS"

Commit message: Add files via upload
Parts:
- added C129: 100nF, symbol PCM_Elektuur:C
- added R292: DNP, symbol Device:R
- added R299, R300: 0, symbol Device:R
- added R373, R374, R375, R376, R377, R378, R380, R381: 4.7k, symbol Device:R
Connections:
- net GND: now also C129.1 (+)
- net IOW#: now also R299.2
- net PNET1: now also R292.1
- net PNET12: now also R292.2, R300.2
- net PNET7: now also R300.1, R373.2, R374.2, R375.2, R376.2, R377.2, R378.2, R380.2, R381.2
- net SD0: now also R375.1
- net SD1: now also R374.1
- net SD2: now also R376.1
- net SD3: now also R373.1
- net SD4: now also R378.1
- net SD5: now also R377.1
- net SD6: now also R381.1
- net at C272.1 (+), F4.1, J11.25 (VCC)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: now also C129.2 (-)
- net at J11.20 (IOW#), R290.2: now also R299.1
- new net SD7: R380.1
Other:
- moved on the sheet: C272

Commit message: Add files via upload
Parts:
- C129, C133, C141, C142, C143, C144, C145, C146, C236, C241, C263, C266, C269, C271, C272, C94: footprint (none) -> Capacitor_SMD:C_0402_1005Metric
- C131, C132, C134: footprint (none) -> Capacitor_SMD:C_0603_1608Metric
- C262: footprint (none) -> Capacitor_SMD:C_0805_2012Metric
- F4: footprint (none) -> Fuse:Fuse_1206_3216Metric
- J11: footprint (none) -> PC110:CF-card
- Q37: footprint (none) -> Package_TO_SOT_SMD:SOT-89-3
- R131, R134, R145, R161, R173, R184: footprint (none) -> PCM_Resistor_SMD_AKL:R_0402_1005Metric
- R290, R295, R296, R298, R299, R301, R360, R361, R362, R365, R366, R367, R368, R369, R371, R373, R374, R375, R376, R377, R378, R380, R381: footprint (none) -> Resistor_SMD:R_0402_1005Metric
- R292, R300: footprint (none) -> Resistor_SMD:R_0805_2012Metric
- U27: footprint (none) -> PC110:Flash-32
- U41: footprint (none) -> PC110:SanDisk
- U42: footprint (none) -> PC110:QFN-100
- U56, U68: footprint (none) -> Package_SO:TSSOP-14_4.4x5mm_P0.65mm
- U65: footprint (none) -> PC110:SOT-353
Connections:
- net CF_CD2_Pluto: now also R161.1; no longer R161.2
- net GND: now also C129.2 (-), C131.2, C132.2, C133.2, C236.2, C271.2, C94.2, R131.1, R145.1; no longer C129.1 (+), C131.1, C132.1, C133.1, C236.1, C271.1, C94.1, R131.2, R145.2
- net IOR#: now also R295.2; no longer R295.1
- net IRQ14: now also R365.1; no longer R365.2
- net PNET1: now also R161.2; no longer R161.1
- net PNET12: now also C133.1, C236.1, C271.1, C94.1, F4.1, R134.2, R360.2, R361.2; no longer C133.2, C236.2, C271.2, C94.2, F4.2, R134.1, R360.1, R361.1
- net PNET7: now also R365.2; no longer R365.1
- net at C134.2, U41.10 (Cext1): now also C132.1; no longer C132.2
- net at C272.1 (+), J11.25 (VCC), J11.26 (VCC): now also C129.1 (+), F4.2; no longer C129.2 (-), F4.1
- net at J11.13 (CE1#), R366.1, U42.37 (CE1): now also R361.1; no longer R361.2
- net at J11.14 (CE2#), R367.1, U42.39 (CE2): now also R360.1; no longer R360.2
- net at U27.7 (ROMWEL#), U42.73 (ROMWEL): now also R131.2, R134.1; no longer R131.1, R134.2
- net at C143.1: now also U41.21 (Cext3); no longer U41.26 (Cext8)
- net at C143.2: now also U41.26 (Cext8); no longer U41.21 (Cext3)
- net at C146.1: now also U41.24 (Cext6); no longer U41.27 (Cext9)
- net at C146.2: now also U41.27 (Cext9); no longer U41.24 (Cext6)
- net at Q37.1 (C), U41.28 (VCC): now also C131.1; no longer C131.2
- net at C145.2, U41.23 (Cext5): now also C141.2; no longer C141.1
- net at J11.18 (IOR#), R301.2: now also R295.1; no longer R295.2
- net at U65.4: now also R368.2; no longer R368.1
- net at Q37.2 (B): now also R368.1; no longer R368.2
- net at J11.28 (CSEL#): now also R145.2; no longer R145.1
- net at U41.20 (Cext2): now also C141.1; no longer C141.2
- net at C144.2, U41.22 (Cext4): now also C142.1; no longer C142.2
- net at U41.25 (Cext7): now also C142.2; no longer C142.1
Other:
- moved on the sheet: C129, C131, C132, C141, C142, C143, C146, C236, C271, C94, F4, R295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

Commit message: Add files via upload
Parts:
- removed Q37: BH, Package_TO_SOT_SMD:SOT-89-3, symbol PCM_Generic:Q-BJT-Darlington,PNP,IEEE
- added Q37: BH, symbol PCM_Transistor_BJT_Darlington_AKL:Q_PNP_Darlington_Generic_BCE
Connections:
- net PNET12: now also Q37.3 (E)
- net at C131.1, U41.28 (VCC): now also Q37.2 (C)
- net at R368.1: now also Q37.1 (B)
Changed lines of the file:
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@@
 	)
 	(junction
-		(at 431.8 69.85)
-		(diameter 0)
-		(color 0 0 0 0)
-	)
-	(junction
 		(at 304.8 245.11)
 		(diameter 0)
@@
 	)
 	(junction
+		(at 431.8 69.85)
+		(diameter 0)
+		(color 0 0 0 0)
+	)
+	(junction
 		(at 438.15 176.53)
 		(diameter 0)
@@
 	)
 	(junction
+		(at 431.8 99.06)
+		(diameter 0)
+		(color 0 0 0 0)
+	)
+	(junction
 		(at 430.53 176.53)
 		(diameter 0)
@@
 	)
 	(junction
-		(at 431.8 99.06)
-		(diameter 0)
-		(color 0 0 0 0)
-	)
-	(junction
 		(at 87.63 274.32)
 		(diameter 0)
@@
 	(wire
 		(pts
+			(xy 431.8 93.98) (xy 431.8 99.06)
+		)
+		(stroke
+			(width 0)
+			(type default)
+		)
+	)
+	(wire
+		(pts
 			(xy 218.44 243.84) (xy 209.55 243.84)
 		)
@@
 	(wire
 		(pts
+			(xy 431.8 69.85) (xy 431.8 78.74)
+		)
+		(stroke
+			(width 0)
+			(type default)
+		)
+	)
+	(wire
+		(pts
 			(xy 331.47 196.85) (xy 407.67 196.85)
 		)
@@
 	(wire
 		(pts
-			(xy 431.8 69.85) (xy 431.8 82.55)
-		)
-		(stroke
-			(width 0)
-			(type default)
-		)
-	)
-	(wire
-		(pts
 			(xy 209.55 243.84) (xy 209.55 231.14)
 		)
@@
 		)
 	)
-	(wire
-		(pts
-			(xy 431.8 92.71) (xy 431.8 99.06)
-		)
-		(stroke
-			(width 0)
-			(type default)
-		)
-	)
 	(bus
 		(pts
@@
 	(wire
 		(pts
-			(xy 449.58 99.06) (xy 431.8 99.06)
+			(xy 431.8 99.06) (xy 449.58 99.06)
 		)
 		(stroke
@@
 	)
 	(symbol
+		(lib_id "PCM_Transistor_BJT_Darlington_AKL:Q_PNP_Darlington_Generic_BCE")
+		(at 429.26 86.36 0)
+		(unit 1)
+		(exclude_from_sim no)
+		(in_bom yes)
+		(on_board yes)
+		(dnp no)
+		(fields_autoplaced yes)
+		(property "Reference" "Q37"
+			(at 435.61 85.0899 0)
+			(effects
+				(font
+					(size 1.27 1.27)
+				)
+				(justify left)
+			)
+		)
+		(property "Value" "BH"
+			(at 435.61 87.6299 0)
+			(effects
+				(font
+					(size 1.27 1.27)
+				)
+				(justify left)
+			)
+		)
+		(property "Footprint" ""
+			(at 434.34 88.9 0)
+			(effects
+				(font
+					(size 1.27 1.27)
+				)
+				(hide yes)
+			)
+		)
+		(property "Datasheet" "~"
+			(at 429.26 85.09 0)
+			(effects
+				(font
+					(size 1.27 1.27)
+				)
+				(hide yes)
+			)
+		)
+		(property "Description" "PNP Darlington transistor, Generic symbol, Alternate KiCAD Library"
+			(at 429.26 86.36 0)
+			(effects
+				(font
+					(size 1.27 1.27)
+				)
+				(hide yes)
+			)
+		)
+		(pin "1"
+		)
+		(pin "3"
+		)
+		(pin "2"
+		)
+		(instances
+			(project ""
+				(path "/45c7911f-b027-440e-9e3e-77a146b41944/00000000-0000-0000-0000-00006e2d8c88"
+					(reference "Q37")
+					(unit 1)
+				)
+			)
+		)
+	)
+	(symbol
 		(lib_id "Device:R")
 		(at 121.92 279.4 90)
@@
 					(unit 1)
 				)
-			)
-		)
-	)
-	(symbol
-		(lib_id "PCM_Generic:Q-BJT-Darlington,PNP,IEEE")
-		(at 426.72 87.63 0)
-		(unit 1)
-		(exclude_from_sim no)
-		(in_bom yes)
-		(on_board yes)
-		(dnp no)
-		(property "Reference" "Q37"
-			(at 435.61 85.0899 0)
-			(effects
-				(font
-					(size 2.54 2.54)
-				)
-				(justify left)
-			)
-		)
-		(property "Value" "BH"
-			(at 435.61 90.1699 0)
-			(effects
-				(font
-					(size 2.54 2.54)
-				)
-				(justify left)
-			)
-		)
-		(property "Footprint" "Package_TO_SOT_SMD:SOT-89-3"
-			(at 426.72 87.63 0)
-			(effects
-				(font
-					(size 2.54 2.54)
-				)
-				(hide yes)
-			)
-		)
-		(property "Datasheet" ""
-			(at 426.72 87.63 0)
-			(effects
-				(font
-					(size 2.54 2.54)
-				)
-				(hide yes)
-			)
-		)
-		(property "Description" "bipolar junction transistor (BJT) Darlington pair: PNP (IEEE with envelope)"
-			(at 426.72 87.63 0)
-			(effects
-				(font
-					(size 1.27 1.27)
-				)
-				(hide yes)
-			)
-		)
-		(property "Sim.Pins" "1=1 2=2 3=3"
-			(at 426.72 87.63 0)
-			(effects
-				(font
-					(size 1.27 1.27)
-				)
-				(hide yes)
-			)
-		)
-		(property "Sim.Device" "SPICE"
-			(at 434.34 85.09 0)
-			(effects
-				(font
-					(size 2.54 2.54)
-				)
-				(justify left)
-				(hide yes)
-			)
-		)
-		(property "Sim.Params" "type=\"X\" model=\"Q-BJT-Darlington,PNP,IEEE\" lib=\"\""
-			(at 426.72 87.63 0)
-			(effects
-				(font
-					(size 1.27 1.27)
-				)
-				(hide yes)
-			)
-		)
-		(pin "2"
-		)
-		(pin "1"
-		)
-		(pin "3"
-		)
-		(instances
-			(project "PC110"
-				(path "/45c7911f-b027-440e-9e3e-77a146b41944/00000000-0000-0000-0000-00006e2d8c88"
-					(reference "Q37")
-					(unit 1)
-				)

Commit message: Add files via upload
Parts:
- Q37: footprint (none) -> Package_TO_SOT_SMD:SOT-89-3
Changed lines of the file:
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@@
 			)
 		)
-		(property "Footprint" ""
+		(property "Footprint" "Package_TO_SOT_SMD:SOT-89-3"
 			(at 434.34 88.9 0)
 			(effects

Commit message: Add files via upload
Parts:
- C129, C272: Indicator + -> (none); Rating V -> (none)
- C269: value 180pF -> 220pF
- J11: value ~ -> CF-card
- Q37: value BH -> BH RT
- R131, R184: now not fitted
- U27: value AT29LV512 -> AT29LV512-12TU
- U41: value SDBL-4 -> SDLB-4

Commit message: Add files via upload
Connections:
- no-connect marks 18 -> 20
Other:
- note added: "Schtokey diode between YellowWire4 (Anode) and YwlloWire5 (Cathode)"
- note added: "YellowWire4"
- note added: "YellowWire5"
Changed lines of the file:
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@@
 		)
 	)
+	(text "YellowWire5"
+		(exclude_from_sim no)
+		(at 471.932 112.268 0)
+		(effects
+			(font
+				(size 1.27 1.27)
+			)
+		)
+	)
 	(text "Device_Data_BUS"
 		(exclude_from_sim no)
@@
 		)
 	)
+	(text "YellowWire4"
+		(exclude_from_sim no)
+		(at 464.566 98.552 0)
+		(effects
+			(font
+				(size 1.27 1.27)
+			)
+		)
+	)
 	(text "Device_Address_BUS"
 		(exclude_from_sim no)
@@
 		)
 	)
+	(text "Schtokey diode between YellowWire4 (Anode) and YwlloWire5 (Cathode)"
+		(exclude_from_sim no)
+		(at 498.348 105.156 0)
+		(effects
+			(font
+				(size 1.27 1.27)
+			)
+		)
+	)
 	(junction
 		(at 114.3 358.14)
@@
 	)
 	(junction
+		(at 449.58 99.06)
+		(diameter 0)
+		(color 0 0 0 0)
+	)
+	(junction
 		(at 431.8 99.06)
 		(diameter 0)
@@
 	)
 	(junction
+		(at 461.01 120.65)
+		(diameter 0)
+		(color 0 0 0 0)
+	)
+	(junction
 		(at 158.75 139.7)
 		(diameter 0)
@@
 	)
 	(no_connect
+		(at 471.17 99.06)
+	)
+	(no_connect
+		(at 478.79 113.03)
+	)
+	(no_connect
 		(at 334.01 127)
 	)
@@
 	(wire
 		(pts
+			(xy 461.01 113.03) (xy 478.79 113.03)
+		)
+		(stroke
+			(width 0)
+			(type default)
+		)
+	)
+	(wire
+		(pts
 			(xy 125.73 279.4) (xy 135.89 279.4)
 		)
@@
 		)
 	)
+	(wire
+		(pts
+			(xy 449.58 99.06) (xy 471.17 99.06)
+		)
+		(stroke
+			(width 0)
+			(type default)
+		)
+	)
 	(bus
 		(pts
@@
 		)
 		(stroke
+			(width 0)
+			(type default)
+		)
+	)
+	(wire
+		(pts
+			(xy 461.01 120.65) (xy 461.01 113.03)
+		)
+		(stroke
