File: PCB/Mainboard/Processor.kicad_sch (KiCad schematic)
At the start: 16 parts, among them U16 Intel_P24T

Commit message: Add files via upload
Parts:
- removed JP10: SMI Enable, My_Components:Conn_Pin_Header_2x1_2.54mm, symbol Jumper:Jumper_2_Open
- removed JP11: Reset Select, My_Components:Conn_Pin_Header_3x1_2.54mm, symbol Jumper:Jumper_3_Open
- removed JP12: CPU Select 1, My_Components:Conn_Pin_Header_3x1_2.54mm, symbol Jumper:Jumper_3_Open
- removed JP13: FERR Select, My_Components:Conn_Pin_Header_3x1_2.54mm, symbol Jumper:Jumper_3_Open
- removed JP19: CPU Select 2, My_Components:Conn_Pin_Header_3x1_2.54mm, symbol Jumper:Jumper_3_Open
- removed JP20: STPCLK, My_Components:Conn_Pin_Header_2x1_2.54mm, symbol Jumper:Jumper_2_Open
- removed JP21, JP30: CPU Select 3, My_Components:Conn_Pin_Header_3x1_2.54mm, symbol Jumper:Jumper_3_Open
- removed JP23: NMI/IGNNE#, My_Components:Conn_Pin_Header_4x1_2.54mm, symbol Connector_Generic:Conn_01x04
- removed JP32: CPU Select 4, My_Components:Conn_Pin_Header_3x1_2.54mm, symbol Jumper:Jumper_3_Open
- removed JP9: Intel/Cyrix, My_Components:Conn_Pin_Header_2x1_2.54mm, symbol Jumper:Jumper_2_Open
- removed R35: 100, Resistor_SMD:R_0612_1632Metric_Pad1.18x3.40mm_HandSolder, symbol Device:R
- removed R42, R68: 10k, Resistor_SMD:R_0612_1632Metric_Pad1.18x3.40mm_HandSolder, symbol Device:R
- removed R47: 1k, Resistor_SMD:R_0612_1632Metric_Pad1.18x3.40mm_HandSolder, symbol Device:R
- U16: value Intel_P24T -> Intel_486sx
Connections:
- net A20M#: no longer names the net of U16.E16 (A20M#)
- net ADS#: no longer names the net of U16.T18 (ADS#)
- net AHOLD: no longer names the net of U16.B18 (AHOLD)
- net BE0#: no longer names the net of U16.L16 (BE0#)
- net BE1#: no longer names the net of U16.K17 (BE1#)
- net BE2#: no longer names the net of U16.K16 (BE2#)
- net BE3#: no longer names the net of U16.G18 (BE3#)
- net BLAST#: no longer names the net of U16.S17 (BLAST#)
- net BRDY#: no longer names the net of U16.J16 (BRDY#)
- net BS16#: no longer names the net of U16.D18 (BS16#)
- net BS8#_PU: no longer names the net of U16.E17 (BS8#)
- net BS8#_PU: no longer U16.E18 (BOFF#)
- net CA10: no longer names the net of U16.T14 (A10)
- net CA11: no longer names the net of U16.S13 (A11)
- net CA12: no longer names the net of U16.T8 (A12)
- net CA13: no longer names the net of U16.R11 (A13)
- net CA14: no longer names the net of U16.T6 (A14)
- net CA15: no longer names the net of U16.S8 (A15)
- net CA16: no longer names the net of U16.R10 (A16)
- net CA17: no longer names the net of U16.R4 (A17)
- net CA18: no longer names the net of U16.S6 (A18)
- net CA19: no longer names the net of U16.R5 (A19)
- net CA2: no longer names the net of U16.R15 (A2)
- net CA20: no longer names the net of U16.R9 (A20)
- net CA21: no longer names the net of U16.R6 (A21)
- net CA22: no longer names the net of U16.R8 (A22)
- net CA23: no longer names the net of U16.T4 (A23)
- net CA24: no longer names the net of U16.R7 (A24)
- net CA25: no longer names the net of U16.S3 (A25)
- net CA26: no longer names the net of U16.T3 (A26)
- net CA27: no longer names the net of U16.T2 (A27)
- net CA28: no longer names the net of U16.S2 (A28)
- net CA29: no longer names the net of U16.Q3 (A29)
- net CA3: no longer names the net of U16.S16 (A3)
- net CA30: no longer names the net of U16.Q4 (A30)
- net CA31: no longer names the net of U16.R2 (A31)
- net CA4: no longer names the net of U16.T17 (A4)
- net CA5: no longer names the net of U16.R13 (A5)
- net CA6: no longer names the net of U16.T16 (A6)
- net CA7: no longer names the net of U16.R14 (A7)
- net CA8: no longer names the net of U16.S14 (A8)
- net CA9: no longer names the net of U16.R12 (A9)
- net CD0: no longer names the net of U16.Q2 (D0)
- net CD1: no longer names the net of U16.P3 (D1)
- net CD10: no longer names the net of U16.F4 (GND)
- net CD11: no longer names the net of U16.D2 (D11)
- net CD12: no longer names the net of U16.H4 (GND)
- net CD13: no longer names the net of U16.E3 (VCC)
- net CD14: no longer names the net of U16.L4 (GND)
- net CD15: no longer names the net of U16.G4 (GND)
- net CD16: no longer names the net of U16.K4 (GND)
- net CD17: no longer names the net of U16.E4 (VCC)
- net CD18: no longer names the net of U16.D3 (VCC)
- net CD19: no longer names the net of U16.C2 (D19)
- net CD2: no longer names the net of U16.P2 (D2)
- net CD20: no longer names the net of U16.B2 (D20)
- net CD21: no longer names the net of U16.C3 (D21)
- net CD22: no longer names the net of U16.B3 (D22)
- net CD23: no longer names the net of U16.B5 (D23)
- net CD24: no longer names the net of U16.B7 (D24)
- net CD25: no longer names the net of U16.C7 (D25)
- net CD26: no longer names the net of U16.D8 (VCC)
- net CD27: no longer names the net of U16.D7 (VCC)
- net CD28: no longer names the net of U16.D9 (VCC)
- net CD29: no longer names the net of U16.B9 (D29)
- net CD3: no longer names the net of U16.J3 (VCC)
- net CD30: no longer names the net of U16.D10 (VCC)
- net CD31: no longer names the net of U16.C9 (D31)
- net CD4: no longer names the net of U16.N4 (VCC)
- net CD5: no longer names the net of U16.K3 (VCC)
- net CD6: no longer names the net of U16.M3 (VCC)
- net CD7: no longer names the net of U16.M4 (VCC)
- net CD8: no longer names the net of U16.G3 (VCC)
- net CD9: no longer names the net of U16.E2 (D9)
- net CPUCLK: no longer names the net of U16.D4 (VCC)
- net CPURST: no longer names the net of U16.F19 (INIT)
- net DP0_PU: no longer names the net of U16.P4 (DP0)
- net DP1_PU: no longer names the net of U16.G2 (DP1)
- net DP2_PU: no longer names the net of U16.J4 (GND)
- net DP3_PU: no longer names the net of U16.B6 (DP3)
- net D_C#: no longer names the net of U16.N16 (D/C#)
- net EADS#: no longer names the net of U16.C18 (EADS#)
- net FLUSH#: no longer names the net of U16.D16 (FLUSH#)
- removed net GND: U16.A12 (GND), U16.A13 (GND), U16.A14 (GND), U16.A15 (GND), U16.A17 (GND), U16.A5 (GND), U16.A7 (BLEN#), U16.A8 (GND), U16.B10 (GND), U16.B12 (GND), U16.B8 (GND), U16.C19 (GND), U16.C4 (GND), U16.C5 (GND), U16.C6 (GND), U16.E1 (GND), U16.E19 (GND), U16.F18 (GND), U16.F2 (GND), U16.G19 (GND), U16.H1 (GND), U16.H18 (GND), U16.H19 (GND), U16.H2 (GND), U16.J18 (GND), U16.J2 (GND), U16.L18 (GND), U16.L2 (GND), U16.M1 (GND), U16.M18 (GND), U16.M19 (GND), U16.M2 (GND), U16.N18 (GND), U16.N19 (GND), U16.N2 (GND), U16.P1 (EWBE#), U16.Q1 (GND), U16.Q18 (GND), U16.Q19 (GND), U16.R3 (GND), U16.S1 (GND), U16.S19 (GND), U16.S5 (GND), U16.T10 (GND), U16.T11 (GND), U16.T12 (GND), U16.T13 (GND), U16.T15 (GND), U16.T7 (GND), U16.T9 (GND), U16.U12 (GND), U16.U13 (GND), U16.U14 (GND), U16.U15 (GND), U16.U17 (GND), U16.U3 (GND), U16.U5 (GND), U16.U6 (GND), U16.U7 (GND), U16.U8 (GND)
- net HITM#: no longer names the net of U16.U1 (HITM#)
- net HLDA: no longer names the net of U16.Q16 (HLDA)
- net HOLD: no longer names the net of U16.F16 (HOLD)
- net IBM_SMI#: no longer names the net of U16.B13 (INC/HITM#)
- net INTR: no longer names the net of U16.B17 (INTR)
- net KEN#: no longer names the net of U16.G16 (KEN#)
- net M_IO#: no longer names the net of U16.P17 (M/IO#)
- net PIN_B14: no longer names the net of U16.B14 (FERR#)
- net PIN_B16: no longer names the net of U16.B16 (IGNNE#)
- net PIN_C14: no longer names the net of U16.C14 (INC/WB/WT#)
- net PIN_C16: no longer names the net of U16.C16 (NMI)
- net PIN_D11: no longer names the net of U16.D11 (INC/INIT/SRESET)
- net PIN_D13: no longer names the net of U16.D13 (SMIACT#)
- net PIN_D15: no longer names the net of U16.D15 (INC/FERR#)
- net PIN_D17: no longer names the net of U16.D17 (RESET)
- net PIN_H16: no longer names the net of U16.H16 (STPCLK#)
- net PIN_R16: no longer names the net of U16.R16 (BREQ)
- net PIN_S18: no longer names the net of U16.S18 (CLKMUL)
- net PIN_T5: no longer names the net of U16.T5 (VOLDET)
- net RDY#: no longer names the net of U16.G17 (RDY#)
- net SMI#: no longer names the net of U16.C11 (SMI#)
- removed net VCC: U16.A10 (VCC), U16.A11 (VCC), U16.A16 (VCC), U16.A9 (VCC), U16.D1 (VCC), U16.D19 (VCC), U16.J1 (VCC), U16.J19 (VCC), U16.K1 (VCC), U16.K19 (VCC), U16.L1 (VCC), U16.L19 (VCC), U16.N1 (INV), U16.R1 (VCC), U16.R19 (VCC), U16.U10 (VCC), U16.U11 (VCC), U16.U16 (VCC), U16.U4 (VCC), U16.U9 (VCC)
- removed net VCPU: U16.C10 (VCC), U16.C12 (VCC), U16.C8 (VCC), U16.D5 (VCC), U16.D6 (VCC), U16.F17 (VCC), U16.F3 (VCC), U16.H17 (VCC), U16.H3 (VCC), U16.J17 (VCC), U16.L17 (VCC), U16.L3 (VCC), U16.M17 (VCC), U16.N17 (VCC), U16.N3 (VCC), U16.Q17 (VCC), U16.S10 (VCC), U16.S11 (VCC), U16.S12 (VCC), U16.S15 (VCC), U16.S4 (VCC), U16.S7 (VCC), U16.S9 (VCC)
- net WB_WT#: no longer names the net of U16.T1 (WB/WT#)
- net W_R#: no longer names the net of U16.P18 (W/R#)
- no-connect marks 14 -> 9
Other:
- note removed: "JP9 - Pin T5 - VOLDET connection Intel/AMD: Open; Cyrix/IBM: Closed JP10 - Pin C11 - SMI# connection Non-SL CPU: Open; SL-enabled CPU: Closed JP11 - Pin D17 - Reset connection CPURST: 1-2; RSTDRV: 2-3 JP12 - Pin D11/C13 - CPURST connection Pin D11: 1-2; Pin C14: 2-3 JP13 - Pin D15/B14 - FERR# connection 486DX/ODPR/5x86: 1-2; 487DX/ODP/P24T: 2-3; 486SX: Open or 2-3? JP19 - Pin C14 - CPU select 1-2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"
- note removed: "Pin C15 is connected to JP22 (not populated) JP22 is connected to 10k pull-up (to VCC)"
- note removed: "Pins A3, C3 are connected to GND Pins A4, D1 are connected to VCC/5V"

Commit message: Add files via upload
Parts:
- removed U16: Intel_486sx, My_Components:IC_PGA_SOCKET3, symbol my_components:Intel_P24T
- added U76: 80486SX, symbol PC110:80486SX
Connections:
- new net GND: U76.F10 (GND), U76.F11 (GND), U76.F12 (GND), U76.F13 (GND), U76.F4 (GND), U76.F5 (GND), U76.F6 (GND), U76.F7 (GND), U76.F8 (GND), U76.F9 (GND), U76.G10 (GND), U76.G11 (GND), U76.G12 (GND), U76.G13 (GND), U76.G4 (GND), U76.G5 (GND), U76.G6 (GND), U76.G7 (GND), U76.G8 (GND), U76.G9 (GND), U76.H10 (GND), U76.H11 (GND), U76.H12 (GND), U76.H13 (GND), U76.H4 (GND), U76.H6 (GND), U76.H7 (GND), U76.H8 (GND), U76.H9 (GND), U76.J10 (GND), U76.J11 (GND), U76.J12 (GND), U76.J13 (GND), U76.J4 (GND), U76.J5 (GND), U76.J6 (GND), U76.J7 (GND), U76.J8 (GND), U76.J9 (GND), U76.K10 (GND), U76.K11 (GND), U76.K12 (GND), U76.K13 (GND), U76.K4 (GND), U76.K5 (GND), U76.K6 (GND), U76.K7 (GND), U76.K8 (GND), U76.K9 (GND), U76.L10 (GND), U76.L11 (GND), U76.L12 (GND), U76.L13 (GND), U76.L4 (GND), U76.L5 (GND), U76.L6 (GND), U76.L7 (GND), U76.L8 (GND), U76.L9 (GND)
- new net PNET1: U76.D10 (VCC), U76.D11 (VCC), U76.D12 (VCC), U76.D13 (VCC), U76.D14 (VCC), U76.D2 (VCC), U76.D4 (VCC), U76.D5 (VCC), U76.D6 (VCC), U76.D7 (VCC), U76.D8 (VCC), U76.D9 (VCC), U76.E10 (VCC), U76.E11 (VCC), U76.E12 (VCC), U76.E13 (VCC), U76.E14 (VCC), U76.E3 (VCC), U76.E4 (VCC), U76.E5 (VCC), U76.E6 (VCC), U76.E7 (VCC), U76.E8 (VCC), U76.E9 (VCC), U76.F14 (VCC), U76.F3 (VCC), U76.G14 (VCC), U76.G3 (VCC), U76.H14 (VCC), U76.H3 (VCC), U76.J14 (VCC), U76.J3 (VCC), U76.K14 (VCC), U76.K3 (VCC), U76.L14 (VCC), U76.L3 (VCC), U76.M10 (VCC), U76.M11 (VCC), U76.M12 (VCC), U76.M13 (VCC), U76.M14 (VCC), U76.M3 (VCC), U76.M4 (VCC), U76.M5 (VCC), U76.M6 (VCC), U76.M7 (VCC), U76.M8 (VCC), U76.M9 (VCC), U76.N10 (VCC), U76.N11 (VCC), U76.N12 (VCC), U76.N13 (VCC), U76.N14 (VCC), U76.N3 (VCC), U76.N4 (VCC), U76.N5 (VCC), U76.N6 (VCC), U76.N7 (VCC), U76.N8 (VCC), U76.N9 (VCC)
- no-connect marks 9 -> 30

Commit message: Add files via upload
Parts:
- added R252: 33, symbol Device:R
- added R253: DNP, symbol Device:R
- added R395: 10k, symbol Device:R
- added RA3: 22k, symbol Device:R_Pack04
- added RA4: 10k, symbol Device:R_Pack04
Connections:
- net GND: now also R395.1, RA3.5 (R4.2), RA3.6 (R3.2), RA3.7 (R2.2), RA3.8 (R1.2), RA4.5 (R4.2), RA4.6 (R3.2), RA4.7 (R2.2), RA4.8 (R1.2)
- net CPU_A2: now reaches U76.A3 (A2)
- net at U76.A9 (CLK_CPU): now also R252.1, R253.1
- net CPU_RESET: now reaches U76.C13 (RSTCPU)
- net CPU_A4: now reaches U76.D1 (A4)
- net SRESET: now reaches U76.E15 (SRESET)
- net CPU_SMIACT#: now reaches U76.E16 (SMIACT#)
- net CPU_A5: now reaches U76.E2 (A5)
- net CPU_A7: now reaches U76.F1 (A7)
- net CPU_SMI#: now reaches U76.F15 (SMI#)
- net CPU_A6: now reaches U76.F2 (A6)
- net CPU_A9: now reaches U76.G1 (A9)
- net CPU_STPCLK#: now reaches U76.G15 (STPCLK#)
- net CPU_D31: now reaches U76.G16 (D31)
- net CPU_A8: now reaches U76.G2 (A8)
- net CPU_A11: now reaches U76.H1 (A11)
- net CPU_D30: now reaches U76.H15 (D30)
- net CPU_D29: now reaches U76.H16 (D29)
- net CPU_A10: now reaches U76.H2 (A10)
- net CPU_A12: now reaches U76.J1 (A12)
- net CPU_D28: now reaches U76.J15 (D28)
- net CPU_D27: now reaches U76.J16 (D27)
- net CPU_A14: now reaches U76.K1 (A14)
- net CPU_D26: now reaches U76.K15 (D26)
- net CPU_D25: now reaches U76.K16 (D25)
- net CPU_A13: now reaches U76.K2 (A13)
- net CPU_A16: now reaches U76.L1 (A16)
- net CPU_D24: now reaches U76.L15 (D24)
- net at U76.L16 (DP3): now also RA3.1 (R1.1)
- net CPU_A15: now reaches U76.L2 (A15)
- net CPU_D23: now reaches U76.M15 (D23)
- net CPU_D22: now reaches U76.M16 (D22)
- net CPU_A17: now reaches U76.M2 (A17)
- net CPU_A18: now reaches U76.N1 (A18)
- net CPU_D21: now reaches U76.N15 (D21)
- net CPU_D20: now reaches U76.N16 (D20)
- net CPU_A20: now reaches U76.P1 (A20)
- net CPU_D9: now reaches U76.P10 (D9)
- net CPU_D11: now reaches U76.P11 (D11)
- net CPU_D14: now reaches U76.P12 (D14)
- net CPU_D16: now reaches U76.P13 (D16)
- net CPU_D19: now reaches U76.P15 (D19)
- net CPU_D18: now reaches U76.P16 (D18)
- net CPU_A19: now reaches U76.P2 (A19)
- net CPU_A23: now reaches U76.P3 (A23)
- net at U76.P4 (A26): now also RA4.1 (R1.1)
- net at U76.P5 (A29): now also RA4.4 (R4.1)
- net CPU_D1: now reaches U76.P7 (D1)
- net CPU_D4: now reaches U76.P8 (D4)
- net CPU_D8: now reaches U76.R10 (D8)
- net CPU_D10: now reaches U76.R11 (D10)
- net CPU_D13: now reaches U76.R12 (D13)
- net at U76.R13 (DP2): now also RA3.2 (R2.1)
- net CPU_D17: now reaches U76.R16 (D17)
- net CPU_A22: now reaches U76.R3 (A22)
- net CPU_A25: now reaches U76.R4 (A25)
- net at U76.R5 (A28): now also RA4.3 (R3.1)
- net CPU_A31: now reaches U76.R6 (A31)
- net CPU_D0: now reaches U76.R7 (D0)
- net CPU_D3: now reaches U76.R8 (D3)
- net CPU_D6: now reaches U76.R9 (D6)
- net at U76.T10 (DP1): now also RA3.3 (R3.1)
- net CPU_D12: now reaches U76.T12 (D12)
- net CPU_D15: now reaches U76.T13 (D15)
- net CPU_A21: now reaches U76.T3 (A21)
- net CPU_A24: now reaches U76.T4 (A24)
- net at U76.T5 (A27): now also RA4.2 (R2.1)
- net at U76.T6 (A30): now also R395.2
- net at U76.T7 (DP0): now also RA3.4 (R4.1)
- net CPU_D2: now reaches U76.T8 (D2)
- net CPU_D5: now reaches U76.T9 (D5)
- new net CPU_A3: U76.D2 (VCC)
- new net CPU_D7: U76.D9 (VCC)
- new net Chipset_CPU_CLK: R252.2
- new net Chipset_CPU_CLK_Sense: R253.2
- no-connect marks 30 -> 35
Other:
- moved on the sheet: U76

Commit message: Add files via upload
Parts:
- added J12: ~, symbol PC110:CPU_Debug6
- added J9: ~, symbol PC110:CPU_Debug10
Connections:
- net CPU_A31: now also J12.6
- net CPU_BE2#: now reaches U76.A11 (BE2#)
- net CPU_BE2#: now also J9.8
- net CPU_DC#: now reaches U76.A12 (DC#)
- net CPU_EADS#: now reaches U76.A13 (EADS#)
- net CPU_EADS#: now also J12.4
- net CPU_BS16#: now reaches U76.A6 (BS16#)
- net CPU_AHOLD: now reaches U76.A8 (AHOLD)
- net CPU_AHOLD: now also J12.5
- net CPU_BE0#: now reaches U76.B10 (BE0#)
- net CPU_BE0#: now also J9.6
- net CPU_BE3#: now reaches U76.B11 (BE3#)
- net CPU_BE3#: now also J9.5
- net CPU_A20M#: now reaches U76.B13 (A20M#)
- net CPU_A20M#: now also J9.7
- net CPU_ADS#: now reaches U76.B3 (ADS#)
- net CPU_BRDY#: now reaches U76.B5 (BRDY#)
- net CPU_BRDY#: now also J9.2
- net CPU_KEN#: now reaches U76.B7 (KEN#)
- net CPU_KEN#: now also J12.3
- net CPU_HLDA: now reaches U76.B9 (HLDA)
- net CPU_HLDA: now also J9.4
- net CPU_BE1#: now reaches U76.C10 (BE1#)
- net CPU_BE1#: now also J9.3
- net CPU_MIO#: now reaches U76.C11 (MIO#)
- net CPU_FLUSH#: now reaches U76.C16 (FLUSH#)
- net CPU_FLUSH#: now also J12.2
- net CPU_BLAST#: now reaches U76.C3 (BLAST#)
- net CPU_BLAST#: now also J12.1
- net CPU_HOLD: now reaches U76.C7 (HOLD)
- net CPU_HOLD: now also J9.1
- net CPU_WR#: now reaches U76.C9 (WR#)
- net CPU_INTR: now reaches U76.D15 (INTR)
- net CPU_NMI: now reaches U76.D16 (NMI)
- net CPU_NMI: now also J9.10
- new net CPU_SRESET#: J9.9
- no-connect marks 35 -> 43
Other:
- moved on the sheet: R252, R253, R395, RA3, RA4, U76

Commit message: Add files via upload
Other:
- moved on the sheet: R252, R253
Changed lines of the file:
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@@
 	(wire
 		(pts
-			(xy 326.39 203.2) (xy 360.68 203.2)
+			(xy 330.2 207.01) (xy 360.68 207.01)
 		)
 		(stroke
@@
 	(wire
 		(pts
-			(xy 318.77 195.58) (xy 314.96 195.58)
+			(xy 322.58 199.39) (xy 314.96 199.39)
 		)
 		(stroke
@@
 	(wire
 		(pts
-			(xy 326.39 195.58) (xy 360.68 195.58)
+			(xy 330.2 199.39) (xy 360.68 199.39)
 		)
 		(stroke
@@
 	(wire
 		(pts
-			(xy 314.96 203.2) (xy 318.77 203.2)
+			(xy 314.96 207.01) (xy 322.58 207.01)
 		)
 		(stroke
@@
 	(wire
 		(pts
-			(xy 314.96 195.58) (xy 314.96 203.2)
+			(xy 314.96 199.39) (xy 314.96 203.2)
 		)
 		(stroke
@@
 	(wire
 		(pts
+			(xy 314.96 207.01) (xy 314.96 203.2)
+		)
+		(stroke
+			(width 0)
+			(type default)
+		)
+	)
+	(wire
+		(pts
 			(xy 207.01 36.83) (xy 207.01 50.8)
 		)
@@
 	)
 	(label "Chipset_CPU_CLK_Sense"
-		(at 336.55 195.58 0)
+		(at 336.55 199.39 0)
 		(effects
 			(font
@@
 	)
 	(label "Chipset_CPU_CLK"
-		(at 342.9 203.2 0)
+		(at 342.9 207.01 0)
 		(effects
 			(font
@@
 	(symbol
 		(lib_id "Device:R")
-		(at 322.58 195.58 90)
+		(at 326.39 199.39 90)
 		(unit 1)
 		(exclude_from_sim no)
@@
 		(dnp no)
 		(property "Reference" "R253"
-			(at 324.612 191.77 90)
+			(at 328.422 195.58 90)
 			(effects
 				(font
@@
 		)
 		(property "Value" "DNP"
-			(at 324.104 193.548 90)
+			(at 327.914 197.358 90)
 			(effects
 				(font
@@
 		)
 		(property "Footprint" ""
-			(at 322.58 197.358 90)
+			(at 326.39 201.168 90)
 			(effects
 				(font
@@
 		)
 		(property "Datasheet" "~"
-			(at 322.58 195.58 0)
+			(at 326.39 199.39 0)
 			(effects
 				(font
@@
 		)
 		(property "Description" "Resistor"
-			(at 322.58 195.58 0)
+			(at 326.39 199.39 0)
 			(effects
 				(font
@@
 	(symbol
 		(lib_id "Device:R")
-		(at 322.58 203.2 90)
+		(at 326.39 207.01 90)
 		(unit 1)
 		(exclude_from_sim no)
@@
 		(dnp no)
 		(property "Reference" "R252"
-			(at 324.612 199.39 90)
+			(at 328.422 203.2 90)
 			(effects
 				(font
@@
 		)
 		(property "Value" "33"
-			(at 324.104 201.168 90)
+			(at 327.914 204.978 90)
 			(effects
 				(font
@@
 		)
 		(property "Footprint" ""
-			(at 322.58 204.978 90)
+			(at 326.39 208.788 90)
 			(effects
 				(font
@@
 		)
 		(property "Datasheet" "~"
-			(at 322.58 203.2 0)
+			(at 326.39 207.01 0)
 			(effects
 				(font
@@
 		)
 		(property "Description" "Resistor"
-			(at 322.58 203.2 0)
+			(at 326.39 207.01 0)
 			(effects
 				(font

Commit message: Add files via upload
Changed lines of the file:
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@@
 	)
 	(junction
+		(at 62.23 198.12)
+		(diameter 0)
+		(color 0 0 0 0)
+	)
+	(junction
 		(at 199.39 36.83)
 		(diameter 0)
@@
 	)
 	(bus_entry
+		(at 62.23 224.79)
+		(size 2.54 -2.54)
+		(stroke
+			(width 0)
+			(type default)
+		)
+	)
+	(bus_entry
 		(at 62.23 158.75)
 		(size 2.54 2.54)
@@
 		)
 	)
+	(bus
+		(pts
+			(xy 35.56 198.12) (xy 62.23 198.12)
+		)
+		(stroke
+			(width 0)
+			(type default)
+		)
+	)
 	(wire
 		(pts
@@
 	(wire
 		(pts
-			(xy 66.04 222.25) (xy 82.55 222.25)
+			(xy 64.77 222.25) (xy 82.55 222.25)
 		)
 		(stroke
@@
 		)
 	)
+	(bus
+		(pts
+			(xy 62.23 232.41) (xy 35.56 232.41)
+		)
+		(stroke
+			(width 0)
+			(type default)
+		)
+	)
 	(wire
 		(pts
@@
 	(bus
 		(pts
-			(xy 62.23 199.39) (xy 62.23 196.85)
+			(xy 62.23 199.39) (xy 62.23 198.12)
 		)
 		(stroke
@@
 		)
 	)
+	(bus
+		(pts
+			(xy 62.23 198.12) (xy 62.23 196.85)
+		)
+		(stroke
+			(width 0)
+			(type default)
+		)
+	)
 	(wire
 		(pts
@@
 		)
 	)
+	(bus
+		(pts
+			(xy 62.23 224.79) (xy 62.23 232.41)
+		)
+		(stroke
+			(width 0)
+			(type default)
+		)
+	)
 	(wire
 		(pts
@@
 		)
 		(stroke
+			(width 0)
+			(type default)
+		)
+	)
+	(bus
+		(pts
+			(xy 35.56 232.41) (xy 35.56 198.12)
+		)
+		(stroke

Commit message: Add files via upload
Connections:
- net SRESET is gone; now on net CPU_SRESET: U76.E15 (SRESET)
- net CPU_RDY#: now reaches U76.A7 (RDY#)
- net CPU_SRESET# renamed CPU_SRESET
Changed lines of the file:
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@@
 	(wire
 		(pts
+			(xy 289.56 142.24) (xy 309.88 142.24)
+		)
+		(stroke
+			(width 0)
+			(type default)
+		)
+	)
+	(wire
+		(pts
 			(xy 240.03 36.83) (xy 240.03 50.8)
 		)
@@
 		)
 	)
+	(label "CPU_SRESET"
+		(at 379.73 125.73 0)
+		(effects
+			(font
+				(size 1.27 1.27)
+			)
+			(justify left bottom)
+		)
+	)
 	(label "CPU_BE2#"
 		(at 299.72 88.9 0)
@@
 		)
 	)
-	(label "SRESET"
-		(at 300.99 208.28 0)
+	(label "CPU_SRESET"
+		(at 297.18 208.28 0)
 		(effects
 			(font
@@
 		)
 	)
+	(label "CPU_RDY#"
+		(at 299.72 142.24 0)
+		(effects
+			(font
+				(size 1.27 1.27)
+			)
+			(justify left bottom)
+		)
+	)
 	(label "CPU_D19"
 		(at 67.31 113.03 0)
@@
 		)
 	)
-	(label "CPU_SRESET#"
-		(at 378.46 125.73 0)
-		(effects
-			(font
-				(size 1.27 1.27)
-			)
-			(justify left bottom)
-		)
-	)
 	(label "CPU_BLAST#"
 		(at 340.36 142.24 0)
@@
 		(on_board yes)
 		(dnp no)
-		(fields_autoplaced yes)
 		(property "Reference" "J9"
-			(at 365.76 106.68 0)
+			(at 365.76 108.966 0)
 			(effects
 				(font

Commit message: Add files via upload
Other:
- company: (none) -> Recreated by: Ahmad Byagowi
Changed lines of the file:
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@@
 	(title_block
 		(title "PC110")
+		(company "Recreated by: Ahmad Byagowi")
 	)
 	(junction
