File: PCB/Mainboard/Processor.kicad_sch (KiCad schematic)
At the start: 8 parts, among them U76 80486SX

Commit message: Add files via upload
Connections:
- net CPU_D7: now also U76.P9 (D7); no longer U76.D9 (VCC)
- net GND: now also U76.H5 (GND)
- net PNET1: now also U76.D3 (VCC); no longer U76.D2 (VCC)
- no-connect marks 43 -> 13
Other:
- note added: "CPU_ADDRESS_BUS"
- note added: "CPU_DATA_BUS"
Changed lines of the file:
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@@
 		(company "Recreated by: Ahmad Byagowi")
 	)
+	(text "CPU_ADDRESS_BUS"
+		(exclude_from_sim no)
+		(at 52.578 144.018 0)
+		(effects
+			(font
+				(size 1.27 1.27)
+			)
+		)
+	)
+	(text "CPU_DATA_BUS"
+		(exclude_from_sim no)
+		(at 52.832 59.944 0)
+		(effects
+			(font
+				(size 1.27 1.27)
+			)
+		)
+	)
 	(junction
 		(at 158.75 36.83)
@@
 	)
 	(no_connect
-		(at 247.65 50.8)
-	)
-	(no_connect
-		(at 252.73 236.22)
-	)
-	(no_connect
-		(at 262.89 50.8)
-	)
-	(no_connect
-		(at 280.67 50.8)
-	)
-	(no_connect
-		(at 252.73 50.8)
-	)
-	(no_connect
 		(at 289.56 67.31)
 	)
 	(no_connect
-		(at 257.81 236.22)
-	)
-	(no_connect
 		(at 289.56 214.63)
 	)
 	(no_connect
-		(at 267.97 50.8)
-	)
-	(no_connect
 		(at 292.1 134.62)
 	)
@@
 	)
 	(no_connect
-		(at 275.59 50.8)
-	)
-	(no_connect
 		(at 292.1 116.84)
 	)
 	(no_connect
-		(at 250.19 50.8)
-	)
-	(no_connect
 		(at 292.1 119.38)
 	)
 	(no_connect
-		(at 242.57 236.22)
-	)
-	(no_connect
-		(at 265.43 236.22)
-	)
-	(no_connect
 		(at 289.56 219.71)
 	)
@@
 	)
 	(no_connect
-		(at 273.05 50.8)
-	)
-	(no_connect
-		(at 278.13 50.8)
-	)
-	(no_connect
-		(at 245.11 236.22)
-	)
-	(no_connect
-		(at 250.19 236.22)
-	)
-	(no_connect
-		(at 273.05 236.22)
-	)
-	(no_connect
-		(at 262.89 236.22)
-	)
-	(no_connect
-		(at 260.35 50.8)
-	)
-	(no_connect
-		(at 245.11 50.8)
-	)
-	(no_connect
 		(at 292.1 173.99)
 	)
 	(no_connect
-		(at 267.97 236.22)
-	)
-	(no_connect
 		(at 292.1 185.42)
 	)
@@
 	)
 	(no_connect
-		(at 278.13 236.22)
-	)
-	(no_connect
-		(at 255.27 236.22)
-	)
-	(no_connect
-		(at 270.51 50.8)
-	)
-	(no_connect
-		(at 257.81 50.8)
-	)
-	(no_connect
-		(at 275.59 236.22)
-	)
-	(no_connect
-		(at 270.51 236.22)
-	)
-	(no_connect
-		(at 265.43 50.8)
-	)
-	(no_connect
-		(at 255.27 50.8)
-	)
-	(no_connect
-		(at 260.35 236.22)
-	)
-	(no_connect
 		(at 289.56 217.17)
 	)
@@
 		(at 292.1 171.45)
 	)
-	(no_connect
-		(at 247.65 236.22)
-	)
 	(bus_entry
 		(at 62.23 97.79)
@@
 	)
 	(bus_entry
+		(at 339.09 156.21)
+		(size 2.54 2.54)
+		(stroke
+			(width 0)
+			(type default)
+		)
+	)
+	(bus_entry
 		(at 62.23 163.83)
 		(size 2.54 2.54)
@@
 	(wire
 		(pts
-			(xy 354.33 154.94) (xy 359.41 154.94)
+			(xy 341.63 158.75) (xy 354.33 158.75)
 		)
 		(stroke
@@
 	(wire
 		(pts
+			(xy 354.33 154.94) (xy 359.41 154.94)
+		)
+		(stroke
+			(width 0)
+			(type default)
+		)
+	)
+	(wire
+		(pts
 			(xy 102.87 36.83) (xy 105.41 36.83)
 		)
@@
 		)
 	)
+	(bus
+		(pts
+			(xy 339.09 156.21) (xy 339.09 165.1)
+		)
+		(stroke
+			(width 0)
+			(type default)
+		)
+	)
+	(wire
+		(pts
+			(xy 354.33 158.75) (xy 354.33 154.94)
+		)
+		(stroke
+			(width 0)
+			(type default)
+		)
+	)
 	(wire
 		(pts
@@
 		)
 	)
+	(bus
+		(pts
+			(xy 339.09 165.1) (xy 346.71 165.1)
+		)
+		(stroke
+			(width 0)
+			(type default)
+		)
+	)
 	(wire
 		(pts
@@
 	(bus
 		(pts
-			(xy 45.72 144.78) (xy 62.23 144.78)
+			(xy 41.91 144.78) (xy 62.23 144.78)
 		)
 		(stroke
@@
 		)
 	)
+	(label "CPU_A31"
+		(at 341.63 158.75 0)
+		(effects
+			(font
+				(size 1.27 1.27)
+			)
+			(justify left bottom)
+		)
+	)
 	(label "CPU_A6"
 		(at 67.31 158.75 0)
@@
 		)
 	)
-	(global_label "CPU_A31"
-		(shape input)
-		(at 354.33 154.94 180)
-		(fields_autoplaced yes)
-		(effects
-			(font
-				(size 1.27 1.27)
-			)
-			(justify right)
-		)
-		(property "Intersheetrefs" "${INTERSHEET_REFS}"
-			(at 342.9991 154.94 0)
-			(effects
-				(font
-					(size 1.27 1.27)
-				)
-				(justify right)
-				(hide yes)
-			)
-		)
-	)
 	(global_label "CPU_MIO#"
 		(shape input)
@@
 		)
 	)
-	(global_label "CPU_ADDRESS_BUS"
+	(global_label "CPU_A[2..31]"
 		(shape input)
-		(at 45.72 144.78 180)
+		(at 41.91 144.78 180)
 		(fields_autoplaced yes)
 		(effects
@@
 		)
 		(property "Intersheetrefs" "${INTERSHEET_REFS}"
-			(at 24.6525 144.78 0)
+			(at 26.4666 144.78 0)
 			(effects
 				(font
@@
 		)
 	)
-	(global_label "CPU_DATA_BUS"
+	(global_label "CPU_D[0..31]"
 		(shape input)
 		(at 41.91 60.96 180)
@@
 		)
 		(property "Intersheetrefs" "${INTERSHEET_REFS}"
-			(at 24.8943 60.96 0)
+			(at 26.2852 60.96 0)
 			(effects
 				(font
@@
 		)
 	)
+	(global_label "CPU_A[2..31]"
+		(shape input)
+		(at 346.71 165.1 0)
+		(fields_autoplaced yes)
+		(effects
+			(font
+				(size 1.27 1.27)
+			)
+			(justify left)
+		)
+		(property "Intersheetrefs" "${INTERSHEET_REFS}"
+			(at 362.1534 165.1 0)
+			(effects
+				(font
+					(size 1.27 1.27)
+				)
+				(justify left)
+				(hide yes)
+			)
+		)
+	)
 	(global_label "CPU_HLDA"
 		(shape input)
@@
 		(pin "F14"
 		)
-		(pin "H4"
+		(pin "P9"
 		)
 		(pin "E14"
@@
 		(pin "L13"
 		)
-		(pin "D2"
+		(pin "H5"
 		)
 		(pin "A15"
@@
 		(pin "R7"
 		)
-		(pin "D9"
+		(pin "D3"
 		)
 		(pin "T9"

Commit message: Add files via upload
Parts:
- added C107: 1nF, symbol Device:C
- added C112: 150nF, symbol Device:C
Connections:
- net GND: now also C107.2, C112.2
- net PNET1: now also C107.1, C112.1

Commit message: Add files via upload
Parts:
- C107, C112: footprint (none) -> Capacitor_SMD:C_0402_1005Metric
- J12: footprint (none) -> PC110:Debug-6
- J9: footprint (none) -> PC110:Debug-10
- R252, R253: footprint (none) -> PCM_Resistor_SMD_AKL:R_0402_1005Metric
- R395: footprint (none) -> Resistor_SMD:R_0402_1005Metric
- RA3, RA4: footprint (none) -> PC110:R-array
- U76: footprint (none) -> PC110:BGA-256
Connections:
- net Chipset_CPU_CLK: now also R252.1; no longer R252.2
- net GND: now also C107.1, C112.1; no longer C107.2, C112.2
- net PNET1: now also C107.2, C112.2; no longer C107.1, C112.1
- net at R253.1, U76.A9 (CLK_CPU): now also R252.2; no longer R252.1
Other:
- moved on the sheet: C107, C112, R252
Changed lines of the file:
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@@
 			)
 		)
-		(property "Footprint" ""
+		(property "Footprint" "PCM_Resistor_SMD_AKL:R_0402_1005Metric"
 			(at 326.39 201.168 90)
 			(effects
@@
 			)
 		)
-		(property "Footprint" ""
+		(property "Footprint" "Resistor_SMD:R_0402_1005Metric"
 			(at 54.61 219.202 90)
 			(effects
@@
 	(symbol
 		(lib_id "Device:C")
-		(at 256.54 30.48 0)
-		(mirror y)
+		(at 256.54 30.48 180)
 		(unit 1)
 		(exclude_from_sim no)
@@
 		(dnp no)
 		(property "Reference" "C112"
-			(at 261.874 29.464 0)
+			(at 261.874 31.496 0)
 			(effects
 				(font
@@
 		)
 		(property "Value" "150nF"
-			(at 262.636 31.75 0)
-			(effects
-				(font
-					(size 1.27 1.27)
-				)
-			)
-		)
-		(property "Footprint" ""
-			(at 255.5748 34.29 0)
+			(at 262.636 29.21 0)
+			(effects
+				(font
+					(size 1.27 1.27)
+				)
+			)
+		)
+		(property "Footprint" "Capacitor_SMD:C_0402_1005Metric"
+			(at 255.5748 26.67 0)
 			(effects
 				(font
@@
 			)
 		)
-		(property "Footprint" ""
+		(property "Footprint" "PC110:BGA-256"
 			(at 184.15 144.78 0)
 			(effects
@@
 			)
 		)
-		(property "Footprint" ""
+		(property "Footprint" "PC110:R-array"
 			(at 54.61 221.615 90)
 			(effects
@@
 			)
 		)
-		(property "Footprint" ""
+		(property "Footprint" "PC110:Debug-10"
 			(at 365.76 119.38 0)
 			(effects
@@
 	(symbol
 		(lib_id "Device:R")
-		(at 326.39 207.01 90)
+		(at 326.39 207.01 270)
+		(mirror x)
 		(unit 1)
 		(exclude_from_sim no)
@@
 		(dnp no)
 		(property "Reference" "R252"
-			(at 328.422 203.2 90)
+			(at 324.358 203.2 90)
 			(effects
 				(font
@@
 		)
 		(property "Value" "33"
-			(at 327.914 204.978 90)
+			(at 324.866 204.978 90)
 			(effects
 				(font
@@
 			)
 		)
-		(property "Footprint" ""
+		(property "Footprint" "PCM_Resistor_SMD_AKL:R_0402_1005Metric"
 			(at 326.39 208.788 90)
 			(effects
@@
 			)
 		)
-		(property "Footprint" ""
+		(property "Footprint" "PC110:Debug-6"
 			(at 365.76 148.59 0)
 			(effects
@@
 			)
 		)
-		(property "Footprint" ""
+		(property "Footprint" "PC110:R-array"
 			(at 307.34 65.405 90)
 			(effects
@@
 	(symbol
 		(lib_id "Device:C")
-		(at 275.59 30.48 0)
-		(mirror y)
+		(at 275.59 30.48 180)
 		(unit 1)
 		(exclude_from_sim no)
@@
 		(dnp no)
 		(property "Reference" "C107"
-			(at 280.924 29.464 0)
+			(at 280.924 31.496 0)
 			(effects
 				(font
@@
 		)
 		(property "Value" "1nF"
-			(at 281.686 31.75 0)
-			(effects
-				(font
-					(size 1.27 1.27)
-				)
-			)
-		)
-		(property "Footprint" ""
-			(at 274.6248 34.29 0)
-			(effects
-				(font
+			(at 281.686 29.21 0)
+			(effects
+				(font
+					(size 1.27 1.27)
+				)
+			)
+		)
+		(property "Footprint" "Capacitor_SMD:C_0402_1005Metric"
+			(at 274.6248 26.67 0)
+			(effects
+				(font

Commit message: Add files via upload
Parts:
- J12: value ~ -> Debug-6
- J9: value ~ -> Debug-10
- U76: value 80486SX -> 486SX-33
Changed lines of the file:
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@@
 			)
 		)
-		(property "Description" "Resistor"
+		(property "Description" ""
 			(at 326.39 199.39 0)
 			(effects
@@
 			)
 		)
-		(property "Description" "Resistor"
+		(property "Description" ""
 			(at 54.61 220.98 0)
 			(effects
@@
 			)
 		)
-		(property "Description" "Unpolarized capacitor"
+		(property "Description" ""
 			(at 256.54 30.48 0)
 			(effects
@@
 			)
 		)
-		(property "Value" "80486SX"
+		(property "Value" "486SX-33"
 			(at 287.528 51.816 0)
 			(effects
@@
 			)
 		)
-		(property "Datasheet" ""
+		(property "Datasheet" "http://github.com/ahmadexp/PC110-Mainboard-Schematic/blob/main/datasheets/bottom/4-486SX-33.pdf"
 			(at 184.15 144.78 0)
 			(effects
@@
 			)
 		)
-		(property "Description" ""
+		(property "Description" "Intel 486 SX"
 			(at 184.15 144.78 0)
 			(effects
@@
 			)
 		)
-		(property "Description" "4 resistor network, parallel topology"
+		(property "Description" ""
 			(at 54.61 214.63 0)
 			(effects
@@
 			)
 		)
-		(property "Value" "~"
+		(property "Value" "Debug-10"
 			(at 365.76 109.22 0)
 			(effects
@@
 			)
 		)
-		(property "Description" "Resistor"
+		(property "Description" ""
 			(at 326.39 207.01 0)
 			(effects
@@
 			)
 		)
-		(property "Value" "~"
+		(property "Value" "Debug-6"
 			(at 370.84 149.86 0)
 			(effects
@@
 			)
 		)
-		(property "Description" "4 resistor network, parallel topology"
+		(property "Description" ""
 			(at 307.34 72.39 0)
 			(effects
@@
 			)
 		)
-		(property "Description" "Unpolarized capacitor"
+		(property "Description" ""
 			(at 275.59 30.48 0)
 			(effects
