File: PCB/Mainboard/DockStation.kicad_sch (KiCad schematic)
At the start: 1 part, among them J13 Docking Station

Commit message: Add files via upload
Parts:
- added C238: 1uF, symbol PCM_Elektuur:C
- added C243: 120nF, symbol PCM_Elektuur:C
- added F2: 1.0A, symbol Device:Fuse
- added J8: ~, symbol PC110:Modem_Conn
- added Q32: 8B, symbol Simulation_SPICE:NPN
- added Q33: BH, symbol PCM_Generic:Q-BJT-Darlington,PNP,IEEE
- added R122, R123, R124, R125, R130, R139, R302, R306: 470k, symbol Device:R
- added R181, R289: 10k, symbol Device:R
- added R291, R297: 220, symbol Device:R
- added R293: 22k, symbol Device:R
- added U20: 7W14, symbol 74xGxx:74LVC3G14
- added U57: SN74LVT125, symbol 74xx:74LS125
- added U71: SN74LV32, symbol 74xx:74LS32
Connections:
- net GND: now reaches J13.1 (GND)
- net GND: now also J13.100 (GND), J13.50 (GND), J13.51 (GND), J13.64 (GND), J13.66 (GND), J13.68 (GND), J13.70 (GND), J13.75 (GND), J13.85 (GND), C243.2 (-), J8.1 (GND), J8.13 (GND), J8.14 (GND), J8.26 (GND), Q32.3 (E), U20.4 (GND), U57.7 (GND)
- net FDC_WRTPRT#: now reaches J13.10 (FDC_WRTPRT#)
- net FDC_WRTPRT#: now also R125.1
- net FDC_HDSEL#: now reaches J13.11 (FDC_HDSEL#)
- net FDC_DSKCHG#: now reaches J13.12 (FDC_DSKCHG#)
- net FDC_DSKCHG#: now also R122.1
- net at J13.13 (Q33_2): now also J13.88 (Q33_2), J13.89 (Q33_2)
- net Pluto_Dock_IO1: now reaches J13.2 (Pluto_IO1)
- net Pluto_Dock_IO1: now also R139.1
- net at J13.3 (FDD_DRATE1): now also U57.11
- net FDD_INDEX#: now reaches J13.4 (FDD_INDEX#)
- net FDD_INDEX#: now also R123.1
- net FDD_DRSEL: now reaches J13.5 (FDD_DRSEL)
- net FDD_MOTEN: now reaches J13.6 (FDD_MOTEN)
- net FDC_DIR#: now reaches J13.7 (FDC_DIR#)
- net Pluto_Dock_IO3: now reaches J13.79 (J13_79)
- net FDC_TRK0#: now reaches J13.9 (FDC_TRK0)
- net FDC_TRK0#: now also R124.1
- net FDC_WGATE#: now reaches J13.93 (FDC_WGATE#)
- net FDC_STEP#: now reaches J13.94 (FDC_STEP#)
- net at J13.96 (FDD_DRATE0): now also U57.3
- net Pluto_Dock_IO2: now reaches J13.99 (Pluto_IO2)
- net Pluto_Dock_IO2: now also R130.1
- new net: C238.1 (+), Q33.2 (B), R293.1, R297.2
- new net: C238.2 (-), Q33.1 (C)
- new net: Q32.1 (C), R291.1
- new net: Q32.2 (B), R289.2
- new net: U20.6, U57.1, U57.13, U71.3
- new net: F2.2, Q33.3 (E), R293.2
- new net: R289.1, U20.2
- new net: R291.2, R297.1
- new net FDC_DRATE0: R302.1, U57.2
- new net FDC_DRATE1: R306.1, U57.12
- new net MN195_U1RD#: J8.3 (U1RD#)
- new net PNET5: C243.1 (+), F2.1, R122.2, R123.2, R124.2, R125.2, R302.2, R306.2, U20.8 (VCC), U57.14 (VCC)
- new net PNET7: R130.2, R139.2
- new net PWRGD_shift_buff: R181.1, U71.1
- new net Pluto_Switched_PNET5: J8.12 (PNET5_Pluto), J8.15 (PNET5_Pluto)
- new net U71_OR1_IN2: U71.2
- new net VCC: J8.1 (GND), J8.25 (VCC)
- new net YellowWire1_2: R181.2
- no-connect marks 0 -> 9
Other:
- moved on the sheet: J13

Commit message: Add files via upload
Parts:
- added C163, C167, C170, C199: 220pF, symbol PCM_Elektuur:C
- added C198, C92: 120nF, symbol PCM_Elektuur:C
- added C240: 330nF, symbol PCM_Elektuur:C
- added C256: 150nF, symbol PCM_Elektuur:C
- added C7: 100nF, symbol PCM_Elektuur:C
- added EMI5: EMI, symbol Device:Filter_EMI_LLLL_15263748
- added F3: 0.5A, symbol Device:Fuse
- added J1: ~, symbol PC110:PS2_Conn
- added L1: 1.5uH, symbol Device:L
- added L12: 300nH, symbol Device:L
- added Q34: BH, symbol PCM_Generic:Q-BJT-Darlington,PNP,IEEE
- added R231: 0, symbol Device:R
- added R294: 1.2k, symbol Device:R
- added RA2: 10k, symbol Device:R_Pack04
Connections:
- net GND: now also U71.7 (GND), C163.2 (-), C167.2 (-), C170.2 (-), C198.2 (-), C199.2 (-), C256.2 (-), C7.2 (-), C92.2 (-), R231.1
- net PNET5: now also U71.14 (VCC), C256.1 (+), Q34.3 (E)
- net KB_INIT1: now reaches J13.14 (KB_INT1)
- net KB_INIT1: now also EMI5.5, RA2.5 (R4.2)
- new net: C92.1 (+), F3.2, L12.2, RA2.1 (R1.1), RA2.2 (R2.1), RA2.3 (R3.1), RA2.4 (R4.1)
- new net: C7.1 (+), J1.7 (PS2_Pluto), L1.1
- new net: C240.2 (-), F3.1, Q34.1 (C)
- new net: C240.1 (+), Q34.2 (B), R294.2
- new net: C170.1 (+), EMI5.1, J1.5 (KB_INIT3)
- new net: C198.1 (+), J1.4 (5V), L12.1
- new net: J1.1 (GND), J1.8 (GND), R231.2
- new net: C167.1 (+), EMI5.4, J1.2 (KB_INIT1)
- new net: C199.1 (+), EMI5.2, J1.3 (KB_INIT4)
- new net: C163.1 (+), EMI5.3, J1.6 (KB_INIT2)
- new net KB_INIT2: EMI5.6, RA2.6 (R3.2)
- new net KB_INIT3: EMI5.8, RA2.8 (R1.2)
- new net KB_INIT4: EMI5.7, RA2.7 (R2.2)
- new net KB_SRDY#_shift: R294.1
Other:
- moved on the sheet: J8, U20A, U20C, U57B, U57C, U71B

Commit message: Add files via upload
Parts:
- added C235, C237: 150nF, symbol PCM_Elektuur:C
- added C89: 470nF, symbol PCM_Elektuur:C
- added C90: 120nF, symbol PCM_Elektuur:C
- added D39, D55: s.3 5F, symbol Device:D
- added D52, D53, D54, D56, D57: K, symbol Device:D_Dual_Series_KAC
- added R127, R135, R144, R183, R187, R189, R191, R194, R228, R303, R305, R307, R309, R311: 470k, symbol Device:R
- added R188, R192, R193: 10k, symbol Device:R
- added U26: 7W126, symbol 74xGxx:74AUC1G74
- added U64: 74LV126, symbol 74xx:74LS126
Connections:
- net FDC_TRK0# is gone; now on net FDC_DSKCHG#: J13.9 (FDC_TRK0), R124.1
- net GND: now also C235.2 (-), C237.2 (-), C90.2 (-), D52.1 (A), D53.1 (A), D54.1 (A), D56.1 (A), D57.1 (A), U26.4 (GND), U64.7 (GND)
- net KB_INIT2: now also J13.15 (KB_INT2)
- net KB_INIT3: now also J13.86 (KB_INT3)
- net KB_INIT4: now also J13.87 (KB_INT4)
- net PNET5: now also J13.40 (PNET5), C90.1 (+), R135.2, R188.2, R192.2, R193.2, R303.2, R305.2, R307.2, R309.2, R311.2, U26.8 (VCC)
- net PNET7: now also R144.2
- net VCC: now also D52.2 (K), D53.2 (K), D54.2 (K), D56.2 (K), D57.2 (K)
- net at C92.1 (+), F3.2, L12.2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: now also J13.16 (PNET5_Q1)
- net at C238.2 (-), Q33.1 (C): now also J13.13 (Q33_2), J13.88 (Q33_2), J13.89 (Q33_2)
- net FDC_DCD2#: now reaches J13.17 (DCD2#)
- net FDC_DCD2#: now also R309.1
- net at J13.18 (RXD2): now also R135.1, U26.5 (Q)
- net at J13.19 (TXD2): now also U26.6 (~{CLR})
- net FDC_DTR2#: now reaches J13.20 (DTR2#)
- net PNET2: now reaches J13.21 (PNET2)
- net PNET2: now also J13.80 (PNET2), C235.1 (+), C237.1 (+), R183.2
- net FDC_BUSY: now reaches J13.22 (BUSY)
- net FDC_SLCT: now reaches J13.23 (SLCT)
- net FDC_PD7: now reaches J13.24 (PD7)
- net FDC_PD5: now reaches J13.25 (PD5)
- net FDC_PD4: now reaches J13.26 (PD4)
- net FDC_PD3: now reaches J13.27 (PD3)
- net FDC_PD2: now reaches J13.28 (PD2)
- net FDC_PD1: now reaches J13.29 (PD1)
- net FDC_PD0: now reaches J13.30 (PD0)
- net FDC_STROBE#: now reaches J13.31 (STROBE#)
- net VGA_VSync: now reaches J13.33 (VGA_VSync)
- net VGA_VSync: now also D57.3 (common)
- net VGA_HSync: now reaches J13.36 (VGA_HSync)
- net VGA_HSync: now also D56.3 (common)
- net M38_P34: now reaches J13.38 (M38_P34)
- net M38_P46: now reaches J13.39 (M38_P46)
- net at J13.41 (Modem_RSRVD2): now also J8.24 (RSRVD1)
- net at J13.42 (Modem_RSRVD1): now also J8.23 (RSRVD2)
- net at J13.46 (PNET4): now also D39.2 (A)
- net at J13.48 (PNET4): now also D55.2 (A)
- net at J13.52 (Modem_VPDA#): now also J8.19 (VPDA#)
- net J13_53: now reaches J13.53 (J13_53)
- net J13_53: now also J13.54 (J13_53), J13.55 (J13_53), J13.56 (J13_53), J13.57 (J13_53)
- net at J13.58 (Modem_S11): now also J8.22 (S11)
- net at J13.59 (Modem_ADCK#): now also J8.21 (ADCK#)
- net at J13.60 (Modem_IRQ1#): now also J8.20 (IRQ1#)
- net M38_P67: now reaches J13.61 (M38_P67)
- net M38_P16_R86: now reaches J13.62 (M38_P16)
- net KB_SPKUP_DN: now reaches J13.63 (KB_SPKUP_DN)
- net VGA_Blue: now reaches J13.65 (VGA_Blue)
- net VGA_Blue: now also D54.3 (common)
- net VGA_Green: now reaches J13.67 (VGA_Green)
- net VGA_Green: now also D53.3 (common)
- net VGA_Red: now reaches J13.69 (VGA_Red)
- net VGA_Red: now also D52.3 (common)
- net FDC_ACK#: now reaches J13.71 (ACK#)
- net FDC_INIT#: now reaches J13.72 (INIT#)
- net FDC_AUTOFD#: now reaches J13.73 (AUTOFD#)
- net FDC_SLCTIN#: now reaches J13.74 (SLCTIN#)
- net FDC_PD6: now reaches J13.76 (PD6)
- net FDC_ERROR#: now reaches J13.77 (ERROR#)
- net FDC_PE: now reaches J13.78 (PE)
- net FDC_WDATA#: now reaches J13.8 (FDC_WDATA#)
- net FDC_RI2#: now reaches J13.81 (RI2#)
- net FDC_RI2#: now also R311.1
- net FDC_CTS2#: now reaches J13.82 (CTS2#)
- net FDC_CTS2#: now also R303.1
- net FDC_RTS2#: now reaches J13.83 (RTS2#)
- net FDC_DSR2#: now reaches J13.84 (DSR2#)
- net FDC_DSR2#: now also R305.1
- net FDD_Bowman: now reaches J13.90 (FDD_Bowman)
- net FDD_Bowman: now also R144.1
- net FDC_RDATA#: now reaches J13.91 (FDC_RDATA#)
- net FDC_RDATA#: now also R307.1
- net FDD_Pluto4: now reaches J13.92 (FDD_Pluto4)
- net FDD_Pluto3: now reaches J13.95 (FDD_Pluto3)
- net FDD_Pluto2: now reaches J13.97 (FDD_Pluto2)
- net FDD_Pluto1: now reaches J13.98 (FDD_Pluto1)
- net PS2_L1_Pluto: now reaches L1.2
- net PS2_L1_Pluto: now also R228.1
- net FDC_RXD1: now reaches J8.10 (RXD1)
- net FDC_RXD1: now also R194.1
- net at J8.11 (TXD1): now also U64.3
- net MN192_VSEN#: now reaches J8.16 (VSEN#)
- net Modem_VSDA#: now reaches J8.17 (VSDA#)
- net Modem_VSDA#: now also R127.1
- net at J8.18 (VPCK#): now also C89.1 (+)
- net FDC_DCD1#: now reaches J8.4 (DCD1#)
- net FDC_RI1#: now reaches J8.5 (RI1#)
- net FDC_RI1#: now also R187.1
- net at J8.6 (DRT1#): now also U64.8
- net FDC_DSR1: now reaches J8.7 (DSR1)
- net FDC_DSR1: now also R189.1
- net FDC_CTS1#: now reaches J8.8 (CTS1#)
- net FDC_CTS1#: now also R191.1
- net at J8.9 (RTS1#): now also U64.6
- new net: U64.1, U64.10, U64.4
- new net: U26.1 (C), U26.7 (~{PRE})
- new net FDC_DTR1#: R192.1, U64.9
- new net FDC_IRTX_TXD2: R183.1, U26.2 (D)
- new net FDC_RTS1#: R193.1, U64.5
- new net FDC_TXD1: R188.1, U64.2
- new net Modem_Audio_Out: C89.2 (-)
- new net PNET1: R127.2, R228.2, U64.14 (VCC)
- new net PNET4: D39.1 (K), D55.1 (K)
- new net Pluto_enabled_PNET5: R187.2, R189.2, R191.2, R194.2
Other:
- moved on the sheet: C163, C167, C170, C198, C199, C238, C240, C243, C256, C7, C92, EMI5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

Commit message: Add files via upload
Parts:
- removed unit 3 of U20
- removed unit 1 of U20
- added C1: DNP, symbol PCM_Elektuur:C
- added C168: 1uF, symbol PCM_Elektuur:C
- added C197: 300nF, symbol PCM_Elektuur:C
- added C2, C202: 150nF, symbol PCM_Elektuur:C
- added C200, C201: 10uF, symbol PCM_Elektuur:C
- added C4: 1nF, symbol PCM_Elektuur:C
- added D1, D59: 3D, symbol Device:D_Dual_CommonCathode_AKA
- added Q24: 6D, symbol Simulation_SPICE:PNP
- added Q25: BH, symbol PCM_Generic:Q-BJT-Darlington,PNP,IEEE
- added R238: 56, symbol Device:R
- added R241: 8.2, symbol Device:R
- added R242: 7.5k, symbol Device:R
- added R4: 4.7k, symbol Device:R
- added R8: 300, symbol Device:R
- added U1: EA, symbol 74xGxx:74AHC1G14
- added U2: 7W32, symbol 74xGxx:74LVC2G32
- added U3: HSDL-1000 X03, symbol PC110:IRDA
- renumbered C256 to C265, EMI5 to EM5
Connections:
- net FDC_IRTX_TXD2: now also U57.5
- net GND: now also D52.2 (A), D53.2 (A), D54.2 (A), D56.2 (A), D57.2 (A), U71.4, U71.5, C1.2 (-), C168.2 (-), C197.2 (-), C2.2 (-), C200.2 (-), C201.2 (-), C202.2 (-), C4.2 (-), U1.3 (GND), U2.4 (GND), U3.2 (GND); no longer D52.1 (A), D53.1 (A), D54.1 (A), D56.1 (A), D57.1 (A)
- net KB_INIT1: now also EM5.8; no longer EM5.5
- net KB_INIT2: now also EM5.7; no longer EM5.6
- net KB_INIT3: now also EM5.5; no longer EM5.8
- net KB_INIT4: now also EM5.6; no longer EM5.7
- net KB_SPKUP_DN: now also D59.3 (A)
- net PNET2: now also C2.1 (+), U1.5 (VCC), U2.8 (VCC)
- net PNET5: now also Q24.3 (E), Q25.3 (E)
- net VCC: now also D52.1 (K), D53.1 (K), D54.1 (K), D56.1 (K), D57.1 (K); no longer D52.2 (K), D53.2 (K), D54.2 (K), D56.2 (K), D57.2 (K)
- net Enable_IRDA_Buf: now reaches U57.10
- net Enable_IRDA_Buf: now also U26.1 (C), U26.7 (~{PRE}), U57.4, Q24.2 (B), R242.2
- net FDC_IRRX_RXD2: now reaches U57.8
- net FDC_IRRX_RXD2: now also U26.3 (~{Q})
- net at U57.9: now also U2.7
- net FDC_TXD2_EN: now reaches U57.6
- net FDC_TXD2_EN: now also R8.1, U2.5
- new net: C1.1 (+), U2.1, U3.1 (IRDA_RXA)
- new net: U1.4, U2.2
- new net: C4.1 (+), D1.1 (A), D1.3 (A), R4.2, U1.2
- new net: C200.1 (+), R241.1, U3.8 (IRDA_LED_A)
- new net: C168.1 (+), U3.3 (PIN_Bypass)
- new net: D1.2 (K), R4.1, U2.3
- new net: Q24.1 (C), R238.2
- new net: C201.1 (+), C202.1 (+), R238.1, U3.6 (IRDA_Supply)
- new net: Q25.1 (C), R241.2
- new net: Q25.2 (B), R242.1
- new net: C197.1 (+), U3.5 (Daylight_Cancellation)
- new net: R8.2, U3.7 (IRDA_TXD)
- new net Pluto_IRDA_OUT: U2.6
- new net YellowWire2_1: D59.1 (A)
- new net YellowWire2_3: D59.2 (K)
- no-connect marks 9 -> 11
Other:
- moved on the sheet: C163, C167, C170, C198, C199, C235, C237, C238, C240, C243, C265, C7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

Commit message: Add files via upload
Other:
- moved on the sheet: L12
Changed lines of the file:
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@@
 	(wire
 		(pts
-			(xy 186.69 114.3) (xy 181.61 114.3)
+			(xy 195.58 114.3) (xy 181.61 114.3)
 		)
 		(stroke
@@
 	(wire
 		(pts
-			(xy 194.31 114.3) (xy 217.17 114.3)
+			(xy 203.2 114.3) (xy 217.17 114.3)
 		)
 		(stroke
@@
 	(symbol
 		(lib_id "Device:L")
-		(at 190.5 114.3 90)
+		(at 199.39 114.3 90)
 		(unit 1)
 		(exclude_from_sim no)
@@
 		(dnp no)
 		(property "Reference" "L12"
-			(at 190.5 117.348 90)
+			(at 199.39 117.348 90)
 			(effects
 				(font
@@
 		)
 		(property "Value" "300nH"
-			(at 190.5 115.316 90)
+			(at 199.39 115.316 90)
 			(effects
 				(font
@@
 		)
 		(property "Footprint" ""
-			(at 190.5 114.3 0)
+			(at 199.39 114.3 0)
 			(effects
 				(font
@@
 		)
 		(property "Datasheet" "~"
-			(at 190.5 114.3 0)
+			(at 199.39 114.3 0)
 			(effects
 				(font
@@
 		)
 		(property "Description" "Inductor"
-			(at 190.5 114.3 0)
+			(at 199.39 114.3 0)
 			(effects
 				(font

Commit message: Add files via upload
Other:
- moved on the sheet: C2, C243, C265, U20D, U2C, U57E, U64E, U71B, U71E

Commit message: Add files via upload
Other:
- company: (none) -> Recreated by: Ahmad Byagowi
Changed lines of the file:
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@@
 	(title_block
 		(title "PC110")
+		(company "Recreated by: Ahmad Byagowi")
 	)
 	(junction

Commit message: Add files via upload
Connections:
- net Pluto_Dock_IO3 renamed EN_RS232
Other:
- note added: "Enables all external PS/2 devices; PS/2 conn on PC110 and dock"
Changed lines of the file:
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@@
 		(company "Recreated by: Ahmad Byagowi")
 	)
+	(text "Enables all external PS/2 devices; \nPS/2 conn on PC110 and dock"
+		(exclude_from_sim no)
+		(at 281.94 84.074 0)
+		(effects
+			(font
+				(size 1.27 1.27)
+			)
+		)
+	)
 	(junction
 		(at 589.28 378.46)
@@
 		)
 	)
-	(label "Pluto_Dock_IO3"
-		(at 467.36 307.34 0)
+	(label "EN_RS232"
+		(at 472.44 307.34 0)
 		(effects
 			(font
