File: PCB/Mainboard/DockStation.kicad_sch (KiCad schematic)
At the start: 91 parts, among them J13 Docking Station, Q24 MUN2114, Q25 BH, Q32 8B, Q33 BH, Q34 BH, U1 EA, U2 7W32, U20 7W14, U26 7W126, U3 HSDL-1000 X03, U57 SN74LVT125, U64 74LV126, U71 SN74LV32

Commit message: Add files via upload
Connections:
- net Pluto_enabled_PNET5 is gone; now on net Pluto_Switched_PNET5: R187.2, R189.2, R191.2, R194.2
- net FDC_DSKCHG#: no longer J13.9 (FDC_TRK0), R124.1
- net VCC: now also J8.2 (VCC); no longer J8.1 (GND)
- new net FDC_TRK0#: J13.9 (FDC_TRK0), R124.1
- no-connect marks 11 -> 2

Commit message: Add files via upload
Connections:
- net FDC_UART1_EN: now reaches U64.1, U64.10, U64.4
Other:
- moved on the sheet: D59, R181
Changed lines of the file:
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@@
 	)
 	(junction
-		(at 334.01 408.94)
-		(diameter 0)
-		(color 0 0 0 0)
-	)
-	(junction
 		(at 302.26 351.79)
 		(diameter 0)
@@
 	)
 	(junction
+		(at 646.43 360.68)
+		(diameter 0)
+		(color 0 0 0 0)
+	)
+	(junction
 		(at 521.97 260.35)
 		(diameter 0)
@@
 	(wire
 		(pts
-			(xy 334.01 403.86) (xy 334.01 408.94)
-		)
-		(stroke
-			(width 0)
-			(type default)
-		)
-	)
-	(wire
-		(pts
 			(xy 431.8 85.09) (xy 416.56 85.09)
 		)
@@
 		)
 	)
-	(bus
+	(wire
 		(pts
-			(xy 328.93 312.42) (xy 328.93 309.88)
+			(xy 651.51 350.52) (xy 646.43 350.52)
 		)
 		(stroke
@@
 		)
 	)
-	(wire
+	(bus
 		(pts
-			(xy 299.72 414.02) (xy 299.72 420.37)
+			(xy 328.93 312.42) (xy 328.93 309.88)
 		)
 		(stroke
@@
 	(wire
 		(pts
+			(xy 646.43 350.52) (xy 646.43 360.68)
+		)
+		(stroke
+			(width 0)
+			(type default)
+		)
+	)
+	(wire
+		(pts
 			(xy 386.08 407.67) (xy 383.54 407.67)
 		)
@@
 	(wire
 		(pts
-			(xy 299.72 420.37) (xy 312.42 420.37)
-		)
-		(stroke
-			(width 0)
-			(type default)
-		)
-	)
-	(wire
-		(pts
 			(xy 449.58 99.06) (xy 449.58 152.4)
 		)
@@
 	(wire
 		(pts
+			(xy 355.6 430.53) (xy 344.17 430.53)
+		)
+		(stroke
+			(width 0)
+			(type default)
+		)
+	)
+	(wire
+		(pts
 			(xy 214.63 388.62) (xy 346.71 388.62)
 		)
@@
 	(wire
 		(pts
-			(xy 317.5 403.86) (xy 334.01 403.86)
-		)
-		(stroke
-			(width 0)
-			(type default)
-		)
-	)
-	(wire
-		(pts
 			(xy 204.47 358.14) (xy 204.47 360.68)
 		)
@@
 	(wire
 		(pts
-			(xy 646.43 361.95) (xy 656.59 361.95)
+			(xy 646.43 360.68) (xy 656.59 360.68)
 		)
 		(stroke
@@
 	(wire
 		(pts
+			(xy 339.09 443.23) (xy 339.09 438.15)
+		)
+		(stroke
+			(width 0)
+			(type default)
+		)
+	)
+	(wire
+		(pts
 			(xy 331.47 309.88) (xy 346.71 309.88)
 		)
@@
 	(wire
 		(pts
-			(xy 307.34 408.94) (xy 334.01 408.94)
-		)
-		(stroke
-			(width 0)
-			(type default)
-		)
-	)
-	(wire
-		(pts
 			(xy 381 242.57) (xy 381 250.19)
 		)
@@
 	(wire
 		(pts
-			(xy 547.37 243.84) (xy 560.07 243.84)
+			(xy 542.29 243.84) (xy 560.07 243.84)
 		)
 		(stroke
@@
 	(wire
 		(pts
-			(xy 646.43 391.16) (xy 646.43 361.95)
+			(xy 646.43 391.16) (xy 646.43 360.68)
 		)
 		(stroke
@@
 	(wire
 		(pts
-			(xy 339.09 392.43) (xy 339.09 408.94)
+			(xy 339.09 392.43) (xy 339.09 422.91)
 		)
 		(stroke
@@
 	(wire
 		(pts
-			(xy 334.01 408.94) (xy 339.09 408.94)
-		)
-		(stroke
-			(width 0)
-			(type default)
-		)
-	)
-	(wire
-		(pts
 			(xy 365.76 255.27) (xy 365.76 267.97)
 		)
@@
 	(wire
 		(pts
-			(xy 519.43 243.84) (xy 539.75 243.84)
+			(xy 515.62 243.84) (xy 534.67 243.84)
 		)
 		(stroke
@@
 	(wire
 		(pts
+			(xy 656.59 360.68) (xy 656.59 361.95)
+		)
+		(stroke
+			(width 0)
+			(type default)
+		)
+	)
+	(wire
+		(pts
 			(xy 589.28 361.95) (xy 589.28 378.46)
 		)
@@
 	(wire
 		(pts
-			(xy 283.21 408.94) (xy 292.1 408.94)
+			(xy 317.5 443.23) (xy 339.09 443.23)
 		)
 		(stroke
@@
 		)
 	)
-	(label "YellowWire1_2"
-		(at 519.43 243.84 0)
-		(effects
-			(font
-				(size 1.27 1.27)
-			)
-			(justify left bottom)
-		)
-	)
 	(label "FDC_PD3"
 		(at 331.47 309.88 0)
@@
 		)
 	)
-	(label "YellowWire2_2"
-		(at 317.5 403.86 0)
-		(effects
-			(font
-				(size 1.27 1.27)
-			)
-			(justify left bottom)
-		)
-	)
 	(label "J13_53"
 		(at 414.02 283.21 180)
@@
 		)
 	)
+	(global_label "FDC_UART1_EN"
+		(shape input)
+		(at 651.51 350.52 0)
+		(fields_autoplaced yes)
+		(effects
+			(font
+				(size 1.27 1.27)
+			)
+			(justify left)
+		)
+		(property "Intersheetrefs" "${INTERSHEET_REFS}"
+			(at 668.4047 350.52 0)
+			(effects
+				(font
+					(size 1.27 1.27)
+				)
+				(justify left)
+				(hide yes)
+			)
+		)
+	)
 	(global_label "KB_INIT2"
 		(shape input)
@@
 		)
 	)
+	(global_label "YellowWire1_2"
+		(shape input)
+		(at 515.62 243.84 180)
+		(fields_autoplaced yes)
+		(effects
+			(font
+				(size 1.27 1.27)
+			)
+			(justify right)
+		)
+		(property "Intersheetrefs" "${INTERSHEET_REFS}"
+			(at 499.3301 243.84 0)
+			(effects
+				(font
+					(size 1.27 1.27)
+				)
+				(justify right)
+				(hide yes)
+			)
+		)
+	)
 	(global_label "KB_INIT4"
 		(shape input)
@@
 	(global_label "YellowWire2_3"
 		(shape input)
-		(at 312.42 420.37 0)
+		(at 355.6 430.53 0)
 		(fields_autoplaced yes)
 		(effects
@@
 		)
 		(property "Intersheetrefs" "${INTERSHEET_REFS}"
-			(at 328.7099 420.37 0)
+			(at 371.8899 430.53 0)
 			(effects
 				(font
@@
 	(global_label "YellowWire2_1"
 		(shape input)
-		(at 283.21 408.94 180)
+		(at 317.5 443.23 180)
 		(fields_autoplaced yes)
 		(effects
@@
 		)
 		(property "Intersheetrefs" "${INTERSHEET_REFS}"
-			(at 266.9201 408.94 0)
+			(at 301.2101 443.23 0)
 			(effects
 				(font
@@
 	(symbol
 		(lib_id "Device:D_Schottky_Dual_CommonCathode_AKA")
-		(at 299.72 408.94 0)
+		(at 339.09 430.53 90)
 		(unit 1)
 		(exclude_from_sim no)
@@
 		(dnp no)
 		(property "Reference" "D59"
-			(at 299.72 402.59 0)
+			(at 334.264 429.768 90)
 			(effects
 				(font
@@
 		)
 		(property "Value" "RB715F"
-			(at 299.72 405.13 0)
+			(at 332.74 432.054 90)
 			(effects
 				(font
@@
 		)
 		(property "Footprint" ""
-			(at 299.72 408.94 0)
+			(at 339.09 430.53 0)
 			(effects
 				(font
@@
 		)
 		(property "Datasheet" "~"
-			(at 299.72 408.94 0)
+			(at 339.09 430.53 0)
 			(effects
 				(font
@@
 		)
 		(property "Description" "Dual Schottky diode, common cathode on pin 2"
-			(at 299.72 408.94 0)
+			(at 339.09 430.53 0)
 			(effects
 				(font
@@
 		)
 		(property "Topmark" "3D"
-			(at 299.72 408.94 0)
+			(at 339.09 430.53 0)
 			(effects
 				(font
@@
 	(symbol
 		(lib_id "Device:R")
-		(at 543.56 243.84 270)
+		(at 538.48 243.84 270)
 		(mirror x)
 		(unit 1)
@@
 		(dnp no)
 		(property "Reference" "R181"
-			(at 545.592 240.03 90)
+			(at 540.512 240.03 90)
 			(effects
 				(font
@@
 		)
 		(property "Value" "10k"
-			(at 545.084 241.808 90)
+			(at 540.004 241.808 90)
 			(effects
 				(font
@@
 		)
 		(property "Footprint" ""
-			(at 543.56 245.618 90)
+			(at 538.48 245.618 90)
 			(effects
 				(font
@@
 		)
 		(property "Datasheet" "~"
-			(at 543.56 243.84 0)
+			(at 538.48 243.84 0)
 			(effects
 				(font
@@
 		)
 		(property "Description" "Resistor"
-			(at 543.56 243.84 0)
+			(at 538.48 243.84 0)
 			(effects
 				(font

Commit message: Add files via upload
Parts:
- added C239: 150nF, symbol PCM_Elektuur:C
- added C86, C88: 180nF, symbol PCM_Elektuur:C
- added C91, C93: 100nF, symbol PCM_Elektuur:C
- added R187: 470k, symbol Device:R
- added R230: 0, symbol Device:R
- renumbered R187 to R190
Connections:
- net FDC_DCD1#: now also R187.1
- net GND: now also C239.1 (+), C86.1 (+), C88.1 (+), C91.1 (+), C93.1 (+), R230.1
- net PNET5: now also C91.2 (-)
- net Pluto_Switched_PNET5: now also C86.2 (-), R187.2
- net VCC: now also C88.2 (-)
- net at C238.2 (-), J13.13 (FDD_PWR), J13.88 (FDD_PWR)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: now also C239.2 (-), C93.2 (-)
- net at J1.1 (GND), R231.2: no longer J1.8 (GND)
- new net: J1.8 (GND), R230.2
Other:
- moved on the sheet: F2, R188, R189, R190, R191, R192, R193, R194, R231, U64A, U64B, U64C

Commit message: Add files via upload
Parts:
- added C3: 100nF, symbol PCM_Elektuur:C
Connections:
- net GND: now also C3.2 (-)
- net PNET2: now also C3.1 (+)
Changed lines of the file:
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@@
 	)
 	(junction
+		(at 567.69 81.28)
+		(diameter 0)
+		(color 0 0 0 0)
+	)
+	(junction
 		(at 293.37 114.3)
 		(diameter 0)
@@
 	(wire
 		(pts
+			(xy 549.91 81.28) (xy 567.69 81.28)
+		)
+		(stroke
+			(width 0)
+			(type default)
+		)
+	)
+	(wire
+		(pts
 			(xy 528.32 119.38) (xy 528.32 109.22)
 		)
@@
 	(wire
 		(pts
-			(xy 567.69 96.52) (xy 567.69 99.06)
+			(xy 567.69 78.74) (xy 567.69 81.28)
 		)
 		(stroke
@@
 	(wire
 		(pts
+			(xy 549.91 83.82) (xy 549.91 81.28)
+		)
+		(stroke
+			(width 0)
+			(type default)
+		)
+	)
+	(wire
+		(pts
 			(xy 674.37 391.16) (xy 674.37 389.89)
 		)
@@
 	(wire
 		(pts
+			(xy 567.69 81.28) (xy 567.69 99.06)
+		)
+		(stroke
+			(width 0)
+			(type default)
+		)
+	)
+	(wire
+		(pts
 			(xy 373.38 278.13) (xy 373.38 293.37)
 		)
@@
 	(wire
 		(pts
+			(xy 549.91 93.98) (xy 549.91 96.52)
+		)
+		(stroke
+			(width 0)
+			(type default)
+		)
+	)
+	(wire
+		(pts
 			(xy 533.4 297.18) (xy 533.4 302.26)
 		)
@@
 	(symbol
 		(lib_id "power:VCC")
-		(at 567.69 96.52 0)
+		(at 567.69 78.74 0)
 		(unit 1)
 		(exclude_from_sim no)
@@
 		(fields_autoplaced yes)
 		(property "Reference" "#PWR0270"
-			(at 567.69 100.33 0)
+			(at 567.69 82.55 0)
 			(effects
 				(font
@@
 		)
 		(property "Value" "PNET2"
-			(at 567.69 91.44 0)
+			(at 567.69 73.66 0)
 			(effects
 				(font
@@
 		)
 		(property "Footprint" ""
-			(at 567.69 96.52 0)
+			(at 567.69 78.74 0)
 			(effects
 				(font
@@
 		)
 		(property "Datasheet" ""
-			(at 567.69 96.52 0)
+			(at 567.69 78.74 0)
 			(effects
 				(font
@@
 		)
 		(property "Description" "Power symbol creates a global label with name \"VCC\""
-			(at 567.69 96.52 0)
+			(at 567.69 78.74 0)
 			(effects
 				(font
@@
 	)
 	(symbol
+		(lib_id "power:GND")
+		(at 549.91 96.52 0)
+		(mirror y)
+		(unit 1)
+		(exclude_from_sim no)
+		(in_bom yes)
+		(on_board yes)
+		(dnp no)
+		(fields_autoplaced yes)
+		(property "Reference" "#PWR0707"
+			(at 549.91 102.87 0)
+			(effects
+				(font
+					(size 1.27 1.27)
+				)
+				(hide yes)
+			)
+		)
+		(property "Value" "GND"
+			(at 549.91 101.6 0)
+			(effects
+				(font
+					(size 1.27 1.27)
+				)
+			)
+		)
+		(property "Footprint" ""
+			(at 549.91 96.52 0)
+			(effects
+				(font
+					(size 1.27 1.27)
+				)
+				(hide yes)
+			)
+		)
+		(property "Datasheet" ""
+			(at 549.91 96.52 0)
+			(effects
+				(font
+					(size 1.27 1.27)
+				)
+				(hide yes)
+			)
+		)
+		(property "Description" "Power symbol creates a global label with name \"GND\" , ground"
+			(at 549.91 96.52 0)
+			(effects
+				(font
+					(size 1.27 1.27)
+				)
+				(hide yes)
+			)
+		)
+		(pin "1"
+		)
+		(instances
+			(project "PC110"
+				(path "/45c7911f-b027-440e-9e3e-77a146b41944/6dbc8bfb-047e-469c-b9e0-4e168250e555"
+					(reference "#PWR0707")
+					(unit 1)
+				)
+			)
+		)
+	)
+	(symbol
 		(lib_id "PC110:IRDA")
 		(at 421.64 146.05 0)
@@
 					(unit 1)
 				)
+			)
+		)
+	)
+	(symbol
+		(lib_id "PCM_Elektuur:C")
+		(at 549.91 88.9 0)
+		(unit 1)
+		(exclude_from_sim no)
+		(in_bom yes)
+		(on_board yes)
+		(dnp no)
+		(property "Reference" "C3"
+			(at 553.72 87.6299 0)
+			(effects
+				(font
+					(size 1.27 1.27)
+				)
+				(justify left)
+			)
+		)
+		(property "Value" "100nF"
+			(at 553.72 90.1699 0)
+			(effects
+				(font
+					(size 1.27 1.27)
+				)
+				(justify left)
+			)
+		)
+		(property "Footprint" ""
+			(at 549.91 88.9 0)
+			(effects
+				(font
+					(size 1.27 1.27)
+				)
+				(hide yes)
+			)
+		)
+		(property "Datasheet" ""
+			(at 549.91 88.9 0)
+			(effects
+				(font
+					(size 1.27 1.27)
+				)
+				(hide yes)
+			)
+		)
+		(property "Description" "capacitor, non-polarized/bipolar"
+			(at 549.91 88.9 0)
+			(effects
+				(font
+					(size 1.27 1.27)
+				)
+				(hide yes)
+			)
+		)
+		(property "Indicator" "+"
+			(at 548.64 85.725 0)
+			(effects
+				(font
+					(size 1.27 1.27)
+				)
+				(hide yes)
+			)
+		)
+		(property "Rating" "V"
+			(at 549.275 92.075 0)
+			(effects
+				(font
+					(size 1.27 1.27)
+				)
+				(justify right)
+				(hide yes)
+			)
+		)
+		(pin "1"
+		)
+		(pin "2"
+		)
+		(instances
+			(project "PC110"
+				(path "/45c7911f-b027-440e-9e3e-77a146b41944/6dbc8bfb-047e-469c-b9e0-4e168250e555"
+					(reference "C3")
+					(unit 1)
+				)

Commit message: Add files via upload
Parts:
- C1, C163, C167, C170, C198, C199, C2, C235, C237, C239, C243, C265, C3, C4, C7, C86, C88, C90, C91, C92, C93: footprint (none) -> Capacitor_SMD:C_0402_1005Metric
- C168, C197, C202, C238, C240, C89: footprint (none) -> Capacitor_SMD:C_0603_1608Metric
- C200, C201: footprint (none) -> Capacitor_SMD:C_1206_3216Metric
- D1: footprint (none) -> PC110:3D
- D39, D55: footprint (none) -> PC110:Diode
- D52, D53, D54, D56, D57, Q32: footprint (none) -> Package_TO_SOT_SMD:SOT-416
- D59: footprint (none) -> PC110:SOT-416L
- EM5, RA2: footprint (none) -> PC110:R-array
- F2, F3: footprint (none) -> Fuse:Fuse_1206_3216Metric
- J1: footprint (none) -> PC110:PS2
- J13: footprint (none) -> PC110:Docking Port
- J8: footprint (none) -> PC110:Modem-Connector
- L1: footprint (none) -> Inductor_SMD:L_0603_1608Metric
- L12: footprint (none) -> Inductor_SMD:L_0805_2012Metric
- Q24: footprint (none) -> PCM_Package_TO_SOT_SMD_AKL:SOT-23
- Q25, Q33, Q34: footprint (none) -> Package_TO_SOT_SMD:SOT-89-3
- R122, R123, R124, R125, R127, R130, R135, R139, R144, R181, R183, R187, R188, R189, R190, R191, R192, R193, R194, R228, R242, R4, R8: footprint (none) -> PCM_Resistor_SMD_AKL:R_0402_1005Metric
- R230: footprint (none) -> PCM_Resistor_SMD_AKL:R_0805_2012Metric
- R231: footprint (none) -> PCM_Resistor_SMD_AKL:R_0603_1608Metric
- R238: footprint (none) -> Resistor_SMD:R_0603_1608Metric
- R241: footprint (none) -> Resistor_SMD:R_1206_3216Metric_Pad1.30x1.75mm_HandSolder
- R289, R291, R293, R294, R297, R302, R303, R305, R306, R307, R309, R311: footprint (none) -> Resistor_SMD:R_0402_1005Metric
- U1: footprint (none) -> PC110:SOT-353
- U2, U20, U26: footprint (none) -> PC110:sso-8
- U3: footprint (none) -> PC110:IRDA
- U57, U64, U71: footprint (none) -> Package_SO:TSSOP-14_4.4x5mm_P0.65mm
Connections:
- net FDC_CTS2#: now also R303.2; no longer R303.1
- net FDC_DCD2#: now also R309.2; no longer R309.1
- net FDC_DRATE0: now also R302.2; no longer R302.1
- net FDC_DRATE1: now also R306.2; no longer R306.1
- net FDC_DSKCHG#: now also R122.2; no longer R122.1
- net FDC_DSR2#: now also R305.2; no longer R305.1
- net FDC_IRTX_TXD2: now also R183.2; no longer R183.1
- net FDC_RDATA#: now also R307.2; no longer R307.1
- net FDC_TRK0#: now also R124.2; no longer R124.1
- net FDD_Bowman: now also R144.2; no longer R144.1
- net FDD_INDEX#: now also R123.2; no longer R123.1
- net GND: now also C163.1 (+), C167.1 (+), C168.1 (+), C197.1 (+), C200.1 (+), C202.1 (+), C243.1 (+), C265.1 (+), C86.2 (-), C90.1 (+), C91.2 (-), C92.1 (+); no longer C163.2 (-), C167.2 (-), C168.2 (-), C197.2 (-), C200.2 (-), C202.2 (-), C243.2 (-), C265.2 (-), C86.1 (+), C90.2 (-), C91.1 (+), C92.2 (-)
- net Modem_Audio_Out: now also C89.1 (+); no longer C89.2 (-)
- net PNET2: now also R183.1; no longer R183.2
- net PNET5: now also C243.2 (-), C265.2 (-), C90.2 (-), C91.1 (+), F2.2, R122.1, R123.1, R124.1, R302.1, R303.1, R305.1, R306.1, R307.1, R309.1; no longer C243.1 (+), C265.1 (+), C90.1 (+), C91.2 (-), F2.1, R122.2, R123.2, R124.2, R302.2, R303.2, R305.2, R306.2, R307.2, R309.2
- net PNET7: now also R130.1, R139.1, R144.1; no longer R130.2, R139.2, R144.2
- net PWRGD_shift_buff: now also R181.2; no longer R181.1
- net Pluto_Dock_IO1: now also R139.2; no longer R139.1
- net Pluto_Dock_IO2: now also R130.2; no longer R130.1
- net Pluto_Switched_PNET5: now also C86.1 (+); no longer C86.2 (-)
- net YellowWire1_2: now also R181.1; no longer R181.2
- net at J13.16 (PS/2_Power), RA2.1 (R1.1), RA2.2 (R2.1)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: now also C92.2 (-), F3.1, L12.1; no longer C92.1 (+), F3.2, L12.2
- net at C4.1 (+), D1.1 (A), D1.3 (A)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: now also R4.1; no longer R4.2
- net at C240.2 (-), Q34.1 (C): now also F3.2; no longer F3.1
- net at C198.1 (+), J1.4 (5V): now also L12.2; no longer L12.1
- net at R241.1, U3.8 (IRDA_LED_A): now also C200.2 (-); no longer C200.1 (+)
- net at U3.3 (PIN_Bypass): now also C168.2 (-); no longer C168.1 (+)
- net at Q33.3 (E), R293.2: now also F2.1; no longer F2.2
- net at EM5.4, J1.2 (KB_INIT1): now also C167.2 (-); no longer C167.1 (+)
- net at EM5.3, J1.6 (KB_INIT2): now also C163.2 (-); no longer C163.1 (+)
- net at C201.1 (+), R238.1, U3.6 (IRDA_Supply): now also C202.2 (-); no longer C202.1 (+)
- net at D1.2 (K), U2.3: now also R4.2; no longer R4.1
- net at J8.18 (VPCK#): now also C89.2 (-); no longer C89.1 (+)
- net at U3.5 (Daylight_Cancellation): now also C197.2 (-); no longer C197.1 (+)
Other:
- moved on the sheet: C265, C86, C91, C92, F2, F3, L12, R181, R4

Commit message: Add files via upload
Parts:
- removed D52, D53, D54, D56, D57: DA204U, Package_TO_SOT_SMD:SOT-416, symbol Device:D_Dual_Series_KAC
- removed Q25, Q33, Q34: BH, Package_TO_SOT_SMD:SOT-89-3, symbol PCM_Generic:Q-BJT-Darlington,PNP,IEEE
- removed Q32: 8B, Package_TO_SOT_SMD:SOT-416, symbol Simulation_SPICE:NPN
- added D52, D53, D54, D56, D57: DA204U, Package_TO_SOT_SMD:SOT-323_SC-70, symbol Diode:BAT54SW
- added Q25, Q33, Q34: BH, symbol PCM_Transistor_BJT_Darlington_AKL:Q_PNP_Darlington_Generic_BCE
- added Q32: 8B, symbol PCM_Transistor_BJT_AKL:Q_NPN_Generic_BEC
Connections:
- net GND: now also D52.1 (A), D53.1 (A), D54.1 (A), D56.1 (A), D57.1 (A), Q32.2 (E)
- net PNET1: now also D52.2 (K), D53.2 (K), D54.2 (K), D56.2 (K), D57.2 (K)
- net PNET5: now also Q25.3 (E), Q34.3 (E)
- net VGA_Blue: now also D54.3 (COM)
- net VGA_Green: now also D53.3 (COM)
- net VGA_HSync: now also D56.3 (COM)
- net VGA_Red: now also D52.3 (COM)
- net VGA_VSync: now also D57.3 (COM)
- net at C238.1 (+), R293.1, R297.2: now also Q33.1 (B)
- net at C238.2 (-), C239.2 (-), C93.2 (-)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: now also Q33.2 (C)
- net at C240.2 (-), F3.2: now also Q34.2 (C)
- net at C240.1 (+), R294.2: now also Q34.1 (B)
- net at R291.1: now also Q32.3 (C)
- net at R289.2: now also Q32.1 (B)
- net at F2.1, R293.2: now also Q33.3 (E)
- net at R241.2: now also Q25.2 (C)
- net at R242.1: now also Q25.1 (B)

Commit message: Add files via upload
Connections:
- net PNET1: now also R228.1; no longer R228.2
- net PS2_L1_Pluto: now also R228.2; no longer R228.1
Changed lines of the file:
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@@
 		(lib_id "Device:R")
 		(at 281.94 135.89 0)
-		(mirror x)
 		(unit 1)
 		(exclude_from_sim no)
@@
 		(dnp no)
 		(property "Reference" "R228"
-			(at 279.4 134.6199 0)
+			(at 279.4 137.1601 0)
 			(effects
 				(font
@@
 		)
 		(property "Value" "470k"
-			(at 279.4 137.1599 0)
+			(at 279.4 134.6201 0)
 			(effects
 				(font

Commit message: Add files via upload
Parts:
- D52, D53, D54, D56, D57: footprint Package_TO_SOT_SMD:SOT-323_SC-70 -> Package_TO_SOT_SMD:SOT-416
- Q25, Q33, Q34: footprint (none) -> Package_TO_SOT_SMD:SOT-89-3
- Q32: footprint (none) -> Package_TO_SOT_SMD:SOT-416
Changed lines of the file:
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@@
 			)
 		)
-		(property "Footprint" "Package_TO_SOT_SMD:SOT-323_SC-70"
+		(property "Footprint" "Package_TO_SOT_SMD:SOT-416"
 			(at 525.145 520.065 0)
 			(effects
@@
 			)
 		)
-		(property "Footprint" ""
+		(property "Footprint" "Package_TO_SOT_SMD:SOT-89-3"
 			(at 452.12 59.69 0)
 			(effects
@@
 			)
 		)
-		(property "Footprint" "Package_TO_SOT_SMD:SOT-323_SC-70"
+		(property "Footprint" "Package_TO_SOT_SMD:SOT-416"
 			(at 596.265 484.505 0)
 			(effects
@@
 			)
 		)
-		(property "Footprint" ""
+		(property "Footprint" "Package_TO_SOT_SMD:SOT-416"
 			(at 421.64 257.81 0)
 			(effects
@@
 			)
 		)
-		(property "Footprint" "Package_TO_SOT_SMD:SOT-323_SC-70"
+		(property "Footprint" "Package_TO_SOT_SMD:SOT-416"
 			(at 551.815 484.505 0)
 			(effects
@@
 			)
 		)
-		(property "Footprint" ""
+		(property "Footprint" "Package_TO_SOT_SMD:SOT-89-3"
 			(at 228.6 81.28 0)
 			(effects
@@
 			)
 		)
-		(property "Footprint" ""
+		(property "Footprint" "Package_TO_SOT_SMD:SOT-89-3"
 			(at 363.22 251.46 0)
 			(effects
@@
 			)
 		)
-		(property "Footprint" "Package_TO_SOT_SMD:SOT-323_SC-70"
+		(property "Footprint" "Package_TO_SOT_SMD:SOT-416"
 			(at 504.825 484.505 0)
 			(effects
@@
 			)
 		)
-		(property "Footprint" "Package_TO_SOT_SMD:SOT-323_SC-70"
+		(property "Footprint" "Package_TO_SOT_SMD:SOT-416"
 			(at 572.135 520.065 0)
 			(effects
