File: PCB/Mainboard/Clock.kicad_sch (KiCad schematic)
At the start: 34 parts, among them Q31 MUN2114, U16 BD53E31? QC01, U62 74LS125, U63 AV9154A-27, U66 74LS02, X4 59G3482

Commit message: Add files via upload
Parts:
- U62: value SN74LVT125 -> 74LS125
Changed lines of the file:
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@@
 			)
 		)
-		(property "Value" "SN74LVT125"
+		(property "Value" "74LS125"
 			(at 107.95 245.1099 0)
 			(effects

Commit message: Add files via upload
Parts:
- U16: value BD53E31? QC01 -> BD53E31
Connections:
- no-connect marks 3 -> 2
Changed lines of the file:
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@@
-	)
-	(no_connect
-		(at 255.27 114.3)
 	)
 	(no_connect
@@
 		(pts
 			(xy 101.6 100.33) (xy 92.71 100.33)
-		)
-		(stroke
-			(width 0)
-			(type default)
-		)
-	)
-	(wire
-		(pts
-			(xy 255.27 114.3) (xy 252.73 114.3)
 		)
 		(stroke
@@
 			)
 		)
-		(property "Value" "BD53E31? QC01"
+		(property "Value" "BD53E31"
 			(at 244.094 104.14 0)
 			(effects
@@
 			)
 		)
-		(property "Description" ""
+		(property "Description" "QC01"
 			(at 242.57 110.49 0)
 			(effects

Commit message: Add files via upload
Parts:
- C227, C230, C242, C254, C256, C257, C258, C260, C261, C56: footprint (none) -> Capacitor_SMD:C_0402_1005Metric
- C232: footprint (none) -> Capacitor_SMD:C_1206_3216Metric
- C259, C59: footprint (none) -> Capacitor_SMD:C_0603_1608Metric
- D9: footprint (none) -> PC110:3D
- Q31: footprint (none) -> PCM_Package_TO_SOT_SMD_AKL:SOT-23
- R275, R332, R340, R341, R344, R348, R350, R353, R357, R358, R359, R79, R91: footprint (none) -> PCM_Resistor_SMD_AKL:R_0402_1005Metric
- R284: footprint (none) -> PCM_Resistor_SMD_AKL:R_0805_2012Metric
- U16: footprint (none) -> Package_TO_SOT_SMD:SOT-23-5
- U62, U66: footprint (none) -> Package_SO:TSSOP-14_4.4x5mm_P0.65mm
- U63: footprint (none) -> PC110:SOIC-16W
- X4: footprint (none) -> PC110:XTAL-6
Connections:
- net Chipset_2XCPU_CLK: now also R359.2; no longer R359.1
- net Chipset_CLK: now also R341.1; no longer R341.2
- net GND: now also C227.1 (+), C230.1 (+), C232.1 (+), C242.1 (+), C254.1 (+), C256.1 (+), C258.1 (+), C259.1 (+), C260.1 (+), C56.2, C59.2; no longer C227.2 (-), C230.2 (-), C232.2 (-), C242.2 (-), C254.2 (-), C256.2 (-), C258.2 (-), C259.2 (-), C260.2 (-), C56.1, C59.1
- net PNET1: now also C242.2 (-), C254.2 (-), C256.2 (-); no longer C242.1 (+), C254.1 (+), C256.1 (+)
- net Pluto_CLK: now also R348.1; no longer R348.2
- net VGA_CLK: now also R350.1; no longer R350.2
- net at D9.2 (K), Q31.3 (C), R275.1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: now also C227.2 (-); no longer C227.1 (+)
- net at U62.12, U62.2, U62.5: now also R357.1; no longer R357.2
- net at U62.3: now also R350.2; no longer R350.1
- net at D9.1 (A), R79.2, U16.2 (VDD): now also C56.1; no longer C56.2
- net at D9.3 (A), U16.5 (CD): now also C59.1; no longer C59.2
- net at U63.11 (14.318MHz): now also R357.2; no longer R357.1
- net at C261.1 (+), U63.3 (X1), X4.1: now also C257.1 (+); no longer C257.2 (-)
- net at U63.2 (X2), X4.2: now also C230.2 (-), C257.2 (-); no longer C230.1 (+), C257.1 (+)
- net at U63.14 (3XCPUCLK): now also R359.1; no longer R359.2
- new net: C232.2 (-), C258.2 (-), C259.2 (-), C260.2 (-), R284.2, U63.13 (VCC), U63.4 (VCC)
- new net: R341.2, R348.2, U62.6
Other:
- moved on the sheet: C227, C230, C232, C258, C259, C260, R341, R348, R350, R359

Commit message: Add files via upload
Parts:
- C227, C232, C242, C254, C256, C258, C259, C260: Indicator + -> (none); Rating V -> (none)
- C230, C257, C261: Indicator + -> (none); Rating V -> (none); now not fitted
- D9, R344: now not fitted
- Q31: value MUN2114 -> 6D; Topmark 6D -> (none)
- R357: value 47 -> 33
- U16: value BD53E31 -> 8C01
- U62: value 74LS125 -> SN74LVT125
- U66: value 74LS02 -> SN74LV02
- X4: Frequency 14.318MHz -> (none)
