File: PCB/Mainboard/PC110.kicad_pcb (KiCad board)
At the start: 10 copper layers, 150.1 x 107.4 mm, 936 parts, among them J1 PS2, J10 PCMCIA, J11 CF-card, J12 Debug-6, J13 Docking Port, J14 TestPoint_Pad_D1.5mm, J15 RAM Module, J16 Flat-20, J17 Flat-8, J18 Flat-4, J19 Flat-18, J2 LCD_connector, J3 Audio-Jack, J4 connector-4, J5 PSU_Connector, J6 BridgeBatt, J7 SPKR, J8 Modem-Connector, J9 Debug-10, Q1 IS6, Q10 8C, Q11 IS6, Q12 8C, Q13 IS6, Q14 8C, Q15 8B, Q16 IS6, Q17 6D, Q18 8C, Q19 8B, Q2 8C, Q20 7C, Q21 8B, Q22 YQ, Q23 8B, Q24 6D, Q25 BH RT, Q26 8C, Q27 8C, Q28 8LR, Q29 DNP, Q3 582 B74, Q30 8C, Q31 6D, Q32 8B, Q33 BH RT, Q34 BH RT, Q35 8C, Q36 7C, Q37 BH RT, Q38 8C, Q39 HQ, Q4 YQ, Q40 HQ, Q41 CQ, Q42 CQ, Q43 8B, Q44 8B, Q5 HQ, Q6 ST3, Q7 8C, Q8 6D, Q9 8C, SW1 Switch, SW2 LidSwitch, U1 EA, U10 YM3812, U11 NJM2904M, U12 LM4861, U13 8C01, U14 EA, U15 EA, U16 8C01, U17 3E00, U18 VT74, U19 7W126, U2 7W32, U20 7W14, U21 Bowman, U22 FDC37C665IR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

Commit message: Personal notes for PSU understanding
Connections:
- net Net-(SW2-B) renamed SW2-2
- R354 pad 2: PNET2 -> U21-99
- U21 pad 99: PNET2 -> U21-99
- U3 pad 10: (no net) -> GND
- U3 pad 9: (no net) -> GND
- U35 pad 31: RAM_ID0 -> RAM_ID1
- U35 pad 32: RAM_ID1 -> RAM_ID0
- U36 pad 34: (no net) -> GND
Routing:
- net PNET2: track 494.6 -> 406.1 mm, vias 32 -> 21
- net U21-99: track 0.00 -> 87.7 mm, vias 0 -> 11
